File: Hardware/MaxiCarrierPCB/DC-DC.kicad_sch (KiCad schematic)
At the start: 8 parts

Commit message: more sch + some footprints
Parts:
- added C6: 0.1uF, symbol Device:C
- added JP1: SNS+, Jumper:SolderJumper-2_P1.3mm_Open_TrianglePad1.0x1.5mm, symbol Jumper:SolderJumper_2_Open
- added JP2: SNS-, Jumper:SolderJumper-2_P1.3mm_Open_TrianglePad1.0x1.5mm, symbol Jumper:SolderJumper_2_Open
- added R3: Ru, Capacitor_SMD:C_0603_1608Metric_Pad1.08x0.95mm_HandSolder, symbol Device:R
- added R4: Rd, Capacitor_SMD:C_0603_1608Metric_Pad1.08x0.95mm_HandSolder, symbol Device:R
- added U1: ~, UTSVT_Connectors:Vicor_Maxi_Brick, symbol utsvt_connectors:Vicor_Maxi_Brick
- D3: value D_Zener -> TVS; footprint (none) -> Diode_SMD:D_SMB_Handsoldering
- F1: footprint (none) -> Fuse:Fuseholder_Clip-6.3x32mm_Littelfuse_122_Inline_P34.21x7.62mm_D2.54mm_Horizontal
- H1: footprint (none) -> MountingHole:MountingHole_3.2mm_M3_Pad_TopBottom
Connections:
- net IN+: now also U1.1 (IN+)
- net IN-: now also U1.4 (IN-)
- net OUT+: now also C6.1, JP1.1 (A), U1.9 (OUT+); no longer C5.2
- net BKPLN renamed PLATE
- net PLATE: now also U1.10 (PLATE)
- new net OUT-: C5.2, C6.2, JP2.1 (A), U1.5 (OUT-)
- new net PC: U1.2 (PC)
- new net SC: R3.1, R4.1, U1.7 (SC)
- new net SNS+: JP1.2 (B), R3.2, U1.8 (SENSE+)
- new net SNS-: JP2.2 (B), R4.2, U1.6 (SENSE-)
- no-connect marks 0 -> 1
Other:
- note added: "Baseplate chassis tie point"
- note added: "Jumpers must be closed to enable local sensing"
- note added: "SMBJ150D-M3/I for 135v"
- note added: "Vicor Maxi Converter"
- note removed: "Backplane chassis tie point"
- note removed: "Mounting"
- note removed: "Need more input capacitance?? Eval board has big input cap"
- title: (none) -> DC-DC
- moved on the sheet: H1

Commit message: holy fatass
Parts:
- removed C6: 0.1uF, symbol Device:C
- C1: footprint (none) -> Capacitor_SMD:C_1812_4532Metric_Pad1.57x3.40mm_HandSolder; PN (none) -> C1812X204KDRLCAUTO
- C2, C3, C4, C5: footprint (none) -> Capacitor_SMD:C_1812_4532Metric_Pad1.57x3.40mm_HandSolder; PN (none) -> GA343DR7GD472KW01L
Other:
- note removed: "Caps must be rated >150v"
Changed lines of the file:
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@@
 		)
 	)
-	(text "Caps must be rated >150v"
-		(exclude_from_sim no)
-		(at 83.312 31.75 0)
-		(effects
-			(font
-				(size 1.27 1.27)
-			)
-		)
-	)
 	(text "Vicor Maxi Converter"
 		(exclude_from_sim no)
@@
 	)
 	(junction
-		(at 100.33 38.1)
-		(diameter 0)
-		(color 0 0 0 0)
-	)
-	(junction
 		(at 59.69 25.4)
 		(diameter 0)
@@
 	)
 	(junction
-		(at 100.33 25.4)
-		(diameter 0)
-		(color 0 0 0 0)
-	)
-	(junction
 		(at 80.01 38.1)
 		(diameter 0)
@@
 	(wire
 		(pts
-			(xy 100.33 35.56) (xy 100.33 38.1)
-		)
-		(stroke
-			(width 0)
-			(type default)
-		)
-	)
-	(wire
-		(pts
 			(xy 59.69 38.1) (xy 66.04 38.1)
 		)
@@
 	(wire
 		(pts
-			(xy 100.33 27.94) (xy 100.33 25.4)
-		)
-		(stroke
-			(width 0)
-			(type default)
-		)
-	)
-	(wire
-		(pts
 			(xy 73.66 25.4) (xy 80.01 25.4)
 		)
@@
 			)
 		)
-		(property "Footprint" ""
+		(property "Footprint" "Capacitor_SMD:C_1812_4532Metric_Pad1.57x3.40mm_HandSolder"
 			(at 73.66 37.1348 0)
 			(effects
@@
 			)
 		)
+		(property "PN" "GA343DR7GD472KW01L"
+			(at 69.85 38.1 90)
+			(effects
+				(font
+					(size 1.27 1.27)
+				)
+				(hide yes)
+			)
+		)
 		(pin "1"
 		)
@@
 			)
 		)
-		(property "Footprint" ""
+		(property "Footprint" "Capacitor_SMD:C_1812_4532Metric_Pad1.57x3.40mm_HandSolder"
 			(at 93.98 37.1348 0)
 			(effects
@@
 			)
 		)
+		(property "PN" "GA343DR7GD472KW01L"
+			(at 90.17 38.1 90)
+			(effects
+				(font
+					(size 1.27 1.27)
+				)
+				(hide yes)
+			)
+		)
 		(pin "1"
 		)
@@
 			)
 		)
-		(property "Footprint" ""
+		(property "Footprint" "Capacitor_SMD:C_1812_4532Metric_Pad1.57x3.40mm_HandSolder"
 			(at 73.66 24.4348 0)
 			(effects
@@
 			)
 		)
+		(property "PN" "GA343DR7GD472KW01L"
+			(at 69.85 25.4 90)
+			(effects
+				(font
+					(size 1.27 1.27)
+				)
+				(hide yes)
+			)
+		)
 		(pin "1"
 		)
@@
 	)
 	(symbol
-		(lib_id "Device:C")
-		(at 100.33 31.75 0)
-		(unit 1)
-		(exclude_from_sim no)
-		(in_bom yes)
-		(on_board yes)
-		(dnp no)
-		(fields_autoplaced yes)
-		(property "Reference" "C6"
-			(at 104.14 30.4799 0)
-			(effects
-				(font
-					(size 1.27 1.27)
-				)
-				(justify left)
-			)
-		)
-		(property "Value" "0.1uF"
-			(at 104.14 33.0199 0)
-			(effects
-				(font
-					(size 1.27 1.27)
-				)
-				(justify left)
-			)
-		)
-		(property "Footprint" ""
-			(at 101.2952 35.56 0)
-			(effects
-				(font
-					(size 1.27 1.27)
-				)
-				(hide yes)
-			)
-		)
-		(property "Datasheet" "~"
-			(at 100.33 31.75 0)
-			(effects
-				(font
-					(size 1.27 1.27)
-				)
-				(hide yes)
-			)
-		)
-		(property "Description" "Unpolarized capacitor"
-			(at 100.33 31.75 0)
-			(effects
-				(font
-					(size 1.27 1.27)
-				)
-				(hide yes)
-			)
-		)
-		(pin "1"
-		)
-		(pin "2"
-		)
-		(instances
-			(project "MaxiCarrier"
-				(path "/9822b44e-a9c2-4c7f-86ac-4edcd1d27dc4/89fb0e6b-6d5f-4609-8215-b6408236ae89"
-					(reference "C6")
-					(unit 1)
-				)
-			)
-		)
-	)
-	(symbol
 		(lib_id "power:VCC")
 		(at 22.86 22.86 0)
@@
 			)
 		)
-		(property "Footprint" ""
+		(property "Footprint" "Capacitor_SMD:C_1812_4532Metric_Pad1.57x3.40mm_HandSolder"
 			(at 93.98 24.4348 0)
 			(effects
@@
 			)
 		)
+		(property "PN" "GA343DR7GD472KW01L"
+			(at 90.17 25.4 90)
+			(effects
+				(font
+					(size 1.27 1.27)
+				)
+				(hide yes)
+			)
+		)
 		(pin "1"
 		)
@@
 			)
 		)
-		(property "Footprint" ""
+		(property "Footprint" "Capacitor_SMD:C_1812_4532Metric_Pad1.57x3.40mm_HandSolder"
 			(at 60.6552 35.56 0)
 			(effects
@@
 			(at 59.69 31.75 0)
 			(effects
+				(font
+					(size 1.27 1.27)
+				)
+				(hide yes)
+			)
+		)
+		(property "P/N" ""
+			(at 59.69 31.75 0)
+			(effects
+				(font
+					(size 1.27 1.27)
+				)
+				(hide yes)
+			)
+		)
+		(property "PN" "C1812X204KDRLCAUTO"
+			(at 59.69 31.75 0)
+			(effects

Commit message: more fix
Parts:
- removed JP1: SNS+, Jumper:SolderJumper-2_P1.3mm_Open_TrianglePad1.0x1.5mm, symbol Jumper:SolderJumper_2_Open
- removed JP2: SNS-, Jumper:SolderJumper-2_P1.3mm_Open_TrianglePad1.0x1.5mm, symbol Jumper:SolderJumper_2_Open
- added R5, R6: 0, Resistor_SMD:R_0603_1608Metric_Pad0.98x0.95mm_HandSolder, symbol Device:R
- R3, R4: footprint Capacitor_SMD:C_0603_1608Metric_Pad1.08x0.95mm_HandSolder -> Resistor_SMD:R_0603_1608Metric_Pad0.98x0.95mm_HandSolder
Connections:
- net OUT+: now also R5.2
- net OUT-: now also R6.2
- net SNS+: now also R5.1
- net SNS-: now also R6.1
Other:
- moved on the sheet: R3, R4
