File: Hardware/BasePCB/LV Carrier Board/LV Carrier Board.kicad_sch (KiCad schematic)
At the start: 44 parts, among them J1 52465-2470, J4 CarCANConnector, J5 Ext_Power, J6 CarCANConnector, Q5 PMOS, Q7 PMOS, U1 TPS27SA08-Q1, U2 DCDC, U3 SUPP Charger, U5 LeaderSOM

Commit message: More Updates
Parts:
- removed J5: Ext_Power, symbol Connector_Generic:Conn_01x03
- added J2, J7: Conn_01x02, symbol Connector_Generic:Conn_01x02
- added R18, R20: 62k, symbol Device:R
- added R19, R21: 10k, symbol Device:R
Connections:
- net GND: now also J2.1 (Pin_1), J7.1 (Pin_1), R19.1, R21.1
- net LV_EN_PS: now also U5.45 (ADC1_IN8), R20.2, R21.2
- net LV_EN_SUPP: now also U5.47 (ADC1_IN6), R18.2, R19.2
- net PS: now also J2.2 (Pin_2), R20.1
- net SUPP_IN: now also J7.2 (Pin_2), R18.1
- net LoadSw_Rd: now reaches R11.2, U1.4 (EN)
- net LoadSw_Rd: now also U5.11 (I2C3_SCL)
- no-connect marks 24 -> 22
Other:
- note removed: "ADD ARRAY"
- note removed: "mCU pin"
- moved on the sheet: U5A, U5B

Commit message: Update
Parts:
- removed J2, J7: Conn_01x02, symbol Connector_Generic:Conn_01x02
- removed J6: CarCANConnector, UTSVT_Connectors:Molex_Nano-Fit_105309-xx02_1x02_P2.50mm_Vertical, symbol utsvt_connectors:CarCANConnector
- removed R18, R20: 62k, symbol Device:R
- removed R19, R21: 10k, symbol Device:R
- added J2: Conn_01x04, symbol Connector_Generic:Conn_01x04
- added J5, J8: Conn_01x02, symbol Connector_Generic:Conn_01x02
Connections:
- net CANH: now also J2.1 (Pin_1)
- net CANL: now also J2.2 (Pin_2)
- net CHARGER_OUT: no longer D5.2 (A), F1.2, R1.4
- net GND: now also J5.1 (Pin_1), J8.1 (Pin_1)
- net LV_EN_PS: now also J2.3 (Pin_3)
- net LV_EN_SUPP: now also J2.4 (Pin_4)
- net PS: now also J8.2 (Pin_2)
- net SUPP_IN: now also J5.2 (Pin_2)
- new net: D5.2 (A), F1.2, R1.4
Other:
- note added: "Enable Logic"
- note removed: "Can In"
- note removed: "Power Supply"
- moved on the sheet: D1, D2, D5, D6, J1, J4, Q5, Q7, R13, R14, R15, R16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

Commit message: Updates to footprints
Parts:
- 120V Conn1: footprint (none) -> Connector_AMASS:AMASS_XT30U-M_1x02_P5.0mm_Vertical
- J2: footprint (none) -> Connector_Molex:Molex_Nano-Fit_105309-xx04_1x04_P2.50mm_Vertical
- J5: footprint (none) -> Connector_AMASS:AMASS_XT30U-M_1x02_P5.0mm_Vertical
- J8: footprint (none) -> Connector_AMASS:AMASS_XT60-M_1x02_P7.20mm_Vertical
- TP12, TP13: footprint (none) -> UTSVT_Special:TestPoint_HEX_3mmID
- U2, U3, U4: footprint UTSVT_Connectors:Maxi_Carrier_Connector -> LV Carrier Library:Maxi_Carrier_Connector
Changed lines of the file:
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@@
 			)
 		)
-		(property "Footprint" ""
+		(property "Footprint" "Connector_AMASS:AMASS_XT30U-M_1x02_P5.0mm_Vertical"
 			(at 26.67 175.26 0)
 			(effects
@@
 			)
 		)
-		(property "Footprint" ""
+		(property "Footprint" "Connector_AMASS:AMASS_XT60-M_1x02_P7.20mm_Vertical"
 			(at 24.13 46.99 0)
 			(effects
@@
 			)
 		)
-		(property "Footprint" "UTSVT_Connectors:Maxi_Carrier_Connector"
+		(property "Footprint" "LV Carrier Library:Maxi_Carrier_Connector"
 			(at 81.28 170.18 0)
 			(effects
@@
 			)
 		)
-		(property "Footprint" ""
+		(property "Footprint" "UTSVT_Special:TestPoint_HEX_3mmID"
 			(at 200.66 74.93 0)
 			(effects
@@
 			)
 		)
-		(property "Footprint" "UTSVT_Connectors:Maxi_Carrier_Connector"
+		(property "Footprint" "LV Carrier Library:Maxi_Carrier_Connector"
 			(at 120.65 120.65 0)
 			(effects
@@
 			)
 		)
-		(property "Footprint" "UTSVT_Connectors:Maxi_Carrier_Connector"
+		(property "Footprint" "LV Carrier Library:Maxi_Carrier_Connector"
 			(at 129.54 29.21 0)
 			(effects
@@
 			)
 		)
-		(property "Footprint" ""
+		(property "Footprint" "UTSVT_Special:TestPoint_HEX_3mmID"
 			(at 200.66 64.77 0)
 			(effects
@@
 			)
 		)
-		(property "Footprint" ""
+		(property "Footprint" "Connector_AMASS:AMASS_XT30U-M_1x02_P5.0mm_Vertical"
 			(at 24.13 36.83 0)
 			(effects
@@
 			)
 		)
-		(property "Footprint" ""
+		(property "Footprint" "Connector_Molex:Molex_Nano-Fit_105309-xx04_1x04_P2.50mm_Vertical"
 			(at 31.75 81.28 0)
 			(effects
