File: Hardware/SupplementalMonitoringPCB/CurrentBefore.kicad_sch (KiCad schematic)
At the start: 12 parts, among them IC2 TLV9002QDRQ1, IC5 INA241A5IDR

Commit message: Draft
Connections:
- net +1V renamed VRef
Changed lines of the file:
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@@
+		)
+	)
+	(hierarchical_label "VRef"
+		(shape input)
+		(at 62.23 138.43 180)
+		(effects
+			(font
+				(size 1.27 1.27)
+			)
+			(justify right)
 		)
 	)
@@
 					(unit 1)
 				)
-			)
-		)
-	)
-	(symbol
-		(lib_id "power:+1V0")
-		(at 62.23 138.43 0)
-		(unit 1)
-		(exclude_from_sim no)
-		(in_bom yes)
-		(on_board yes)
-		(dnp no)
-		(property "Reference" "#PWR025"
-			(at 62.23 142.24 0)
-			(effects
-				(font
-					(size 1.27 1.27)
-				)
-				(hide yes)
-			)
-		)
-		(property "Value" "+1V"
-			(at 57.404 137.922 0)
-			(effects
-				(font
-					(size 1.27 1.27)
-				)
-			)
-		)
-		(property "Footprint" ""
-			(at 62.23 138.43 0)
-			(effects
-				(font
-					(size 1.27 1.27)
-				)
-				(hide yes)
-			)
-		)
-		(property "Datasheet" ""
-			(at 62.23 138.43 0)
-			(effects
-				(font
-					(size 1.27 1.27)
-				)
-				(hide yes)
-			)
-		)
-		(property "Description" "Power symbol creates a global label with name \"+1V0\""
-			(at 62.23 138.43 0)
-			(effects
-				(font
-					(size 1.27 1.27)
-				)
-				(hide yes)
-			)
-		)
-		(pin "1"
-		)
-		(instances
-			(project "Supplemental Monitoring PCB"
-				(path "/4b30d391-cf39-434b-85dc-df89b45eb2b2/1c9c40d1-9135-4b24-beff-d2d4ce45e42f"
-					(reference "#PWR025")
-					(unit 1)
-				)

Commit message: labels
Connections:
- net I_Current renamed Initial_Current
- net I_Input renamed Initial_Input
- net I_Shunt renamed Initial_Shunt
Changed lines of the file:
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@@
 		)
 	)
-	(text "200 gain\n OpAmp"
+	(text "200 gain OpAmp"
 		(exclude_from_sim no)
-		(at 31.496 59.436 0)
+		(at 35.306 57.15 0)
 		(effects
 			(font
@@
 		)
 	)
-	(hierarchical_label "I_Input"
+	(hierarchical_label "Initial_Input"
 		(shape input)
 		(at 119.38 45.72 0)
@@
 		)
 	)
-	(hierarchical_label "I_Shunt"
+	(hierarchical_label "Initial_Shunt"
 		(shape input)
 		(at 92.71 45.72 0)
@@
 		)
 	)
-	(hierarchical_label "I_Current"
+	(hierarchical_label "Initial_Current"
 		(shape output)
 		(at 240.03 130.81 0)

Commit message: 9/27 Workday
Other:
- note added: "1.75 x 1.8 = 3.15"
- note added: "18(1/1+4.5) = 3.27"
- note added: "200(-0.00125) = -0.25"
- note added: "200(0.0075) = 1.5"
- note added: "30(1/1+4.5) = 5.45"
- note added: "Max Current: 30(250E-6)"
- note added: "Min Current: -5(250E-6)"
- note added: "Op Amp Gain of 1.8"
- note added: "Range of 1.75 V (-.25 to 1.5)"
- note added: "Voltage Difference Range:"
- note added: "Voltage input Range for OpAmp: 3.27-5.45"
- note added: "Vout = 1.75 + 1.024 (close to 3.3)"
- note removed: "shunt resistor: ULR3N-R00025JT2"
- moved on the sheet: R20, R21, R22, R23

Commit message: Address Reviews
Parts:
- added TP10, TP11, TP12, TP13, TP14, TP9: TestPoint, symbol Connector:TestPoint
Connections:
- net VRef is gone; now on net 1.024V: IC5.3 (REF2)
- net Initial_Current: now also TP14.1
- net Out1: now also TP12.1, TP9.1
- net Out2: now also TP13.1
- net Sense+: now also IC5.8 (IN+), TP11.1; no longer IC5.1 (IN-)
- net Sense-: now also IC5.1 (IN-), TP10.1; no longer IC5.8 (IN+)
- net +1V0 renamed 1.024V
- net Initial_Input renamed Unregulated_Initial_V
- net Initial_Shunt renamed Unregulated_Initial_Sense
Other:
- note added: "I have resistor dividers here becuase the max voltage that the op amp can handle is 20v and the max possible voltage is 30v"

Commit message: 10/2 changes
Parts:
- added C27, C28: 1u, symbol Device:C
- C11: value 1u -> .1u
- UnregulatedCurrentIn1: renamed from TP12; value TestPoint -> Test Point
- UnregulatedCurrentOut1: renamed from TP9; value TestPoint -> Test Point
- UnregulatedSense+: renamed from TP11; value TestPoint -> Test Point
- renumbered TP13 to UnregulatedCurrentOut2, TP14 to UnregulatedCurrentOut3, TP10 to UnregulatedSense-
Connections:
- net +3.3V: now also C27.1, C28.1
- net GND: now also C27.2, C28.2
Other:
- moved on the sheet: C13

Commit message: starting layout now
Parts:
- removed R20, R22: 4.5k, symbol Device:R
- removed R21, R23: 1k, symbol Device:R
- C11, C12, C13, C27, C28: footprint (none) -> Capacitor_SMD:C_0603_1608Metric_Pad1.08x0.95mm_HandSolder
- IC2, IC5: footprint SOIC127P600X175-8N -> TLV9002QDRQ1:SOIC127P600X175-8N
- R3, R4, R5: footprint (none) -> Resistor_SMD:R_0603_1608Metric_Pad0.98x0.95mm_HandSolder
- UnregulatedCurrentIn1, UnregulatedCurrentOut1, UnregulatedCurrentOut2, UnregulatedCurrentOut3: footprint (none) -> TestPoint:TestPoint_Pad_1.0x1.0mm
- UnregulatedSense+1: renamed from UnregulatedSense+; footprint (none) -> TestPoint:TestPoint_Pad_1.0x1.0mm
- UnregulatedSense-1: renamed from UnregulatedSense-; footprint (none) -> TestPoint:TestPoint_Pad_1.0x1.0mm
Connections:
- net Sense+ is gone; now on net Unregulated_Initial_V: IC5.8 (IN+), UnregulatedSense+1.1
- net Sense- is gone; now on net Unregulated_Initial_Sense: IC5.1 (IN-), UnregulatedSense-1.1
Other:
- note removed: "18(1/1+4.5) = 3.27"
- note removed: "30(1/1+4.5) = 5.45"
- note removed: "I have resistor dividers here becuase the max voltage that the op amp can handle is 20v and the max possible voltage is 30v"
- note removed: "Voltage input Range for OpAmp: 3.27-5.45"

Commit message: layout,fixedschematic
Parts:
- removed UnregulatedCurrentIn1, UnregulatedCurrentOut1, UnregulatedSense+1: Test Point, TestPoint:TestPoint_Pad_1.0x1.0mm, symbol Connector:TestPoint
- removed UnregulatedCurrentOut2, UnregulatedCurrentOut3, UnregulatedSense-1: TestPoint, TestPoint:TestPoint_Pad_1.0x1.0mm, symbol Connector:TestPoint
- added Unreg_CurrentIn1: Test Point, TestPoint:TestPoint_Pad_1.0x1.0mm, symbol Connector:TestPoint
- added Unreg_Current_Filter1: TestPoint, TestPoint:TestPoint_Pad_1.0x1.0mm, symbol Connector:TestPoint
Connections:
- net Out1: now also Unreg_CurrentIn1.1
- net Out2: now also Unreg_Current_Filter1.1
- net Initial_Current renamed Unreg_Current
- net Unregulated_Initial_Sense renamed Unreg_Sense-
- net Unregulated_Initial_V renamed Unreg_Sense+
Other:
- moved on the sheet: C11, C27, C28
