File: Hardware/SupplementalMonitoringPCB/SevenSegment.kicad_sch (KiCad schematic)
At the start: 9 parts, among them U1 SN74HC595N, U2 SN74HC595N, U3 SN74HC595N, U4 SN74HC595N

Commit message: Draft
Parts:
- added R11, R12, R14, R24, R25, R26, R27, R28, R29, R30, R33, R34, R35, R36, R37, R38, R39, R42, R43, R44, R45, R46, R47, R48, R49, R50, R51, R52, R53, R54, R55, R56: 560, symbol Device:R
Connections:
- net +5V: now also DS1.22 (COMMON_ANODE_DIG_4), DS1.23 (COMMON_ANODE_DIG_3), DS1.31 (COMMON_ANODE_DIG_2), DS1.32 (COMMON_ANODE_DIG_1)
- net 1a: now also R29.2; no longer DS1.34 (CATHODE_A_DIG_1)
- net 1b: now also R30.2; no longer DS1.33 (CATHODE_B_DIG_1)
- net 1c: now also R14.1; no longer DS1.3 (CATHODE_C_DIG_1)
- net 1d: now also R12.1; no longer DS1.2 (CATHODE_D_DIG_1)
- net 1e: now also R11.1; no longer DS1.1 (CATHODE_E_DIG_1)
- net 1f: now also R27.2; no longer DS1.36 (CATHODE_F_DIG_1)
- net 1g: now also R28.2; no longer DS1.35 (CATHODE_G_DIG_1)
- net 1h: now also R24.1
- net 3b: now reaches U3.1 (QB)
- net 3b: now also R39.2
- net 3a: now reaches U3.15 (QA)
- net 3a: now also R38.2
- net 3c: now reaches U3.2 (QC)
- net 3c: now also R50.1
- net 3d: now reaches U3.3 (QD)
- net 3d: now also R49.1
- net 3e: now reaches U3.4 (QE)
- net 3e: now also R48.1
- net 3f: now reaches U3.5 (QF)
- net 3f: now also R36.2
- net 3g: now reaches U3.6 (QG)
- net 3g: now also R37.2
- net 3h: now reaches U3.7 (QH)
- net 3h: now also R51.1
- net 4b: now reaches U4.1 (QB)
- net 4b: now also R44.2
- net 4a: now reaches U4.15 (QA)
- net 4a: now also R43.2
- net 4c: now reaches U4.2 (QC)
- net 4c: now also R55.1
- net 4d: now reaches U4.3 (QD)
- net 4d: now also R53.1
- net 4e: now reaches U4.4 (QE)
- net 4e: now also R52.1
- net 4f: now reaches U4.5 (QF)
- net 4f: now also R42.2
- net 4g: now reaches U4.6 (QG)
- net 4g: now also R54.1
- net 4h: now reaches U4.7 (QH)
- net 4h: now also R56.1
- net 2b: now reaches U2.1 (QB)
- net 2b: now also R35.2
- net 2a: now reaches U2.15 (QA)
- net 2a: now also R34.2
- net 2c: now reaches U2.2 (QC)
- net 2c: now also R46.1
- net 2d: now reaches U2.3 (QD)
- net 2d: now also R26.1
- net 2e: now reaches U2.4 (QE)
- net 2e: now also R25.1
- net 2f: now reaches U2.5 (QF)
- net 2f: now also R33.2
- net 2g: now reaches U2.6 (QG)
- net 2g: now also R45.1
- net 2h: now reaches U2.7 (QH)
- net 2h: now also R47.1
- net at DS1.10 (CATHODE_E_DIG_3): now also R48.2
- net at DS1.11 (CATHODE_D_DIG_3): now also R49.2
- net at DS1.12 (CATHODE_C_DIG_3): now also R50.2
- net at DS1.13 (CATHODE_DP3_DIG_3): now also R51.2
- net at DS1.14 (CATHODE_E_DIG_4): now also R52.2
- net at DS1.15 (CATHODE_D_DIG_4): now also R53.2
- net at DS1.16 (CATHODE_G_DIG_4): now also R54.2
- net at DS1.17 (CATHODE_C_DIG_4): now also R55.2
- net at DS1.18 (CATHODE_DP4_DIG_4): now also R56.2
- net at DS1.19 (CATHODE_B_DIG_4): now also R44.1
- net at DS1.20 (CATHODE_A_DIG_4): now also R43.1
- net at DS1.21 (CATHODE_F_DIG_4): now also R42.1
- net at DS1.24 (CATHODE_B_DIG_3): now also R39.1
- net at DS1.25 (CATHODE_A_DIG_3): now also R38.1
- net at DS1.26 (CATHODE_G_DIG_3): now also R37.1
- net at DS1.27 (CATHODE_F_DIG_3): now also R36.1
- net at DS1.28 (CATHODE_B_DIG_2): now also R35.1
- net at DS1.29 (CATHODE_A_DIG_2): now also R34.1
- net at DS1.30 (CATHODE_F_DIG_2): now also R33.1
- net at DS1.4 (CATHODE_DP1_DIG_1): now also R24.2
- net at DS1.5 (CATHODE_E_DIG_2): now also R25.2
- net at DS1.6 (CATHODE_D_DIG_2): now also R26.2
- net at DS1.7 (CATHODE_G_DIG_2): now also R45.2
- net at DS1.8 (CATHODE_CDIG_2): now also R46.2
- net at DS1.9 (CATHODE_DP2_DIG_2): now also R47.2
- new net: DS1.35 (CATHODE_G_DIG_1), R28.1
- new net: DS1.33 (CATHODE_B_DIG_1), R30.1
- new net: DS1.1 (CATHODE_E_DIG_1), R11.2
- new net: DS1.2 (CATHODE_D_DIG_1), R12.2
- new net: DS1.3 (CATHODE_C_DIG_1), R14.2
- new net: DS1.36 (CATHODE_F_DIG_1), R27.1
- new net: DS1.34 (CATHODE_A_DIG_1), R29.1
- no-connect marks 0 -> 1
Other:
- note added: "Seven Segment"

Commit message: labels
Other:
- moved on the sheet: DS1, R11, R12, R14, R24, R25, R26, R27, R28, R29, R30, R33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

Commit message: 9/27 Workday
Connections:
- net +5V renamed +3.3V

Commit message: Address Reviews
Parts:
- added J1: Conn_01x18, symbol Connector_Generic:Conn_01x18
- added J2: Conn_01x14, symbol Connector_Generic:Conn_01x14
Connections:
- net +3.3V: no longer C18.1
- net 1a: now also J2.3 (Pin_3)
- net 1b: now also J2.4 (Pin_4)
- net 1c: now also J1.16 (Pin_16)
- net 1d: now also J1.17 (Pin_17)
- net 1e: now also J1.18 (Pin_18)
- net 1f: now also J2.1 (Pin_1)
- net 1g: now also J2.2 (Pin_2)
- net 1h: now also J1.15 (Pin_15)
- net 2a: now also J2.6 (Pin_6)
- net 2b: now also J2.7 (Pin_7)
- net 2c: now also J1.11 (Pin_11)
- net 2d: now also J1.13 (Pin_13)
- net 2e: now also J1.14 (Pin_14)
- net 2f: now also J2.5 (Pin_5)
- net 2g: now also J1.12 (Pin_12)
- net 2h: now also J1.10 (Pin_10)
- net 3a: now also J2.10 (Pin_10)
- net 3b: now also J2.11 (Pin_11)
- net 3c: now also J1.7 (Pin_7)
- net 3d: now also J1.8 (Pin_8)
- net 3e: now also J1.9 (Pin_9)
- net 3f: now also J2.8 (Pin_8)
- net 3g: now also J2.9 (Pin_9)
- net 3h: now also J1.6 (Pin_6)
- net 4a: now also J2.13 (Pin_13)
- net 4b: now also J2.14 (Pin_14)
- net 4c: now also J1.2 (Pin_2)
- net 4d: now also J1.4 (Pin_4)
- net 4e: now also J1.5 (Pin_5)
- net 4f: now also J2.12 (Pin_12)
- net 4g: now also J1.3 (Pin_3)
- net 4h: now also J1.1 (Pin_1)
- net GND: now also C18.2
- net at U4.10 (~{SRCLR}), U4.16 (VCC): now also C18.1; no longer C18.2
Other:
- note added: "Headers for test points."
- moved on the sheet: C18

Commit message: 10/2 changes
Parts:
- removed C16, C17, C8: 1u, symbol Device:C
- added C19, C20, C31: .1u, symbol Device:C
- C18: value 1u -> .1u
- renumbered J1 to SevenSegmentTestPoint1, J2 to SevenSegmentTestPoint2
Connections:
- net GND is gone; now on net +3.3V: C18.2, U1.13 (~{OE}), U1.8 (GND), U2.10 (~{SRCLR}), U2.13 (~{OE}), U2.16 (VCC), U2.8 (GND), U3.13 (~{OE}), U3.8 (GND), U4.13 (~{OE}), U4.8 (GND)
- net +3.3V: now also C18.1, U1.10 (~{SRCLR}), U1.16 (VCC), U3.10 (~{SRCLR}), U3.16 (VCC), U4.10 (~{SRCLR}), U4.16 (VCC), C19.1, C19.2, C20.1, C20.2, C31.1, C31.2
Other:
- moved on the sheet: C18

Commit message: starting layout now
Parts:
- removed SevenSegmentTestPoint1: Conn_01x18, symbol Connector_Generic:Conn_01x18
- removed SevenSegmentTestPoint2: Conn_01x14, symbol Connector_Generic:Conn_01x14
- added RCLK1, SER1, SRCLK1: Test Point, TestPoint:TestPoint_Pad_1.0x1.0mm, symbol Connector:TestPoint
- C18, C19, C20, C31: footprint (none) -> Capacitor_SMD:C_0603_1608Metric_Pad1.08x0.95mm_HandSolder
- DS1: footprint CA5611GWA -> CA5611:CA5611GWA
- R11, R12, R14, R24, R25, R26, R27, R28, R29, R30, R33, R34, R35, R36, R37, R38, R39, R42, R43, R44, R45, R46, R47, R48, R49, R50, R51, R52, R53, R54, R55, R56: footprint (none) -> Resistor_SMD:R_0603_1608Metric_Pad0.98x0.95mm_HandSolder
Connections:
- net RCLK: now also SER1.1
- net SER: now also RCLK1.1
- net SRCLK: now also SRCLK1.1

Commit message: layout,fixedschematic
Parts:
- removed RCLK1, SER1, SRCLK1: Test Point, TestPoint:TestPoint_Pad_1.0x1.0mm, symbol Connector:TestPoint
- U1, U2, U3, U4: footprint SN74HC595N:DIP794W45P254L1969H508Q16 -> SN74HC594DR:SOIC127P600X175-16N
Connections:
- net +3.3V: no longer C18.2, C19.2, C20.2, C31.2, U1.13 (~{OE}), U1.8 (GND), U2.13 (~{OE}), U2.8 (GND), U3.13 (~{OE}), U3.8 (GND), U4.13 (~{OE}), U4.8 (GND)
- new net GND: C18.2, C19.2, C20.2, C31.2, U1.13 (~{OE}), U1.8 (GND), U2.13 (~{OE}), U2.8 (GND), U3.13 (~{OE}), U3.8 (GND), U4.13 (~{OE}), U4.8 (GND)

Commit message: Reviews
Parts:
- DS1: footprint CA5611:CA5611GWA -> CA56_11GWA:CA5611GWA
Changed lines of the file:
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@@
 			)
 		)
-		(property "Footprint" "CA5611:CA5611GWA"
+		(property "Footprint" "CA56_11GWA:CA5611GWA"
 			(at 172.72 200.33 0)
 			(effects
