File: Hardware/SupplementalMonitoringPCB/Supplemental Monitoring PCB.kicad_sch (KiCad schematic)
At the start: 6 parts, among them J6 52465-2470

Commit message: Draft
Parts:
- removed LED1: LDQ-M516RI, LED_LDQ-M516RI_LUM, symbol 2025-09-27_20-00-42:LDQ-M516RI
- added C3, C4, C6: 1uF, Capacitor_SMD:C_0603_1608Metric_Pad1.08x0.95mm_HandSolder, symbol Device:C
- added IC6: REF35102QDBVR, SOT95P280X145-6N, symbol REF35102QDBVR:REF35102QDBVR
Connections:
- net +3.3V: now also C6.1, IC6.3 (EN), IC6.4 (VIN)
- net GND: now also C3.2, C4.2, C6.2, IC6.1 (GND_1), IC6.2 (GND_2)
- net SRCLK: now also J6.4; no longer J6.6
- net RCLK: now reaches J6.2
- new net: C4.1, IC6.5 (NR)
- new net VRef: C3.1, IC6.6 (VREF)
Other:
- sheet CurrentAfter ports: added VRef; removed none
- sheet CurrentBefore ports: added VRef; removed none
- sheet Seven Segment ports: added RCLK, SER, SRCLK; removed none
- note added: "Reference Voltage"

Commit message: labels
Connections:
- net I_Current renamed Initial_Current
- net I_Input renamed Initial_Input
- net I_Shunt renamed Initial_Shunt
- net I_Voltage renamed Initial_Voltage
- net R_Current renamed Regulated_Current
- net R_Input renamed Regulated_Input
- net R_Shunt renamed Regulated_Shunt
- net R_Voltage renamed Regulated_Voltage
Other:
- sheet CurrentAfter ports: added Regulated_Current, Regulated_Input, Regulated_Shunt; removed R_Current, R_Input, R_Shunt
- sheet CurrentBefore ports: added Initial_Current, Initial_Input, Initial_Shunt; removed I_Current, I_Input, I_Shunt
- sheet Voltage ports: added Initial_Input, Initial_Voltage, Regulated_Input, Regulated_Voltage; removed I_Input, I_Voltage, R_Input, R_Voltage
- note added: "Reference Voltage of 1.024V"
Changed lines of the file:
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@@
 	(text "Seven Segment"
 		(exclude_from_sim no)
-		(at 108.966 108.966 0)
+		(at 108.966 111.506 0)
 		(effects
 			(font
@@
 		(exclude_from_sim no)
 		(at 38.608 25.908 0)
+		(effects
+			(font
+				(size 1.27 1.27)
+			)
+		)
+	)
+	(text "Reference Voltage of 1.024V"
+		(exclude_from_sim no)
+		(at 250.952 105.41 0)
 		(effects
 			(font
@@
 		)
 	)
-	(label "I_Input"
-		(at 24.13 125.73 180)
+	(label "Initial_Input"
+		(at 30.48 129.54 180)
 		(effects
 			(font
@@
 	)
 	(label "RCLK"
-		(at 97.79 127 180)
+		(at 97.79 129.54 180)
 		(effects
 			(font
@@
 		)
 	)
-	(label "I_Voltage"
+	(label "Initial_Voltage"
+		(at 69.85 132.08 0)
+		(effects
+			(font
+				(size 1.27 1.27)
+			)
+			(justify left bottom)
+		)
+	)
+	(label "Initial_Voltage"
 		(at 68.58 50.8 0)
 		(effects
@@
 		)
 	)
-	(label "R_Input"
-		(at 24.13 149.86 180)
+	(label "Regulated_Input"
+		(at 30.48 153.67 180)
 		(effects
 			(font
@@
 		)
 	)
-	(label "R_Current"
-		(at 63.5 151.13 0)
+	(label "Regulated_Current"
+		(at 69.85 154.94 0)
 		(effects
 			(font
@@
 	)
 	(label "SRCLK"
-		(at 97.79 132.08 180)
+		(at 97.79 134.62 180)
 		(effects
 			(font
@@
 		)
 	)
-	(label "R_Voltage"
-		(at 63.5 128.27 0)
+	(label "Regulated_Voltage"
+		(at 69.85 129.54 0)
 		(effects
 			(font
@@
 		)
 	)
-	(label "R_Input"
+	(label "Regulated_Input"
 		(at 45.72 45.72 180)
 		(effects
@@
 		)
 	)
-	(label "R_Shunt"
+	(label "Regulated_Shunt"
 		(at 45.72 55.88 180)
 		(effects
@@
 		)
 	)
-	(label "R_Shunt"
-		(at 24.13 152.4 180)
+	(label "Regulated_Shunt"
+		(at 30.48 156.21 180)
 		(effects
 			(font
@@
 		)
 	)
-	(label "I_Current"
+	(label "Initial_Current"
 		(at 68.58 55.88 0)
 		(effects
@@
 	)
 	(label "SER"
-		(at 97.79 129.54 180)
+		(at 97.79 132.08 180)
 		(effects
 			(font
@@
 		)
 	)
-	(label "R_Voltage"
+	(label "Regulated_Voltage"
 		(at 68.58 45.72 0)
 		(effects
@@
 		)
 	)
-	(label "R_Current"
+	(label "Regulated_Current"
 		(at 68.58 40.64 0)
 		(effects
@@
 		)
 	)
-	(label "R_Input"
-		(at 24.13 128.27 180)
+	(label "Regulated_Input"
+		(at 30.48 132.08 180)
 		(effects
 			(font
@@
 		)
 	)
-	(label "I_Current"
-		(at 63.5 102.87 0)
+	(label "Initial_Current"
+		(at 69.85 106.68 0)
 		(effects
 			(font
@@
 		)
 	)
-	(label "I_Voltage"
-		(at 63.5 125.73 0)
-		(effects
-			(font
-				(size 1.27 1.27)
-			)
-			(justify left bottom)
-		)
-	)
 	(label "VRef"
-		(at 24.13 106.68 180)
+		(at 30.48 110.49 180)
 		(effects
 			(font
@@
 		)
 	)
-	(label "I_Input"
+	(label "Initial_Input"
 		(at 45.72 40.64 180)
 		(effects
@@
 		)
 	)
-	(label "I_Shunt"
+	(label "Initial_Shunt"
 		(at 45.72 50.8 180)
 		(effects
@@
 		)
 	)
-	(label "I_Shunt"
-		(at 24.13 104.14 180)
+	(label "Initial_Shunt"
+		(at 30.48 107.95 180)
 		(effects
 			(font
@@
 		)
 	)
-	(label "I_Input"
-		(at 24.13 101.6 180)
+	(label "Initial_Input"
+		(at 30.48 105.41 180)
 		(effects
 			(font
@@
 	)
 	(label "VRef"
-		(at 24.13 154.94 180)
+		(at 30.48 158.75 180)
 		(effects
 			(font
@@
 	)
 	(sheet
-		(at 24.13 95.25)
+		(at 30.48 99.06)
 		(size 39.37 15.24)
 		(exclude_from_sim no)
@@
 		)
 		(property "Sheetname" "CurrentBefore"
-			(at 24.13 94.5384 0)
+			(at 30.48 98.3484 0)
 			(effects
 				(font
@@
 		)
 		(property "Sheetfile" "CurrentBefore.kicad_sch"
-			(at 24.13 111.0746 0)
+			(at 30.48 114.8846 0)
 			(effects
 				(font
@@
 			)
 		)
-		(pin "I_Input" input
-			(at 24.13 101.6 180)
+		(pin "Initial_Input" input
+			(at 30.48 105.41 180)
 			(effects
 				(font
@@
 			)
 		)
-		(pin "I_Shunt" input
-			(at 24.13 104.14 180)
+		(pin "Initial_Shunt" input
+			(at 30.48 107.95 180)
 			(effects
 				(font
@@
 		)
 		(pin "VRef" input
-			(at 24.13 106.68 180)
+			(at 30.48 110.49 180)
 			(effects
 				(font
@@
 			)
 		)
-		(pin "I_Current" output
-			(at 63.5 102.87 0)
+		(pin "Initial_Current" output
+			(at 69.85 106.68 0)
 			(effects
 				(font
@@
 	)
 	(sheet
-		(at 97.79 121.92)
+		(at 97.79 124.46)
 		(size 35.56 13.97)
 		(exclude_from_sim no)
@@
 		)
 		(property "Sheetname" "Seven Segment"
-			(at 97.79 121.2084 0)
+			(at 97.79 123.7484 0)
 			(effects
 				(font
@@
 		)
 		(property "Sheetfile" "SevenSegment.kicad_sch"
-			(at 97.79 136.4746 0)
+			(at 97.79 139.0146 0)
 			(effects
 				(font
@@
 		)
 		(pin "RCLK" input
-			(at 97.79 127 180)
+			(at 97.79 129.54 180)
 			(effects
 				(font
@@
 		)
 		(pin "SER" input
-			(at 97.79 129.54 180)
+			(at 97.79 132.08 180)
 			(effects
 				(font
@@
 		)
 		(pin "SRCLK" input
-			(at 97.79 132.08 180)
+			(at 97.79 134.62 180)
 			(effects
 				(font
@@
 	)
 	(sheet
-		(at 24.13 119.38)
+		(at 30.48 123.19)
 		(size 39.37 15.24)
 		(exclude_from_sim no)
@@
 		)
 		(property "Sheetname" "Voltage"
-			(at 24.13 118.6684 0)
+			(at 30.48 122.4784 0)
 			(effects
 				(font
@@
 		)
 		(property "Sheetfile" "VoltageBefore.kicad_sch"
-			(at 24.13 135.2046 0)
+			(at 30.48 139.0146 0)
 			(effects
 				(font
@@
 			)
 		)
-		(pin "I_Input" input
-			(at 24.13 125.73 180)
+		(pin "Initial_Input" input
+			(at 30.48 129.54 180)
 			(effects
 				(font
@@
 			)
 		)
-		(pin "R_Input" input
-			(at 24.13 128.27 180)
+		(pin "Regulated_Input" input
+			(at 30.48 132.08 180)
 			(effects
 				(font
@@
 			)
 		)
-		(pin "R_Voltage" output
-			(at 63.5 125.73 0)
+		(pin "Regulated_Voltage" output
+			(at 69.85 129.54 0)
 			(effects
 				(font
@@
 			)
 		)
-		(pin "I_Voltage" output
-			(at 63.5 128.27 0)
+		(pin "Initial_Voltage" output
+			(at 69.85 132.08 0)
 			(effects
 				(font
@@
 	)
 	(sheet
-		(at 24.13 143.51)
+		(at 30.48 147.32)
 		(size 39.37 15.24)
 		(exclude_from_sim no)
@@
 		)
 		(property "Sheetname" "CurrentAfter"
-			(at 24.13 142.7984 0)
+			(at 30.48 146.6084 0)
 			(effects
 				(font
@@
 		)
 		(property "Sheetfile" "currentAfter.kicad_sch"
-			(at 24.13 159.3346 0)
+			(at 30.48 163.1446 0)
 			(effects
 				(font
@@
 			)
 		)
-		(pin "R_Shunt" input
-			(at 24.13 152.4 180)
+		(pin "Regulated_Shunt" input
+			(at 30.48 156.21 180)
 			(effects
 				(font
@@
 			)
 		)
-		(pin "R_Input" input
-			(at 24.13 149.86 180)
+		(pin "Regulated_Input" input
+			(at 30.48 153.67 180)
 			(effects
 				(font
@@
 			)
 		)
-		(pin "R_Current" output
-			(at 63.5 151.13 0)
+		(pin "Regulated_Current" output
+			(at 69.85 154.94 0)
 			(effects
 				(font
@@
 		)
 		(pin "VRef" input
-			(at 24.13 154.94 180)
-			(effects
-				(font
+			(at 30.48 158.75 180)
+			(effects
+				(font

Commit message: 9/27 Workday
Parts:
- removed C2, C9: 1uF, Capacitor_SMD:C_0603_1608Metric_Pad1.08x0.95mm_HandSolder, symbol Device:C
- removed LED3, LED7: WS2812B, WS2812B:WS2812B, symbol WS2812B:WS2812B
Connections:
- no-connect marks 1 -> 11
Other:
- note added: "rip"

Commit message: Address Reviews
Connections:
- net +3.3V: now also J6.7; no longer J6.3
- net GND: now also J6.3, J6.5
- net Initial_Input renamed Unregulated_Initial_V
- net Initial_Shunt renamed Unregulated_Initial_Sense
- net Regulated_Input renamed Regulated_24V
- net Regulated_Shunt renamed Regulated_24V_Sense
- net VRef renamed 1.024V
- no-connect marks 11 -> 9
Other:
- sheet CurrentAfter ports: added 1.024V; removed Regulated_Input, Regulated_Shunt, VRef
- sheet CurrentBefore ports: added 1.024V; removed Initial_Input, Initial_Shunt, VRef
- sheet Voltage ports: added none; removed Initial_Input, Regulated_Input

Commit message: 10/2 changes
Other:
- sheet CurrentAfter ports: added Regulated_24V, Regulated_24V_Sense; removed none
- sheet CurrentBefore ports: added Unregulated_Initial_Sense, Unregulated_Initial_V; removed none
- sheet Voltage ports: added Regulated_24V, Regulated_Out, Unregulated_Initial_V, Unregulated_Out; removed Initial_Voltage, Regulated_Voltage
- note removed: "Adressable LED"
- note removed: "rip"
Changed lines of the file:
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@@
 	(generator_version "9.0")
 	(paper "A4")
-	(text "rip"
-		(exclude_from_sim no)
-		(at 201.422 50.038 0)
-		(effects
-			(font
-				(size 1.27 1.27)
-			)
-		)
-	)
 	(text "Reference Voltage"
 		(exclude_from_sim no)
@@
 		(exclude_from_sim no)
 		(at 68.834 86.36 0)
-		(effects
-			(font
-				(face "FF Comma Trial")
-				(size 1.905 1.905)
-			)
-		)
-	)
-	(text "Adressable LED"
-		(exclude_from_sim no)
-		(at 200.406 21.336 0)
 		(effects
 			(font
@@
 	)
 	(label "Unregulated_Initial_V"
-		(at 34.29 130.81 180)
+		(at 34.29 128.27 180)
 		(effects
 			(font
@@
 			)
 		)
+		(pin "Unregulated_Initial_Sense" input
+			(at 34.29 109.22 180)
+			(effects
+				(font
+					(size 1.27 1.27)
+				)
+				(justify left)
+			)
+		)
+		(pin "Unregulated_Initial_V" input
+			(at 34.29 106.68 180)
+			(effects
+				(font
+					(size 1.27 1.27)
+				)
+				(justify left)
+			)
+		)
 		(instances
 			(project "Supplemental Monitoring PCB"
@@
 			)
 		)
-		(pin "Regulated_Voltage" output
+		(pin "Regulated_24V" input
+			(at 34.29 133.35 180)
+			(effects
+				(font
+					(size 1.27 1.27)
+				)
+				(justify left)
+			)
+		)
+		(pin "Unregulated_Initial_V" input
+			(at 34.29 128.27 180)
+			(effects
+				(font
+					(size 1.27 1.27)
+				)
+				(justify left)
+			)
+		)
+		(pin "Regulated_Out" output
 			(at 73.66 130.81 0)
 			(effects
@@
 			)
 		)
-		(pin "Initial_Voltage" output
+		(pin "Unregulated_Out" output
 			(at 73.66 133.35 0)
 			(effects
@@
 			(effects
 				(font
+					(size 1.27 1.27)
+				)
+				(justify left)
+			)
+		)
+		(pin "Regulated_24V" input
+			(at 34.29 154.94 180)
+			(effects
+				(font
+					(size 1.27 1.27)
+				)
+				(justify left)
+			)
+		)
+		(pin "Regulated_24V_Sense" input
+			(at 34.29 157.48 180)
+			(effects
+				(font

Commit message: starting layout now
Parts:
- IC6: footprint SOT95P280X145-6N -> KiCad:SOT95P280X145-6N
Changed lines of the file:
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@@
 			)
 		)
-		(property "Footprint" "SOT95P280X145-6N"
+		(property "Footprint" "KiCad:SOT95P280X145-6N"
 			(at 223.52 207.95 0)
 			(effects

Commit message: layout,fixedschematic
Parts:
- added H1, H2, H3, H4: MountingHole, MountingHole:MountingHole_3.2mm_M3, symbol Mechanical:MountingHole
- added RCLK1, Reg_Current1, Reg_Sense+1, SER1, SRCLK1, Unreg_Sense+1: Test Point, TestPoint:TestPoint_Pad_1.0x1.0mm, symbol Connector:TestPoint
- added Reg_Sense-1, Reg_V1, Unreg_Current1, Unreg_Sense-1, Unreg_V1: TestPoint, TestPoint:TestPoint_Pad_1.0x1.0mm, symbol Connector:TestPoint
Connections:
- net RCLK: now also RCLK1.1
- net SER: now also SER1.1
- net SRCLK: now also SRCLK1.1
- net RegSense-: now reaches J6.13
- net RegSense-: now also Reg_Sense-1.1
- net Unreg_Sense+: now reaches J6.17
- net Unreg_Sense+: now also Unreg_Sense+1.1
- net Initial_Current renamed Reg_Current
- net Reg_Current: now also Reg_Current1.1
- net Initial_Voltage renamed Unreg_Current
- net Unreg_Current: now also Unreg_Current1.1
- net Regulated_24V renamed Unreg_Sense-
- net Unreg_Sense-: now also Unreg_Sense-1.1
- net Regulated_24V_Sense renamed Reg_Sense+
- net Reg_Sense+: now also Reg_Sense+1.1
- net Regulated_Current renamed Unreg_V
- net Unreg_V: now also Unreg_V1.1
- net Regulated_Voltage renamed Reg_V
- net Reg_V: now also Reg_V1.1
- net Unregulated_Initial_Sense: no longer names the net of J6.15
- net Unregulated_Initial_V renamed Supp_Vin
- no-connect marks 9 -> 8
Other:
- sheet CurrentAfter ports: added Reg_Current, Reg_Sense+, Reg_Sense-; removed Regulated_24V, Regulated_24V_Sense, Regulated_Current
- sheet CurrentBefore ports: added Unreg_Current, Unreg_Sense+, Unreg_Sense-; removed Initial_Current, Unregulated_Initial_Sense, Unregulated_Initial_V
- sheet Voltage ports: added Reg_Sense+, Reg_V, SuppVin, Unreg_V; removed Regulated_24V, Regulated_Out, Unregulated_Initial_V, Unregulated_Out
- moved on the sheet: C3, C4

Commit message: Reviews
Parts:
- added LOGO1: Dr. Hallock, UTSVT_Logos:LHRs_LOGO, symbol utsvt_misc:Logo_Placeholder
- IC6: footprint KiCad:SOT95P280X145-6N -> REF35102QDBVR:SOT95P280X145-6N
Changed lines of the file:
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@@
+	)
+	(symbol
+		(lib_id "utsvt_misc:Logo_Placeholder")
+		(at 200.66 64.77 0)
+		(unit 1)
+		(exclude_from_sim no)
+		(in_bom yes)
+		(on_board yes)
+		(dnp no)
+		(fields_autoplaced yes)
+		(property "Reference" "LOGO1"
+			(at 200.66 60.96 0)
+			(effects
+				(font
+					(size 1.27 1.27)
+				)
+				(hide yes)
+			)
+		)
+		(property "Value" "Dr. Hallock"
+			(at 204.47 64.7699 0)
+			(effects
+				(font
+					(size 1.27 1.27)
+				)
+				(justify left)
+			)
+		)
+		(property "Footprint" "UTSVT_Logos:LHRs_LOGO"
+			(at 200.66 62.865 0)
+			(effects
+				(font
+					(size 1.27 1.27)
+				)
+				(hide yes)
+			)
+		)
+		(property "Datasheet" ""
+			(at 200.66 62.865 0)
+			(effects
+				(font
+					(size 1.27 1.27)
+				)
+				(hide yes)
+			)
+		)
+		(property "Description" "Graph footprint placeholder"
+			(at 200.66 64.77 0)
+			(effects
+				(font
+					(size 1.27 1.27)
+				)
+				(hide yes)
+			)
+		)
+		(property "PN" ""
+			(at 200.66 64.77 0)
+			(effects
+				(font
+					(size 1.27 1.27)
+				)
+				(hide yes)
+			)
+		)
+		(property "p/n" ""
+			(at 200.66 64.77 0)
+			(effects
+				(font
+					(size 1.27 1.27)
+				)
+				(hide yes)
+			)
+		)
+		(instances
+			(project ""
+				(path "/4b30d391-cf39-434b-85dc-df89b45eb2b2"
+					(reference "LOGO1")
+					(unit 1)
+				)
+			)
+		)
 	)
 	(symbol
@@
 			)
 		)
-		(property "Footprint" "KiCad:SOT95P280X145-6N"
+		(property "Footprint" "REF35102QDBVR:SOT95P280X145-6N"
 			(at 223.52 207.95 0)
 			(effects
