File: Hardware/SupplementalMonitoringPCB/VoltageBefore.kicad_sch (KiCad schematic)
At the start: 7 parts, among them IC1 TLV9002QDRQ1

Commit message: Draft
Changed lines of the file:
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@@
 	)
 	(hierarchical_label "I_Voltage"
-		(shape input)
+		(shape output)
 		(at 52.07 121.92 180)
 		(effects

Commit message: labels
Connections:
- net I_Input renamed Initial_Input
- net I_Voltage renamed Initial_Voltage
- net R_Input renamed Regulated_Input
- net R_Voltage renamed Regulated_Voltage
Changed lines of the file:
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@@
 		)
 	)
-	(hierarchical_label "I_Input"
+	(hierarchical_label "Initial_Input"
 		(shape input)
 		(at 66.04 36.83 0)
@@
 		)
 	)
-	(hierarchical_label "R_Voltage"
+	(hierarchical_label "Regulated_Voltage"
 		(shape output)
 		(at 92.71 124.46 0)
@@
 		)
 	)
-	(hierarchical_label "R_Input"
+	(hierarchical_label "Regulated_Input"
 		(shape input)
 		(at 34.29 36.83 0)
@@
 		)
 	)
-	(hierarchical_label "I_Voltage"
+	(hierarchical_label "Initial_Voltage"
 		(shape output)
 		(at 52.07 121.92 180)

Commit message: 9/27 Workday
Parts:
- R10, R8: value 45k -> 9k
- R13, R19: value 10k -> 1k
Other:
- note added: "24(1/1+9) = 2.4"
- note added: "30(10/10+45) = 3.0 18(10/10+45) = 1.8"
- note added: "OpAmp+ -> Input Range: 1.8 V-3.0 V"
- note added: "OpAmp2+ -> Input Range: 2.4 V"
- moved on the sheet: R10, R13, R19, R8

Commit message: Address Reviews
Parts:
- removed C5, C7: 1u, symbol Device:C
- added C19, C20: 1u, symbol Device:C
- added TP5, TP6, TP7, TP8: TestPoint, symbol Connector:TestPoint
Connections:
- net GND: now also C19.2, C20.2
- net OpAmp+: now also TP7.1
- net OpAmp2+: now also TP6.1
- net Initial_Input renamed Unregulated_Initial_V
- net Initial_Voltage renamed Unregulated_Out
- net Unregulated_Out: now also C20.1, TP8.1
- net Regulated_Input renamed Regulated_24V
- net Regulated_Voltage renamed Regulated_Out
- net Regulated_Out: now also C19.1, TP5.1

Commit message: 10/2 changes
Parts:
- removed C19, C20: 1u, symbol Device:C
- added C21, C24: 4.64u, symbol Device:C
- added C22, C23: 2.05u, symbol Device:C
- added C25, C26: 1u, symbol Device:C
- added IC7: TLV9002QDRQ1, SOIC127P600X175-8N, symbol TLV9002QDRQ1:TLV9002QDRQ1
- added R31, R40: 9.53k, symbol Device:R
- added R32, R41: 13k, symbol Device:R
- added RegulatedVoltageIn2, RegulatedVoltageOut2, UnegulatedVoltageOut2, UnregulatedVoltageIn2: TestPoint, symbol Connector:TestPoint
- renumbered TP6 to RegulatedVoltageIn1, TP5 to RegulatedVoltageOut1, TP8 to UnegulatedVoltageOut1, TP7 to UnregulatedVoltageIn1
Connections:
- net +3.3V: now also C25.1, C26.1
- net GND: now also C21.2, C24.2, C25.2, C26.2, IC7.3 (IN1+), IC7.4 (V-), IC7.5 (IN2+), IC7.6 (IN2-)
- net Regulated_Out: now also C23.2, IC7.8 (V+), RegulatedVoltageOut2.1; no longer IC1.6 (IN2-), IC1.7 (OUT2), RegulatedVoltageOut1.1
- net Unregulated_Out: now also C22.2, IC7.1 (OUT1), UnegulatedVoltageOut2.1; no longer IC1.1 (OUT1), IC1.2 (IN1-), UnegulatedVoltageOut1.1
- new net: C22.1, R31.2, R32.1
- new net: C23.1, R40.2, R41.1
- new net: C24.1, IC7.7 (OUT2), R41.2
- new net: C21.1, IC7.2 (IN1-), R32.2
- new net Out1: IC1.1 (OUT1), IC1.2 (IN1-), R31.1, UnegulatedVoltageOut1.1, UnregulatedVoltageIn2.1
- new net Out2: IC1.6 (IN2-), IC1.7 (OUT2), R40.1, RegulatedVoltageIn2.1, RegulatedVoltageOut1.1
Other:
- note added: "Low Pass Filter"
- note added: "Op Amp Gain of 0"

Commit message: starting layout now
Parts:
- C21, C22, C23, C24, C25, C26: footprint (none) -> Capacitor_SMD:C_0603_1608Metric_Pad1.08x0.95mm_HandSolder
- IC1, IC7: footprint SOIC127P600X175-8N -> TLV9002QDRQ1:SOIC127P600X175-8N
- R10, R13, R19, R31, R32, R40, R41, R8: footprint (none) -> Resistor_SMD:R_0603_1608Metric_Pad0.98x0.95mm_HandSolder
- RegulatedVoltageIn1, RegulatedVoltageIn2, RegulatedVoltageOut1, RegulatedVoltageOut2, UnegulatedVoltageOut1, UnegulatedVoltageOut2, UnregulatedVoltageIn1, UnregulatedVoltageIn2: footprint (none) -> TestPoint:TestPoint_Pad_1.0x1.0mm
Changed lines of the file:
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@@
 			"AAAAAAAAAAAAAAAAAAAAAAAAAAAAAAAAAAAAAAAAAAAAAAAAAAAAAAAAAAAAAAAAAAAAAAAAAAAA"
 			"AAAAAAAAAAAAAAAAAAAAAAAAAAAAAAAAAAAAAAAAAAAAAAAAAAAAAAAAAAAAAAAAAAAAAAAAAAAA"
-			"AAAAAAAAAAAAAAAAAAAAAAAAAAAAAAAAAAAAAA=="
+			"AAAAAAAAAAAAAAAAAAAAAAAAAAAAAAAAAAAAAAClzi1YAB4BgAAAAAAAAAAABAAAAAAAAAABAAAA"
+			"AAAAAAEAAAAAAAAAAAAAAAAAAACgzihYAB8BgAAAAAAAAAAAAwAAAAAAAACwQTjA5QEAAAEAAAAA"
+			"AAAAAAAAAAAAAACjzidYACABgJDkR8DlAQAAAwAAAAAAAAAgVh/A5QEAAAEAAAAAAAAAAAAAAAAA"
+			"AAC+ziJYACEBgJDnR8DlAQAAAwAAAAAAAADQVR/A5QEAAAEAAAAAAAAAAAAAAAAAAAC5ziFYACIB"
+			"gHDpR8DlAQAAAwAAAAAAAAAQVh/A5QEAAAEAAAAAAAAAAAAAAAAAAAC0zjxYACMBgIDlR8DlAQAA"
+			"AwAAAAAAAAAwVh/A5QEAAAEAAAAAAAAAAAAAAAAAAAC3zjtYACQBgGDnR8DlAQAAAwAAAAAAAAAg"
+			"Ux/A5QEAAAEAAAAAAAAAAAAAAAAAAACyzjZYACUBgFDiR8DlAQAAAwAAAAAAAAAQRzjA5QEAAAEA"
+			"AAAAAAAAAAAAAAAAAABNzjVYACYBgAAAAAAAAAAAAwAAAAAAAAAQVB/A5QEAAAEAAAAAAAAAAAAA"
+			"AAAAAABIzjBYACcBgAAAAAAAAAAACAAAAAAAAABQ4UbA5QEAAAEAAAAAAAAAAAAAAAAAAABLzs9Y"
+			"ACgBgAAAAAAAAAAACAAAAAAAAACQ70bA5QEAAAEAAAAAAAAAAAAAAAAAAABGzspYACkBgPDnR8Dl"
+			"AQAAAwAAAAAAAACQRzjA5QEAAAEAAAAAAAAAAAAAAAAAAABBzslYACoBgEDpR8DlAQAAAwAAAAAA"
+			"AACgVR/A5QEAAAEAAAAAAAAAAAAAAAAAAABczsRYACsBgJDhR8DlAQAAAwAAAAAAAADQQTjA5QEA"
+			"AAEAAAAAAAAAAAAAAAAAAABfzsNYACwBgFDlR8DlAQAAAwAAAAAAAABAUx/A5QEAAAEAAAAAAAAA"
+			"AAAAAAAAAABazt5YAC0BgAAAAAAAAAAAAwAAAAAAAAAwUx/A5QEAAAEAAAAAAAAAAAAAAAAAAABV"
+			"zt1YAC4BgAAAAAAAAAAAAwAAAAAAAAAgVR/A5QEAAAEAAAAAAAAAAAAAAAAAAABQzthYAC8BgHDs"
+			"R8DlAQAAAwAAAAAAAACQVB/A5QEAAAEAAAAAAAAAAAAAAAAAAABTztdYADABgEM6L1dJTkRPV1Mv"
+			"Zm9udHNcQlJMTlNEQi5UVEYAAAAAAAAAAAAAAABuztJYADEBgGDqR8DlAQAAAwAAAAAAAACgUx/A"
+			"5QEAAAEAAAAAAAAAAAAAAAAAAABpztFYADIBgJDqR8DlAQAAAwAAAAAAAABwVh/A5QEAAAEAAAAA"
+			"AAAAAAAAAAAAAABkzuxYADMBgMDqR8DlAQAAAwAAAAAAAAAAAAAAAAAAAHWMuYUA0AKAAAAAAAAA"
+			"AAAIAAAAAAAAANAhvOmsAQAAAQAAAAAAAAAAAAAAAAAAAHaMRIUA0QKAAAAAAAAAAAADAAAAAAAA"
+			"AJCN/umsAQAAAQAAAAAAAAAAAAAAAAAAAHuMQ4UA0gKAAAAAAAAAAAAEAAAAAAAAAAEAAAAAAAAA"
+			"AQAAAAAAAAAAAAAAAAAAAHyMToUA0wKA0I/+6awBAAADAAAAAAAAAFD1/emsAQAAAQAAAAAAAAAA"
+			"AAAAAAAAAGGMTYUA1AKAAAAAAAAAAAADAAAAAAAAAFD4/emsAQAAAQAAAAAAAAAAAAAAAAAAAGKM"
+			"SIUA1QKAAAAAAAAAAAADAAAAAAAAAHCJ/umsAQAAAQAAAAAAAAAAAAAAAAAAAGeMV4UA1gKAQzov"
+			"V0lORE9XUy9mb250c1xDYW5kYXJhbC50dGYAAAAAAAAAAAAAAGiMUoUA1wKAAAAAAAAAAAADAAAA"
+			"AAAAAMD4/emsAQAAAQAAAAAAAAAAAAAAAAAAAG2MUYUA2AKAAAAAAAAAAAAEAAAAAAAAAAEAAAAA"
+			"AAAAAQAAAAAAAAAAAAAAAAAAAG6MXIUA2QKAQzovV0lORE9XUy9mb250c1xDYW5kYXJhbGkudHRm"
+			"AAAAAAAAAAAAAFOMW4UA2gKAAAAAAAAAAAAIAAAAAAAAAFAovOmsAQAAAQAAAAAAAAAAAAAAAAAA"
+			"AFSMZoUA2wKAsIX+6awBAAADAAAAAAAAAPD0/emsAQAAAQAAAAAAAAAAAAAAAAAAAFmMZYUA3AKA"
+			"AAAAAAAAAAADAAAAAAAAALD3/emsAQAAAQAAAAAAAAAAAAAAAAAAAFqMYIUA3QKAgI7+6awBAAAD"
+			"AAAAAAAAAFC+8+msAQAAAQAAAAAAAAAAAAAAAAAAAF+Mb4UA3gKAAAAAAAAAAAAEAAAAAAAAAAEA"
+			"AAAAAAAAAQAAAAAAAAAAAAAAAAAAAECMaoUA3wKAYJD+6awBAAADAAAAAAAAAJC98+msAQAAAQAA"
+			"AAAAAAAAAAAAAAAAAEWMaYUA4AKAoI/+6awBAAADAAAAAAAAAHDA8+msAQAAAQAAAAAAAAAAAAAA"
+			"AAAAAEaMdIUA4QKAAAAAAAAAAAADAAAAAAAAAHC68+msAQAAAQAAAAAAAAAAAAAAAAAAAEuMc4UA"
+			"4gKAwIr+6awBAAADAAAAAAAAAED3/emsAQAAAQAAAAAAAAAAAAAAAAAAAEyMfoUA4wKAAAAAAAAA"
+			"AAADAAAAAAAAAGD4/emsAQAAAQAAAAAAAAAAAAAAAAAAADGMfYUA5AKAQzovV0lORE9XUy9mb250"
+			"c1xDVVJMWl9fXy5UVEYAAAAAAAAAAAAAADKMeA=="
 		)
 	)
@@
 			)
 		)
-		(property "Footprint" ""
+		(property "Footprint" "TestPoint:TestPoint_Pad_1.0x1.0mm"
 			(at 40.64 121.92 0)
 			(effects
@@
 			)
 		)
-		(property "Footprint" ""
+		(property "Footprint" "Resistor_SMD:R_0603_1608Metric_Pad0.98x0.95mm_HandSolder"
 			(at 171.45 130.048 90)
 			(effects
@@
 			)
 		)
-		(property "Footprint" "SOIC127P600X175-8N"
+		(property "Footprint" "TLV9002QDRQ1:SOIC127P600X175-8N"
 			(at 82.55 216.84 0)
 			(effects
@@
 			)
 		)
-		(property "Footprint" ""
+		(property "Footprint" "TestPoint:TestPoint_Pad_1.0x1.0mm"
 			(at 275.59 128.27 0)
 			(effects
@@
 			)
 		)
-		(property "Footprint" ""
+		(property "Footprint" "Resistor_SMD:R_0603_1608Metric_Pad0.98x0.95mm_HandSolder"
 			(at 192.532 53.34 90)
 			(effects
@@
 			)
 		)
-		(property "Footprint" ""
+		(property "Footprint" "Resistor_SMD:R_0603_1608Metric_Pad0.98x0.95mm_HandSolder"
 			(at 160.782 53.34 90)
 			(effects
@@
 			)
 		)
-		(property "Footprint" ""
+		(property "Footprint" "TestPoint:TestPoint_Pad_1.0x1.0mm"
 			(at 63.5 127 0)
 			(effects
@@
 			)
 		)
-		(property "Footprint" ""
+		(property "Footprint" "TestPoint:TestPoint_Pad_1.0x1.0mm"
 			(at 105.41 124.46 0)
 			(effects
@@
 			)
 		)
-		(property "Footprint" ""
+		(property "Footprint" "Capacitor_SMD:C_0603_1608Metric_Pad1.08x0.95mm_HandSolder"
 			(at 191.77 110.7948 0)
 			(effects
@@
 			)
 		)
-		(property "Footprint" ""
+		(property "Footprint" "TestPoint:TestPoint_Pad_1.0x1.0mm"
 			(at 81.28 132.08 0)
 			(effects
@@
 			)
 		)
-		(property "Footprint" ""
+		(property "Footprint" "Resistor_SMD:R_0603_1608Metric_Pad0.98x0.95mm_HandSolder"
 			(at 251.46 130.048 90)
 			(effects
@@
 			)
 		)
-		(property "Footprint" ""
+		(property "Footprint" "Resistor_SMD:R_0603_1608Metric_Pad0.98x0.95mm_HandSolder"
 			(at 182.88 130.048 90)
 			(effects
@@
 			)
 		)
-		(property "Footprint" ""
+		(property "Footprint" "Capacitor_SMD:C_0603_1608Metric_Pad1.08x0.95mm_HandSolder"
 			(at 242.57 110.7948 0)
 			(effects
@@
 			)
 		)
-		(property "Footprint" ""
+		(property "Footprint" "Capacitor_SMD:C_0603_1608Metric_Pad1.08x0.95mm_HandSolder"
 			(at 188.9252 135.89 0)
 			(effects
@@
 			)
 		)
-		(property "Footprint" ""
+		(property "Footprint" "Capacitor_SMD:C_0603_1608Metric_Pad1.08x0.95mm_HandSolder"
 			(at 277.8252 153.67 0)
 			(effects
@@
 			)
 		)
-		(property "Footprint" "SOIC127P600X175-8N"
+		(property "Footprint" "TLV9002QDRQ1:SOIC127P600X175-8N"
 			(at 227.33 220.65 0)
 			(effects
@@
 			)
 		)
-		(property "Footprint" ""
+		(property "Footprint" "Resistor_SMD:R_0603_1608Metric_Pad0.98x0.95mm_HandSolder"
 			(at 153.67 46.228 90)
 			(effects
@@
 			)
 		)
-		(property "Footprint" ""
+		(property "Footprint" "TestPoint:TestPoint_Pad_1.0x1.0mm"
 			(at 158.75 128.27 0)
 			(effects
@@
 			)
 		)
-		(property "Footprint" ""
+		(property "Footprint" "Capacitor_SMD:C_0603_1608Metric_Pad1.08x0.95mm_HandSolder"
 			(at 124.1552 161.29 0)
 			(effects
@@
 			)
 		)
-		(property "Footprint" ""
+		(property "Footprint" "TestPoint:TestPoint_Pad_1.0x1.0mm"
 			(at 205.74 125.73 0)
 			(effects
@@
 			)
 		)
-		(property "Footprint" ""
+		(property "Footprint" "Resistor_SMD:R_0603_1608Metric_Pad0.98x0.95mm_HandSolder"
 			(at 262.89 130.048 90)
 			(effects
@@
 			)
 		)
-		(property "Footprint" ""
+		(property "Footprint" "Capacitor_SMD:C_0603_1608Metric_Pad1.08x0.95mm_HandSolder"
 			(at 245.4148 135.89 0)
 			(effects
@@
 			)
 		)
-		(property "Footprint" ""
+		(property "Footprint" "TestPoint:TestPoint_Pad_1.0x1.0mm"
 			(at 228.6 125.73 0)
 			(effects
@@
 			)
 		)
-		(property "Footprint" ""
+		(property "Footprint" "Resistor_SMD:R_0603_1608Metric_Pad0.98x0.95mm_HandSolder"
 			(at 185.42 46.228 90)
 			(effects

Commit message: layout,fixedschematic
Parts:
- removed RegulatedVoltageIn2, RegulatedVoltageOut1, RegulatedVoltageOut2, UnegulatedVoltageOut1, UnegulatedVoltageOut2, UnregulatedVoltageIn2: TestPoint, TestPoint:TestPoint_Pad_1.0x1.0mm, symbol Connector:TestPoint
- renumbered RegulatedVoltageIn1 to RegVdiv1, UnregulatedVoltageIn1 to Unreg_Vdiv1
Connections:
- net Regulated_24V renamed Reg_Sense+
- net Regulated_Out renamed Reg_V
- net Unregulated_Initial_V renamed SuppVin
- net Unregulated_Out renamed Unreg_V
Other:
- moved on the sheet: C21, C24, C26, R40, RegVdiv1, Unreg_Vdiv1
