File: Hardware/SupplementalMonitoringPCB/currentAfter.kicad_sch (KiCad schematic)
At the start: 12 parts, among them IC3 TLV9002QDRQ1, IC4 INA241A5IDR

Commit message: Draft
Connections:
- net +1V0: no longer IC4.3 (REF2)
- new net VRef: IC4.3 (REF2)
Changed lines of the file:
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@@
+		)
+	)
+	(hierarchical_label "VRef"
+		(shape input)
+		(at 58.42 137.16 180)
+		(effects
+			(font
+				(size 1.27 1.27)
+			)
+			(justify right)
 		)
 	)
@@
 					(unit 1)
 				)
-			)
-		)
-	)
-	(symbol
-		(lib_id "power:+1V0")
-		(at 58.42 137.16 0)
-		(unit 1)
-		(exclude_from_sim no)
-		(in_bom yes)
-		(on_board yes)
-		(dnp no)
-		(property "Reference" "#PWR020"
-			(at 58.42 140.97 0)
-			(effects
-				(font
-					(size 1.27 1.27)
-				)
-				(hide yes)
-			)
-		)
-		(property "Value" "+1V0"
-			(at 53.594 136.652 0)
-			(effects
-				(font
-					(size 1.27 1.27)
-				)
-			)
-		)
-		(property "Footprint" ""
-			(at 58.42 137.16 0)
-			(effects
-				(font
-					(size 1.27 1.27)
-				)
-				(hide yes)
-			)
-		)
-		(property "Datasheet" ""
-			(at 58.42 137.16 0)
-			(effects
-				(font
-					(size 1.27 1.27)
-				)
-				(hide yes)
-			)
-		)
-		(property "Description" "Power symbol creates a global label with name \"+1V0\""
-			(at 58.42 137.16 0)
-			(effects
-				(font
-					(size 1.27 1.27)
-				)
-				(hide yes)
-			)
-		)
-		(pin "1"
-		)
-		(instances
-			(project "Supplemental Monitoring PCB"
-				(path "/4b30d391-cf39-434b-85dc-df89b45eb2b2/e6ad27a4-998d-404c-8222-a3ba4eac724d"
-					(reference "#PWR020")
-					(unit 1)
-				)

Commit message: labels
Connections:
- net R_Current renamed Regulated_Current
- net R_Input renamed Regulated_Input
- net R_Shunt renamed Regulated_Shunt
Changed lines of the file:
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@@
 		)
 	)
-	(text "200 gain\n OpAmp"
+	(text "200 gain OpAmp"
 		(exclude_from_sim no)
-		(at 27.686 58.166 0)
+		(at 30.734 56.388 0)
 		(effects
 			(font
@@
 		)
 	)
-	(hierarchical_label "R_Input"
+	(hierarchical_label "Regulated_Input"
 		(shape input)
 		(at 115.57 44.45 0)
@@
 		)
 	)
-	(hierarchical_label "R_Current"
+	(hierarchical_label "Regulated_Current"
 		(shape output)
 		(at 238.76 130.81 0)
@@
 		)
 	)
-	(hierarchical_label "R_Shunt"
+	(hierarchical_label "Regulated_Shunt"
 		(shape input)
 		(at 88.9 44.45 0)

Commit message: 9/27 Workday
Other:
- note added: "1.75 x 1.8 = 3.15"
- note added: "18(1/1+4.5) = 3.27"
- note added: "200(-0.00125) = -0.25"
- note added: "200(0.0075) = 1.5"
- note added: "30(1/1+4.5) = 5.45"
- note added: "Max Current: 30(250E-6)"
- note added: "Min Current: -5(250E-6)"
- note added: "Op Amp Gain of 1.8"
- note added: "Range of 1.75 V (-.25 to 1.5)"
- note added: "Voltage Difference Range:"
- note added: "Voltage input Range for OpAmp: 3.27-5.45"
- note added: "Vout = 1.75 + 1.024 (close to 3.3)"
- note removed: "shunt resistor: ULR3N-R00025JT2"
- moved on the sheet: R15, R16, R17, R18

Commit message: Address Reviews
Parts:
- added TP15, TP16, TP17, TP18, TP19, TP20: TestPoint, symbol Connector:TestPoint
Connections:
- net VRef is gone; now on net 1.024V: IC4.3 (REF2)
- net Out1: now also TP17.1, TP18.1
- net Out2: now also TP19.1
- net Regulated_Current: now also TP20.1
- net Sense+: now also IC4.8 (IN+), TP16.1; no longer IC4.1 (IN-)
- net Sense-: now also IC4.1 (IN-), TP15.1; no longer IC4.8 (IN+)
- net +1V0 renamed 1.024V
- net Regulated_Input renamed Regulated_24V
- net Regulated_Shunt renamed Regulated_24V_Sense

Commit message: 10/2 changes
Parts:
- added C29, C30: 1u, symbol Device:C
- C10: value 1u -> .1u
- RegulatedCurentOut3: renamed from TP20; value TestPoint -> Test Point
- RegulatedCurrentIn1: renamed from TP18; value TestPoint -> Test Point
- TP16: value TestPoint -> RegulatedSense+
- renumbered TP19 to RegulatedCurentOut2, TP15 to RegulatedSense-, TP17 to UnregulatedCurrentOut1
Connections:
- net +3.3V: now also C29.1, C30.1
- net GND: now also C29.2, C30.2
Other:
- moved on the sheet: C14

Commit message: starting layout now
Parts:
- removed R15, R17: 4.5k, symbol Device:R
- removed R16, R18: 1k, symbol Device:R
- C10, C14, C15, C29, C30: footprint (none) -> Capacitor_SMD:C_0603_1608Metric_Pad1.08x0.95mm_HandSolder
- IC3, IC4: footprint SOIC127P600X175-8N -> TLV9002QDRQ1:SOIC127P600X175-8N
- R6, R7, R9: footprint (none) -> Resistor_SMD:R_0603_1608Metric_Pad0.98x0.95mm_HandSolder
- RegulatedCurentOut2, RegulatedCurentOut3, RegulatedCurrentIn1, TP16: footprint (none) -> TestPoint:TestPoint_Pad_1.0x1.0mm
- RegulatedCurrentOut1: renamed from UnregulatedCurrentOut1; footprint (none) -> TestPoint:TestPoint_Pad_1.0x1.0mm
- RegulatedSense-1: renamed from RegulatedSense-; footprint (none) -> TestPoint:TestPoint_Pad_1.0x1.0mm
Connections:
- net Sense+ is gone; now on net Regulated_24V: IC4.8 (IN+), TP16.1
- net Sense- is gone; now on net Regulated_24V_Sense: IC4.1 (IN-), RegulatedSense-1.1
Other:
- note removed: "18(1/1+4.5) = 3.27"
- note removed: "30(1/1+4.5) = 5.45"
- note removed: "Voltage input Range for OpAmp: 3.27-5.45"

Commit message: layout,fixedschematic
Parts:
- removed RegulatedCurentOut3: Test Point, TestPoint:TestPoint_Pad_1.0x1.0mm, symbol Connector:TestPoint
- removed RegulatedCurrentOut1, RegulatedSense-1: TestPoint, TestPoint:TestPoint_Pad_1.0x1.0mm, symbol Connector:TestPoint
- removed TP16: RegulatedSense+, TestPoint:TestPoint_Pad_1.0x1.0mm, symbol Connector:TestPoint
- renumbered RegulatedCurrentIn1 to Reg_CurrentIn1, RegulatedCurentOut2 to Reg_Current_Filter1
Connections:
- net Regulated_24V renamed Reg_Sense+
- net Regulated_24V_Sense renamed Reg_Sense-
- net Regulated_Current renamed Reg_Current
Other:
- moved on the sheet: C10, Reg_CurrentIn1, Reg_Current_Filter1
