File: Hardware/SuppMonTesterPCB/SuppMonTester.kicad_pcb (KiCad board)
At the start: 2 copper layers, 18 parts, among them J1 53307-2471, J2 UNREG+, J3 SHIFT_REG, J4 REG+, J5 GND, J6 UNREG-, J7 REG-

Commit message: layout or smth
Parts:
- moved J6 104.0 mm to (88.5, 44.5)
- moved R4 99.3 mm to (38.6, 53.5), turned to 180 degrees
- moved R6 97.3 mm to (40.4, 93.2), turned to 180 degrees
- moved R5 95.4 mm to (41.1, 111.2), turned to 180 degrees
- moved R3 94.5 mm to (39.6, 69.7), turned to 180 degrees
- moved TP1 81.9 mm to (101.8, 123.2)
- moved TP2 79.9 mm to (108.8, 123.2)
- moved TP3 77.6 mm to (116.2, 123.2)
- moved TP4 75.5 mm to (123.8, 123.2)
- moved TPe 66.7 mm to (145.0, 123.5)
- moved J3 62.1 mm to (133.0, 123.2), turned to 90 degrees
- moved J1 48.6 mm to (118.9, 83.6)
- moved J7 24.7 mm to (88.5, 122.5)
- renumbered TP5 to TPe
Other:
- board outline added: 140.2 x 101 mm
- board text added: "GND"
- board text added: "RCLK"
- board text added: "REG CURRENT"
- board text added: "REG VOLTAGE"
- board text added: "SER"
- board text added: "SHIFT REGISTER"
- board text added: "SRCLK"
- board text added: "UNREG CURRENT"
- board text added: "UNREG VOLTAGE"

Commit message: smth
Parts:
- moved R1 23.2 mm to (53.2, 62.8), turned to 180 degrees
- moved R2 23.2 mm to (53.2, 104.0), turned to 180 degrees
- moved R6 3.25 mm to (40.4, 96.5)
- moved R4 2.47 mm to (40.4, 55.2)
- moved R3 0.92 mm to (40.4, 70.2)
- moved R5 0.92 mm to (40.4, 111.8)
Routing:
- added copper zone on F.Cu, net GND
Other:
- board size 140.2 x 101 mm -> 140.2 x 93.8 mm
- board text added: "REG SENSE+"
- board text added: "REG SENSE-"
- board text added: "UNREG SENSE+"
- board text added: "UNREG SENSE-"
Changed lines of the file:
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@@
 	(footprint "Resistor_SMD:R_1225_3264Metric_Pad1.47x6.45mm_HandSolder"
 		(layer "F.Cu")
-		(at 76.5 62.75)
+		(at 53.25 62.75 180)
 		(descr "Resistor SMD 1225 (3264 Metric), square (rectangular) end terminal, IPC-7351 nominal with elongated pad for handsoldering. (Body size source: https://www.koaspeer.com/pdfs/WK73S.pdf), generated with kicad-footprint-generator")
 		(tags "resistor handsolder")
@@
 		)
 		(property "P/N" "ULR3N-R00025JT2"
-			(at 0 0 0)
+			(at 0 0 180)
 			(unlocked yes)
 			(layer "F.Fab")
@@
 		(attr smd)
 		(fp_line
-			(start -0.502064 -3.26)
-			(end 0.502064 -3.26)
+			(start -0.502064 3.26)
+			(end 0.502064 3.26)
 			(stroke
 				(width 0.12)
@@
 		)
 		(fp_line
-			(start -0.502064 3.26)
-			(end 0.502064 3.26)
+			(start -0.502064 -3.26)
+			(end 0.502064 -3.26)
 			(stroke
 				(width 0.12)
@@
 		)
 		(fp_line
-			(start -2.4 -3.48)
-			(end 2.4 -3.48)
+			(start 2.4 3.48)
+			(end -2.4 3.48)
 			(stroke
 				(width 0.05)
@@
 		)
 		(fp_line
-			(start -2.4 3.48)
-			(end -2.4 -3.48)
+			(start 2.4 -3.48)
+			(end 2.4 3.48)
 			(stroke
 				(width 0.05)
@@
 		)
 		(fp_line
-			(start 2.4 -3.48)
-			(end 2.4 3.48)
+			(start -2.4 3.48)
+			(end -2.4 -3.48)
 			(stroke
 				(width 0.05)
@@
 		)
 		(fp_line
-			(start 2.4 3.48)
-			(end -2.4 3.48)
+			(start -2.4 -3.48)
+			(end 2.4 -3.48)
 			(stroke
 				(width 0.05)
@@
 		)
 		(fp_line
-			(start -1.55 -3.15)
-			(end 1.55 -3.15)
+			(start 1.55 3.15)
+			(end -1.55 3.15)
 			(stroke
 				(width 0.1)
@@
 		)
 		(fp_line
-			(start -1.55 3.15)
-			(end -1.55 -3.15)
+			(start 1.55 -3.15)
+			(end 1.55 3.15)
 			(stroke
 				(width 0.1)
@@
 		)
 		(fp_line
-			(start 1.55 -3.15)
-			(end 1.55 3.15)
+			(start -1.55 3.15)
+			(end -1.55 -3.15)
 			(stroke
 				(width 0.1)
@@
 		)
 		(fp_line
-			(start 1.55 3.15)
-			(end -1.55 3.15)
+			(start -1.55 -3.15)
+			(end 1.55 -3.15)
 			(stroke
 				(width 0.1)
@@
 		)
 		(pad "1" smd roundrect
-			(at -1.4125 0)
+			(at -1.4125 0 180)
 			(size 1.475 6.45)
 			(layers "F.Cu" "F.Mask" "F.Paste")
@@
 		)
 		(pad "2" smd roundrect
-			(at 1.4125 0)
+			(at 1.4125 0 180)
 			(size 1.475 6.45)
 			(layers "F.Cu" "F.Mask" "F.Paste")
@@
 	(footprint "Parts:RES_PWR263S-35-3300F"
 		(layer "F.Cu")
-		(at 40.365 93.21 180)
+		(at 40.365 96.46 180)
 		(property "Reference" "R6"
 			(at 0.175 -6.135 0)
@@
 	(footprint "Parts:RES_PWR263S-35-3300F"
 		(layer "F.Cu")
-		(at 41.115 111.21 180)
+		(at 40.365 111.75 180)
 		(property "Reference" "R5"
 			(at 0.175 -6.135 0)
@@
 	(footprint "Resistor_SMD:R_1225_3264Metric_Pad1.47x6.45mm_HandSolder"
 		(layer "F.Cu")
-		(at 76.5 104)
+		(at 53.25 104 180)
 		(descr "Resistor SMD 1225 (3264 Metric), square (rectangular) end terminal, IPC-7351 nominal with elongated pad for handsoldering. (Body size source: https://www.koaspeer.com/pdfs/WK73S.pdf), generated with kicad-footprint-generator")
 		(tags "resistor handsolder")
@@
 		)
 		(property "P/N" "ULR3N-R00025JT2"
-			(at 0 0 0)
+			(at 0 0 180)
 			(unlocked yes)
 			(layer "F.Fab")
@@
 		(attr smd)
 		(fp_line
-			(start -0.502064 -3.26)
-			(end 0.502064 -3.26)
+			(start -0.502064 3.26)
+			(end 0.502064 3.26)
 			(stroke
 				(width 0.12)
@@
 		)
 		(fp_line
-			(start -0.502064 3.26)
-			(end 0.502064 3.26)
+			(start -0.502064 -3.26)
+			(end 0.502064 -3.26)
 			(stroke
 				(width 0.12)
@@
 		)
 		(fp_line
-			(start -2.4 -3.48)
-			(end 2.4 -3.48)
+			(start 2.4 3.48)
+			(end -2.4 3.48)
 			(stroke
 				(width 0.05)
@@
 		)
 		(fp_line
-			(start -2.4 3.48)
-			(end -2.4 -3.48)
+			(start 2.4 -3.48)
+			(end 2.4 3.48)
 			(stroke
 				(width 0.05)
@@
 		)
 		(fp_line
-			(start 2.4 -3.48)
-			(end 2.4 3.48)
+			(start -2.4 3.48)
+			(end -2.4 -3.48)
 			(stroke
 				(width 0.05)
@@
 		)
 		(fp_line
-			(start 2.4 3.48)
-			(end -2.4 3.48)
+			(start -2.4 -3.48)
+			(end 2.4 -3.48)
 			(stroke
 				(width 0.05)
@@
 		)
 		(fp_line
-			(start -1.55 -3.15)
-			(end 1.55 -3.15)
+			(start 1.55 3.15)
+			(end -1.55 3.15)
 			(stroke
 				(width 0.1)
@@
 		)
 		(fp_line
-			(start -1.55 3.15)
-			(end -1.55 -3.15)
+			(start 1.55 -3.15)
+			(end 1.55 3.15)
 			(stroke
 				(width 0.1)
@@
 		)
 		(fp_line
-			(start 1.55 -3.15)
-			(end 1.55 3.15)
+			(start -1.55 3.15)
+			(end -1.55 -3.15)
 			(stroke
 				(width 0.1)
@@
 		)
 		(fp_line
-			(start 1.55 3.15)
-			(end -1.55 3.15)
+			(start -1.55 -3.15)
+			(end 1.55 -3.15)
 			(stroke
 				(width 0.1)
@@
 		)
 		(pad "1" smd roundrect
-			(at -1.4125 0)
+			(at -1.4125 0 180)
 			(size 1.475 6.45)
 			(layers "F.Cu" "F.Mask" "F.Paste")
@@
 		)
 		(pad "2" smd roundrect
-			(at 1.4125 0)
+			(at 1.4125 0 180)
 			(size 1.475 6.45)
 			(layers "F.Cu" "F.Mask" "F.Paste")
@@
 	(footprint "Parts:RES_PWR263S-35-3300F"
 		(layer "F.Cu")
-		(at 39.615 69.71 180)
+		(at 40.365 70.25 180)
 		(property "Reference" "R3"
 			(at 0.175 -6.135 0)
@@
 	(footprint "Parts:RES_PWR263S-35-3300F"
 		(layer "F.Cu")
-		(at 38.615 53.46 180)
+		(at 40.365 55.21 180)
 		(property "Reference" "R4"
 			(at 0.175 -6.135 0)
@@
 	)
 	(gr_rect
-		(start 26 33.25)
-		(end 166.25 134.25)
+		(start 26 37.5)
+		(end 166.25 131.25)
 		(stroke
 			(width 0.05)
@@
 		)
 	)
+	(gr_text "GND"
+		(at 55 83.5 0)
+		(layer "F.SilkS" knockout)
+		(effects
+			(font
+				(size 1 1)
+				(thickness 0.15)
+			)
+		)
+	)
 	(gr_text "UNREG\nVOLTAGE"
 		(at 101.75 127.5 0)
@@
 		)
 	)
+	(gr_text "REG\nSENSE+"
+		(at 62.75 111 0)
+		(layer "F.SilkS" knockout)
+		(effects
+			(font
+				(size 1 1)
+				(thickness 0.15)
+			)
+		)
+	)
+	(gr_text "UNREG\nSENSE-"
+		(at 79.25 44.5 0)
+		(layer "F.SilkS" knockout)
+		(effects
+			(font
+				(size 1 1)
+				(thickness 0.15)
+			)
+		)
+	)
 	(gr_text "SER"
 		(at 133 119.75 90)
@@
 		)
 	)
+	(gr_text "UNREG\nSENSE+"
+		(at 62.75 55.75 0)
+		(layer "F.SilkS" knockout)
+		(effects
+			(font
+				(size 1 1)
+				(thickness 0.15)
+			)
+		)
+	)
+	(gr_text "REG\nSENSE-"
+		(at 79.5 122.5 0)
+		(layer "F.SilkS" knockout)
+		(effects
+			(font
+				(size 1 1)
+				(thickness 0.15)
+			)
+		)
+	)
 	(gr_text "RCLK"
 		(at 138 119.25 90)
@@
 			)
 		)
+	)
+	(zone
+		(net 12)
+		(net_name "GND")
+		(layer "F.Cu")
+		(hatch edge 0.5)
+		(connect_pads yes
+			(clearance 0.5)
+		)
+		(min_thickness 0.25)
+		(filled_areas_thickness no)
+		(fill yes
+			(thermal_gap 0.5)
+			(thermal_bridge_width 0.5)
+		)
+		(polygon
+			(pts
+				(xy 169.25 34) (xy 169.25 133.5) (xy 22.75 134.5) (xy 23.75 34)
+			)
+		)

Commit message: fin
Parts:
- removed TPe: GND, UTSVT_Special:TestPoint_HEX_3mmID
- added H1: MountingHole_Pad_MP, MountingHole:MountingHole_3.2mm_M3_Pad, F.Cu at (30.0, 40.5)
- added H2: MountingHole_Pad_MP, MountingHole:MountingHole_3.2mm_M3_Pad, F.Cu at (154.5, 59.2)
- added H3: MountingHole_Pad_MP, MountingHole:MountingHole_3.2mm_M3_Pad, F.Cu at (29.8, 127.5)
- added H4: MountingHole_Pad_MP, MountingHole:MountingHole_3.2mm_M3_Pad, F.Cu at (154.5, 108.5)
- added J8: GND, Parts:5754, F.Cu at (154.8, 123.2)
- added J9: 3V3, Parts:5754, F.Cu at (154.8, 45.5)
- added TP5: GND, UTSVT_Special:TestPoint_HEX_3mmID, F.Cu at (145.0, 123.2)
- J3: footprint Connector_PinHeader_2.54mm:PinHeader_1x03_P2.54mm_Vertical -> Connector_PinHeader_2.54mm:PinHeader_1x04_P2.54mm_Vertical
- moved J5 2.50 mm to (60.2, 83.4)
Routing:
- net /UNREG_SENSE+: track 0.00 -> 137.0 mm, vias 0 -> 1
- net /REG_SENSE+: track 0.00 -> 79.2 mm
- net /REG_SENSE-: track 0.00 -> 79.2 mm
- net /UNREG_SENSE-: track 0.00 -> 76.4 mm
- net +3.3V: track 0.00 -> 50.9 mm
- net /UNREG_VOLTAGE: track 0.00 -> 44.4 mm
- net /RCLK: track 0.00 -> 43.6 mm
- net /SRCLK: track 0.00 -> 42.8 mm
- net /SER: track 0.00 -> 42.4 mm
- net /REG_VOLTAGE: track 0.00 -> 42.4 mm
- net /REG_CURRENT: track 0.00 -> 41.0 mm
- net /UNREG_CURRENT: track 0.00 -> 38.0 mm
- net GND: vias 0 -> 30
- added copper zone on F.Cu, net /REG_SENSE+
- added copper zone on F.Cu, net /REG_SENSE-
- added copper zone on F.Cu, net /THERMAL_PAD
- added copper zone on F.Cu, net /UNREG_SENSE+
- added copper zone on F.Cu, net /UNREG_SENSE-
- added copper zone on B.Cu, net GND
Other:
- board size 140.2 x 93.8 mm -> 138.5 x 94.8 mm
- board text added: "3V3"
