File: Hardware/SuppMonTesterPCB/SuppMonTester.kicad_sch (KiCad schematic)
At the start: 0 parts

Commit message: some sch
Parts:
- added J1: 53307-2471, UTSVT_Connectors:533072471, symbol utsvt_connectors:53307-2471
- added J2: UNREG+, Parts:5754, symbol Connector_Generic:Conn_01x01
- added J3: SHIFT_REG, Connector_PinHeader_2.54mm:PinHeader_1x03_P2.54mm_Vertical, symbol Connector_Generic:Conn_01x03
- added J4: REG+, Parts:5754, symbol Connector_Generic:Conn_01x01
- added J5: GND, Parts:5754, symbol Connector_Generic:Conn_01x01
- added J6: UNREG-, Parts:5754, symbol Connector_Generic:Conn_01x01
- added J7: REG-, Parts:5754, symbol Connector_Generic:Conn_01x01
- added R1, R2: 250u, Resistor_SMD:R_1225_3264Metric_Pad1.47x6.45mm_HandSolder, symbol Device:R
- added R3, R4, R5, R6: 20, Parts:RES_PWR263S-35-3300F, symbol Precharge-R:PWR263S-35-3300F
- added TP1: UNREG_VOLTAGE, UTSVT_Special:TestPoint_HEX_3mmID, symbol Connector:TestPoint
- added TP2: REG_VOLTAGE, UTSVT_Special:TestPoint_HEX_3mmID, symbol Connector:TestPoint
- added TP3: UNREG_CURRENT, UTSVT_Special:TestPoint_HEX_3mmID, symbol Connector:TestPoint
- added TP4: REG_CURRENT, UTSVT_Special:TestPoint_HEX_3mmID, symbol Connector:TestPoint
- added TP5: GND, UTSVT_Special:TestPoint_HEX_3mmID, symbol Connector:TestPoint
Connections:
- new net +3.3V: J1.7, J1.9
- new net GND: J1.1, J1.3, J1.5, J5.1 (Pin_1), R3.1, R4.1, R5.1, R6.1, TP5.1
- new net RCLK: J1.2, J3.3 (Pin_3)
- new net REG_CURRENT: J1.12, TP4.1
- new net REG_SENSE+: J1.11, J4.1 (Pin_1), R2.1
- new net REG_SENSE-: J1.13, J7.1 (Pin_1), R2.2, R5.2, R6.2
- new net REG_VOLTAGE: J1.20, TP2.1
- new net SER: J1.8, J3.1 (Pin_1)
- new net SRCLK: J1.4, J3.2 (Pin_2)
- new net THERMAL_PAD: R3.3, R4.3, R5.3, R6.3
- new net UNREG_CURRENT: J1.16, TP3.1
- new net UNREG_SENSE+: J1.17, J1.23, J2.1 (Pin_1), R1.1
- new net UNREG_SENSE-: J1.19, J6.1 (Pin_1), R1.2, R3.2, R4.2
- new net UNREG_VOLTAGE: J1.24, TP1.1
- no-connect marks 0 -> 7
Other:
- note added: "Current Measurement"
- note added: "Load Resistance"
- note added: "Testpoints"
- note added: "total r = 10ohm i = v/r = 24/10 = 2.4A p = iv = 2.4 * 24 = 57.6w max disp of 70w so we chillin"

Commit message: fin
Parts:
- added H1, H2, H3, H4: MountingHole_Pad_MP, MountingHole:MountingHole_3.2mm_M3_Pad, symbol Mechanical:MountingHole_Pad_MP
- added J8: GND, Parts:5754, symbol Connector_Generic:Conn_01x01
- added J9: 3V3, Parts:5754, symbol Connector_Generic:Conn_01x01
- J3: footprint Connector_PinHeader_2.54mm:PinHeader_1x03_P2.54mm_Vertical -> Connector_PinHeader_2.54mm:PinHeader_1x04_P2.54mm_Vertical; symbol Connector_Generic:Conn_01x03 -> Connector_Generic:Conn_01x04
Connections:
- net +3.3V: now also J9.1 (Pin_1)
- net GND: now also J3.4 (Pin_4), J8.1 (Pin_1)
- no-connect marks 7 -> 11
