File: Hardware/BasePCB/SUPP Charger.kicad_sch (KiCad schematic)
At the start: 6 parts, among them J7 52465-2470, Q6 FDD6637, Q8 STD35NF06T4

Commit message: Changes
Parts:
- removed J7: 52465-2470, UTSVT_Connectors:524652470, symbol utsvt_connectors:52465-2470
- removed R18: R, LV Carrier Library:RESC1005X40N, symbol Device:R
- added J7: 53307-2471, UTSVT_Connectors:533072471, symbol utsvt_connectors:53307-2471
- added R19: ERJ3BWFR050V, ERJ3BWFR050V:RES_ERJ3BWFR050V, symbol ERJ3BWFR050V:ERJ3BWFR050V
- D8: footprint DIOM5226X223N -> LV Carrier Library:DIOM5226X223N
- L1: footprint WE-LHMI_7030/705048 -> LV Carrier Library:WE-LHMI_7030_705048
- Q6: footprint DPAK3-CASE-369AS -> LV Carrier Library:DPAK3-CASE-369AS
- Q8: footprint STD35NF06T4 -> LV Carrier Library:STD35NF06T4
Connections:
- net Bgate: now also J7.15
- net Chrg: now also J7.22
- net DCin: now also J7.23
- net Fault: now also J7.24
- net GND: now also J7.10, J7.8, J7.9
- net PGND: now also J7.11
- net Ready: now also J7.18
- net Tgate: now also J7.17
- net Toc: now also J7.20
- net SUPPCHRG_Out: now reaches L1.2
- net SUPPCHRG_Out: now also J7.3, J7.5, R19.1, R19.2

Commit message: Changes
Parts:
- R19: footprint ERJ3BWFR050V:RES_ERJ3BWFR050V -> LV Carrier Library:RES_ERJ3BWFR050V
Connections:
- net DCin renamed DCIN
- net PGND renamed PGnd
Changed lines of the file:
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@@
-	)
-	(junction
-		(at 64.77 55.88)
-		(diameter 0)
-		(color 0 0 0 0)
 	)
 	(junction
@@
 	)
 	(junction
-		(at 64.77 58.42)
+		(at 95.25 58.42)
 		(diameter 0)
 		(color 0 0 0 0)
@@
 		(color 0 0 0 0)
 	)
-	(junction
-		(at 95.25 58.42)
-		(diameter 0)
-		(color 0 0 0 0)
-	)
 	(no_connect
 		(at 64.77 60.96)
@@
 	(wire
 		(pts
-			(xy 62.23 58.42) (xy 64.77 58.42)
+			(xy 168.91 71.12) (xy 168.91 68.58)
+		)
+		(stroke
+			(width 0)
+			(type default)
+		)
+	)
+	(wire
+		(pts
+			(xy 149.86 43.18) (xy 175.26 43.18)
+		)
+		(stroke
+			(width 0)
+			(type default)
+		)
+	)
+	(wire
+		(pts
+			(xy 128.27 43.18) (xy 149.86 43.18)
+		)
+		(stroke
+			(width 0)
+			(type default)
+		)
+	)
+	(wire
+		(pts
+			(xy 110.49 41.91) (xy 110.49 43.18)
+		)
+		(stroke
+			(width 0)
+			(type default)
+		)
+	)
+	(wire
+		(pts
+			(xy 175.26 96.52) (xy 175.26 97.79)
+		)
+		(stroke
+			(width 0)
+			(type default)
+		)
+	)
+	(wire
+		(pts
+			(xy 38.1 40.64) (xy 41.91 40.64)
+		)
+		(stroke
+			(width 0)
+			(type default)
+		)
+	)
+	(wire
+		(pts
+			(xy 38.1 35.56) (xy 41.91 35.56)
+		)
+		(stroke
+			(width 0)
+			(type default)
+		)
+	)
+	(wire
+		(pts
+			(xy 119.38 63.5) (xy 128.27 63.5)
+		)
+		(stroke
+			(width 0)
+			(type default)
+		)
+	)
+	(wire
+		(pts
+			(xy 64.77 55.88) (xy 95.25 55.88)
+		)
+		(stroke
+			(width 0)
+			(type default)
+		)
+	)
+	(wire
+		(pts
+			(xy 64.77 48.26) (xy 71.12 48.26)
+		)
+		(stroke
+			(width 0)
+			(type default)
+		)
+	)
+	(wire
+		(pts
+			(xy 69.85 26.67) (xy 110.49 26.67)
+		)
+		(stroke
+			(width 0)
+			(type default)
+		)
+	)
+	(wire
+		(pts
+			(xy 41.91 53.34) (xy 38.1 53.34)
+		)
+		(stroke
+			(width 0)
+			(type default)
+		)
+	)
+	(wire
+		(pts
+			(xy 95.25 55.88) (xy 95.25 58.42)
+		)
+		(stroke
+			(width 0)
+			(type default)
+		)
+	)
+	(wire
+		(pts
+			(xy 110.49 43.18) (xy 128.27 43.18)
+		)
+		(stroke
+			(width 0)
+			(type default)
+		)
+	)
+	(wire
+		(pts
+			(xy 114.3 53.34) (xy 120.65 53.34)
+		)
+		(stroke
+			(width 0)
+			(type default)
+		)
+	)
+	(wire
+		(pts
+			(xy 149.86 59.69) (xy 149.86 63.5)
+		)
+		(stroke
+			(width 0)
+			(type default)
+		)
+	)
+	(wire
+		(pts
+			(xy 38.1 38.1) (xy 41.91 38.1)
+		)
+		(stroke
+			(width 0)
+			(type default)
+		)
+	)
+	(wire
+		(pts
+			(xy 95.25 96.52) (xy 175.26 96.52)
+		)
+		(stroke
+			(width 0)
+			(type default)
+		)
+	)
+	(wire
+		(pts
+			(xy 175.26 66.04) (xy 175.26 68.58)
+		)
+		(stroke
+			(width 0)
+			(type default)
+		)
+	)
+	(wire
+		(pts
+			(xy 64.77 33.02) (xy 69.85 33.02)
+		)
+		(stroke
+			(width 0)
+			(type default)
+		)
+	)
+	(wire
+		(pts
+			(xy 97.79 36.83) (xy 102.87 36.83)
 		)
 		(stroke
@@
 	(wire
 		(pts
-			(xy 168.91 71.12) (xy 168.91 68.58)
-		)
-		(stroke
-			(width 0)
-			(type default)
-		)
-	)
-	(wire
-		(pts
-			(xy 149.86 43.18) (xy 175.26 43.18)
-		)
-		(stroke
-			(width 0)
-			(type default)
-		)
-	)
-	(wire
-		(pts
-			(xy 128.27 43.18) (xy 149.86 43.18)
-		)
-		(stroke
-			(width 0)
-			(type default)
-		)
-	)
-	(wire
-		(pts
-			(xy 62.23 55.88) (xy 64.77 55.88)
-		)
-		(stroke
-			(width 0)
-			(type default)
-		)
-	)
-	(wire
-		(pts
-			(xy 110.49 41.91) (xy 110.49 43.18)
-		)
-		(stroke
-			(width 0)
-			(type default)
-		)
-	)
-	(wire
-		(pts
-			(xy 175.26 96.52) (xy 175.26 97.79)
-		)
-		(stroke
-			(width 0)
-			(type default)
-		)
-	)
-	(wire
-		(pts
-			(xy 38.1 40.64) (xy 41.91 40.64)
-		)
-		(stroke
-			(width 0)
-			(type default)
-		)
-	)
-	(wire
-		(pts
-			(xy 38.1 35.56) (xy 41.91 35.56)
-		)
-		(stroke
-			(width 0)
-			(type default)
-		)
-	)
-	(wire
-		(pts
-			(xy 119.38 63.5) (xy 128.27 63.5)
-		)
-		(stroke
-			(width 0)
-			(type default)
-		)
-	)
-	(wire
-		(pts
-			(xy 64.77 48.26) (xy 71.12 48.26)
-		)
-		(stroke
-			(width 0)
-			(type default)
-		)
-	)
-	(wire
-		(pts
-			(xy 69.85 26.67) (xy 110.49 26.67)
-		)
-		(stroke
-			(width 0)
-			(type default)
-		)
-	)
-	(wire
-		(pts
-			(xy 41.91 53.34) (xy 38.1 53.34)
-		)
-		(stroke
-			(width 0)
-			(type default)
-		)
-	)
-	(wire
-		(pts
 			(xy 95.25 58.42) (xy 95.25 71.12)
-		)
-		(stroke
-			(width 0)
-			(type default)
-		)
-	)
-	(wire
-		(pts
-			(xy 64.77 55.88) (xy 95.25 55.88)
-		)
-		(stroke
-			(width 0)
-			(type default)
-		)
-	)
-	(wire
-		(pts
-			(xy 110.49 43.18) (xy 128.27 43.18)
-		)
-		(stroke
-			(width 0)
-			(type default)
-		)
-	)
-	(wire
-		(pts
-			(xy 114.3 53.34) (xy 120.65 53.34)
-		)
-		(stroke
-			(width 0)
-			(type default)
-		)
-	)
-	(wire
-		(pts
-			(xy 149.86 59.69) (xy 149.86 63.5)
-		)
-		(stroke
-			(width 0)
-			(type default)
-		)
-	)
-	(wire
-		(pts
-			(xy 38.1 38.1) (xy 41.91 38.1)
-		)
-		(stroke
-			(width 0)
-			(type default)
-		)
-	)
-	(wire
-		(pts
-			(xy 95.25 96.52) (xy 175.26 96.52)
-		)
-		(stroke
-			(width 0)
-			(type default)
-		)
-	)
-	(wire
-		(pts
-			(xy 175.26 66.04) (xy 175.26 68.58)
-		)
-		(stroke
-			(width 0)
-			(type default)
-		)
-	)
-	(wire
-		(pts
-			(xy 64.77 33.02) (xy 69.85 33.02)
-		)
-		(stroke
-			(width 0)
-			(type default)
-		)
-	)
-	(wire
-		(pts
-			(xy 97.79 36.83) (xy 102.87 36.83)
-		)
-		(stroke
-			(width 0)
-			(type default)
-		)
-	)
-	(wire
-		(pts
-			(xy 95.25 55.88) (xy 95.25 58.42)
 		)
 		(stroke
@@
 		)
 	)
-	(hierarchical_label "DCin"
+	(hierarchical_label "DCIN"
 		(shape input)
 		(at 66.04 33.02 90)
@@
 			)
 		)
-		(property "Footprint" "ERJ3BWFR050V:RES_ERJ3BWFR050V"
+		(property "Footprint" "LV Carrier Library:RES_ERJ3BWFR050V"
 			(at 175.26 83.82 0)
 			(effects
@@
 			)
 		)
-		(property "Value" "PGND"
+		(property "Value" "PGnd"
 			(at 128.27 69.85 0)
 			(effects

Commit message: lakshay and changxu bullied me incessantly for hours
Parts:
- removed D8: STPS140A, LV Carrier Library:DIOM5226X223N, symbol STPS140A:STPS140A
- removed L1: 74437349100, LV Carrier Library:WE-LHMI_7030_705048, symbol 74437349100:74437349100
- removed Q6: FDD6637, LV Carrier Library:DPAK3-CASE-369AS, symbol FDD6637:FDD6637
- removed Q8: STD35NF06T4, LV Carrier Library:STD35NF06T4, symbol STD35NF06T4:STD35NF06T4
- removed R19: ERJ3BWFR050V, LV Carrier Library:RES_ERJ3BWFR050V, symbol ERJ3BWFR050V:ERJ3BWFR050V
- J7: footprint UTSVT_Connectors:533072471 -> LV Carrier Library:SuppCharger
Connections:
- net DCIN: no longer names the net of J7.23
- net SUPPCHRG_Out: no longer names the net of J7.3
- net SUPPCHRG_Out: no longer J7.5

Commit message: mostly done
Changed lines of the file:
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@@
-	(wire
-		(pts
-			(xy 64.77 58.42) (xy 92.71 58.42)
-		)
-		(stroke
-			(width 0)
-			(type default)
-		)
-	)
 	(wire
 		(pts
@@
 		)
 		(stroke
-			(width 0)
-			(type default)
-		)
-	)
-	(wire
-		(pts
-			(xy 64.77 55.88) (xy 95.25 55.88)
-		)
-		(stroke
