File: Hardware/SuppChargerPCB/ChargerICPCB.kicad_pcb (KiCad board)
At the start: 4 copper layers, 59 x 22.1 mm, 65 parts, among them J1 SLIMSTACK, J2 SLIMSTACK, Q1 NMOS, Q2 PMOS, U1 LTC4011CFE

Commit message: cosmetic changes
Parts:
- removed the LOGO5 at (101.6, 148.9)
Routing:
- net PGND: track 8.91 -> 7.07 mm, vias 39 -> 62
- net /3V3_THERM: track 9.07 -> 9.76 mm
- net BAT: vias 18 -> 20
- net +24V: vias 5 -> 13
- removed copper zone on In2.Cu, net GND
Other:
- board size 59 x 22.1 mm -> 58.6 x 21.8 mm

Commit message: more cosmetic changes
Parts:
- moved LOGO7 0.89 mm to (110.0, 130.1)
- moved LOGO9 0.89 mm to (113.3, 130.5)
Changed lines of the file:
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@@
 	(footprint "CustomLib:mid"
 		(layer "F.Cu")
-		(at 114.190172 130.53805)
+		(at 113.3 130.53805)
 		(property "Reference" "LOGO9"
 			(at 0 0 0)
@@
 	(footprint "CustomLib:sunderland"
 		(layer "F.Cu")
-		(at 110.87 130.1)
+		(at 109.979828 130.1)
 		(property "Reference" "LOGO7"
 			(at 0 0 0)
@@
 	)
 	(gr_text "9 - 1"
-		(at 111.22 129.27 0)
+		(at 110.1 129.27 0)
 		(layer "F.SilkS")
 		(effects

Commit message: cosmetology
Other:
- board text added: "BAT"
- board text added: "BGATE"
- board text added: "DCIN"
- board text added: "GND"
- board text added: "SENSE"
- board text added: "TGATE"
