File: Hardware/SuppChargerPCB/SuppChargerPCB.kicad_pcb (KiCad board)
At the start: 4 copper layers, 59.4 x 45.4 mm, 100 parts, among them J1 SLIMSTACK, J2 SLIMSTACK, Q1 NMOS, Q11 NMOS, Q12 NMOS, Q13 NMOS, Q14 NMOS, Q2 NMOS, Q3 NMOS, Q4 NMOS, Q5 NMOS, U1 BQ25756ERRVR

Commit message: should b good
Parts:
- L4: value 2.2uH -> 10uH; footprint Components:BMRA000606302R2MA1 -> Components:WE-HCC_807021
- Q1, Q2, Q3, Q4, Q5: value NMOS -> PMOS; footprint Components:SOT95P237X112-3N -> Package_TO_SOT_SMD:SOT-23
- R12: value 7.06k -> 7k
- R13: footprint Resistor_SMD:R_1218_3246Metric_Pad1.22x4.75mm_HandSolder -> Resistor_SMD:R_1210_3225Metric_Pad1.30x2.65mm_HandSolder
- R41: value 14.2K -> 14k
- moved G*** 5.96 mm to (94.7, 105.4)
- moved R51 5.89 mm to (106.0, 115.0), turned to 180 degrees
- moved R12 5.14 mm to (101.8, 112.8), turned to 180 degrees
- moved OUT3 4.69 mm to (110.8, 115.0)
- moved ACOV5 3.60 mm to (122.5, 114.9)
- moved LOGO2 2.01 mm to (117.5, 109.9)
- moved C15 1.91 mm to (96.6, 112.0)
- moved ACUV2 1.67 mm to (119.6, 114.9)
- moved ACOV2 1.55 mm to (116.8, 114.9)
- moved R34 1.20 mm to (108.9, 109.2), turned to 90 degrees
- moved C14 1.18 mm to (125.5, 101.1)
- moved Q12 1.08 mm to (109.9, 105.6)
- moved ACOV3 1.08 mm to (125.6, 109.3)
- moved C16 1.06 mm to (87.9, 112.0)
- moved Q11 1.05 mm to (114.3, 105.6)
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Connections:
- R51 pad 1: +3V3 -> PGND
Routing:
- net /LODRV1: track 21.3 -> 27.9 mm
- net /LODRV2: track 12.4 -> 17.3 mm
- net Net-(U1-ILIM_HIZ): track 6.55 -> 2.16 mm, vias 2 -> 0
- net +24V: track 36.6 -> 32.4 mm
- net /REGN: track 21.4 -> 17.6 mm
- net /ACUV: track 18.9 -> 15.7 mm
- net /Converter/BOOST_LOW: track 4.56 -> 1.78 mm
- net PGND: track 16.8 -> 14.2 mm, vias 77 -> 70
- net /FB: track 28.7 -> 30.8 mm
- net /Converter/BUCK_LOW: track 7.01 -> 5.10 mm
- net /Converter/BOOST_HIGH: track 5.08 -> 3.79 mm
- net /SW2: track 18.5 -> 17.4 mm
- net /HIDRV1: track 20.8 -> 19.8 mm
- net /DRV_SUP: track 13.4 -> 14.4 mm
- net Net-(U1-FSW_SYNC): track 1.83 -> 2.69 mm
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Other:
- board text added: "INT"
- board text added: "Rev B"
- board text added: "Supp Charger PCB"
- board text added: "march 1st 2026"
- board text removed: "Supp Charger Board"
- board text removed: "december 2026"

Commit message: fixed 24v
Routing:
- net +24V: vias 2 -> 8
Changed lines of the file:
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@@
+	)
+	(via
+		(at 120.3 84.5)
+		(size 0.6)
+		(drill 0.3)
+		(layers "F.Cu" "B.Cu")
+		(free yes)
+		(net 1)
+	)
+	(via
+		(at 118.7 83)
+		(size 0.6)
+		(drill 0.3)
+		(layers "F.Cu" "B.Cu")
+		(free yes)
+		(net 1)
+	)
+	(via
+		(at 118.7 84.5)
+		(size 0.6)
+		(drill 0.3)
+		(layers "F.Cu" "B.Cu")
+		(free yes)
+		(net 1)
 	)
 	(via
@@
 		(net 1)
 	)
+	(via
+		(at 120.3 83)
+		(size 0.6)
+		(drill 0.3)
+		(layers "F.Cu" "B.Cu")
+		(free yes)
+		(net 1)
+	)
+	(via
+		(at 120.3 85.8)
+		(size 0.6)
+		(drill 0.3)
+		(layers "F.Cu" "B.Cu")
+		(free yes)
+		(net 1)
+	)
+	(via
+		(at 118.7 85.8)
+		(size 0.6)
+		(drill 0.3)
+		(layers "F.Cu" "B.Cu")
+		(free yes)
+		(net 1)
+	)
