File: Hardware/PowerMuxPCB/LVMuxPCB.kicad_sch (KiCad schematic)
At the start: 58 parts, among them Q1 PMOS, U1 LTC4421CG-PBF

Commit message: blah blah blah
Parts:
- C4: value 470p -> 0p
Other:
- note added: "Need to recalc"
Changed lines of the file:
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@@
 		)
 	)
+	(text "Need to recalc"
+		(exclude_from_sim no)
+		(at 151.638 190.754 0)
+		(effects
+			(font
+				(size 1.27 1.27)
+			)
+		)
+	)
 	(text "Notes:  \n  t_QUAL = C_QUAL * 16 (ms/nF)\n  t_QUAL = 8 ms"
 		(exclude_from_sim no)
@@
 			)
 		)
-		(property "Value" "470p"
+		(property "Value" "0p"
 			(at 125.73 92.7162 0)
 			(effects

Commit message: inital layout
Parts:
- CCPO1: footprint Capacitor_SMD:C_0805_2012Metric -> Capacitor_SMD:C_0603_1608Metric
- Q1: footprint footprints:SOT95P237X112-3N -> footprints1:PMOSGSD_SOT-23_TO-236_VIS
- R1, R10, R11, R12, R13, R14, R2, R4, R5, R6, R7, R9: footprint (none) -> Resistor_SMD:R_0603_1608Metric
- R18, R25: footprint Resistor_SMD:R_0805_2012Metric -> Resistor_SMD:R_0603_1608Metric
- U1: footprint PowerBoardLib:QFN50P600X500X80-37N -> PowerBoardLib:G_05-08-1640_ADI
Changed lines of the file:
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@@
 	)
 	(junction
-		(at 31.75 30.48)
+		(at 31.75 33.02)
 		(diameter 0)
 		(color 0 0 0 0)
@@
 	)
 	(junction
-		(at 31.75 33.02)
-		(diameter 0)
-		(color 0 0 0 0)
-	)
-	(junction
 		(at 49.53 171.45)
 		(diameter 0)
@@
 	(wire
 		(pts
-			(xy 24.13 30.48) (xy 31.75 30.48)
-		)
-		(stroke
-			(width 0)
-			(type default)
-		)
-	)
-	(wire
-		(pts
 			(xy 64.77 82.55) (xy 64.77 90.17)
 		)
@@
 	(wire
 		(pts
+			(xy 16.51 29.21) (xy 16.51 33.02)
+		)
+		(stroke
+			(width 0)
+			(type default)
+		)
+	)
+	(wire
+		(pts
 			(xy 29.21 68.58) (xy 31.75 68.58)
 		)
@@
 		)
 	)
-	(label "CPOREF"
-		(at 24.13 30.48 0)
-		(effects
-			(font
-				(size 1.27 1.27)
-			)
-			(justify left bottom)
-		)
-	)
 	(label "CPO"
 		(at 106.68 31.75 270)
@@
 		)
 	)
+	(label "CPOREF"
+		(at 16.51 33.02 0)
+		(effects
+			(font
+				(size 1.27 1.27)
+			)
+			(justify left bottom)
+		)
+	)
 	(label "V2"
 		(at 198.12 43.18 180)
@@
 		)
 	)
+	(label "OUT"
+		(at 16.51 29.21 0)
+		(effects
+			(font
+				(size 1.27 1.27)
+			)
+			(justify left bottom)
+		)
+	)
 	(label "VALID1"
 		(at 223.52 99.06 90)
@@
 		(exclude_from_sim no)
 		(in_bom yes)
-		(on_board no)
+		(on_board yes)
 		(dnp yes)
 		(fields_autoplaced yes)
@@
 			)
 		)
-		(property "Footprint" ""
+		(property "Footprint" "Resistor_SMD:R_0603_1608Metric"
 			(at 35.56 166.37 0)
 			(effects
@@
 		(exclude_from_sim no)
 		(in_bom yes)
-		(on_board no)
+		(on_board yes)
 		(dnp yes)
 		(fields_autoplaced yes)
@@
 			)
 		)
-		(property "Footprint" ""
+		(property "Footprint" "Resistor_SMD:R_0603_1608Metric"
 			(at 15.24 166.37 0)
 			(effects
@@
 			)
 		)
-		(property "Footprint" "Resistor_SMD:R_0805_2012Metric"
+		(property "Footprint" "Resistor_SMD:R_0603_1608Metric"
 			(at 123.698 161.29 90)
 			(effects
@@
 		(exclude_from_sim no)
 		(in_bom yes)
-		(on_board no)
+		(on_board yes)
 		(dnp yes)
 		(fields_autoplaced yes)
@@
 			)
 		)
-		(property "Footprint" ""
+		(property "Footprint" "Resistor_SMD:R_0603_1608Metric"
 			(at 25.4 166.37 0)
 			(effects
@@
 		(exclude_from_sim no)
 		(in_bom yes)
-		(on_board no)
+		(on_board yes)
 		(dnp yes)
 		(fields_autoplaced yes)
@@
 			)
 		)
-		(property "Footprint" ""
+		(property "Footprint" "Resistor_SMD:R_0603_1608Metric"
 			(at 59.69 175.26 0)
 			(effects
@@
 		(exclude_from_sim no)
 		(in_bom yes)
-		(on_board no)
+		(on_board yes)
 		(dnp yes)
 		(fields_autoplaced yes)
@@
 			)
 		)
-		(property "Footprint" ""
+		(property "Footprint" "Resistor_SMD:R_0603_1608Metric"
 			(at 15.24 175.26 0)
 			(effects
@@
 		(exclude_from_sim no)
 		(in_bom yes)
-		(on_board no)
+		(on_board yes)
 		(dnp yes)
 		(fields_autoplaced yes)
@@
 			)
 		)
-		(property "Footprint" ""
+		(property "Footprint" "Resistor_SMD:R_0603_1608Metric"
 			(at 49.53 166.37 0)
 			(effects
@@
 		(exclude_from_sim no)
 		(in_bom yes)
-		(on_board no)
+		(on_board yes)
 		(dnp yes)
 		(fields_autoplaced yes)
@@
 			)
 		)
-		(property "Footprint" ""
+		(property "Footprint" "Resistor_SMD:R_0603_1608Metric"
 			(at 49.53 175.26 0)
 			(effects
@@
 		(exclude_from_sim no)
 		(in_bom yes)
-		(on_board no)
+		(on_board yes)
 		(dnp yes)
 		(fields_autoplaced yes)
@@
 			)
 		)
-		(property "Footprint" ""
+		(property "Footprint" "Resistor_SMD:R_0603_1608Metric"
 			(at 69.85 166.37 0)
 			(effects
@@
 		(exclude_from_sim no)
 		(in_bom yes)
-		(on_board no)
+		(on_board yes)
 		(dnp yes)
 		(fields_autoplaced yes)
@@
 			)
 		)
-		(property "Footprint" ""
+		(property "Footprint" "Resistor_SMD:R_0603_1608Metric"
 			(at 25.4 175.26 0)
 			(effects
@@
 		(exclude_from_sim no)
 		(in_bom yes)
-		(on_board no)
+		(on_board yes)
 		(dnp yes)
 		(fields_autoplaced yes)
@@
 			)
 		)
-		(property "Footprint" ""
+		(property "Footprint" "Resistor_SMD:R_0603_1608Metric"
 			(at 59.69 166.37 0)
 			(effects
@@
 			)
 		)
-		(property "Footprint" "Resistor_SMD:R_0805_2012Metric"
+		(property "Footprint" "Resistor_SMD:R_0603_1608Metric"
 			(at 94.488 161.29 90)
 			(effects
@@
 			)
 		)
-		(property "Footprint" "footprints:SOT95P237X112-3N"
+		(property "Footprint" "footprints1:PMOSGSD_SOT-23_TO-236_VIS"
 			(at 39.37 83.82 0)
 			(effects
@@
 		(exclude_from_sim no)
 		(in_bom yes)
-		(on_board no)
+		(on_board yes)
 		(dnp yes)
 		(fields_autoplaced yes)
@@
 			)
 		)
-		(property "Footprint" ""
+		(property "Footprint" "Resistor_SMD:R_0603_1608Metric"
 			(at 35.56 175.26 0)
 			(effects
@@
 		(exclude_from_sim no)
 		(in_bom yes)
-		(on_board no)
+		(on_board yes)
 		(dnp yes)
 		(fields_autoplaced yes)
@@
 			)
 		)
-		(property "Footprint" ""
+		(property "Footprint" "Resistor_SMD:R_0603_1608Metric"
 			(at 69.85 175.26 0)
 			(effects
@@
 			)
 		)
-		(property "Footprint" "PowerBoardLib:QFN50P600X500X80-37N"
+		(property "Footprint" "PowerBoardLib:G_05-08-1640_ADI"
 			(at 31.75 27.94 0)
 			(effects
@@
 			)
 		)
-		(property "Footprint" "Capacitor_SMD:C_0805_2012Metric"
+		(property "Footprint" "Capacitor_SMD:C_0603_1608Metric"
 			(at 107.6452 46.99 0)
 			(effects

Commit message: ts is so aids
Parts:
- removed Q1: PMOS, footprints1:PMOSGSD_SOT-23_TO-236_VIS, symbol Simulation_SPICE:PMOS
- removed R24: 0, Resistor_SMD:R_0603_1608Metric, symbol Device:R
- added Q1: SQ2315CES-T1_GE3, PMOSGSD_SOT-23_TO-236_VIS, symbol sumStuff1:SQ2315CES-T1_GE3
- added TP14, TP15, TP16, TP17, TP18, TP19: TestPoint, TestPoint:TestPoint_Pad_D1.0mm, symbol Connector:TestPoint
- R26: renamed from R3; value 10K -> 1K
- renumbered CQUAL1 to C5, R11 to R10, R12 to R11, R13 to R12, R14 to R13, R18 to R14, R17 to R15, R15 to R17, R42 to R18, R43 to R19, R25 to R20, R44 to R21, R45 to R22, R46 to R23, R23 to R24, R26 to R27, R27 to R28, R28 to R29, R4 to R3, R29 to R30, R30 to R31, R31 to R32, R32 to R33, R33 to R34, R34 to R35, R35 to R36, R5 to R4, R6 to R5, R7 to R6, R8 to R7, R9 to R8, R10 to R9
Connections:
- net INTVCC: now also Q1.3 (D)
- net OV1: now also TP14.1
- net OV2: now also TP17.1
- net SHDN: now also Q1.2 (S)
- net UVF1: now also TP16.1
- net UVF2: now also TP19.1
- net UVR1: now also TP15.1
- net UVR2: now also TP18.1
- net at R26.2: now also Q1.1 (G)
Other:
- moved on the sheet: R26, R7, TP2, TP3, TP4, TP5, TP6, TP7

Commit message: lakshay is ragebaiting
Parts:
- removed C4: 0p, Capacitor_SMD:C_0603_1608Metric, symbol Device:C_Small
- removed R24: 0, Resistor_SMD:R_0603_1608Metric, symbol Device:R

Commit message: Merge LTC Mux Branches (#6)
* this board isn't performative lakshay :sob:

* ts performative

* step

* ninja fix shutdown circuitry

* ninja fix the ninja fix for double nmos

* lil guy alert

---------

Co-authored-by: Frank Li <fxl77@my.utexas.edu>
Co-authored-by: sodaplayzz <sc.seaofthieves@gmail.com>
Parts:
- removed Q1: SQ2315CES-T1_GE3, PMOSGSD_SOT-23_TO-236_VIS, symbol sumStuff1:SQ2315CES-T1_GE3
- removed R7: 10K, Resistor_SMD:R_0603_1608Metric, symbol Device:R_Small
- added MH1, MH2, MH3, MH4: M3, MountingHole:MountingHole_3.2mm_M3_Pad_TopBottom, symbol Mechanical:MountingHole
- added Q10, Q9: IRLML0030, Package_TO_SOT_SMD:SOT-23, symbol Transistor_FET:IRLML0030
- added R43: 1K, Resistor_SMD:R_0603_1608Metric, symbol Device:R_Small
- added R44: 100k, Resistor_SMD:R_0603_1608Metric, symbol Device:R_Small
- TP1, TP2, TP3, TP4, TP5, TP6, TP7: footprint UTSVT_Special:TestPoint_HEX_3mmID -> TestPoint:TestPoint_Pad_D1.0mm
Connections:
- net GND: now also Q10.2 (S), Q9.2 (S)
- net INTVCC: now also R44.1
- net SHDN: now also Q9.3 (D)
- net SHDNOUT: now also R43.1; no longer R26.1
- net at R26.2: now also Q9.1 (G)
- new net: Q10.1 (G), R43.2
- new net: Q10.3 (D), R26.1, R44.2
Other:
- sheet IO_CONN ports: added none; removed INTVCC
- note added: "Mounting Holes"
- note added: "Shutdown pulled LOW disables chip NMOS gate needs to be pulled HIGH by default to turn off car in an unknown state"
- moved on the sheet: R26

Commit message: final changes
Parts:
- removed C1: .1u, Capacitor_SMD:C_0603_1608Metric, symbol Device:C_Small
- removed C2: 10u, Capacitor_SMD:C_0603_1608Metric, symbol Device:C_Small
- removed COUT1: 1.2m, PowerBoardLib:EEUFS1C122LB, symbol Device:C_Polarized_US
- TP1, TP2, TP3, TP4, TP5, TP6, TP7: footprint TestPoint:TestPoint_Pad_D1.0mm -> TestPoint:TestPoint_Pad_D2.0mm
Connections:
- net CPOREF: no longer U1.34 (OUT2)
- new net OUT2: U1.34 (OUT2)
Other:
- sheet IO_CONN ports: added OUT1, OUT2; removed OUT
- note removed: "Decoupling Capacitors"
- note removed: "Notes: - As per datasheet, using 10uf to 50 uf of output capacitance per Ampere of maximum load current achieves a reasonable tradeoff. As such: 40 uf * 20 = 8 mF - Need to look more closely into this."
- note removed: "Output Capacitor"
- note removed: "Values for Output Capacitor"

Commit message: silk + roosters
Parts:
- added LOGO1: Dr. Hallock, UTSVT_Logos:Hallock_Image_Tiny, symbol utsvt-misc:Logo_Placeholder
- added LOGO2: Dr. Hallock, UTSVT_Logos:LHRs_LOGO, symbol utsvt-misc:Logo_Placeholder
- U1: footprint PowerBoardLib:G_05-08-1640_ADI -> LTC4421:G_05-08-1640_ADI

Commit message: cleaned up power mux
Parts:
- removed CCPO1: 1u, Capacitor_SMD:C_0603_1608Metric, symbol ECE319K:C
- removed U1: LTC4421CG-PBF, LTC4421:G_05-08-1640_ADI, symbol PowerBoardLib:LTC4421CG-PBF
- added CCPO1: 1u, Capacitor_SMD:C_0603_1608Metric, symbol Device:C
- added U1: LTC4421CG-PBF, PowerMuxLib:LTC4421CG-PBF, symbol PowerMuxLib:LTC4421CG-PBF
Connections:
- net CH1: now also U1.13 (*CH1)
- net CH2: now also U1.24 (*CH2)
- net CPO: now also CCPO1.1, U1.1 (CPO)
- net CPOREF: now also CCPO1.2, U1.2 (CPOREF), U1.3 (OUT1)
- net DISABLE1: now also U1.12 (*DISABLE1)
- net DISABLE2: now also U1.25 (*DISABLE2)
- net FAULT1: now also U1.15 (*FAULT1)
- net FAULT2: now also U1.22 (*FAULT2)
- net GATE1: now also U1.6 (GATE1)
- net GATE2: now also U1.31 (GATE2)
- net GND: now also U1.35 (GND), U1.36 (EXTVCC)
- net INTVCC: now also U1.16 (CASIN), U1.17 (INTVCC)
- net OUT2: now also U1.34 (OUT2)
- net OV1: now also U1.10 (OV1)
- net OV2: now also U1.27 (OV2)
- net QUAL: now also U1.19 (QUAL)
- net RETRY: now also U1.20 (RETRY)
- net SENSE1: now also U1.4 (SENSE1)
- net SENSE2: now also U1.33 (SENSE2)
- net SHDN: now also U1.21 (*SHDN)
- net SOURCE1: now also U1.5 (SOURCE1)
- net SOURCE2: now also U1.32 (SOURCE2)
- net TMR1: now also U1.11 (TMR1)
- net TMR2: now also U1.26 (TMR2)
- net UVF1: now also U1.8 (UVF1)
- net UVF2: now also U1.29 (UVF2)
- net UVR1: now also U1.9 (UVR1)
- net UVR2: now also U1.28 (UVR2)
- net V1: now also U1.7 (V1)
- net V2: now also U1.30 (V2)
- net VALID1: now also U1.14 (*VALID1)
- net VALID2: now also U1.23 (*VALID2)
Other:
- moved on the sheet: Q9
