File: hardware/PS-LVCarrier.kicad_sch (KiCad schematic)
At the start: 0 parts

Commit message: finished LTC calcs
Other:
- sheet HV -> 24V ports: added DCDC_OUT, HV_PROTECTED; removed none
- sheet HV Input Protection ports: added GND_HV_ISO, HV_PROTECTED; removed none
- sheet LV -> 24V ports: added LV_PROTECTED, LV_REGULATED; removed none
- sheet LV Input Protection ports: added GND_LV, LV_PROTECTED; removed none
- sheet Priority Combiner ports: added HV_24V, LV_24V, {CTRL_INPUTS}, {STATS_OUTPUTS}; removed none

Commit message: added gpios, root page clean up then switch to laptop
Other:
- sheet Priority Combiner ports: added 24V_VOUT; removed none
- note added: "Application Notes"
- note added: "RevB Notes"
Changed lines of the file:
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@@
 	(generator_version "10.0")
 	(paper "A3")
+	(rectangle
+		(start 300.99 104.775)
+		(end 403.86 164.465)
+		(stroke
+			(width 0)
+			(type default)
+		)
+		(fill
+			(type none)
+		)
+	)
+	(rectangle
+		(start 300.99 169.545)
+		(end 403.86 247.65)
+		(stroke
+			(width 0)
+			(type default)
+		)
+		(fill
+			(type none)
+		)
+	)
+	(text "Application Notes\n"
+		(exclude_from_sim no)
+		(at 312.928 173.482 0)
+		(effects
+			(font
+				(size 1.27 1.27)
+			)
+		)
+	)
+	(text "RevB Notes"
+		(exclude_from_sim no)
+		(at 309.118 108.204 0)
+		(effects
+			(font
+				(size 1.27 1.27)
+			)
+		)
+	)
 	(bus
 		(pts
 			(xy 151.13 88.9) (xy 176.53 88.9)
+		)
+		(stroke
+			(width 0)
+			(type default)
+		)
+	)
+	(wire
+		(pts
+			(xy 232.41 54.61) (xy 256.54 54.61)
 		)
 		(stroke
@@
 			)
 		)
+		(pin "24V_VOUT" output
+			(at 232.41 54.61 0)
+			(effects
+				(font
+					(size 1.27 1.27)
+				)
+				(justify right)
+			)
+		)
 		(instances
 			(project "PS-LVCarrier"
@@
 	(sheet
 		(at 256.54 49.53)
-		(size 39.37 41.91)
+		(size 36.195 41.91)
 		(exclude_from_sim no)
 		(in_bom yes)

Commit message: small changes
Changed lines of the file:
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@@
+		)
+	)
+	(bus_entry
+		(at 153.67 154.94)
+		(size -2.54 2.54)
+		(stroke
+			(width 0)
+			(type default)
+		)
+	)
+	(bus_entry
+		(at 153.67 157.48)
+		(size -2.54 2.54)
+		(stroke
+			(width 0)
+			(type default)
+		)
+	)
+	(bus_entry
+		(at 153.67 160.02)
+		(size -2.54 2.54)
+		(stroke
+			(width 0)
+			(type default)
+		)
+	)
+	(bus_entry
+		(at 153.67 149.86)
+		(size -2.54 2.54)
+		(stroke
+			(width 0)
+			(type default)
+		)
+	)
+	(bus_entry
+		(at 153.67 152.4)
+		(size -2.54 2.54)
+		(stroke
+			(width 0)
+			(type default)
+		)
+	)
+	(bus_entry
+		(at 153.67 157.48)
+		(size -2.54 2.54)
+		(stroke
+			(width 0)
+			(type default)
+		)
+	)
+	(bus_entry
+		(at 153.67 149.86)
+		(size -2.54 2.54)
+		(stroke
+			(width 0)
+			(type default)
+		)
+	)
+	(wire
+		(pts
+			(xy 142.24 157.48) (xy 151.13 157.48)
+		)
+		(stroke
+			(width 0)
+			(type default)
+		)
+	)
+	(wire
+		(pts
+			(xy 142.24 162.56) (xy 151.13 162.56)
+		)
+		(stroke
+			(width 0)
+			(type default)
+		)
+	)
+	(wire
+		(pts
+			(xy 142.24 160.02) (xy 151.13 160.02)
+		)
+		(stroke
+			(width 0)
+			(type default)
+		)
+	)
+	(wire
+		(pts
+			(xy 232.41 54.61) (xy 256.54 54.61)
+		)
+		(stroke
+			(width 0)
+			(type default)
+		)
+	)
+	(wire
+		(pts
+			(xy 130.81 54.61) (xy 176.53 54.61)
+		)
+		(stroke
+			(width 0)
+			(type default)
+		)
+	)
+	(wire
+		(pts
+			(xy 135.89 59.69) (xy 176.53 59.69)
+		)
+		(stroke
+			(width 0)
+			(type default)
 		)
 	)
 	(bus
 		(pts
-			(xy 151.13 88.9) (xy 176.53 88.9)
-		)
-		(stroke
-			(width 0)
-			(type default)
-		)
-	)
-	(wire
-		(pts
-			(xy 232.41 54.61) (xy 256.54 54.61)
-		)
-		(stroke
-			(width 0)
-			(type default)
-		)
-	)
-	(wire
-		(pts
-			(xy 130.81 54.61) (xy 176.53 54.61)
-		)
-		(stroke
-			(width 0)
-			(type default)
-		)
-	)
-	(wire
-		(pts
-			(xy 135.89 59.69) (xy 176.53 59.69)
+			(xy 156.21 195.58) (xy 156.21 106.68)
 		)
 		(stroke
@@
 	(bus
 		(pts
-			(xy 151.13 80.01) (xy 176.53 80.01)
+			(xy 153.67 104.14) (xy 176.53 104.14)
+		)
+		(stroke
+			(width 0)
+			(type default)
+		)
+	)
+	(bus
+		(pts
+			(xy 153.67 104.14) (xy 153.67 163.83)
+		)
+		(stroke
+			(width 0)
+			(type default)
+		)
+	)
+	(bus
+		(pts
+			(xy 156.21 106.68) (xy 176.53 106.68)
 		)
 		(stroke
@@
 	(wire
 		(pts
+			(xy 142.24 152.4) (xy 151.13 152.4)
+		)
+		(stroke
+			(width 0)
+			(type default)
+		)
+	)
+	(wire
+		(pts
+			(xy 142.24 154.94) (xy 151.13 154.94)
+		)
+		(stroke
+			(width 0)
+			(type default)
+		)
+	)
+	(wire
+		(pts
 			(xy 40.64 102.87) (xy 40.64 104.14)
 		)
@@
 			(width 0)
 			(type default)
+		)
+	)
+	(label "DISABLE2"
+		(at 142.24 157.48 0)
+		(effects
+			(font
+				(size 1.27 1.27)
+			)
+			(justify left bottom)
+		)
+	)
+	(label "RETRY"
+		(at 142.24 152.4 0)
+		(effects
+			(font
+				(size 1.27 1.27)
+			)
+			(justify left bottom)
+		)
+	)
+	(label "DISABLE1"
+		(at 142.24 154.94 0)
+		(effects
+			(font
+				(size 1.27 1.27)
+			)
+			(justify left bottom)
+		)
+	)
+	(label "CASIN"
+		(at 142.24 162.56 0)
+		(effects
+			(font
+				(size 1.27 1.27)
+			)
+			(justify left bottom)
+		)
+	)
+	(label "SHDN"
+		(at 142.24 160.02 0)
+		(effects
+			(font
+				(size 1.27 1.27)
+			)
+			(justify left bottom)
 		)
 	)
@@
 		)
 		(pin "{CTRL_INPUTS}" input
-			(at 176.53 80.01 180)
+			(at 176.53 104.14 180)
 			(effects
 				(font
@@
 		)
 		(pin "{STATS_OUTPUTS}" input
-			(at 176.53 88.9 180)
-			(effects
-				(font
+			(at 176.53 106.68 180)
+			(effects
+				(font
