File: hardware/LV_protection.kicad_sch (KiCad schematic)
At the start: 0 parts

Commit message: finished LTC calcs
Parts:
- added D2: D_Zener, symbol Device:D_Zener
- added F2: Fuse, symbol Device:Fuse
- added J2: Conn_01x02, symbol Connector_Generic:Conn_01x02
- added Q2: NMOS, symbol Simulation_SPICE:NMOS
Connections:
- new net: F2.1, J2.2 (Pin_2)
- new net LV_GND: J2.1 (Pin_1)
- new net LV_PROTECTED: F2.2
Other:
- note added: "need supp battery voltage range"

Commit message: more changes, switch to pc
Other:
- note added: "LV (20V-28V) 24V nominal"
Changed lines of the file:
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@@
+		)
+	)
+	(text "LV (20V-28V)\n24V nominal"
+		(exclude_from_sim no)
+		(at 40.386 39.878 0)
+		(effects
+			(font
+				(size 1.27 1.27)
+			)
 		)
 	)

Commit message: did fan circuits, added MCU design block, made buck converter, added VIP sensing + soft start?
Parts:
- added C40: 0.1u, symbol Device:C_Small
- added R46: R_Shunt, symbol Device:R_Shunt
- added U9: INA228, Package_SO:TSSOP-10_3x3mm_P0.5mm, symbol Sensor_Energy:INA228
Connections:
- net LV_GND: now also C40.2, U9.1 (A1), U9.7 (GND)
- net LV_PROTECTED: now also R46.1, U9.8 (Vbus); no longer F2.2
- new net: R46.2, U9.10 (Vin+)
- new net: R46.3, U9.9 (Vin-)
- new net: F2.2, R46.4
- new net +3V3: C40.1, U9.2 (A0), U9.6 (VS)
- new net ALERT: U9.3 (~{Alert})
- new net SCL: U9.5 (SCL)
- new net SDA: U9.4 (SDA)
Other:
- note added: "0x41"
- note added: "route tightly"
- moved on the sheet: D2, F2, J2, Q2

Commit message: switch to pc
Parts:
- F2: value Fuse -> 20A
- R46: value R_Shunt -> 2m
Other:
- note added: "17^2V/2mohm = 578m W = .6W"
- note added: "300W/20V = 15A worst case scenario"
- note removed: "need supp battery voltage range"
- moved on the sheet: C40, D2, F2, J2, Q2, R46, U9

Commit message: changes
Parts:
- removed D2: D_Zener, symbol Device:D_Zener
- removed Q2: NMOS, symbol Simulation_SPICE:NMOS
Changed lines of the file:
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@@
-	)
-	(symbol
-		(lib_id "Device:D_Zener")
-		(at 77.47 85.09 180)
-		(unit 1)
-		(body_style 1)
-		(exclude_from_sim no)
-		(in_bom yes)
-		(on_board yes)
-		(in_pos_files yes)
-		(dnp no)
-		(fields_autoplaced yes)
-		(property "Reference" "D2"
-			(at 77.47 78.74 0)
-			(show_name no)
-			(do_not_autoplace no)
-			(effects
-				(font
-					(size 1.27 1.27)
-				)
-			)
-		)
-		(property "Value" "D_Zener"
-			(at 77.47 81.28 0)
-			(show_name no)
-			(do_not_autoplace no)
-			(effects
-				(font
-					(size 1.27 1.27)
-				)
-			)
-		)
-		(property "Footprint" ""
-			(at 77.47 85.09 0)
-			(hide yes)
-			(show_name no)
-			(do_not_autoplace no)
-			(effects
-				(font
-					(size 1.27 1.27)
-				)
-			)
-		)
-		(property "Datasheet" ""
-			(at 77.47 85.09 0)
-			(hide yes)
-			(show_name no)
-			(do_not_autoplace no)
-			(effects
-				(font
-					(size 1.27 1.27)
-				)
-			)
-		)
-		(property "Description" "Zener diode"
-			(at 77.47 85.09 0)
-			(hide yes)
-			(show_name no)
-			(do_not_autoplace no)
-			(effects
-				(font
-					(size 1.27 1.27)
-				)
-			)
-		)
-		(pin "2"
-		)
-		(pin "1"
-		)
-		(instances
-			(project "PS-LVCarrier"
-				(path "/9bab2d9d-20f3-40ef-8545-e1299efec47e/a5bb0fbd-5072-4239-af04-5df171469b26"
-					(reference "D2")
-					(unit 1)
-				)
-			)
-		)
 	)
 	(symbol
@@
 					(unit 1)
 				)
-			)
-		)
-	)
-	(symbol
-		(lib_id "Simulation_SPICE:NMOS")
-		(at 57.15 85.09 180)
-		(unit 1)
-		(body_style 1)
-		(exclude_from_sim no)
-		(in_bom yes)
-		(on_board yes)
-		(in_pos_files yes)
-		(dnp no)
-		(fields_autoplaced yes)
-		(property "Reference" "Q2"
-			(at 50.8 83.8199 0)
-			(show_name no)
-			(do_not_autoplace no)
-			(effects
-				(font
-					(size 1.27 1.27)
-				)
-				(justify left)
-			)
-		)
-		(property "Value" "NMOS"
-			(at 50.8 86.3599 0)
-			(show_name no)
-			(do_not_autoplace no)
-			(effects
-				(font
-					(size 1.27 1.27)
-				)
-				(justify left)
-			)
-		)
-		(property "Footprint" ""
-			(at 52.07 87.63 0)
-			(hide yes)
-			(show_name no)
-			(do_not_autoplace no)
-			(effects
-				(font
-					(size 1.27 1.27)
-				)
-			)
-		)
-		(property "Datasheet" "https://ngspice.sourceforge.io/docs/ngspice-html-manual/manual.xhtml#cha_MOSFETs"
-			(at 57.15 72.39 0)
-			(hide yes)
-			(show_name no)
-			(do_not_autoplace no)
-			(effects
-				(font
-					(size 1.27 1.27)
-				)
-			)
-		)
-		(property "Description" "N-MOSFET transistor, drain/source/gate"
-			(at 57.15 85.09 0)
-			(hide yes)
-			(show_name no)
-			(do_not_autoplace no)
-			(effects
-				(font
-					(size 1.27 1.27)
-				)
-			)
-		)
-		(property "Sim.Device" "NMOS"
-			(at 57.15 67.945 0)
-			(hide yes)
-			(show_name no)
-			(do_not_autoplace no)
-			(effects
-				(font
-					(size 1.27 1.27)
-				)
-			)
-		)
-		(property "Sim.Type" "VDMOS"
-			(at 57.15 66.04 0)
-			(hide yes)
-			(show_name no)
-			(do_not_autoplace no)
-			(effects
-				(font
-					(size 1.27 1.27)
-				)
-			)
-		)
-		(property "Sim.Pins" "1=D 2=G 3=S"
-			(at 57.15 69.85 0)
-			(hide yes)
-			(show_name no)
-			(do_not_autoplace no)
-			(effects
-				(font
-					(size 1.27 1.27)
-				)
-			)
-		)
-		(pin "2"
-		)
-		(pin "1"
-		)
-		(pin "3"
-		)
-		(instances
-			(project "PS-LVCarrier"
-				(path "/9bab2d9d-20f3-40ef-8545-e1299efec47e/a5bb0fbd-5072-4239-af04-5df171469b26"
-					(reference "Q2")
-					(unit 1)
-				)

Commit message: cleaned up root page, reviewed subsheets, pretty much ready for a review ig
Parts:
- added C58: .1u, Capacitor_SMD:C_0603_1608Metric_Pad1.08x0.95mm_HandSolder, symbol Device:C
- added C60: 1 uF, Capacitor_SMD:C_0603_1608Metric_Pad1.08x0.95mm_HandSolder, symbol Device:C
- added C65: 220n, symbol Device:C_Small
- added D10: HPZR-C3V0-QX, LV Carrier Library:HPZRC3V0QX, symbol Device:D_Zener
- added D26: SMBJ33D, LV Carrier Library:SMBJ15DM3, symbol LV-Carrier:SMBJ15D-M3I
- added IC1: AP74502QTA8-7, LV Carrier Library:AP74502HQTA87, symbol LV-Carrier:AP74502HQTA8-7
- added Q10, Q9: NVMFWS1D7N04XMT1G, LV Carrier Library:NVMFWS3D0P04M8LT1G, symbol LV-Carrier:NVMFWS1D7N04XMT1G
- added Q11: IRLML0030, Package_TO_SOT_SMD:SOT-23, symbol Transistor_FET:IRLML0030
- added R60: 1k, Resistor_SMD:R_0603_1608Metric_Pad0.98x0.95mm_HandSolder, symbol Device:R
- added R61, R62, R65: 10k, Resistor_SMD:R_0603_1608Metric_Pad0.98x0.95mm_HandSolder, symbol Device:R
- added R63: 100k, Resistor_SMD:R_0603_1608Metric_Pad0.98x0.95mm_HandSolder, symbol Device:R
- added R64: 255k, Resistor_SMD:R_0603_1608Metric_Pad0.98x0.95mm_HandSolder, symbol Device:R
- added TP7, TP8: TestPoint, TestPoint:TestPoint_Pad_D2.5mm, symbol Connector:TestPoint
Connections:
- net LV_GND: now also C58.2, C60.2, D10.2 (A), D26.1 (K), IC1.2 (GND), Q11.2 (S), R62.2, R65.2
- net at R46.4: now also C60.1, Q10.5, Q10.6, Q10.7, Q10.8, Q10.9; no longer F2.2
- new net: D10.1 (K), Q11.1 (G), R60.2, R61.2, R62.1, TP7.1
- new net DIODE_EN: IC1.1 (EN/UVLO), Q11.3 (D), R63.2, TP8.1
- new net GATE: IC1.6 (GATE), Q10.4, Q9.4
- new net LV_EN: R60.1, R61.1
- new net OVLO: IC1.7 (OVLO), R64.2, R65.1
- new net SRC: IC1.8 (SRC), Q10.1, Q10.2, Q10.3, Q9.1, Q9.2, Q9.3
- new net VCP: C65.2, IC1.4 (VCP)
- new net VIN: C58.1, C65.1, D26.2 (A), F2.2, IC1.5 (VIN), Q9.5, Q9.6, Q9.7, Q9.8, Q9.9, R63.1, R64.1
Other:
- note added: "1.25 x (1 + 255/10) = 33.3V"
- note added: "Diode clips gate voltage at 3.3V (max vgs of IRLML is 20V) Divider in case diode doesn't work"
- note added: "OV comp threshold = 1.25V"
- note added: "Positive Logic"
- note added: "Vicor input limit 36V"
- note added: "inverted logic?"
- note added: "keep trace short"
- note added: "use q instead of hq, slow gate for inrush limiting"
- moved on the sheet: C40, F2, J2, R46, U9

Commit message: checkout
Parts:
- renumbered C58 to C18, C65 to C19, C60 to C20, C40 to C21, D10 to D2, D26 to D3, Q11 to Q1, Q9 to Q2, Q10 to Q3, R60 to R12, R61 to R13, R62 to R14, R63 to R15, R64 to R16, R65 to R17, R46 to R18, TP7 to TP1, TP8 to TP2, U9 to U6

Commit message: fixes switch to laptop
Parts:
- C18: value .1u -> 1u
Other:
- note added: "Indicator LEDs"
- note added: "Testpoints"
- moved on the sheet: C18, C19, R16, R17
