File: hardware/powersupply.kicad_sch (KiCad schematic)
At the start: 1 part, among them J13 PS

Commit message: initial review again
Parts:
- added F3: Fuse, symbol Device:Fuse
Connections:
- net PS_OUT: now also F3.2; no longer J13.1 (Pin_1)
- new net: F3.1, J13.1 (Pin_1)
Changed lines of the file:
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@@
 	(wire
 		(pts
-			(xy 92.71 67.31) (xy 107.95 67.31)
+			(xy 113.03 67.31) (xy 124.46 67.31)
+		)
+		(stroke
+			(width 0)
+			(type default)
+		)
+	)
+	(wire
+		(pts
+			(xy 92.71 67.31) (xy 105.41 67.31)
 		)
 		(stroke
@@
 	(hierarchical_label "PS_OUT"
 		(shape output)
-		(at 107.95 67.31 0)
+		(at 124.46 67.31 0)
 		(effects
 			(font
@@
 					(unit 1)
 				)
+			)
+		)
+	)
+	(symbol
+		(lib_id "Device:Fuse")
+		(at 109.22 67.31 90)
+		(unit 1)
+		(body_style 1)
+		(exclude_from_sim no)
+		(in_bom yes)
+		(on_board yes)
+		(in_pos_files yes)
+		(dnp no)
+		(fields_autoplaced yes)
+		(property "Reference" "F3"
+			(at 109.22 60.96 90)
+			(show_name no)
+			(do_not_autoplace no)
+			(effects
+				(font
+					(size 1.27 1.27)
+				)
+			)
+		)
+		(property "Value" "Fuse"
+			(at 109.22 63.5 90)
+			(show_name no)
+			(do_not_autoplace no)
+			(effects
+				(font
+					(size 1.27 1.27)
+				)
+			)
+		)
+		(property "Footprint" ""
+			(at 109.22 69.088 90)
+			(hide yes)
+			(show_name no)
+			(do_not_autoplace no)
+			(effects
+				(font
+					(size 1.27 1.27)
+				)
+			)
+		)
+		(property "Datasheet" ""
+			(at 109.22 67.31 0)
+			(hide yes)
+			(show_name no)
+			(do_not_autoplace no)
+			(effects
+				(font
+					(size 1.27 1.27)
+				)
+			)
+		)
+		(property "Description" "Fuse"
+			(at 109.22 67.31 0)
+			(hide yes)
+			(show_name no)
+			(do_not_autoplace no)
+			(effects
+				(font
+					(size 1.27 1.27)
+				)
+			)
+		)
+		(pin "1"
+		)
+		(pin "2"
+		)
+		(instances
+			(project "PS-LVCarrier"
+				(path "/9bab2d9d-20f3-40ef-8545-e1299efec47e/ccdd180d-924e-4cb4-9ad4-e64fe43b7b98"
+					(reference "F3")
+					(unit 1)
+				)

Commit message: progress!
Connections:
- net PS_OUT renamed PS_12V_FUSED
Other:
- note added: "300W/12V"
Changed lines of the file:
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@@
 	(generator_version "10.0")
 	(paper "A5")
+	(text "300W/12V"
+		(exclude_from_sim no)
+		(at 108.966 50.038 0)
+		(effects
+			(font
+				(size 1.27 1.27)
+			)
+		)
+	)
 	(wire
 		(pts
@@
 		)
 	)
-	(hierarchical_label "PS_OUT"
+	(hierarchical_label "PS_12V_FUSED"
 		(shape output)
 		(at 124.46 67.31 0)

Commit message: review ts
Parts:
- renumbered F3 to F2, J13 to J2
Other:
- moved on the sheet: F2, J2
Changed lines of the file:
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@@
 	(text "300W/12V"
 		(exclude_from_sim no)
-		(at 108.966 50.038 0)
+		(at 88.646 50.038 0)
 		(effects
 			(font
@@
 	(wire
 		(pts
-			(xy 113.03 67.31) (xy 124.46 67.31)
+			(xy 92.71 67.31) (xy 104.14 67.31)
 		)
 		(stroke
@@
 	(wire
 		(pts
-			(xy 92.71 67.31) (xy 105.41 67.31)
+			(xy 72.39 67.31) (xy 85.09 67.31)
 		)
 		(stroke
@@
 	(wire
 		(pts
-			(xy 92.71 69.85) (xy 99.06 69.85)
+			(xy 72.39 69.85) (xy 78.74 69.85)
 		)
 		(stroke
@@
 	(hierarchical_label "PS_12V_FUSED"
 		(shape output)
-		(at 124.46 67.31 0)
+		(at 104.14 67.31 0)
 		(effects
 			(font
@@
 	(hierarchical_label "LV_GND"
 		(shape passive)
-		(at 99.06 69.85 270)
+		(at 78.74 69.85 270)
 		(effects
 			(font
@@
 	(symbol
 		(lib_id "Connector_Generic:Conn_01x02")
-		(at 87.63 67.31 0)
+		(at 67.31 67.31 0)
 		(mirror y)
 		(unit 1)
@@
 		(dnp no)
 		(fields_autoplaced yes)
-		(property "Reference" "J13"
-			(at 87.63 60.96 0)
+		(property "Reference" "J2"
+			(at 67.31 60.96 0)
 			(show_name no)
 			(do_not_autoplace no)
@@
 		)
 		(property "Value" "PS"
-			(at 87.63 63.5 0)
+			(at 67.31 63.5 0)
 			(show_name no)
 			(do_not_autoplace no)
@@
 		)
 		(property "Footprint" ""
-			(at 87.63 67.31 0)
+			(at 67.31 67.31 0)
 			(hide yes)
 			(show_name no)
@@
 		)
 		(property "Datasheet" ""
-			(at 87.63 67.31 0)
+			(at 67.31 67.31 0)
 			(hide yes)
 			(show_name no)
@@
 		)
 		(property "Description" "Generic connector, single row, 01x02, script generated (kicad-library-utils/schlib/autogen/connector/)"
-			(at 87.63 67.31 0)
+			(at 67.31 67.31 0)
 			(hide yes)
 			(show_name no)
@@
 			(project "PS-LVCarrier"
 				(path "/9bab2d9d-20f3-40ef-8545-e1299efec47e/ccdd180d-924e-4cb4-9ad4-e64fe43b7b98"
-					(reference "J13")
+					(reference "J2")
 					(unit 1)
 				)
@@
 	(symbol
 		(lib_id "Device:Fuse")
-		(at 109.22 67.31 90)
+		(at 88.9 67.31 90)
 		(unit 1)
 		(body_style 1)
@@
 		(dnp no)
 		(fields_autoplaced yes)
-		(property "Reference" "F3"
-			(at 109.22 60.96 90)
+		(property "Reference" "F2"
+			(at 88.9 60.96 90)
 			(show_name no)
 			(do_not_autoplace no)
@@
 		)
 		(property "Value" "Fuse"
-			(at 109.22 63.5 90)
+			(at 88.9 63.5 90)
 			(show_name no)
 			(do_not_autoplace no)
@@
 		)
 		(property "Footprint" ""
-			(at 109.22 69.088 90)
+			(at 88.9 69.088 90)
 			(hide yes)
 			(show_name no)
@@
 		)
 		(property "Datasheet" ""
-			(at 109.22 67.31 0)
+			(at 88.9 67.31 0)
 			(hide yes)
 			(show_name no)
@@
 		)
 		(property "Description" "Fuse"
-			(at 109.22 67.31 0)
+			(at 88.9 67.31 0)
 			(hide yes)
 			(show_name no)
@@
 			(project "PS-LVCarrier"
 				(path "/9bab2d9d-20f3-40ef-8545-e1299efec47e/ccdd180d-924e-4cb4-9ad4-e64fe43b7b98"
-					(reference "F3")
+					(reference "F2")
 					(unit 1)
 				)
