File: hardware/lvprecharge.kicad_sch (KiCad schematic)
At the start: 0 parts

Commit message: initial review again
Parts:
- added C7: C_Polarized, symbol Device:C_Polarized
Connections:
- new net LV_GND: C7.2
- new net PCHG_OUT: C7.1
Other:
- added sheet LV EN (LVEN.kicad_sch)
Changed lines of the file:
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@@
 	(generator_version "10.0")
 	(paper "A4")
+	(junction
+		(at 146.05 92.71)
+		(diameter 0)
+		(color 0 0 0 0)
+	)
+	(wire
+		(pts
+			(xy 130.81 92.71) (xy 146.05 92.71)
+		)
+		(stroke
+			(width 0)
+			(type default)
+		)
+	)
+	(wire
+		(pts
+			(xy 100.33 92.71) (xy 106.68 92.71)
+		)
+		(stroke
+			(width 0)
+			(type default)
+		)
+	)
+	(wire
+		(pts
+			(xy 146.05 102.87) (xy 146.05 105.41)
+		)
+		(stroke
+			(width 0)
+			(type default)
+		)
+	)
+	(wire
+		(pts
+			(xy 146.05 95.25) (xy 146.05 92.71)
+		)
+		(stroke
+			(width 0)
+			(type default)
+		)
+	)
+	(wire
+		(pts
+			(xy 146.05 92.71) (xy 163.83 92.71)
+		)
+		(stroke
+			(width 0)
+			(type default)
+		)
+	)
+	(hierarchical_label "LV_GND"
+		(shape input)
+		(at 146.05 105.41 270)
+		(effects
+			(font
+				(size 1.27 1.27)
+			)
+			(justify right)
+		)
+	)
+	(hierarchical_label "PCHG_IN"
+		(shape input)
+		(at 100.33 92.71 180)
+		(effects
+			(font
+				(size 1.27 1.27)
+			)
+			(justify right)
+		)
+	)
+	(hierarchical_label "PCHG_OUT"
+		(shape input)
+		(at 163.83 92.71 0)
+		(effects
+			(font
+				(size 1.27 1.27)
+			)
+			(justify left)
+		)
+	)
+	(symbol
+		(lib_id "Device:C_Polarized")
+		(at 146.05 99.06 0)
+		(unit 1)
+		(body_style 1)
+		(exclude_from_sim no)
+		(in_bom yes)
+		(on_board yes)
+		(in_pos_files yes)
+		(dnp no)
+		(fields_autoplaced yes)
+		(property "Reference" "C7"
+			(at 149.86 96.9009 0)
+			(show_name no)
+			(do_not_autoplace no)
+			(effects
+				(font
+					(size 1.27 1.27)
+				)
+				(justify left)
+			)
+		)
+		(property "Value" "C_Polarized"
+			(at 149.86 99.4409 0)
+			(show_name no)
+			(do_not_autoplace no)
+			(effects
+				(font
+					(size 1.27 1.27)
+				)
+				(justify left)
+			)
+		)
+		(property "Footprint" ""
+			(at 147.0152 102.87 0)
+			(hide yes)
+			(show_name no)
+			(do_not_autoplace no)
+			(effects
+				(font
+					(size 1.27 1.27)
+				)
+			)
+		)
+		(property "Datasheet" ""
+			(at 146.05 99.06 0)
+			(hide yes)
+			(show_name no)
+			(do_not_autoplace no)
+			(effects
+				(font
+					(size 1.27 1.27)
+				)
+			)
+		)
+		(property "Description" "Polarized capacitor"
+			(at 146.05 99.06 0)
+			(hide yes)
+			(show_name no)
+			(do_not_autoplace no)
+			(effects
+				(font
+					(size 1.27 1.27)
+				)
+			)
+		)
+		(pin "2"
+		)
+		(pin "1"
+		)
+		(instances
+			(project "PS-LVCarrier"
+				(path "/9bab2d9d-20f3-40ef-8545-e1299efec47e/aa1bade0-cb25-4e7b-ad0f-e7ef7d6a5bd3"
+					(reference "C7")
+					(unit 1)
+				)
+			)
+		)
+	)
+	(sheet
+		(at 106.68 85.09)
+		(size 24.13 20.32)
+		(exclude_from_sim no)
+		(in_bom yes)
+		(on_board yes)
+		(dnp no)
+		(fields_autoplaced yes)
+		(stroke
+			(width 0.381)
+			(type solid)
+		)
+		(fill
+			(color 0 0 0 0)
+		)
+		(property "Sheetname" "LV EN"
+			(at 106.68 84.2641 0)
+			(show_name no)
+			(do_not_autoplace no)
+			(effects
+				(font
+					(size 1.27 1.27)
+				)
+				(justify left bottom)
+			)
+		)
+		(property "Sheetfile" "LVEN.kicad_sch"
+			(at 106.68 106.1089 0)
+			(show_name no)
+			(do_not_autoplace no)
+			(effects
+				(font
+					(size 1.27 1.27)
+				)
+				(justify left top)
+			)
+		)
+		(instances
+			(project "PS-LVCarrier"
+				(path "/9bab2d9d-20f3-40ef-8545-e1299efec47e/aa1bade0-cb25-4e7b-ad0f-e7ef7d6a5bd3"
+					(page "22")
+				)
+			)
+		)
+	)
 )

Commit message: small change
Parts:
- added F6: Fuse, symbol Device:Fuse
Connections:
- net PCHG_OUT: now also F6.2
Other:
- moved on the sheet: C7
Changed lines of the file:
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@@
 	(paper "A4")
 	(junction
-		(at 146.05 92.71)
+		(at 149.86 92.71)
 		(diameter 0)
 		(color 0 0 0 0)
@@
 	(wire
 		(pts
-			(xy 130.81 92.71) (xy 146.05 92.71)
+			(xy 149.86 92.71) (xy 175.26 92.71)
+		)
+		(stroke
+			(width 0)
+			(type default)
+		)
+	)
+	(wire
+		(pts
+			(xy 130.81 92.71) (xy 135.89 92.71)
+		)
+		(stroke
+			(width 0)
+			(type default)
+		)
+	)
+	(wire
+		(pts
+			(xy 143.51 92.71) (xy 149.86 92.71)
 		)
 		(stroke
@@
 	(wire
 		(pts
-			(xy 146.05 102.87) (xy 146.05 105.41)
-		)
-		(stroke
-			(width 0)
-			(type default)
-		)
-	)
-	(wire
-		(pts
-			(xy 146.05 95.25) (xy 146.05 92.71)
-		)
-		(stroke
-			(width 0)
-			(type default)
-		)
-	)
-	(wire
-		(pts
-			(xy 146.05 92.71) (xy 163.83 92.71)
+			(xy 149.86 102.87) (xy 149.86 105.41)
+		)
+		(stroke
+			(width 0)
+			(type default)
+		)
+	)
+	(wire
+		(pts
+			(xy 149.86 95.25) (xy 149.86 92.71)
 		)
 		(stroke
@@
 	(hierarchical_label "LV_GND"
 		(shape input)
-		(at 146.05 105.41 270)
+		(at 149.86 105.41 270)
 		(effects
 			(font
@@
 	(hierarchical_label "PCHG_OUT"
 		(shape input)
-		(at 163.83 92.71 0)
+		(at 175.26 92.71 0)
 		(effects
 			(font
@@
 	)
 	(symbol
+		(lib_id "Device:Fuse")
+		(at 139.7 92.71 90)
+		(unit 1)
+		(body_style 1)
+		(exclude_from_sim no)
+		(in_bom yes)
+		(on_board yes)
+		(in_pos_files yes)
+		(dnp no)
+		(fields_autoplaced yes)
+		(property "Reference" "F6"
+			(at 139.7 86.36 90)
+			(show_name no)
+			(do_not_autoplace no)
+			(effects
+				(font
+					(size 1.27 1.27)
+				)
+			)
+		)
+		(property "Value" "Fuse"
+			(at 139.7 88.9 90)
+			(show_name no)
+			(do_not_autoplace no)
+			(effects
+				(font
+					(size 1.27 1.27)
+				)
+			)
+		)
+		(property "Footprint" ""
+			(at 139.7 94.488 90)
+			(hide yes)
+			(show_name no)
+			(do_not_autoplace no)
+			(effects
+				(font
+					(size 1.27 1.27)
+				)
+			)
+		)
+		(property "Datasheet" ""
+			(at 139.7 92.71 0)
+			(hide yes)
+			(show_name no)
+			(do_not_autoplace no)
+			(effects
+				(font
+					(size 1.27 1.27)
+				)
+			)
+		)
+		(property "Description" "Fuse"
+			(at 139.7 92.71 0)
+			(hide yes)
+			(show_name no)
+			(do_not_autoplace no)
+			(effects
+				(font
+					(size 1.27 1.27)
+				)
+			)
+		)
+		(pin "1"
+		)
+		(pin "2"
+		)
+		(instances
+			(project "PS-LVCarrier"
+				(path "/9bab2d9d-20f3-40ef-8545-e1299efec47e/aa1bade0-cb25-4e7b-ad0f-e7ef7d6a5bd3"
+					(reference "F6")
+					(unit 1)
+				)
+			)
+		)
+	)
+	(symbol
 		(lib_id "Device:C_Polarized")
-		(at 146.05 99.06 0)
+		(at 149.86 99.06 0)
 		(unit 1)
 		(body_style 1)
@@
 		(fields_autoplaced yes)
 		(property "Reference" "C7"
-			(at 149.86 96.9009 0)
+			(at 153.67 96.9009 0)
 			(show_name no)
 			(do_not_autoplace no)
@@
 		)
 		(property "Value" "C_Polarized"
-			(at 149.86 99.4409 0)
+			(at 153.67 99.4409 0)
 			(show_name no)
 			(do_not_autoplace no)
@@
 		)
 		(property "Footprint" ""
-			(at 147.0152 102.87 0)
+			(at 150.8252 102.87 0)
 			(hide yes)
 			(show_name no)
@@
 		)
 		(property "Datasheet" ""
-			(at 146.05 99.06 0)
+			(at 149.86 99.06 0)
 			(hide yes)
 			(show_name no)
@@
 		)
 		(property "Description" "Polarized capacitor"
-			(at 146.05 99.06 0)
-			(hide yes)
-			(show_name no)
+			(at 149.86 99.06 0)
+			(hide yes)
+			(show_name no)

Commit message: progress!
Changed lines of the file:
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@@
 	(wire
 		(pts
-			(xy 100.33 92.71) (xy 106.68 92.71)
+			(xy 92.71 92.71) (xy 106.68 92.71)
 		)
 		(stroke
@@
 	(hierarchical_label "PCHG_IN"
 		(shape input)
-		(at 100.33 92.71 180)
+		(at 92.71 92.71 180)
 		(effects
 			(font
@@
 		(instances
 			(project "PS-LVCarrier"
-				(path "/9bab2d9d-20f3-40ef-8545-e1299efec47e/aa1bade0-cb25-4e7b-ad0f-e7ef7d6a5bd3"
+				(path "/9bab2d9d-20f3-40ef-8545-e1299efec47e/10a2a81d-fff8-4091-b6ef-9685e4bd9514/eb8c4e9b-3c3c-4615-8f78-813806fe2364"
 					(reference "F6")
 					(unit 1)
@@
 		(instances
 			(project "PS-LVCarrier"
-				(path "/9bab2d9d-20f3-40ef-8545-e1299efec47e/aa1bade0-cb25-4e7b-ad0f-e7ef7d6a5bd3"
+				(path "/9bab2d9d-20f3-40ef-8545-e1299efec47e/10a2a81d-fff8-4091-b6ef-9685e4bd9514/eb8c4e9b-3c3c-4615-8f78-813806fe2364"
 					(reference "C7")
 					(unit 1)
@@
 		(instances
 			(project "PS-LVCarrier"
-				(path "/9bab2d9d-20f3-40ef-8545-e1299efec47e/aa1bade0-cb25-4e7b-ad0f-e7ef7d6a5bd3"
-					(page "22")
-				)
-			)
+				(path "/9bab2d9d-20f3-40ef-8545-e1299efec47e/10a2a81d-fff8-4091-b6ef-9685e4bd9514/eb8c4e9b-3c3c-4615-8f78-813806fe2364"
+					(page "20")
+				)
+			)

Commit message: addressed da review and fixed some stuff, pushhhhhh
Parts:
- removed C7: C_Polarized, symbol Device:C_Polarized
- added C40: C_Polarized_US, symbol Device:C_Polarized_US
Connections:
- net LV_GND: now also C40.2
- net PCHG_OUT: now also C40.1
Other:
- moved on the sheet: F6
Changed lines of the file:
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@@
 	(generator "eeschema")
 	(generator_version "10.0")
-	(paper "A4")
+	(paper "A5")
 	(junction
-		(at 149.86 92.71)
+		(at 123.19 64.77)
 		(diameter 0)
 		(color 0 0 0 0)
@@
 	(wire
 		(pts
-			(xy 149.86 92.71) (xy 175.26 92.71)
-		)
-		(stroke
-			(width 0)
-			(type default)
-		)
-	)
-	(wire
-		(pts
-			(xy 130.81 92.71) (xy 135.89 92.71)
-		)
-		(stroke
-			(width 0)
-			(type default)
-		)
-	)
-	(wire
-		(pts
-			(xy 143.51 92.71) (xy 149.86 92.71)
-		)
-		(stroke
-			(width 0)
-			(type default)
-		)
-	)
-	(wire
-		(pts
-			(xy 92.71 92.71) (xy 106.68 92.71)
-		)
-		(stroke
-			(width 0)
-			(type default)
-		)
-	)
-	(wire
-		(pts
-			(xy 149.86 102.87) (xy 149.86 105.41)
-		)
-		(stroke
-			(width 0)
-			(type default)
-		)
-	)
-	(wire
-		(pts
-			(xy 149.86 95.25) (xy 149.86 92.71)
+			(xy 123.19 64.77) (xy 148.59 64.77)
+		)
+		(stroke
+			(width 0)
+			(type default)
+		)
+	)
+	(wire
+		(pts
+			(xy 104.14 64.77) (xy 109.22 64.77)
+		)
+		(stroke
+			(width 0)
+			(type default)
+		)
+	)
+	(wire
+		(pts
+			(xy 116.84 64.77) (xy 123.19 64.77)
+		)
+		(stroke
+			(width 0)
+			(type default)
+		)
+	)
+	(wire
+		(pts
+			(xy 66.04 64.77) (xy 80.01 64.77)
+		)
+		(stroke
+			(width 0)
+			(type default)
+		)
+	)
+	(wire
+		(pts
+			(xy 123.19 74.93) (xy 123.19 77.47)
+		)
+		(stroke
+			(width 0)
+			(type default)
+		)
+	)
+	(wire
+		(pts
+			(xy 123.19 67.31) (xy 123.19 64.77)
 		)
 		(stroke
@@
 	(hierarchical_label "LV_GND"
 		(shape input)
-		(at 149.86 105.41 270)
+		(at 123.19 77.47 270)
 		(effects
 			(font
@@
 	(hierarchical_label "PCHG_IN"
 		(shape input)
-		(at 92.71 92.71 180)
+		(at 66.04 64.77 180)
 		(effects
 			(font
@@
 	(hierarchical_label "PCHG_OUT"
 		(shape input)
-		(at 175.26 92.71 0)
+		(at 148.59 64.77 0)
 		(effects
 			(font
@@
 	(symbol
 		(lib_id "Device:Fuse")
-		(at 139.7 92.71 90)
+		(at 113.03 64.77 90)
 		(unit 1)
 		(body_style 1)
@@
 		(fields_autoplaced yes)
 		(property "Reference" "F6"
-			(at 139.7 86.36 90)
+			(at 113.03 58.42 90)
 			(show_name no)
 			(do_not_autoplace no)
@@
 		)
 		(property "Value" "Fuse"
-			(at 139.7 88.9 90)
+			(at 113.03 60.96 90)
 			(show_name no)
 			(do_not_autoplace no)
@@
 		)
 		(property "Footprint" ""
-			(at 139.7 94.488 90)
+			(at 113.03 66.548 90)
 			(hide yes)
 			(show_name no)
@@
 		)
 		(property "Datasheet" ""
-			(at 139.7 92.71 0)
+			(at 113.03 64.77 0)
 			(hide yes)
 			(show_name no)
@@
 		)
 		(property "Description" "Fuse"
-			(at 139.7 92.71 0)
+			(at 113.03 64.77 0)
 			(hide yes)
 			(show_name no)
@@
 	)
 	(symbol
-		(lib_id "Device:C_Polarized")
-		(at 149.86 99.06 0)
+		(lib_id "Device:C_Polarized_US")
+		(at 123.19 71.12 0)
 		(unit 1)
 		(body_style 1)
@@
 		(dnp no)
 		(fields_autoplaced yes)
-		(property "Reference" "C7"
-			(at 153.67 96.9009 0)
+		(property "Reference" "C40"
+			(at 127 69.2149 0)
 			(show_name no)
 			(do_not_autoplace no)
@@
 			)
 		)
-		(property "Value" "C_Polarized"
-			(at 153.67 99.4409 0)
+		(property "Value" "C_Polarized_US"
+			(at 127 71.7549 0)
 			(show_name no)
 			(do_not_autoplace no)
@@
 		)
 		(property "Footprint" ""
-			(at 150.8252 102.87 0)
+			(at 123.19 71.12 0)
 			(hide yes)
 			(show_name no)
@@
 		)
 		(property "Datasheet" ""
-			(at 149.86 99.06 0)
-			(hide yes)
-			(show_name no)
-			(do_not_autoplace no)
-			(effects
-				(font
-					(size 1.27 1.27)
-				)
-			)
-		)
-		(property "Description" "Polarized capacitor"
-			(at 149.86 99.06 0)
+			(at 123.19 71.12 0)
+			(hide yes)
+			(show_name no)
+			(do_not_autoplace no)
+			(effects
+				(font
+					(size 1.27 1.27)
+				)
+			)
+		)
+		(property "Description" "Polarized capacitor, US symbol"
+			(at 123.19 71.12 0)
 			(hide yes)
 			(show_name no)
@@
 			(project "PS-LVCarrier"
 				(path "/9bab2d9d-20f3-40ef-8545-e1299efec47e/10a2a81d-fff8-4091-b6ef-9685e4bd9514/eb8c4e9b-3c3c-4615-8f78-813806fe2364"
-					(reference "C7")
+					(reference "C40")
 					(unit 1)
 				)
@@
 	)
 	(sheet
-		(at 106.68 85.09)
+		(at 80.01 57.15)
 		(size 24.13 20.32)
 		(exclude_from_sim no)
@@
 		)
 		(property "Sheetname" "LV EN"
-			(at 106.68 84.2641 0)
+			(at 80.01 56.3241 0)
 			(show_name no)
 			(do_not_autoplace no)
@@
 		)
 		(property "Sheetfile" "LVEN.kicad_sch"
-			(at 106.68 106.1089 0)
-			(show_name no)
-			(do_not_autoplace no)
+			(at 80.01 78.1689 0)
+			(show_name no)
+			(do_not_autoplace no)

Commit message: review ts
Parts:
- renumbered C40 to C43, F6 to F10
Changed lines of the file:
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@@
 		(dnp no)
 		(fields_autoplaced yes)
-		(property "Reference" "F6"
+		(property "Reference" "F10"
 			(at 113.03 58.42 90)
 			(show_name no)
@@
 			(project "PS-LVCarrier"
 				(path "/9bab2d9d-20f3-40ef-8545-e1299efec47e/10a2a81d-fff8-4091-b6ef-9685e4bd9514/eb8c4e9b-3c3c-4615-8f78-813806fe2364"
-					(reference "F6")
+					(reference "F10")
 					(unit 1)
 				)
@@
 		(dnp no)
 		(fields_autoplaced yes)
-		(property "Reference" "C40"
+		(property "Reference" "C43"
 			(at 127 69.2149 0)
 			(show_name no)
@@
 			(project "PS-LVCarrier"
 				(path "/9bab2d9d-20f3-40ef-8545-e1299efec47e/10a2a81d-fff8-4091-b6ef-9685e4bd9514/eb8c4e9b-3c3c-4615-8f78-813806fe2364"
-					(reference "C40")
+					(reference "C43")
 					(unit 1)
 				)

Commit message: save
Connections:
- net PCHG_IN: now also F10.1
Other:
- removed sheet LV EN
Changed lines of the file:
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@@
-	(wire
-		(pts
-			(xy 104.14 64.77) (xy 109.22 64.77)
-		)
-		(stroke
-			(width 0)
-			(type default)
-		)
-	)
 	(wire
 		(pts
@@
 	(wire
 		(pts
-			(xy 66.04 64.77) (xy 80.01 64.77)
+			(xy 66.04 64.77) (xy 109.22 64.77)
 		)
 		(stroke
@@
 				)
 			)
-		)
-	)
-	(sheet
-		(at 80.01 57.15)
-		(size 24.13 20.32)
-		(exclude_from_sim no)
-		(in_bom yes)
-		(on_board yes)
-		(dnp no)
-		(fields_autoplaced yes)
-		(stroke
-			(width 0.381)
-			(type solid)
-		)
-		(fill
-			(color 0 0 0 0)
-		)
-		(property "Sheetname" "LV EN"
-			(at 80.01 56.3241 0)
-			(show_name no)
-			(do_not_autoplace no)
-			(effects
-				(font
-					(size 1.27 1.27)
-				)
-				(justify left bottom)
-			)
-		)
-		(property "Sheetfile" "LVEN.kicad_sch"
-			(at 80.01 78.1689 0)
-			(show_name no)
-			(do_not_autoplace no)
-			(effects
-				(font
-					(size 1.27 1.27)
-				)
-				(justify left top)
-			)
-		)
-		(instances
-			(project "PS-LVCarrier"
-				(path "/9bab2d9d-20f3-40ef-8545-e1299efec47e/10a2a81d-fff8-4091-b6ef-9685e4bd9514/eb8c4e9b-3c3c-4615-8f78-813806fe2364"
-					(page "20")
-				)
-			)
