File: hardware/hvbattery.kicad_sch (KiCad schematic)
At the start: 0 parts

Commit message: initial review again
Other:
- added sheet HV -> 12V (HV_converter.kicad_sch)
- added sheet HV Input (HV_protection.kicad_sch)
- note added: "HV input protection + sensing"
- note added: "HV vicor + sensing"

Commit message: progress!
Parts:
- added F7: TBD until vicor confirmed, LHRS_Power:Fuse-3557-2, symbol Device:Fuse
Connections:
- new net HV -> 12V/HV_24V_OUT: F7.1
- new net HV_12V_FUSED: F7.2

Commit message: addressed da review and fixed some stuff, pushhhhhh
Other:
- sheet HV -> 12V ports: added HV_VICOR_EN; removed none
Changed lines of the file:
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@@
+	(wire
+		(pts
+			(xy 146.05 71.12) (xy 149.86 71.12)
+		)
+		(stroke
+			(width 0)
+			(type default)
+		)
+	)
 	(wire
 		(pts
@@
 		(shape input)
 		(at 149.86 63.5 0)
+		(effects
+			(font
+				(size 1.27 1.27)
+			)
+			(justify left)
+		)
+	)
+	(hierarchical_label "HV_VICOR_EN"
+		(shape input)
+		(at 149.86 71.12 0)
 		(effects
 			(font
@@
 			(effects
 				(font
+					(size 1.27 1.27)
+				)
+				(justify right)
+			)
+		)
+		(pin "HV_VICOR_EN" input
+			(at 146.05 71.12 0)
+			(effects
+				(font

Commit message: review ts
Parts:
- renumbered F7 to F3
Changed lines of the file:
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@@
 		(dnp no)
 		(fields_autoplaced yes)
-		(property "Reference" "#PWR05"
+		(property "Reference" "#PWR014"
 			(at 100.33 87.63 0)
 			(hide yes)
@@
 			(project "PS-LVCarrier"
 				(path "/9bab2d9d-20f3-40ef-8545-e1299efec47e/4f26e4eb-a337-4f9d-865d-e2c0801c36ac"
-					(reference "#PWR05")
+					(reference "#PWR014")
 					(unit 1)
 				)
@@
 		(dnp no)
 		(fields_autoplaced yes)
-		(property "Reference" "F7"
+		(property "Reference" "F3"
 			(at 160.02 52.07 90)
 			(show_name no)
@@
 			(project "PS-LVCarrier"
 				(path "/9bab2d9d-20f3-40ef-8545-e1299efec47e/4f26e4eb-a337-4f9d-865d-e2c0801c36ac"
-					(reference "F7")
+					(reference "F3")
 					(unit 1)
 				)
@@
 		(dnp no)
 		(fields_autoplaced yes)
-		(property "Reference" "#PWR04"
+		(property "Reference" "#PWR013"
 			(at 87.63 87.63 0)
 			(hide yes)
@@
 			(project "PS-LVCarrier"
 				(path "/9bab2d9d-20f3-40ef-8545-e1299efec47e/4f26e4eb-a337-4f9d-865d-e2c0801c36ac"
-					(reference "#PWR04")
+					(reference "#PWR013")
 					(unit 1)
 				)
@@
 		(dnp no)
 		(fields_autoplaced yes)
-		(property "Reference" "#PWR01"
+		(property "Reference" "#PWR012"
 			(at 38.1 87.63 0)
 			(hide yes)
@@
 			(project "PS-LVCarrier"
 				(path "/9bab2d9d-20f3-40ef-8545-e1299efec47e/4f26e4eb-a337-4f9d-865d-e2c0801c36ac"
-					(reference "#PWR01")
+					(reference "#PWR012")
 					(unit 1)
 				)
@@
 		(dnp no)
 		(fields_autoplaced yes)
-		(property "Reference" "#PWR07"
+		(property "Reference" "#PWR015"
 			(at 151.13 87.63 0)
 			(hide yes)
@@
 			(project "PS-LVCarrier"
 				(path "/9bab2d9d-20f3-40ef-8545-e1299efec47e/4f26e4eb-a337-4f9d-865d-e2c0801c36ac"
-					(reference "#PWR07")
-					(unit 1)
-				)
+					(reference "#PWR015")
+					(unit 1)
+				)

Commit message: review me pt2
Changed lines of the file:
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@@
 	)
 	(hierarchical_label "HV_VICOR_TEMP"
-		(shape input)
+		(shape output)
 		(at 149.86 68.58 0)
 		(effects
@@
 	)
 	(hierarchical_label "{HV_DCDC_FLT}"
-		(shape input)
+		(shape output)
 		(at 149.86 66.04 0)
 		(effects
@@
 	)
 	(hierarchical_label "HV_IN_VFAULT"
-		(shape input)
+		(shape output)
 		(at 85.09 66.04 0)
 		(effects
@@
 	)
 	(hierarchical_label "{HV_OUT_ADC}"
-		(shape input)
+		(shape output)
 		(at 149.86 63.5 0)
 		(effects
@@
 	)
 	(hierarchical_label "{HV_IN_ADC}"
-		(shape input)
+		(shape output)
 		(at 85.09 63.5 0)
 		(effects

Commit message: addressed
Changed lines of the file:
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@@
 	(wire
 		(pts
-			(xy 163.83 58.42) (xy 166.37 58.42)
+			(xy 163.83 58.42) (xy 168.91 58.42)
 		)
 		(stroke
@@
 	(hierarchical_label "HV_12V_FUSED"
 		(shape output)
-		(at 166.37 58.42 0)
+		(at 168.91 58.42 0)
 		(effects
 			(font
@@
 			(project "PS-LVCarrier"
 				(path "/9bab2d9d-20f3-40ef-8545-e1299efec47e/4f26e4eb-a337-4f9d-865d-e2c0801c36ac"
-					(page "14")
+					(page "10")
 				)
 			)
@@
 			(project "PS-LVCarrier"
 				(path "/9bab2d9d-20f3-40ef-8545-e1299efec47e/4f26e4eb-a337-4f9d-865d-e2c0801c36ac"
-					(page "15")
-				)
-			)
+					(page "11")
+				)
+			)

Commit message: switch for laptop
Other:
- sheet HV -> 12V ports: added none; removed {HV_DCDC_FLT}
Changed lines of the file:
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@@
 	(wire
 		(pts
-			(xy 146.05 71.12) (xy 149.86 71.12)
+			(xy 146.05 68.58) (xy 149.86 68.58)
 		)
 		(stroke
@@
 		)
 	)
-	(bus
+	(wire
+		(pts
+			(xy 100.33 80.01) (xy 105.41 80.01)
+		)
+		(stroke
+			(width 0.381)
+			(type default)
+		)
+	)
+	(wire
+		(pts
+			(xy 87.63 80.01) (xy 82.55 80.01)
+		)
+		(stroke
+			(width 0.381)
+			(type default)
+		)
+	)
+	(wire
 		(pts
 			(xy 146.05 66.04) (xy 149.86 66.04)
-		)
-		(stroke
-			(width 0)
-			(type default)
-		)
-	)
-	(wire
-		(pts
-			(xy 100.33 80.01) (xy 105.41 80.01)
-		)
-		(stroke
-			(width 0.381)
-			(type default)
-		)
-	)
-	(wire
-		(pts
-			(xy 87.63 80.01) (xy 82.55 80.01)
-		)
-		(stroke
-			(width 0.381)
-			(type default)
-		)
-	)
-	(wire
-		(pts
-			(xy 146.05 68.58) (xy 149.86 68.58)
 		)
 		(stroke
@@
 	(hierarchical_label "HV_VICOR_TEMP"
 		(shape output)
-		(at 149.86 68.58 0)
-		(effects
-			(font
-				(size 1.27 1.27)
-			)
-			(justify left)
-		)
-	)
-	(hierarchical_label "{HV_DCDC_FLT}"
-		(shape output)
 		(at 149.86 66.04 0)
 		(effects
@@
 	(hierarchical_label "HV_VICOR_EN"
 		(shape input)
-		(at 149.86 71.12 0)
+		(at 149.86 68.58 0)
 		(effects
 			(font
@@
 			)
 		)
-		(pin "HV_GND" passive
+		(pin "HV_GND" input
 			(at 105.41 80.01 180)
 			(effects
@@
 		)
 		(pin "HV_VICOR_TEMP" output
-			(at 146.05 68.58 0)
+			(at 146.05 66.04 0)
 			(effects
 				(font
@@
 			)
 		)
-		(pin "LV_GND" passive
+		(pin "LV_GND" input
 			(at 146.05 80.01 0)
 			(effects
@@
 			)
 		)
-		(pin "{HV_DCDC_FLT}" output
-			(at 146.05 66.04 0)
-			(effects
-				(font
-					(size 1.27 1.27)
-				)
-				(justify right)
-			)
-		)
 		(pin "HV_VICOR_EN" input
-			(at 146.05 71.12 0)
-			(effects
-				(font
+			(at 146.05 68.58 0)
+			(effects
+				(font

Commit message: update kicad sharepoint
Other:
- sheet HV -> 12V ports: added HV_DCDC_EN, HV_DCDC_TEMP; removed HV_VICOR_EN, HV_VICOR_TEMP
Changed lines of the file:
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@@
 		)
 	)
-	(hierarchical_label "HV_VICOR_TEMP"
+	(hierarchical_label "HV_DCDC_TEMP"
 		(shape output)
 		(at 149.86 66.04 0)
@@
 		)
 	)
-	(hierarchical_label "HV_VICOR_EN"
+	(hierarchical_label "HV_DCDC_EN"
 		(shape input)
 		(at 149.86 68.58 0)
@@
 		)
 		(property "LCSC P/N" "C352820"
+			(at 160.02 58.42 90)
+			(hide yes)
+			(show_name no)
+			(do_not_autoplace no)
+			(effects
+				(font
+					(size 1.27 1.27)
+				)
+			)
+		)
+		(property "LCSC" ""
 			(at 160.02 58.42 90)
 			(hide yes)
@@
 			)
 		)
-		(pin "HV_IN" input
+		(pin "HV_IN" output
 			(at 105.41 58.42 180)
 			(effects
@@
 			)
 		)
-		(pin "HV_VICOR_TEMP" output
+		(pin "HV_DCDC_TEMP" output
 			(at 146.05 66.04 0)
 			(effects
@@
 			)
 		)
-		(pin "HV_VICOR_EN" input
+		(pin "HV_DCDC_EN" input
 			(at 146.05 68.58 0)
 			(effects
