File: hardware/MCU.kicad_sch (KiCad schematic)
At the start: 5 parts

Commit message: save
Parts:
- added R101, R102, R103, R106, R107: 10k, symbol Device:R
- added R104, R105: 22, symbol Device:R
Connections:
- net DI_MODE: now also R107.2
- net LIMP_HOME: now also R101.2
- net LV_GND: now also R101.1, R102.1, R106.1, R107.1
- net MISO: now also R103.1
- net MOSI: now also R104.2
- net SCLK: now also R105.2
- new net +3V3: R103.2
- new net HSS_MOSI: R102.2, R104.1, R105.1, R106.2

Commit message: review me pt2
Connections:
- no-connect marks 45 -> 49
Changed lines of the file:
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@@
 	)
 	(no_connect
+		(at 287.02 149.86)
+	)
+	(no_connect
 		(at 368.3 86.36)
 	)
@@
 	)
 	(no_connect
+		(at 287.02 118.11)
+	)
+	(no_connect
 		(at 287.02 160.02)
 	)
@@
 	)
 	(no_connect
-		(at 368.3 71.12)
+		(at 287.02 115.57)
 	)
 	(no_connect
@@
 	)
 	(no_connect
+		(at 287.02 154.94)
+	)
+	(no_connect
 		(at 368.3 110.49)
 	)
@@
 	)
 	(no_connect
+		(at 287.02 123.19)
+	)
+	(no_connect
 		(at 287.02 120.65)
 	)
@@
 	)
 	(no_connect
-		(at 368.3 73.66)
-	)
-	(no_connect
 		(at 368.3 88.9)
 	)
@@
 	)
 	(no_connect
+		(at 287.02 152.4)
+	)
+	(no_connect
 		(at 368.3 113.03)
 	)
@@
 	)
 	(no_connect
-		(at 368.3 76.2)
+		(at 368.3 58.42)
 	)
 	(no_connect
@@
 	)
 	(bus_entry
-		(at 273.05 123.19)
-		(size -2.54 -2.54)
-		(stroke
-			(width 0)
-			(type default)
-		)
-	)
-	(bus_entry
 		(at 273.05 95.25)
 		(size 2.54 2.54)
@@
 	)
 	(bus_entry
-		(at 273.05 149.86)
-		(size -2.54 -2.54)
-		(stroke
-			(width 0)
-			(type default)
-		)
-	)
-	(bus_entry
 		(at 273.05 63.5)
 		(size 2.54 2.54)
@@
 	)
 	(bus_entry
-		(at 273.05 115.57)
-		(size -2.54 -2.54)
-		(stroke
-			(width 0)
-			(type default)
-		)
-	)
-	(bus_entry
 		(at 273.05 60.96)
 		(size 2.54 2.54)
@@
 	)
 	(bus_entry
-		(at 273.05 152.4)
-		(size -2.54 -2.54)
-		(stroke
-			(width 0)
-			(type default)
-		)
-	)
-	(bus_entry
-		(at 273.05 118.11)
-		(size -2.54 -2.54)
-		(stroke
-			(width 0)
-			(type default)
-		)
-	)
-	(bus_entry
-		(at 273.05 154.94)
-		(size -2.54 -2.54)
-		(stroke
-			(width 0)
-			(type default)
-		)
-	)
-	(bus_entry
 		(at 274.32 236.22)
 		(size 2.54 2.54)
@@
 	(wire
 		(pts
-			(xy 273.05 154.94) (xy 287.02 154.94)
-		)
-		(stroke
-			(width 0)
-			(type default)
-		)
-	)
-	(wire
-		(pts
 			(xy 292.1 238.76) (xy 292.1 241.3)
 		)
@@
 	(wire
 		(pts
-			(xy 273.05 149.86) (xy 287.02 149.86)
+			(xy 368.3 73.66) (xy 369.57 73.66)
 		)
 		(stroke
@@
 	(wire
 		(pts
-			(xy 273.05 123.19) (xy 287.02 123.19)
-		)
-		(stroke
-			(width 0)
-			(type default)
-		)
-	)
-	(wire
-		(pts
-			(xy 368.3 58.42) (xy 369.57 58.42)
+			(xy 368.3 76.2) (xy 369.57 76.2)
 		)
 		(stroke
@@
 	(wire
 		(pts
-			(xy 273.05 115.57) (xy 287.02 115.57)
-		)
-		(stroke
-			(width 0)
-			(type default)
-		)
-	)
-	(bus
-		(pts
-			(xy 270.51 146.05) (xy 270.51 152.4)
-		)
-		(stroke
-			(width 0)
-			(type default)
-		)
-	)
-	(wire
-		(pts
 			(xy 275.59 95.25) (xy 287.02 95.25)
 		)
@@
 	(wire
 		(pts
-			(xy 273.05 152.4) (xy 287.02 152.4)
+			(xy 368.3 160.02) (xy 373.38 160.02)
 		)
 		(stroke
@@
 	(wire
 		(pts
-			(xy 368.3 160.02) (xy 373.38 160.02)
+			(xy 368.3 71.12) (xy 369.57 71.12)
 		)
 		(stroke
@@
 	(wire
 		(pts
-			(xy 369.57 77.47) (xy 368.3 78.74)
+			(xy 369.57 78.74) (xy 368.3 78.74)
 		)
 		(stroke
@@
 	(wire
 		(pts
-			(xy 273.05 118.11) (xy 287.02 118.11)
-		)
-		(stroke
-			(width 0)
-			(type default)
-		)
-	)
-	(wire
-		(pts
 			(xy 368.3 102.87) (xy 382.27 102.87)
 		)
@@
 		)
 	)
-	(bus
-		(pts
-			(xy 270.51 111.76) (xy 270.51 120.65)
-		)
-		(stroke
-			(width 0)
-			(type default)
-		)
-	)
 	(image
 		(at 131.826 149.352)
@@
 		)
 	)
-	(label "DISPLAY_RST"
-		(at 273.05 152.4 0)
-		(effects
-			(font
-				(size 1.27 1.27)
-			)
-			(justify left bottom)
-		)
-	)
 	(label "MOSI"
 		(at 262.89 189.23 0)
@@
 		)
 	)
-	(label "DISPLAY_MOSI"
-		(at 273.05 123.19 0)
-		(effects
-			(font
-				(size 1.27 1.27)
-			)
-			(justify left bottom)
-		)
-	)
 	(label "HV_OUT_I"
 		(at 275.59 66.04 0)
@@
 		)
 	)
-	(label "DISPLAY_CS"
-		(at 273.05 115.57 0)
-		(effects
-			(font
-				(size 1.27 1.27)
-			)
-			(justify left bottom)
-		)
-	)
 	(label "LIMP_HOME"
 		(at 261.62 215.9 180)
@@
 		)
 	)
-	(label "DISPLAY_SCK"
-		(at 273.05 118.11 0)
-		(effects
-			(font
-				(size 1.27 1.27)
-			)
-			(justify left bottom)
-		)
-	)
 	(label "SCLK"
 		(at 276.86 238.76 0)
@@
 		)
 	)
-	(label "DISPLAY_GPIO"
-		(at 273.05 154.94 0)
-		(effects
-			(font
-				(size 1.27 1.27)
-			)
-			(justify left bottom)
-		)
-	)
 	(label "I2C_SCL"
 		(at 275.59 81.28 0)
@@
 		)
 	)
-	(label "DISPLAY_DC"
-		(at 273.05 149.86 0)
-		(effects
-			(font
-				(size 1.27 1.27)
-			)
-			(justify left bottom)
-		)
-	)
 	(label "HSS_MOSI"
 		(at 285.75 189.23 180)
@@
 	)
 	(hierarchical_label "CHARGE_EN"
-		(shape input)
-		(at 369.57 58.42 0)
+		(shape output)
+		(at 369.57 76.2 0)
 		(effects
 			(font
@@
 	(hierarchical_label "HV_IN_VFAULT"
 		(shape input)
-		(at 369.57 77.47 0)
+		(at 369.57 78.74 0)
 		(effects
 			(font
@@
 		)
 	)
+	(hierarchical_label "LVD_RESET"
+		(shape input)
+		(at 369.57 73.66 0)
+		(effects
+			(font
+				(size 1.27 1.27)
+			)
+			(justify left)
+		)
+	)
 	(hierarchical_label "{SUPP_ADC}"
 		(shape input)
@@
 		)
 	)
+	(hierarchical_label "LV_EN_3V3"
+		(shape input)
+		(at 369.57 71.12 0)
+		(effects
+			(font
+				(size 1.27 1.27)
+			)
+			(justify left)
+		)
+	)
 	(hierarchical_label "{HV_IN_ADC}"
 		(shape input)
@@
 	)
 	(hierarchical_label "{I2C}"
-		(shape input)
+		(shape bidirectional)
 		(at 273.05 77.47 180)
 		(effects
@@
 		)
 	)
-	(hierarchical_label "{DISPLAY_SPI}"
-		(shape bidirectional)
-		(at 270.51 111.76 180)
-		(effects
-			(font
-				(size 1.27 1.27)
-			)
-			(justify right)
-		)
-	)
 	(hierarchical_label "{HV_FAULT}"
 		(shape input)
@@
 	)
 	(hierarchical_label "LV_GND"
-		(shape passive)
+		(shape input)
 		(at 344.17 199.39 270)
 		(effects
@@
 	)
 	(hierarchical_label "{I2C}"
-		(shape input)
+		(shape bidirectional)
 		(at 271.78 105.41 180)
 		(effects
@@
 		)
 	)
-	(hierarchical_label "{DISPLAY_SPI}"
-		(shape bidirectional)
-		(at 270.51 146.05 180)
-		(effects
-			(font
-				(size 1.27 1.27)
-			)
-			(justify right)
-		)
-	)
 	(hierarchical_label "LV_GND"
 		(shape input)
@@
 	)
 	(hierarchical_label "LV_GND"
-		(shape passive)
+		(shape input)
 		(at 373.38 160.02 270)
 		(effects
@@
 	)
 	(hierarchical_label "HV_VICOR_EN"
-		(shape input)
+		(shape output)
 		(at 369.57 60.96 0)
 		(effects
@@
 	)
 	(hierarchical_label "LV_GND"
-		(shape passive)
+		(shape input)
 		(at 327.66 199.39 270)
 		(effects

Commit message: review me pt 3
Connections:
- no-connect marks 49 -> 45
Changed lines of the file:
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@@
 	)
 	(no_connect
-		(at 287.02 90.17)
-	)
-	(no_connect
 		(at 287.02 154.94)
 	)
 	(no_connect
-		(at 368.3 110.49)
-	)
-	(no_connect
 		(at 287.02 78.74)
 	)
@@
 	)
 	(no_connect
-		(at 368.3 113.03)
-	)
-	(no_connect
 		(at 368.3 133.35)
 	)
@@
 		(at 368.3 149.86)
 	)
-	(no_connect
-		(at 287.02 87.63)
-	)
 	(bus_entry
 		(at 383.54 63.5)
@@
 	)
 	(bus_entry
+		(at 273.05 85.09)
+		(size 2.54 2.54)
+		(stroke
+			(width 0)
+			(type default)
+		)
+	)
+	(bus_entry
 		(at 273.05 95.25)
 		(size 2.54 2.54)
@@
 	)
 	(bus_entry
+		(at 384.81 114.3)
+		(size -2.54 -2.54)
+		(stroke
+			(width 0)
+			(type default)
+		)
+	)
+	(bus_entry
 		(at 273.05 63.5)
 		(size 2.54 2.54)
@@
 	)
 	(bus_entry
+		(at 273.05 87.63)
+		(size 2.54 2.54)
+		(stroke
+			(width 0)
+			(type default)
+		)
+	)
+	(bus_entry
 		(at 273.05 58.42)
 		(size 2.54 2.54)
@@
 	)
 	(bus_entry
+		(at 384.81 116.84)
+		(size -2.54 -2.54)
+		(stroke
+			(width 0)
+			(type default)
+		)
+	)
+	(bus_entry
 		(at 270.51 137.16)
 		(size 2.54 2.54)
@@
 	(wire
 		(pts
+			(xy 372.11 114.3) (xy 382.27 114.3)
+		)
+		(stroke
+			(width 0)
+			(type default)
+		)
+	)
+	(wire
+		(pts
 			(xy 368.3 73.66) (xy 369.57 73.66)
 		)
@@
 		)
 	)
+	(bus
+		(pts
+			(xy 384.81 114.3) (xy 384.81 118.11)
+		)
+		(stroke
+			(width 0)
+			(type default)
+		)
+	)
 	(wire
 		(pts
@@
 	(wire
 		(pts
+			(xy 275.59 90.17) (xy 287.02 90.17)
+		)
+		(stroke
+			(width 0)
+			(type default)
+		)
+	)
+	(wire
+		(pts
 			(xy 275.59 58.42) (xy 287.02 58.42)
 		)
@@
 	(wire
 		(pts
+			(xy 372.11 110.49) (xy 368.3 110.49)
+		)
+		(stroke
+			(width 0)
+			(type default)
+		)
+	)
+	(wire
+		(pts
 			(xy 287.02 100.33) (xy 279.4 100.33)
 		)
@@
 	(wire
 		(pts
+			(xy 275.59 87.63) (xy 287.02 87.63)
+		)
+		(stroke
+			(width 0)
+			(type default)
+		)
+	)
+	(wire
+		(pts
 			(xy 275.59 50.8) (xy 276.86 50.8)
 		)
@@
 	(wire
 		(pts
+			(xy 372.11 111.76) (xy 372.11 110.49)
+		)
+		(stroke
+			(width 0)
+			(type default)
+		)
+	)
+	(wire
+		(pts
 			(xy 327.66 179.07) (xy 327.66 180.34)
 		)
@@
 	(wire
 		(pts
+			(xy 372.11 113.03) (xy 372.11 114.3)
+		)
+		(stroke
+			(width 0)
+			(type default)
+		)
+	)
+	(wire
+		(pts
 			(xy 275.59 63.5) (xy 287.02 63.5)
 		)
@@
 	(wire
 		(pts
+			(xy 368.3 113.03) (xy 372.11 113.03)
+		)
+		(stroke
+			(width 0)
+			(type default)
+		)
+	)
+	(wire
+		(pts
 			(xy 369.57 78.74) (xy 368.3 78.74)
 		)
@@
 	(bus
 		(pts
+			(xy 273.05 83.82) (xy 273.05 87.63)
+		)
+		(stroke
+			(width 0)
+			(type default)
+		)
+	)
+	(bus
+		(pts
 			(xy 273.05 62.23) (xy 273.05 63.5)
 		)
@@
 	(wire
 		(pts
+			(xy 372.11 111.76) (xy 382.27 111.76)
+		)
+		(stroke
+			(width 0)
+			(type default)
+		)
+	)
+	(wire
+		(pts
 			(xy 292.1 238.76) (xy 289.56 238.76)
 		)
@@
 		)
 	)
+	(label "LV_ISNS"
+		(at 275.59 87.63 0)
+		(effects
+			(font
+				(size 1.27 1.27)
+			)
+			(justify left bottom)
+		)
+	)
 	(label "DI_MODE"
 		(at 273.05 144.78 0)
@@
 		)
 	)
+	(label "CHG_PG"
+		(at 382.27 111.76 180)
+		(effects
+			(font
+				(size 1.27 1.27)
+			)
+			(justify right bottom)
+		)
+	)
 	(label "DI_MODE"
 		(at 316.23 217.17 0)
@@
 		)
 	)
+	(label "LV_VSNS"
+		(at 275.59 90.17 0)
+		(effects
+			(font
+				(size 1.27 1.27)
+			)
+			(justify left bottom)
+		)
+	)
 	(label "USBD+"
 		(at 378.46 52.07 180)
@@
 		)
 	)
+	(label "CHG_CC"
+		(at 382.27 114.3 180)
+		(effects
+			(font
+				(size 1.27 1.27)
+			)
+			(justify right bottom)
+		)
+	)
 	(label "HV_OUT_V"
 		(at 275.59 68.58 0)
@@
 		)
 	)
+	(hierarchical_label "{CC}"
+		(shape input)
+		(at 384.81 118.11 0)
+		(effects
+			(font
+				(size 1.27 1.27)
+			)
+			(justify left)
+		)
+	)
+	(hierarchical_label "{LV_ADC}"
+		(shape input)
+		(at 273.05 83.82 180)
+		(effects
+			(font
+				(size 1.27 1.27)
+			)
+			(justify right)
+		)
+	)

Commit message: addressed
Parts:
- removed R101, R102, R103, R106, R107: 10k, symbol Device:R
- removed R104, R105: 22, symbol Device:R
- removed TP4: BOOT, symbol Connector:TestPoint
Connections:
- no-connect marks 45 -> 41
Other:
- sheet STM32G491VET ports: added +3V3, BOOT0, NRST, PC13, PC14, PC15, PE10; removed 3V3, BOOT, PA0, PA1, PA2, PG10-NRST

Commit message: try smth on laptop
Parts:
- added TP22: RESET, symbol Connector:TestPoint
- added TP4: BOOT, symbol Connector:TestPoint
Connections:
- net STM32G491VET/BOOT0: now also TP4.1
- net STM32G491VET/NRST: now also TP22.1
- no-connect marks 41 -> 40

Commit message: update kicad sharepoint
Parts:
- added D43: DCDC_EN, LED_SMD:LED_0603_1608Metric_Pad1.05x0.95mm_HandSolder, symbol Device:LED
- added D44, D46: CHARGE_EN, LED_SMD:LED_0603_1608Metric_Pad1.05x0.95mm_HandSolder, symbol Device:LED
- added D45: LV_EN, LED_SMD:LED_0603_1608Metric_Pad1.05x0.95mm_HandSolder, symbol Device:LED
- added R89, R90, R91, R92: 1.3k, Resistor_SMD:R_0603_1608Metric_Pad0.98x0.95mm_HandSolder, symbol Device:R
Connections:
- net CHARGE_EN: now also R90.1
- net LV_EN_3V3: now also R91.1
- net LV_GND: now also D43.1 (K), D44.1 (K), D45.1 (K), D46.1 (K)
- net OUTPUT_EN: now also R92.1
- new net: D43.2 (A), R89.2
- new net: D46.2 (A), R92.2
- new net: D45.2 (A), R91.2
- new net: D44.2 (A), R90.2
- new net HV_DCDC_EN: R89.1
- no-connect marks 40 -> 43
Other:
- moved on the sheet: D6, R18

Commit message: sorry im omw
Parts:
- TP22, TP4: footprint (none) -> TestPoint:TestPoint_THTPad_D3.0mm_Drill1.5mm
Changed lines of the file:
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@@
 			)
 		)
-		(property "Footprint" ""
+		(property "Footprint" "TestPoint:TestPoint_THTPad_D3.0mm_Drill1.5mm"
 			(at 383.54 46.99 0)
 			(hide yes)
@@
 			)
 		)
-		(property "Footprint" ""
+		(property "Footprint" "TestPoint:TestPoint_THTPad_D3.0mm_Drill1.5mm"
 			(at 375.92 44.45 0)
 			(hide yes)

Commit message: craigenyah
Parts:
- renumbered D46 to D37, D44 to D38, D43 to D39, D5 to D40, D6 to D41, D45 to D42, R92 to R122, R90 to R123, R89 to R124, R17 to R125, R18 to R126, R91 to R127, TP4 to TP49, TP22 to TP50
Changed lines of the file:
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@@
 		(dnp no)
 		(fields_autoplaced yes)
-		(property "Reference" "D43"
+		(property "Reference" "D39"
 			(at 314.96 192.0874 90)
 			(show_name no)
@@
 			(project "PS-LVCarrier"
 				(path "/9bab2d9d-20f3-40ef-8545-e1299efec47e/91fef7fd-6fee-4cc6-8387-2fcfef7b7bdf"
-					(reference "D43")
+					(reference "D39")
 					(unit 1)
 				)
@@
 		(dnp no)
 		(fields_autoplaced yes)
-		(property "Reference" "R17"
+		(property "Reference" "R125"
 			(at 330.2 182.8799 0)
 			(show_name no)
@@
 			(project "PS-LVCarrier"
 				(path "/9bab2d9d-20f3-40ef-8545-e1299efec47e/91fef7fd-6fee-4cc6-8387-2fcfef7b7bdf"
-					(reference "R17")
+					(reference "R125")
 					(unit 1)
 				)
@@
 		(dnp no)
 		(fields_autoplaced yes)
-		(property "Reference" "D6"
+		(property "Reference" "D41"
 			(at 345.44 192.0874 90)
 			(show_name no)
@@
 			(project "PS-LVCarrier"
 				(path "/9bab2d9d-20f3-40ef-8545-e1299efec47e/91fef7fd-6fee-4cc6-8387-2fcfef7b7bdf"
-					(reference "D6")
+					(reference "D41")
 					(unit 1)
 				)
@@
 		(dnp no)
 		(fields_autoplaced yes)
-		(property "Reference" "R89"
+		(property "Reference" "R124"
 			(at 313.69 182.8799 0)
 			(show_name no)
@@
 			(project "PS-LVCarrier"
 				(path "/9bab2d9d-20f3-40ef-8545-e1299efec47e/91fef7fd-6fee-4cc6-8387-2fcfef7b7bdf"
-					(reference "R89")
+					(reference "R124")
 					(unit 1)
 				)
@@
 		(in_pos_files yes)
 		(dnp no)
-		(property "Reference" "TP22"
+		(property "Reference" "TP50"
 			(at 379.984 42.418 0)
 			(show_name no)
@@
 			(project "PS-LVCarrier"
 				(path "/9bab2d9d-20f3-40ef-8545-e1299efec47e/91fef7fd-6fee-4cc6-8387-2fcfef7b7bdf"
-					(reference "TP22")
+					(reference "TP50")
 					(unit 1)
 				)
@@
 		(dnp no)
 		(fields_autoplaced yes)
-		(property "Reference" "R92"
+		(property "Reference" "R122"
 			(at 280.67 182.8799 0)
 			(show_name no)
@@
 			(project "PS-LVCarrier"
 				(path "/9bab2d9d-20f3-40ef-8545-e1299efec47e/91fef7fd-6fee-4cc6-8387-2fcfef7b7bdf"
-					(reference "R92")
+					(reference "R122")
 					(unit 1)
 				)
@@
 		(dnp no)
 		(fields_autoplaced yes)
-		(property "Reference" "R91"
+		(property "Reference" "R127"
 			(at 360.68 182.8799 0)
 			(show_name no)
@@
 			(project "PS-LVCarrier"
 				(path "/9bab2d9d-20f3-40ef-8545-e1299efec47e/91fef7fd-6fee-4cc6-8387-2fcfef7b7bdf"
-					(reference "R91")
+					(reference "R127")
 					(unit 1)
 				)
@@
 		(dnp no)
 		(fields_autoplaced yes)
-		(property "Reference" "D46"
+		(property "Reference" "D37"
 			(at 281.94 192.0874 90)
 			(show_name no)
@@
 			(project "PS-LVCarrier"
 				(path "/9bab2d9d-20f3-40ef-8545-e1299efec47e/91fef7fd-6fee-4cc6-8387-2fcfef7b7bdf"
-					(reference "D46")
+					(reference "D37")
 					(unit 1)
 				)
@@
 		(dnp no)
 		(fields_autoplaced yes)
-		(property "Reference" "R18"
+		(property "Reference" "R126"
 			(at 344.17 182.8799 0)
 			(show_name no)
@@
 			(project "PS-LVCarrier"
 				(path "/9bab2d9d-20f3-40ef-8545-e1299efec47e/91fef7fd-6fee-4cc6-8387-2fcfef7b7bdf"
-					(reference "R18")
+					(reference "R126")
 					(unit 1)
 				)
@@
 		(dnp no)
 		(fields_autoplaced yes)
-		(property "Reference" "D45"
+		(property "Reference" "D42"
 			(at 361.95 192.0874 90)
 			(show_name no)
@@
 			(project "PS-LVCarrier"
 				(path "/9bab2d9d-20f3-40ef-8545-e1299efec47e/91fef7fd-6fee-4cc6-8387-2fcfef7b7bdf"
-					(reference "D45")
+					(reference "D42")
 					(unit 1)
 				)
@@
 		(in_pos_files yes)
 		(dnp no)
-		(property "Reference" "TP4"
+		(property "Reference" "TP49"
 			(at 372.364 39.878 0)
 			(show_name no)
@@
 			(project "PS-LVCarrier"
 				(path "/9bab2d9d-20f3-40ef-8545-e1299efec47e/91fef7fd-6fee-4cc6-8387-2fcfef7b7bdf"
-					(reference "TP4")
+					(reference "TP49")
 					(unit 1)
 				)
@@
 		(dnp no)
 		(fields_autoplaced yes)
-		(property "Reference" "R90"
+		(property "Reference" "R123"
 			(at 297.18 182.8799 0)
 			(show_name no)
@@
 			(project "PS-LVCarrier"
 				(path "/9bab2d9d-20f3-40ef-8545-e1299efec47e/91fef7fd-6fee-4cc6-8387-2fcfef7b7bdf"
-					(reference "R90")
+					(reference "R123")
 					(unit 1)
 				)
@@
 		(dnp no)
 		(fields_autoplaced yes)
-		(property "Reference" "D44"
+		(property "Reference" "D38"
 			(at 298.45 192.0874 90)
 			(show_name no)
@@
 			(project "PS-LVCarrier"
 				(path "/9bab2d9d-20f3-40ef-8545-e1299efec47e/91fef7fd-6fee-4cc6-8387-2fcfef7b7bdf"
-					(reference "D44")
+					(reference "D38")
 					(unit 1)
 				)
@@
 		(dnp no)
 		(fields_autoplaced yes)
-		(property "Reference" "D5"
+		(property "Reference" "D40"
 			(at 331.47 192.0874 90)
 			(show_name no)
@@
 			(project "PS-LVCarrier"
 				(path "/9bab2d9d-20f3-40ef-8545-e1299efec47e/91fef7fd-6fee-4cc6-8387-2fcfef7b7bdf"
-					(reference "D5")
+					(reference "D40")
 					(unit 1)
 				)
