File: hardware/STM32G491VET.kicad_sch (KiCad schematic)
At the start: 28 parts, among them J12 SWD_Header_02x02, U15 STM32G491VET6_1, Y1 Crystal

Commit message: switch branch
Parts:
- renumbered C59 to C67, C60 to C68, C61 to C69, C62 to C70, C63 to C71, C64 to C72, C65 to C73, C66 to C74, C67 to C75, C68 to C76, C69 to C77, C70 to C78, C71 to C79, C72 to C80, R97 to R102, R98 to R103, R99 to R104, R100 to R105, R101 to R106
Changed lines of the file:
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@@
 		(in_pos_files yes)
 		(dnp no)
-		(property "Reference" "C61"
+		(property "Reference" "C69"
 			(at 293.751 152.5016 0)
 			(show_name no)
@@
 			(project "PS-LVCarrier"
 				(path "/9bab2d9d-20f3-40ef-8545-e1299efec47e/91fef7fd-6fee-4cc6-8387-2fcfef7b7bdf/296654fd-4fbd-49cb-a2a3-d3a049f14f33"
-					(reference "C61")
+					(reference "C69")
 					(unit 1)
 				)
@@
 		(dnp no)
 		(fields_autoplaced yes)
-		(property "Reference" "C60"
+		(property "Reference" "C68"
 			(at 157.48 83.1849 0)
 			(show_name no)
@@
 			(project "PS-LVCarrier"
 				(path "/9bab2d9d-20f3-40ef-8545-e1299efec47e/91fef7fd-6fee-4cc6-8387-2fcfef7b7bdf/296654fd-4fbd-49cb-a2a3-d3a049f14f33"
-					(reference "C60")
+					(reference "C68")
 					(unit 1)
 				)
@@
 		(dnp no)
 		(fields_autoplaced yes)
-		(property "Reference" "R99"
+		(property "Reference" "R104"
 			(at 292.735 142.2399 0)
 			(show_name no)
@@
 			(project "PS-LVCarrier"
 				(path "/9bab2d9d-20f3-40ef-8545-e1299efec47e/91fef7fd-6fee-4cc6-8387-2fcfef7b7bdf/296654fd-4fbd-49cb-a2a3-d3a049f14f33"
-					(reference "R99")
+					(reference "R104")
 					(unit 1)
 				)
@@
 		(dnp no)
 		(fields_autoplaced yes)
-		(property "Reference" "C72"
+		(property "Reference" "C80"
 			(at 380.365 99.0599 0)
 			(show_name no)
@@
 			(project "PS-LVCarrier"
 				(path "/9bab2d9d-20f3-40ef-8545-e1299efec47e/91fef7fd-6fee-4cc6-8387-2fcfef7b7bdf/296654fd-4fbd-49cb-a2a3-d3a049f14f33"
-					(reference "C72")
+					(reference "C80")
 					(unit 1)
 				)
@@
 		(in_pos_files yes)
 		(dnp no)
-		(property "Reference" "R100"
+		(property "Reference" "R105"
 			(at 336.931 131.826 90)
 			(show_name no)
@@
 			(project "PS-LVCarrier"
 				(path "/9bab2d9d-20f3-40ef-8545-e1299efec47e/91fef7fd-6fee-4cc6-8387-2fcfef7b7bdf/296654fd-4fbd-49cb-a2a3-d3a049f14f33"
-					(reference "R100")
+					(reference "R105")
 					(unit 1)
 				)
@@
 		(dnp no)
 		(fields_autoplaced yes)
-		(property "Reference" "C68"
+		(property "Reference" "C76"
 			(at 330.835 72.3899 0)
 			(show_name no)
@@
 			(project "PS-LVCarrier"
 				(path "/9bab2d9d-20f3-40ef-8545-e1299efec47e/91fef7fd-6fee-4cc6-8387-2fcfef7b7bdf/296654fd-4fbd-49cb-a2a3-d3a049f14f33"
-					(reference "C68")
+					(reference "C76")
 					(unit 1)
 				)
@@
 		(dnp no)
 		(fields_autoplaced yes)
-		(property "Reference" "C59"
+		(property "Reference" "C67"
 			(at 144.78 83.1849 0)
 			(show_name no)
@@
 			(project "PS-LVCarrier"
 				(path "/9bab2d9d-20f3-40ef-8545-e1299efec47e/91fef7fd-6fee-4cc6-8387-2fcfef7b7bdf/296654fd-4fbd-49cb-a2a3-d3a049f14f33"
-					(reference "C59")
+					(reference "C67")
 					(unit 1)
 				)
@@
 		(dnp no)
 		(fields_autoplaced yes)
-		(property "Reference" "C64"
+		(property "Reference" "C72"
 			(at 305.435 72.3899 0)
 			(show_name no)
@@
 			(project "PS-LVCarrier"
 				(path "/9bab2d9d-20f3-40ef-8545-e1299efec47e/91fef7fd-6fee-4cc6-8387-2fcfef7b7bdf/296654fd-4fbd-49cb-a2a3-d3a049f14f33"
-					(reference "C64")
+					(reference "C72")
 					(unit 1)
 				)
@@
 		(in_pos_files yes)
 		(dnp no)
-		(property "Reference" "R98"
+		(property "Reference" "R103"
 			(at 249.555 69.85 90)
 			(show_name no)
@@
 			(project "PS-LVCarrier"
 				(path "/9bab2d9d-20f3-40ef-8545-e1299efec47e/91fef7fd-6fee-4cc6-8387-2fcfef7b7bdf/296654fd-4fbd-49cb-a2a3-d3a049f14f33"
-					(reference "R98")
+					(reference "R103")
 					(unit 1)
 				)
@@
 		(dnp no)
 		(fields_autoplaced yes)
-		(property "Reference" "C66"
+		(property "Reference" "C74"
 			(at 318.135 72.3899 0)
 			(show_name no)
@@
 			(project "PS-LVCarrier"
 				(path "/9bab2d9d-20f3-40ef-8545-e1299efec47e/91fef7fd-6fee-4cc6-8387-2fcfef7b7bdf/296654fd-4fbd-49cb-a2a3-d3a049f14f33"
-					(reference "C66")
+					(reference "C74")
 					(unit 1)
 				)
@@
 		(dnp no)
 		(fields_autoplaced yes)
-		(property "Reference" "C67"
+		(property "Reference" "C75"
 			(at 325.755 97.7899 0)
 			(show_name no)
@@
 			(project "PS-LVCarrier"
 				(path "/9bab2d9d-20f3-40ef-8545-e1299efec47e/91fef7fd-6fee-4cc6-8387-2fcfef7b7bdf/296654fd-4fbd-49cb-a2a3-d3a049f14f33"
-					(reference "C67")
+					(reference "C75")
 					(unit 1)
 				)
@@
 		(dnp no)
 		(fields_autoplaced yes)
-		(property "Reference" "C62"
+		(property "Reference" "C70"
 			(at 294.64 72.3899 0)
 			(show_name no)
@@
 			(project "PS-LVCarrier"
 				(path "/9bab2d9d-20f3-40ef-8545-e1299efec47e/91fef7fd-6fee-4cc6-8387-2fcfef7b7bdf/296654fd-4fbd-49cb-a2a3-d3a049f14f33"
-					(reference "C62")
+					(reference "C70")
 					(unit 1)
 				)
@@
 		(dnp no)
 		(fields_autoplaced yes)
-		(property "Reference" "C65"
+		(property "Reference" "C73"
 			(at 310.515 97.7899 0)
 			(show_name no)
@@
 			(project "PS-LVCarrier"
 				(path "/9bab2d9d-20f3-40ef-8545-e1299efec47e/91fef7fd-6fee-4cc6-8387-2fcfef7b7bdf/296654fd-4fbd-49cb-a2a3-d3a049f14f33"
-					(reference "C65")
+					(reference "C73")
 					(unit 1)
 				)
@@
 		(dnp no)
 		(fields_autoplaced yes)
-		(property "Reference" "C63"
+		(property "Reference" "C71"
 			(at 295.275 97.7899 0)
 			(show_name no)
@@
 			(project "PS-LVCarrier"
 				(path "/9bab2d9d-20f3-40ef-8545-e1299efec47e/91fef7fd-6fee-4cc6-8387-2fcfef7b7bdf/296654fd-4fbd-49cb-a2a3-d3a049f14f33"
-					(reference "C63")
+					(reference "C71")
 					(unit 1)
 				)
@@
 		(dnp no)
 		(fields_autoplaced yes)
-		(property "Reference" "R97"
+		(property "Reference" "R102"
 			(at 249.555 58.42 90)
 			(show_name no)
@@
 			(project "PS-LVCarrier"
 				(path "/9bab2d9d-20f3-40ef-8545-e1299efec47e/91fef7fd-6fee-4cc6-8387-2fcfef7b7bdf/296654fd-4fbd-49cb-a2a3-d3a049f14f33"
-					(reference "R97")
+					(reference "R102")
 					(unit 1)
 				)
@@
 		(dnp no)
 		(fields_autoplaced yes)
-		(property "Reference" "C69"
+		(property "Reference" "C77"
 			(at 340.995 97.7899 0)
 			(show_name no)
@@
 			(project "PS-LVCarrier"
 				(path "/9bab2d9d-20f3-40ef-8545-e1299efec47e/91fef7fd-6fee-4cc6-8387-2fcfef7b7bdf/296654fd-4fbd-49cb-a2a3-d3a049f14f33"
-					(reference "C69")
+					(reference "C77")
 					(unit 1)
 				)
@@
 		(dnp no)
 		(fields_autoplaced yes)
-		(property "Reference" "C70"
+		(property "Reference" "C78"
 			(at 343.535 72.3899 0)
 			(show_name no)
@@
 			(project "PS-LVCarrier"
 				(path "/9bab2d9d-20f3-40ef-8545-e1299efec47e/91fef7fd-6fee-4cc6-8387-2fcfef7b7bdf/296654fd-4fbd-49cb-a2a3-d3a049f14f33"
-					(reference "C70")
+					(reference "C78")
 					(unit 1)
 				)
@@
 		(in_pos_files yes)
 		(dnp no)
-		(property "Reference" "C71"
+		(property "Reference" "C79"
 			(at 356.362 72.263 0)
 			(show_name no)
@@
 			(project "PS-LVCarrier"
 				(path "/9bab2d9d-20f3-40ef-8545-e1299efec47e/91fef7fd-6fee-4cc6-8387-2fcfef7b7bdf/296654fd-4fbd-49cb-a2a3-d3a049f14f33"
-					(reference "C71")
+					(reference "C79")
 					(unit 1)
 				)
@@
 		(dnp no)
 		(fields_autoplaced yes)
-		(property "Reference" "R101"
+		(property "Reference" "R106"
 			(at 346.075 151.7649 0)
 			(show_name no)
@@
 			(project "PS-LVCarrier"
 				(path "/9bab2d9d-20f3-40ef-8545-e1299efec47e/91fef7fd-6fee-4cc6-8387-2fcfef7b7bdf/296654fd-4fbd-49cb-a2a3-d3a049f14f33"
-					(reference "R101")
+					(reference "R106")
 					(unit 1)
 				)

Commit message: review ts
Parts:
- renumbered C67 to C53, C68 to C54, C69 to C55, C70 to C56, C71 to C57, C72 to C58, C73 to C59, C74 to C60, C75 to C61, C76 to C62, C77 to C63, C78 to C64, C79 to C65, C80 to C66, D30 to D19, D31 to D20, J12 to J11, R102 to R53, R103 to R54, R104 to R55, R105 to R56, R106 to R57, U15 to U12
Changed lines of the file:
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@@
 		(in_pos_files yes)
 		(dnp no)
-		(property "Reference" "C69"
+		(property "Reference" "C55"
 			(at 293.751 152.5016 0)
 			(show_name no)
@@
 			(project "PS-LVCarrier"
 				(path "/9bab2d9d-20f3-40ef-8545-e1299efec47e/91fef7fd-6fee-4cc6-8387-2fcfef7b7bdf/296654fd-4fbd-49cb-a2a3-d3a049f14f33"
-					(reference "C69")
+					(reference "C55")
 					(unit 1)
 				)
@@
 		(dnp no)
 		(fields_autoplaced yes)
-		(property "Reference" "C68"
+		(property "Reference" "C54"
 			(at 157.48 83.1849 0)
 			(show_name no)
@@
 			(project "PS-LVCarrier"
 				(path "/9bab2d9d-20f3-40ef-8545-e1299efec47e/91fef7fd-6fee-4cc6-8387-2fcfef7b7bdf/296654fd-4fbd-49cb-a2a3-d3a049f14f33"
-					(reference "C68")
+					(reference "C54")
 					(unit 1)
 				)
@@
 		(dnp no)
 		(fields_autoplaced yes)
-		(property "Reference" "R104"
+		(property "Reference" "R55"
 			(at 292.735 142.2399 0)
 			(show_name no)
@@
 			(project "PS-LVCarrier"
 				(path "/9bab2d9d-20f3-40ef-8545-e1299efec47e/91fef7fd-6fee-4cc6-8387-2fcfef7b7bdf/296654fd-4fbd-49cb-a2a3-d3a049f14f33"
-					(reference "R104")
+					(reference "R55")
 					(unit 1)
 				)
@@
 		(dnp no)
 		(fields_autoplaced yes)
-		(property "Reference" "U15"
+		(property "Reference" "U12"
 			(at 204.47 65.405 0)
 			(hide yes)
@@
 			(project "PS-LVCarrier"
 				(path "/9bab2d9d-20f3-40ef-8545-e1299efec47e/91fef7fd-6fee-4cc6-8387-2fcfef7b7bdf/296654fd-4fbd-49cb-a2a3-d3a049f14f33"
-					(reference "U15")
+					(reference "U12")
 					(unit 1)
 				)
@@
 		(dnp no)
 		(fields_autoplaced yes)
-		(property "Reference" "C80"
+		(property "Reference" "C66"
 			(at 380.365 99.0599 0)
 			(show_name no)
@@
 			(project "PS-LVCarrier"
 				(path "/9bab2d9d-20f3-40ef-8545-e1299efec47e/91fef7fd-6fee-4cc6-8387-2fcfef7b7bdf/296654fd-4fbd-49cb-a2a3-d3a049f14f33"
-					(reference "C80")
+					(reference "C66")
 					(unit 1)
 				)
@@
 		(in_pos_files yes)
 		(dnp no)
-		(property "Reference" "R105"
+		(property "Reference" "R56"
 			(at 336.931 131.826 90)
 			(show_name no)
@@
 			(project "PS-LVCarrier"
 				(path "/9bab2d9d-20f3-40ef-8545-e1299efec47e/91fef7fd-6fee-4cc6-8387-2fcfef7b7bdf/296654fd-4fbd-49cb-a2a3-d3a049f14f33"
-					(reference "R105")
+					(reference "R56")
 					(unit 1)
 				)
@@
 		(dnp no)
 		(fields_autoplaced yes)
-		(property "Reference" "C76"
+		(property "Reference" "C62"
 			(at 330.835 72.3899 0)
 			(show_name no)
@@
 			(project "PS-LVCarrier"
 				(path "/9bab2d9d-20f3-40ef-8545-e1299efec47e/91fef7fd-6fee-4cc6-8387-2fcfef7b7bdf/296654fd-4fbd-49cb-a2a3-d3a049f14f33"
-					(reference "C76")
+					(reference "C62")
 					(unit 1)
 				)
@@
 		(dnp no)
 		(fields_autoplaced yes)
-		(property "Reference" "C67"
+		(property "Reference" "C53"
 			(at 144.78 83.1849 0)
 			(show_name no)
@@
 			(project "PS-LVCarrier"
 				(path "/9bab2d9d-20f3-40ef-8545-e1299efec47e/91fef7fd-6fee-4cc6-8387-2fcfef7b7bdf/296654fd-4fbd-49cb-a2a3-d3a049f14f33"
-					(reference "C67")
+					(reference "C53")
 					(unit 1)
 				)
@@
 		(dnp no)
 		(fields_autoplaced yes)
-		(property "Reference" "C72"
+		(property "Reference" "C58"
 			(at 305.435 72.3899 0)
 			(show_name no)
@@
 			(project "PS-LVCarrier"
 				(path "/9bab2d9d-20f3-40ef-8545-e1299efec47e/91fef7fd-6fee-4cc6-8387-2fcfef7b7bdf/296654fd-4fbd-49cb-a2a3-d3a049f14f33"
-					(reference "C72")
+					(reference "C58")
 					(unit 1)
 				)
@@
 		(in_pos_files yes)
 		(dnp no)
-		(property "Reference" "R103"
+		(property "Reference" "R54"
 			(at 249.555 69.85 90)
 			(show_name no)
@@
 			(project "PS-LVCarrier"
 				(path "/9bab2d9d-20f3-40ef-8545-e1299efec47e/91fef7fd-6fee-4cc6-8387-2fcfef7b7bdf/296654fd-4fbd-49cb-a2a3-d3a049f14f33"
-					(reference "R103")
+					(reference "R54")
 					(unit 1)
 				)
@@
 		(dnp no)
 		(fields_autoplaced yes)
-		(property "Reference" "C74"
+		(property "Reference" "C60"
 			(at 318.135 72.3899 0)
 			(show_name no)
@@
 			(project "PS-LVCarrier"
 				(path "/9bab2d9d-20f3-40ef-8545-e1299efec47e/91fef7fd-6fee-4cc6-8387-2fcfef7b7bdf/296654fd-4fbd-49cb-a2a3-d3a049f14f33"
-					(reference "C74")
+					(reference "C60")
 					(unit 1)
 				)
@@
 		(dnp no)
 		(fields_autoplaced yes)
-		(property "Reference" "C75"
+		(property "Reference" "C61"
 			(at 325.755 97.7899 0)
 			(show_name no)
@@
 			(project "PS-LVCarrier"
 				(path "/9bab2d9d-20f3-40ef-8545-e1299efec47e/91fef7fd-6fee-4cc6-8387-2fcfef7b7bdf/296654fd-4fbd-49cb-a2a3-d3a049f14f33"
-					(reference "C75")
+					(reference "C61")
 					(unit 1)
 				)
@@
 		(dnp no)
 		(fields_autoplaced yes)
-		(property "Reference" "D31"
+		(property "Reference" "D20"
 			(at 358.14 146.0499 90)
 			(show_name no)
@@
 			(project "PS-LVCarrier"
 				(path "/9bab2d9d-20f3-40ef-8545-e1299efec47e/91fef7fd-6fee-4cc6-8387-2fcfef7b7bdf/296654fd-4fbd-49cb-a2a3-d3a049f14f33"
-					(reference "D31")
+					(reference "D20")
 					(unit 1)
 				)
@@
 		(dnp no)
 		(fields_autoplaced yes)
-		(property "Reference" "C70"
+		(property "Reference" "C56"
 			(at 294.64 72.3899 0)
 			(show_name no)
@@
 			(project "PS-LVCarrier"
 				(path "/9bab2d9d-20f3-40ef-8545-e1299efec47e/91fef7fd-6fee-4cc6-8387-2fcfef7b7bdf/296654fd-4fbd-49cb-a2a3-d3a049f14f33"
-					(reference "C70")
+					(reference "C56")
 					(unit 1)
 				)
@@
 		(in_pos_files yes)
 		(dnp no)
-		(property "Reference" "J12"
+		(property "Reference" "J11"
 			(at 267.843 52.832 0)
 			(show_name no)
@@
 			(project "PS-LVCarrier"
 				(path "/9bab2d9d-20f3-40ef-8545-e1299efec47e/91fef7fd-6fee-4cc6-8387-2fcfef7b7bdf/296654fd-4fbd-49cb-a2a3-d3a049f14f33"
-					(reference "J12")
+					(reference "J11")
 					(unit 1)
 				)
@@
 		(dnp no)
 		(fields_autoplaced yes)
-		(property "Reference" "C73"
+		(property "Reference" "C59"
 			(at 310.515 97.7899 0)
 			(show_name no)
@@
 			(project "PS-LVCarrier"
 				(path "/9bab2d9d-20f3-40ef-8545-e1299efec47e/91fef7fd-6fee-4cc6-8387-2fcfef7b7bdf/296654fd-4fbd-49cb-a2a3-d3a049f14f33"
-					(reference "C73")
+					(reference "C59")
 					(unit 1)
 				)
@@
 		(dnp no)
 		(fields_autoplaced yes)
-		(property "Reference" "C71"
+		(property "Reference" "C57"
 			(at 295.275 97.7899 0)
 			(show_name no)
@@
 			(project "PS-LVCarrier"
 				(path "/9bab2d9d-20f3-40ef-8545-e1299efec47e/91fef7fd-6fee-4cc6-8387-2fcfef7b7bdf/296654fd-4fbd-49cb-a2a3-d3a049f14f33"
-					(reference "C71")
+					(reference "C57")
 					(unit 1)
 				)
@@
 		(dnp no)
 		(fields_autoplaced yes)
-		(property "Reference" "D30"
+		(property "Reference" "D19"
 			(at 347.345 141.9224 90)
 			(show_name no)
@@
 			(project "PS-LVCarrier"
 				(path "/9bab2d9d-20f3-40ef-8545-e1299efec47e/91fef7fd-6fee-4cc6-8387-2fcfef7b7bdf/296654fd-4fbd-49cb-a2a3-d3a049f14f33"
-					(reference "D30")
+					(reference "D19")
 					(unit 1)
 				)
@@
 		(dnp no)
 		(fields_autoplaced yes)
-		(property "Reference" "R102"
+		(property "Reference" "R53"
 			(at 249.555 58.42 90)
 			(show_name no)
@@
 			(project "PS-LVCarrier"
 				(path "/9bab2d9d-20f3-40ef-8545-e1299efec47e/91fef7fd-6fee-4cc6-8387-2fcfef7b7bdf/296654fd-4fbd-49cb-a2a3-d3a049f14f33"
-					(reference "R102")
+					(reference "R53")
 					(unit 1)
 				)
@@
 		(dnp no)
 		(fields_autoplaced yes)
-		(property "Reference" "C77"
+		(property "Reference" "C63"
 			(at 340.995 97.7899 0)
 			(show_name no)
@@
 			(project "PS-LVCarrier"
 				(path "/9bab2d9d-20f3-40ef-8545-e1299efec47e/91fef7fd-6fee-4cc6-8387-2fcfef7b7bdf/296654fd-4fbd-49cb-a2a3-d3a049f14f33"
-					(reference "C77")
+					(reference "C63")
 					(unit 1)
 				)
@@
 		(dnp no)
 		(fields_autoplaced yes)
-		(property "Reference" "C78"
+		(property "Reference" "C64"
 			(at 343.535 72.3899 0)
 			(show_name no)
@@
 			(project "PS-LVCarrier"
 				(path "/9bab2d9d-20f3-40ef-8545-e1299efec47e/91fef7fd-6fee-4cc6-8387-2fcfef7b7bdf/296654fd-4fbd-49cb-a2a3-d3a049f14f33"
-					(reference "C78")
+					(reference "C64")
 					(unit 1)
 				)
@@
 		(in_pos_files yes)
 		(dnp no)
-		(property "Reference" "C79"
+		(property "Reference" "C65"
 			(at 356.362 72.263 0)
 			(show_name no)
@@
 			(project "PS-LVCarrier"
 				(path "/9bab2d9d-20f3-40ef-8545-e1299efec47e/91fef7fd-6fee-4cc6-8387-2fcfef7b7bdf/296654fd-4fbd-49cb-a2a3-d3a049f14f33"
-					(reference "C79")
+					(reference "C65")
 					(unit 1)
 				)
@@
 		(dnp no)
 		(fields_autoplaced yes)
-		(property "Reference" "R106"
+		(property "Reference" "R57"
 			(at 346.075 151.7649 0)
 			(show_name no)
@@
 			(project "PS-LVCarrier"
 				(path "/9bab2d9d-20f3-40ef-8545-e1299efec47e/91fef7fd-6fee-4cc6-8387-2fcfef7b7bdf/296654fd-4fbd-49cb-a2a3-d3a049f14f33"
-					(reference "R106")
+					(reference "R57")
 					(unit 1)
 				)

Commit message: addressed
Parts:
- removed C53, C54: 26p, Capacitor_SMD:C_0603_1608Metric_Pad1.08x0.95mm_HandSolder, symbol Device:C
- removed C55, C57, C58, C59, C60, C62, C64, C65, C66: 0.1u, Capacitor_SMD:C_0603_1608Metric_Pad1.08x0.95mm_HandSolder, symbol Device:C
- removed C56: 10u, Capacitor_SMD:C_0805_2012Metric_Pad1.18x1.45mm_HandSolder, symbol Device:C
- removed C61, C63: 1u, Capacitor_SMD:C_0603_1608Metric_Pad1.08x0.95mm_HandSolder, symbol Device:C
- removed D19: LED, LED_SMD:LED_0201_0603Metric, symbol Device:LED
- removed D20: D_TVS, Diode_SMD:D_SOD-323, symbol Device:D_TVS
- removed FB1, FB2: FerriteBead, Capacitor_SMD:C_0603_1608Metric_Pad1.08x0.95mm_HandSolder, symbol Device:FerriteBead
- removed J11: SWD_Header_02x02, LHRS_Connectors:SWD_Conn, symbol 100PinMCU:SWD_Header_02x02
- removed R53, R54: 22, Resistor_SMD:R_0603_1608Metric_Pad0.98x0.95mm_HandSolder, symbol Device:R
- removed R55, R56: 10k, Resistor_SMD:R_0603_1608Metric_Pad0.98x0.95mm_HandSolder, symbol Device:R
- removed R57: 1k, Resistor_SMD:R_0603_1608Metric_Pad0.98x0.95mm_HandSolder, symbol Device:R
- removed Reset1: Reset, LHRS_Special:TL3365AF180QG, symbol Switch:SW_Push
- removed S1: 450406020024, LHRS_Special:BootSW, symbol Switch:SW_SPDT
- removed U12: STM32G491VET6_1, LHRS_ICs:LQFP_491VET6_STM, symbol lhrs_ics:STM32G491VET6_1
- removed Y1: Crystal, LHRS_Passives:Crystal_SMD_Abracon_ABM3-2Pin_5.0x3.2mm, symbol Device:Crystal
- added C26, C32: 26p, Capacitor_SMD:C_0603_1608Metric_Pad1.08x0.95mm_HandSolder, symbol Device:C
- added C34: 10u, Capacitor_SMD:C_0805_2012Metric, symbol Device:C
- added C36, C37, C38, C39, C40, C42, C73, C74, C75: 0.1u, Capacitor_SMD:C_0603_1608Metric_Pad1.08x0.95mm_HandSolder, symbol Device:C
- added C41, C72: 1u, Capacitor_SMD:C_0603_1608Metric_Pad1.08x0.95mm_HandSolder, symbol Device:C
- added D14: TVS, Diode_SMD:D_SOD-323, symbol lhrs_misc:Boot_TVS
- added D15: RGB_LED, LHRS_Special:RGB_LED, symbol lhrs_special:RGB_LED
- added D16: LED, LED_SMD:LED_0603_1608Metric, symbol lhrs_misc:Blue_LED
- added FB3, FB4: FerriteBead, Capacitor_SMD:C_0603_1608Metric_Pad1.08x0.95mm_HandSolder, symbol Device:FerriteBead
- added J12: SWD_Header, LHRS_Connectors:SWD_Conn, symbol 100PinMCU:SWD_Header_02x02
- added J13: SWD, Connector_PinHeader_2.54mm:PinHeader_1x04_P2.54mm_Vertical, symbol Connector_Generic:Conn_01x04
- added R71, R77: 10k, Resistor_SMD:R_0603_1608Metric_Pad0.98x0.95mm_HandSolder, symbol Device:R
- added R72, R73: 22, Resistor_SMD:R_0603_1608Metric_Pad0.98x0.95mm_HandSolder, symbol Device:R
- added R74, R75, R76, R78: 1k, Resistor_SMD:R_0603_1608Metric_Pad0.98x0.95mm_HandSolder, symbol Device:R
- added Reset2: Reset, LHRS_Special:TL3365AF180QG, symbol Switch:SW_Push
- added SW1: SW_SPDT, LHRS_Special:BootSW, symbol Switch:SW_SPDT
- added U7: STM32G473VETx, LHRS_Special:100PinMCU, symbol lhrs_special:STM32G473VET6
- added Y2: Crystal, LHRS_Passives:Crystal_SMD_Abracon_ABM3-2Pin_5.0x3.2mm, symbol Device:Crystal
Connections:
- net GND: now also C26.1, C32.1, C34.2, C37.2, C39.2, C40.2, C42.2, C73.2, C74.2, D14.1 (A1), FB3.2, J12.2 (Pin_2), J13.2 (Pin_2), R74.2, R75.2, R76.2, R78.2, Reset2.2, SW1.3 (C), U7.23 (VSS), U7.48 (VSS), U7.63 (VSS), U7.74 (VSS), U7.99 (VSS)
- net GNDA: now also C36.2, C38.2, C41.2, C72.2, C75.2, FB3.1, U7.35 (VSSA)
- net PA0: now also D15.5, U7.20 (PA0-GPIO_BLUE)
- net PA1: now also D15.3, U7.21 (PA1-GPIO_RED)
- net PA10: now also U7.71 (PA10)
- net PA15: now also U7.78 (PA15)
- net PA2: now also D15.1, U7.22 (PA2-GPIO_GREEN)
- net PA3: now also U7.25 (PA3)
- net PA4: now also U7.26 (PA4)
- net PA5: now also U7.27 (PA5)
- net PA6: now also U7.28 (PA6)
- net PA7: now also U7.29 (PA7)
- net PA8: now also U7.69 (PA8)
- net PA9: now also U7.70 (PA9)
- net PB0: now also U7.32 (PB0)
- net PB1: now also U7.33 (PB1)
- net PB10: now also U7.47 (PB10)
- net PB11: now also U7.50 (PB11)
- net PB12: now also U7.51 (PB12)
- net PB13: now also U7.52 (PB13)
- net PB14: now also U7.53 (PB14)
- net PB15: now also U7.54 (PB15)
- net PB2: now also U7.34 (PB2)
- net PB3: now also U7.90 (PB3)
- net PB4: now also U7.91 (PB4)
- net PB5: now also U7.92 (PB5)
- net PB6: now also U7.93 (PB6)
- net PB7: now also U7.94 (PB7)
- net PB9: now also U7.96 (PB9)
- net PC0: now also U7.15 (PC0)
- net PC1: now also U7.16 (PC1)
- net PC10: now also U7.79 (PC10)
- net PC11: now also U7.80 (PC11)
- net PC12: now also U7.81 (PC12)
- net PC2: now also U7.17 (PC2)
- net PC3: now also U7.18 (PC3)
- net PC4: now also U7.30 (PC4)
- net PC5: now also U7.31 (PC5)
- net PC6: now also U7.65 (PC6)
- net PC7: now also U7.66 (PC7)
- net PC8: now also U7.67 (PC8)
- net PC9: now also U7.68 (PC9)
- net PD0: now also U7.82 (PD0)
- net PD1: now also U7.83 (PD1)
- net PD10: now also U7.57 (PD10)
- net PD11: now also U7.58 (PD11)
- net PD12: now also U7.59 (PD12)
- net PD13: now also U7.60 (PD13)
- net PD14: now also U7.61 (PD14)
- net PD15: now also U7.62 (PD15)
- net PD2: now also U7.84 (PD2)
- net PD3: now also U7.85 (PD3)
- net PD4: now also U7.86 (PD4)
- net PD5: now also U7.87 (PD5)
- net PD6: now also U7.88 (PD6)
- net PD7: now also U7.89 (PD7)
- net PD8: now also U7.55 (PD8)
- net PD9: now also U7.56 (PD9)
- net PE0: now also U7.97 (PE0)
- net PE1: now also U7.98 (PE1)
- net PE11: now also U7.42 (PE11)
- net PE12: now also U7.43 (PE12)
- net PE13: now also U7.44 (PE13)
- net PE14: now also U7.45 (PE14)
- net PE15: now also U7.46 (PE15)
- net PE2: now also U7.1 (PE2)
- net PE3: now also U7.2 (PE3)
- net PE4: now also U7.3 (PE4)
- net PE5: now also U7.4 (PE5)
- net PE6: now also U7.5 (PE6)
- net PE7: now also U7.38 (PE7)
- net PE8: now also U7.39 (PE8)
- net PE9: now also U7.40 (PE9)
- net PF10: now also U7.11 (PF10)
- net PF2: now also U7.19 (PF2)
- net PF9: now also U7.10 (PF9)
- net SWCLK: now also R72.1, U7.77 (PA14)
- net SWDIO: now also R73.1, U7.76 (PA13)
- net USB_DM: now also U7.72 (PA11)
- net USB_DP: now also U7.73 (PA12)
- net VDDA: now also C36.1, C38.1, C41.1, C72.1, C75.1, FB4.2, U7.36 (VREF+), U7.37 (VDDA)
- new net: D16.1 (K), R78.1
- new net: D14.2 (A2), D16.2 (A), R77.2, SW1.2 (B)
- new net: C26.2, U7.12 (PF0-OSC_IN), Y2.2
- new net: C32.2, U7.13 (PF1-OSC_OUT), Y2.1
- new net: J12.4 (Pin_4), J13.4 (Pin_4), R73.2
- new net: J12.3 (Pin_3), J13.3 (Pin_3), R72.2
- new net: D15.2, R74.1
- new net: D15.4, R75.1
- new net: D15.6, R76.1
- new net +3V3: C34.1, C37.1, C40.1, C42.1, C73.1, C74.1, FB4.1, J12.1 (Pin_1), J13.1 (Pin_1), R71.2, SW1.1 (A), U7.100 (VDD), U7.24 (VDD), U7.49 (VDD), U7.6 (VBAT), U7.64 (VDD), U7.75 (VDD)
- new net BOOT0: R77.1, U7.95 (PB8-BOOT0)
- new net NRST: C39.1, R71.1, Reset2.1, U7.14 (PG10-NRST)
- new net PC13: U7.7 (PC13)
- new net PC14: U7.8 (PC14-OSC32_IN)
- new net PC15: U7.9 (PC15-OSC32_OUT)
- new net PE10: U7.41 (PE10)
- no-connect marks 3 -> 0
Other:
- note added: "*Place oscillator circuitry close to MCU"
- note added: "100 Pin MCU"
- note added: "BLUE"
- note added: "BOOT0 low -> Load into app BOOT0 high -> Load into bootloader"
- note added: "Beware, using PC13 - 15 as GPIOs ..."
- note added: "CLK"
- note added: "Conn"
- note added: "GREEN"
- note added: "IO"
- note added: "Main Flash (user code)"
- note added: "Pin Headers"
- note added: "Place these decoupling caps as close as possible to their respective leads."
- note added: "Power Source Filtering/Isolation"
- note added: "RED"
- note added: "RGB LED"
- note added: "Reset BTN + Boot SW"
- note added: "Serial Wire Communication"
- note added: "Sys Memory (bootloader)"
- note added: "Use PA0, PA1, PA2 to PWM RGB LED (TIM2_CH1, TIM2_CH2, TIM2_CH3)"
- note removed: "BOOT = 0 (Logic LOW) Mode: Main Flash Memory. BOOT = 1 (Logic HIGH) Mode: System Memory."
- note removed: "Boot Switch"
- note removed: "Buttons & Stuff (External Reset)"
- note removed: "Bypass/Separation"
- note removed: "C1 = C2 = 2x(CL-CStray) C1 = C2 = 2x(18p-5p) C1 = C2 = 26p"
- note removed: "Place immediately adjacent to OSC_IN/OUT."
- note removed: "Reset"
- note removed: "System"
- note removed: "User"

Commit message: update kicad sharepoint
Parts:
- C34: footprint Capacitor_SMD:C_0805_2012Metric -> Capacitor_SMD:C_0805_2012Metric_Pad1.18x1.45mm_HandSolder
- D15: MANUFACTURER Everlight -> (none); Manufacturer (none) -> Everlight

Commit message: sorry im omw
Parts:
- D16: footprint LED_SMD:LED_0603_1608Metric -> LED_SMD:LED_0603_1608Metric_Pad1.05x0.95mm_HandSolder
Changed lines of the file:
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@@
 			)
 		)
-		(property "Footprint" "LED_SMD:LED_0603_1608Metric"
+		(property "Footprint" "LED_SMD:LED_0603_1608Metric_Pad1.05x0.95mm_HandSolder"
 			(at 332.994 144.78 0)
 			(hide yes)

Commit message: craigenyah
Parts:
- renumbered C26 to C100, C32 to C101, C34 to C102, C36 to C103, C37 to C104, C38 to C105, C39 to C106, C40 to C107, C41 to C108, C42 to C109, C72 to C110, C73 to C111, C74 to C112, C75 to C113, D14 to D43, D15 to D44, D16 to D45, FB3 to FB1, FB4 to FB2, R71 to R128, R72 to R129, R73 to R130, R74 to R131, R75 to R132, R76 to R133, R77 to R134, R78 to R135, Reset2 to Reset1, U7 to U13, Y2 to Y1
