File: hardware/PS-LVCarrier.kicad_pcb (KiCad board)
At the start: 2 copper layers, 0 parts

Commit message: craigenyah
Parts:
- added C1: 47u, Capacitor_SMD:C_0603_1608Metric_Pad1.08x0.95mm_HandSolder, F.Cu at (62.8, 246.7)
- added C10: 22u, Capacitor_SMD:C_0603_1608Metric_Pad1.08x0.95mm_HandSolder, F.Cu at (72.8, 51.3)
- added C100: 26p, Capacitor_SMD:C_0603_1608Metric_Pad1.08x0.95mm_HandSolder, F.Cu at (34.2, 22.2)
- added C101: 26p, Capacitor_SMD:C_0603_1608Metric_Pad1.08x0.95mm_HandSolder, F.Cu at (34.2, 24.7)
- added C102: 10u, Capacitor_SMD:C_0805_2012Metric_Pad1.18x1.45mm_HandSolder, F.Cu at (59.7, 52.4)
- added C103: 0.1u, Capacitor_SMD:C_0603_1608Metric_Pad1.08x0.95mm_HandSolder, F.Cu at (34.2, 27.2)
- added C104: 0.1u, Capacitor_SMD:C_0603_1608Metric_Pad1.08x0.95mm_HandSolder, F.Cu at (34.2, 29.7)
- added C105: 0.1u, Capacitor_SMD:C_0603_1608Metric_Pad1.08x0.95mm_HandSolder, F.Cu at (34.2, 32.2)
- added C106: 0.1u, Capacitor_SMD:C_0603_1608Metric_Pad1.08x0.95mm_HandSolder, F.Cu at (34.2, 34.7)
- added C107: 0.1u, Capacitor_SMD:C_0603_1608Metric_Pad1.08x0.95mm_HandSolder, F.Cu at (34.2, 37.2)
- added C108: 1u, Capacitor_SMD:C_0603_1608Metric_Pad1.08x0.95mm_HandSolder, F.Cu at (34.2, 39.8)
- added C109: 0.1u, Capacitor_SMD:C_0603_1608Metric_Pad1.08x0.95mm_HandSolder, F.Cu at (38.5, 22.2)
- added C11: 22u, Capacitor_SMD:C_0603_1608Metric_Pad1.08x0.95mm_HandSolder, F.Cu at (72.8, 53.8)
- added C110: 1u, Capacitor_SMD:C_0603_1608Metric_Pad1.08x0.95mm_HandSolder, F.Cu at (38.5, 24.7)
- added C111: 0.1u, Capacitor_SMD:C_0603_1608Metric_Pad1.08x0.95mm_HandSolder, F.Cu at (38.5, 27.2)
- added C112: 0.1u, Capacitor_SMD:C_0603_1608Metric_Pad1.08x0.95mm_HandSolder, F.Cu at (38.5, 29.7)
- added C113: 0.1u, Capacitor_SMD:C_0603_1608Metric_Pad1.08x0.95mm_HandSolder, F.Cu at (38.5, 32.2)
- added C12: 22u, Capacitor_SMD:C_0603_1608Metric_Pad1.08x0.95mm_HandSolder, F.Cu at (72.8, 56.4)
- added C13: 22u, Capacitor_SMD:C_0603_1608Metric_Pad1.08x0.95mm_HandSolder, F.Cu at (72.8, 58.9)
- added C14: 0.1u, Capacitor_SMD:C_0402_1005Metric_Pad0.74x0.62mm_HandSolder, F.Cu at (89.4, 73.3)
- added C15: 10n, Capacitor_SMD:C_0603_1608Metric_Pad1.08x0.95mm_HandSolder, F.Cu at (72.8, 61.4)
- added C16: 4.7n, Capacitor_SMD:C_0603_1608Metric_Pad1.08x0.95mm_HandSolder, F.Cu at (72.8, 63.9)
- added C17: 4.7u, Capacitor_SMD:C_0805_2012Metric_Pad1.18x1.45mm_HandSolder, F.Cu at (90.4, 61.1)
- added C18: 0.1u, Capacitor_SMD:C_0603_1608Metric_Pad1.08x0.95mm_HandSolder, F.Cu at (77.1, 51.3)
- added C19: 0.1u, Capacitor_SMD:C_0603_1608Metric_Pad1.08x0.95mm_HandSolder, F.Cu at (77.1, 53.8)
- added C2: 1u, Capacitor_SMD:C_0603_1608Metric_Pad1.08x0.95mm_HandSolder, F.Cu at (62.8, 248.2)
- added C20: 22u, Capacitor_SMD:C_0603_1608Metric_Pad1.08x0.95mm_HandSolder, F.Cu at (77.1, 56.4)
- added C21: 22u, Capacitor_SMD:C_0603_1608Metric_Pad1.08x0.95mm_HandSolder, F.Cu at (77.1, 58.9)
- added C22: 22u, Capacitor_SMD:C_0603_1608Metric_Pad1.08x0.95mm_HandSolder, F.Cu at (77.1, 61.4)
- added C23: 22u, Capacitor_SMD:C_0603_1608Metric_Pad1.08x0.95mm_HandSolder, F.Cu at (77.1, 63.9)
- added C24: 47u, Capacitor_SMD:C_0603_1608Metric_Pad1.08x0.95mm_HandSolder, F.Cu at (95.8, 246.0)
- added C25: 1u, Capacitor_SMD:C_0603_1608Metric_Pad1.08x0.95mm_HandSolder, F.Cu at (95.8, 247.6)
- added C26: 0.1u, Capacitor_SMD:C_0603_1608Metric_Pad1.08x0.95mm_HandSolder, F.Cu at (95.8, 249.2)
- added C27: 1u, Capacitor_SMD:C_0603_1608Metric_Pad1.08x0.95mm_HandSolder, F.Cu at (95.8, 255.9)
- added C28: 100n, Capacitor_SMD:C_0603_1608Metric_Pad1.08x0.95mm_HandSolder, F.Cu at (136.0, 22.2)
- added C29: 47n, Capacitor_SMD:C_0603_1608Metric_Pad1.08x0.95mm_HandSolder, F.Cu at (136.0, 24.7)
- added C3: 0.1u, Capacitor_SMD:C_0603_1608Metric_Pad1.08x0.95mm_HandSolder, F.Cu at (62.8, 249.8)
- added C30: 0.1u, Capacitor_SMD:C_0603_1608Metric_Pad1.08x0.95mm_HandSolder, F.Cu at (136.0, 27.2)
- added C31: 10n, Capacitor_SMD:C_0603_1608Metric_Pad1.08x0.95mm_HandSolder, F.Cu at (155.1, 45.8)
- added C32: 1n, Capacitor_SMD:C_0603_1608Metric_Pad1.08x0.95mm_HandSolder, F.Cu at (123.1, -11.4)
- added C33: 1u, Capacitor_SMD:C_0603_1608Metric_Pad1.08x0.95mm_HandSolder, F.Cu at (123.1, -8.91)
- added C34: 1n, Capacitor_SMD:C_0603_1608Metric_Pad1.08x0.95mm_HandSolder, F.Cu at (123.1, -6.40)
- added C35: 1u, Capacitor_SMD:C_0603_1608Metric_Pad1.08x0.95mm_HandSolder, F.Cu at (123.1, -3.89)
- added C36: 1n, Capacitor_SMD:C_0805_2012Metric_Pad1.18x1.45mm_HandSolder, F.Cu at (133.9, 7.43)
- added C37: 100n, Capacitor_SMD:C_0603_1608Metric_Pad1.08x0.95mm_HandSolder, F.Cu at (123.1, -1.38)
- added C38: 1n, Capacitor_SMD:C_0603_1608Metric_Pad1.08x0.95mm_HandSolder, F.Cu at (127.5, -11.4)
- added C39: 0.1u, Capacitor_SMD:C_0603_1608Metric_Pad1.08x0.95mm_HandSolder, F.Cu at (127.5, -8.91)
- added C4: 1u, Capacitor_SMD:C_0603_1608Metric_Pad1.08x0.95mm_HandSolder, F.Cu at (62.8, 256.6)
- added C40: 1u, Capacitor_SMD:C_0603_1608Metric_Pad1.08x0.95mm_HandSolder, F.Cu at (127.5, -6.40)
- added C41: 47n, Capacitor_SMD:C_0603_1608Metric_Pad1.08x0.95mm_HandSolder, F.Cu at (127.5, -3.89)
- added C42: 1000p, Capacitor_SMD:C_0603_1608Metric_Pad1.08x0.95mm_HandSolder, F.Cu at (127.5, -1.38)
- added C43: 1000p, Capacitor_SMD:C_0805_2012Metric_Pad1.18x1.45mm_HandSolder, F.Cu at (133.9, 10.4)
- added C44: 47n, Capacitor_SMD:C_0603_1608Metric_Pad1.08x0.95mm_HandSolder, F.Cu at (131.8, -11.4)
- added C45: 100n, Capacitor_SMD:C_0603_1608Metric_Pad1.08x0.95mm_HandSolder, F.Cu at (81.7, -1.82)
- added C46: 100u, Capacitor_SMD:CP_Elec_16x22, F.Cu at (90.7, -12.2)
- added C47: 4700p, Capacitor_SMD:C_0603_1608Metric_Pad1.08x0.95mm_HandSolder, F.Cu at (81.7, 0.69)
- added C48: 4700p, Capacitor_SMD:C_0603_1608Metric_Pad1.08x0.95mm_HandSolder, F.Cu at (81.7, 3.20)
- added C49: 0.1u, Capacitor_SMD:C_0603_1608Metric_Pad1.08x0.95mm_HandSolder, F.Cu at (81.7, 5.71)
- added C5: 47u, Capacitor_SMD:C_0603_1608Metric_Pad1.08x0.95mm_HandSolder, F.Cu at (117.6, 93.3)
- added C50: 0.022u, Capacitor_SMD:C_0603_1608Metric_Pad1.08x0.95mm_HandSolder, F.Cu at (81.7, 8.22)
- added C51: 0.022u, Capacitor_SMD:C_0603_1608Metric_Pad1.08x0.95mm_HandSolder, F.Cu at (86.0, -1.82)
- added C52: 2.2u, Capacitor_SMD:C_0603_1608Metric_Pad1.08x0.95mm_HandSolder, F.Cu at (86.0, 0.69)
- added C53: 680u, Capacitor_SMD:C_1812_4532Metric_Pad1.57x3.40mm_HandSolder, F.Cu at (83.2, 11.9)
- added C54: 100n, Capacitor_SMD:C_0603_1608Metric_Pad1.08x0.95mm_HandSolder, F.Cu at (120.6, 22.2)
- added C55: 47n, Capacitor_SMD:C_0603_1608Metric_Pad1.08x0.95mm_HandSolder, F.Cu at (120.6, 24.7)
- added C56: 0.1u, Capacitor_SMD:C_0603_1608Metric_Pad1.08x0.95mm_HandSolder, F.Cu at (120.6, 27.2)
- added C57: 100n, Capacitor_SMD:C_0603_1608Metric_Pad1.08x0.95mm_HandSolder, F.Cu at (72.8, 30.7)
- added C58: 47u, Capacitor_SMD:C_0603_1608Metric_Pad1.08x0.95mm_HandSolder, F.Cu at (137.7, 246.1)
- added C59: 1u, Capacitor_SMD:C_0603_1608Metric_Pad1.08x0.95mm_HandSolder, F.Cu at (137.7, 247.7)
- added C6: 1u, Capacitor_SMD:C_0603_1608Metric_Pad1.08x0.95mm_HandSolder, F.Cu at (117.6, 94.9)
- added C60: 0.1u, Capacitor_SMD:C_0603_1608Metric_Pad1.08x0.95mm_HandSolder, F.Cu at (137.7, 249.3)
- added C61: 1u, Capacitor_SMD:C_0603_1608Metric_Pad1.08x0.95mm_HandSolder, F.Cu at (137.7, 256.0)
- added C62: 47u, Capacitor_SMD:C_0603_1608Metric_Pad1.08x0.95mm_HandSolder, F.Cu at (183.8, 250.3)
- added C63: 1u, Capacitor_SMD:C_0603_1608Metric_Pad1.08x0.95mm_HandSolder, F.Cu at (183.8, 251.9)
- added C64: 0.1u, Capacitor_SMD:C_0603_1608Metric_Pad1.08x0.95mm_HandSolder, F.Cu at (183.8, 253.5)
- added C65: 1u, Capacitor_SMD:C_0603_1608Metric_Pad1.08x0.95mm_HandSolder, F.Cu at (183.7, 260.2)
- added C66: 47u, Capacitor_SMD:C_0603_1608Metric_Pad1.08x0.95mm_HandSolder, F.Cu at (224.8, 247.5)
- added C67: 1u, Capacitor_SMD:C_0603_1608Metric_Pad1.08x0.95mm_HandSolder, F.Cu at (224.8, 249.1)
- added C68: 0.1u, Capacitor_SMD:C_0603_1608Metric_Pad1.08x0.95mm_HandSolder, F.Cu at (224.8, 250.7)
- added C69: 1u, Capacitor_SMD:C_0603_1608Metric_Pad1.08x0.95mm_HandSolder, F.Cu at (224.7, 257.4)
- added C7: 0.1u, Capacitor_SMD:C_0603_1608Metric_Pad1.08x0.95mm_HandSolder, F.Cu at (117.6, 96.5)
- added C70: 1000u, Capacitor_SMD:CP_Elec_10x12.5, F.Cu at (39.4, -15.2)
- added C71: 1000u, Capacitor_SMD:CP_Elec_10x12.5, F.Cu at (39.4, -3.15)
- added C72: 1000u, Capacitor_SMD:CP_Elec_10x12.5, F.Cu at (39.4, 8.90)
- added C73: 22u, Capacitor_SMD:C_0603_1608Metric_Pad1.08x0.95mm_HandSolder, F.Cu at (75.3, -20.0)
- added C74: 22u, Capacitor_SMD:C_0603_1608Metric_Pad1.08x0.95mm_HandSolder, F.Cu at (75.3, -17.5)
- added C75: 47u, Capacitor_SMD:C_0603_1608Metric_Pad1.08x0.95mm_HandSolder, F.Cu at (265.2, 247.8)
- added C76: 1u, Capacitor_SMD:C_0603_1608Metric_Pad1.08x0.95mm_HandSolder, F.Cu at (265.2, 249.4)
- added C77: 0.1u, Capacitor_SMD:C_0603_1608Metric_Pad1.08x0.95mm_HandSolder, F.Cu at (265.2, 251.1)
- added C78: 1u, Capacitor_SMD:C_0603_1608Metric_Pad1.08x0.95mm_HandSolder, F.Cu at (265.2, 257.8)
- added C79: 100n, Capacitor_SMD:C_0603_1608Metric_Pad1.08x0.95mm_HandSolder, F.Cu at (151.5, 98.7)
- added C8: 1u, Capacitor_SMD:C_0603_1608Metric_Pad1.08x0.95mm_HandSolder, F.Cu at (117.6, 103.2)
- added C80: 47n, Capacitor_SMD:C_0603_1608Metric_Pad1.08x0.95mm_HandSolder, F.Cu at (151.5, 101.2)
- added C81: 0.1u, Capacitor_SMD:C_0603_1608Metric_Pad1.08x0.95mm_HandSolder, F.Cu at (151.5, 103.7)
- added C82: 470n, Capacitor_SMD:C_0603_1608Metric_Pad1.08x0.95mm_HandSolder, F.Cu at (34.2, 99.8)
- added C83: 100n, Capacitor_SMD:C_0603_1608Metric_Pad1.08x0.95mm_HandSolder, F.Cu at (34.2, 102.3)
- added C84: 1n, Capacitor_SMD:C_0603_1608Metric_Pad1.08x0.95mm_HandSolder, F.Cu at (34.2, 104.8)
- added C85: 1u, Capacitor_SMD:C_0603_1608Metric_Pad1.08x0.95mm_HandSolder, F.Cu at (34.2, 107.3)
- added C86: 47n, Capacitor_SMD:C_0603_1608Metric_Pad1.08x0.95mm_HandSolder, F.Cu at (34.2, 109.8)
- added C87: 2.2n, Capacitor_SMD:C_0603_1608Metric_Pad1.08x0.95mm_HandSolder, F.Cu at (34.2, 112.3)
- added C88: 4.7u, Capacitor_SMD:C_0805_2012Metric_Pad1.18x1.45mm_HandSolder, F.Cu at (325.8, 201.4)
- added C89: 100n, Capacitor_SMD:C_0603_1608Metric_Pad1.08x0.95mm_HandSolder, F.Cu at (347.3, 192.5)
- added C9: 0.1u, Capacitor_SMD:C_0402_1005Metric_Pad0.74x0.62mm_HandSolder, F.Cu at (89.4, 71.3)
- added C90: 100n, Capacitor_SMD:C_0603_1608Metric, F.Cu at (326.9, 195.4)
- added C91: 22u, Capacitor_SMD:C_1210_3225Metric_Pad1.33x2.70mm_HandSolder, F.Cu at (342.3, 193.4)
- added C92: 22u, Capacitor_SMD:C_1210_3225Metric_Pad1.33x2.70mm_HandSolder, F.Cu at (342.3, 196.8)
- added C93: 3.3u, Capacitor_SMD:C_0805_2012Metric_Pad1.18x1.45mm_HandSolder, F.Cu at (341.7, 199.5)
- added C94: 10u, Capacitor_SMD:C_0805_2012Metric_Pad1.18x1.45mm_HandSolder, F.Cu at (78.2, 102.9)
- added C95: 10u, Capacitor_SMD:C_0805_2012Metric_Pad1.18x1.45mm_HandSolder, F.Cu at (78.2, 105.9)
- added C96: 10u, Capacitor_SMD:C_0805_2012Metric_Pad1.18x1.45mm_HandSolder, F.Cu at (160.7, 29.0)
- added C97: 0.1u, Capacitor_SMD:C_0603_1608Metric_Pad1.08x0.95mm_HandSolder, F.Cu at (151.5, 22.2)
- added C98: 0.1u, Capacitor_SMD:C_0603_1608Metric_Pad1.08x0.95mm_HandSolder, F.Cu at (151.5, 24.7)
- added C99: 0.1u, Capacitor_SMD:C_0603_1608Metric_Pad1.08x0.95mm_HandSolder, F.Cu at (151.5, 27.2)
- added D1: PS_LED, LED_SMD:LED_0603_1608Metric_Pad1.05x0.95mm_HandSolder, F.Cu at (148.0, 83.6)
- added D10: ORB_IN, LED_SMD:LED_0603_1608Metric_Pad1.05x0.95mm_HandSolder, F.Cu at (103.9, 256.5)
- added D11: SMBJ33D, OBBB Footprints:SMBJ15DM3, F.Cu at (100.0, 242.9)
- added D12: SMLJ150A, Diode_SMD:D_SMB-SMC_Universal_Handsoldering, F.Cu at (149.6, 3.16)
- added D13: HV24V_LED, LED_SMD:LED_0603_1608Metric_Pad1.05x0.95mm_HandSolder, F.Cu at (116.3, -1.78)
- added D14: HV24V_LED, LED_SMD:LED_0603_1608Metric_Pad1.05x0.95mm_HandSolder, F.Cu at (116.3, 0.81)
- added D15: HV24V_LED, LED_SMD:LED_0603_1608Metric_Pad1.05x0.95mm_HandSolder, F.Cu at (90.2, 44.1)
- added D16: DISABLE_LED, LED_SMD:LED_0603_1608Metric_Pad1.05x0.95mm_HandSolder, F.Cu at (90.2, 46.7)
- added D17: ORB_IN, LED_SMD:LED_0603_1608Metric_Pad1.05x0.95mm_HandSolder, F.Cu at (144.7, 254.9)
- added D18: SMBJ33D, OBBB Footprints:SMBJ15DM3, F.Cu at (141.9, 243.0)
- added D19: ORB_IN, LED_SMD:LED_0603_1608Metric_Pad1.05x0.95mm_HandSolder, F.Cu at (195.3, 260.8)
- added D2: ORA_OUT, LED_SMD:LED_0603_1608Metric_Pad1.05x0.95mm_HandSolder, F.Cu at (51.4, 85.4)
- added D20: SMBJ33D, OBBB Footprints:SMBJ15DM3, F.Cu at (187.9, 247.2)
- added D21: ORB_IN, LED_SMD:LED_0603_1608Metric_Pad1.05x0.95mm_HandSolder, F.Cu at (236.3, 258.0)
- added D22: SMBJ33D, OBBB Footprints:SMBJ15DM3, F.Cu at (228.9, 244.4)
- added D23: 12V_IN, LED_SMD:LED_0603_1608Metric_Pad1.05x0.95mm_HandSolder, F.Cu at (61.0, 5.72)
- added D24: 12V_IN, LED_SMD:LED_0603_1608Metric_Pad1.05x0.95mm_HandSolder, F.Cu at (61.0, 8.31)
- added D25: HSS_IN, LED_SMD:LED_0603_1608Metric_Pad1.05x0.95mm_HandSolder, F.Cu at (61.0, 10.9)
- added D26: BPS_IN, LED_SMD:LED_0603_1608Metric_Pad1.05x0.95mm_HandSolder, F.Cu at (61.0, 13.5)
- added D27: PDU_IN_LED, LED_SMD:LED_0603_1608Metric_Pad1.05x0.95mm_HandSolder, F.Cu at (61.0, 16.1)
- added D28: ORB_IN, LED_SMD:LED_0603_1608Metric_Pad1.05x0.95mm_HandSolder, F.Cu at (276.8, 258.3)
- added D29: SMBJ33D, OBBB Footprints:SMBJ15DM3, F.Cu at (269.4, 244.8)
- added D30: LED, LED_SMD:LED_0603_1608Metric_Pad1.05x0.95mm_HandSolder, F.Cu at (55.6, 104.8)
- added D31: D_TVS, Diode_SMD:D_SMB, F.Cu at (49.2, 101.3)
- added D32: D_TVS, Diode_SMD:D_SMB, F.Cu at (49.2, 106.8)
- added D33: 5V_LED, LED_SMD:LED_0603_1608Metric_Pad1.05x0.95mm_HandSolder, F.Cu at (89.9, 102.7)
- added D34: 3V3_LED, LED_SMD:LED_0603_1608Metric_Pad1.05x0.95mm_HandSolder, F.Cu at (89.9, 105.3)
- added D35: SBA130CH-AU_R1_000A1, Diode_SMD:D_SOD-323_HandSoldering, F.Cu at (68.5, 111.2)
- added D36: CDSOT23-T24CAN, LHRS_Passives:CDSOT23-T24CAN, F.Cu at (160.7, 32.8)
- added D37: CHARGE_EN, LED_SMD:LED_0603_1608Metric_Pad1.05x0.95mm_HandSolder, F.Cu at (135.8, 98.8)
- added D38: CHARGE_EN, LED_SMD:LED_0603_1608Metric_Pad1.05x0.95mm_HandSolder, F.Cu at (135.8, 101.3)
- added D39: DCDC_EN, LED_SMD:LED_0603_1608Metric_Pad1.05x0.95mm_HandSolder, F.Cu at (135.8, 103.9)
- added D4: ORB_IN, LED_SMD:LED_0603_1608Metric_Pad1.05x0.95mm_HandSolder, F.Cu at (69.9, 257.1)
- added D40: HB_LED, LED_SMD:LED_0603_1608Metric_Pad1.05x0.95mm_HandSolder, F.Cu at (135.8, 106.5)
- added D41: FAULT_LED, LED_SMD:LED_0603_1608Metric_Pad1.05x0.95mm_HandSolder, F.Cu at (135.8, 109.1)
- added D42: LV_EN, LED_SMD:LED_0603_1608Metric_Pad1.05x0.95mm_HandSolder, F.Cu at (135.8, 111.7)
- added D43: TVS, Diode_SMD:D_SOD-323, F.Cu at (42.8, 53.7)
- added D44: RGB_LED, LHRS_Special:RGB_LED, F.Cu at (47.1, 53.8)
- added D45: LED, LED_SMD:LED_0603_1608Metric_Pad1.05x0.95mm_HandSolder, F.Cu at (42.8, 51.0)
- added D5: SMBJ33D, OBBB Footprints:SMBJ15DM3, F.Cu at (67.0, 243.6)
- added D6: ORB_IN, LED_SMD:LED_0603_1608Metric_Pad1.05x0.95mm_HandSolder, F.Cu at (129.2, 103.8)
- added D7: SMBJ33D, OBBB Footprints:SMBJ15DM3, F.Cu at (121.8, 90.2)
- added D8: LED, LED_SMD:LED_0603_1608Metric_Pad1.05x0.95mm_HandSolder, F.Cu at (90.0, 66.4)
- added D9: LED, LED_SMD:LED_0603_1608Metric_Pad1.05x0.95mm_HandSolder, F.Cu at (90.0, 69.0)
- added F1: TBD, LHRS_Power:Fuse-3557-2, F.Cu at (144.3, 73.0)
- added F10: 5A, LHRS_Power:Fuse-3557-2, F.Cu at (42.8, 94.2)
- added F2: TBD, LHRS_Power:Fuse-3557-2, F.Cu at (42.8, 62.2)
- added F3: TBD until vicor confirmed, LHRS_Power:Fuse-3557-2, F.Cu at (144.3, 91.2)
- added F4: 5A, LHRS_Power:Fuse-3557-2, F.Cu at (131.7, -16.9)
- added F5: 5A, LHRS_Power:Fuse-3557-2, F.Cu at (103.3, 1.20)
- added F6: Fuse, LHRS_Power:Fuse-3557-2, F.Cu at (76.7, 25.2)
- added F7: TBD, LHRS_Power:Fuse-3557-2, F.Cu at (57.3, -16.9)
- added F8: TBD, LHRS_Power:Fuse-3557-2, F.Cu at (57.3, -8.40)
- added F9: TBD, LHRS_Power:Fuse-3557-2, F.Cu at (57.3, 0.15)
- added FB1: FerriteBead, Capacitor_SMD:C_0603_1608Metric_Pad1.08x0.95mm_HandSolder, F.Cu at (38.5, 34.7)
- added FB2: FerriteBead, Capacitor_SMD:C_0603_1608Metric_Pad1.08x0.95mm_HandSolder, F.Cu at (38.5, 37.2)
- added IC1: AP74502HQTA8-7, OBBB Footprints:AP74502HQTA87, F.Cu at (63.7, 253.2)
- added IC2: AP74502HQTA8-7, OBBB Footprints:AP74502HQTA87, F.Cu at (118.5, 99.9)
- added IC3: AP74502HQTA8-7, OBBB Footprints:AP74502HQTA87, F.Cu at (96.8, 252.6)
- added IC4: AP74502HQTA8-7, OBBB Footprints:AP74502HQTA87, F.Cu at (138.6, 252.7)
- added IC5: AP74502HQTA8-7, OBBB Footprints:AP74502HQTA87, F.Cu at (184.7, 256.9)
- added IC6: AP74502HQTA8-7, OBBB Footprints:AP74502HQTA87, F.Cu at (225.7, 254.1)
- added IC7: AP74502HQTA8-7, OBBB Footprints:AP74502HQTA87, F.Cu at (266.1, 254.4)
- added IC8: TPS2HCS08AQPWPRQ1, OBBB Footprints:TPS2HCS08AQPWPRQ1, F.Cu at (49.5, 113.0)
- added IC9: TCAN3413DR, LHRS_Passives:TCAN3413DR, F.Cu at (157.9, 24.2)
- added J1: PS, LHRS_Connectors:AMASS_XT30UPB-M_1x02_P5.0mm_Vertical, F.Cu at (137.2, 80.9)
- added J10: PDU_12V, LHRS_Connectors:AMASS_XT30UPB-M_1x02_P5.0mm_Vertical, F.Cu at (50.2, 15.3)
- added J12: SWD_Header, LHRS_Connectors:SWD_Conn, F.Cu at (37.5, 45.3)
- added J13: SWD, Connector_PinHeader_2.54mm:PinHeader_1x04_P2.54mm_Vertical, F.Cu at (47.3, 42.1)
- added J14: FAN2, LHRS_Connectors:Molex_Nano-Fit_105309-xx04_1x04_P2.50mm_Vertical, F.Cu at (80.3, 84.4)
- added J15: FAN1, LHRS_Connectors:Molex_Nano-Fit_105309-xx04_1x04_P2.50mm_Vertical, F.Cu at (88.7, 84.4)
- added J2: LV_ENABLE, LHRS_Connectors:AMASS_XT30UPB-M_1x02_P5.0mm_Vertical, F.Cu at (35.6, 70.1)
- added J3: SUPP, LHRS_Connectors:AMASS_XT30UPB-M_1x02_P5.0mm_Vertical, F.Cu at (35.6, 77.4)
- added J4: PWM/PFM, Connector_PinHeader_1.00mm:PinHeader_1x03_P1.00mm_Vertical, F.Cu at (89.7, 51.6)
- added J5: HV_IN, LHRS_Connectors:AMASS_XT30UPB-M_1x02_P5.0mm_Vertical, F.Cu at (147.0, 10.7)
- added J6: HV_IN, LHRS_Connectors:AMASS_XT30UPB-M_1x02_P5.0mm_Vertical, F.Cu at (110.3, -17.6)
- added J7: HV_IN, LHRS_Connectors:AMASS_XT30UPB-M_1x02_P5.0mm_Vertical, F.Cu at (110.3, -10.3)
- added J8: HV_THERM, LHRS_Connectors:105313-2102, F.Cu at (94.7, 8.22)
- added J9: BPS_12V, LHRS_Connectors:AMASS_XT30UPB-M_1x02_P5.0mm_Vertical, F.Cu at (50.2, 8.05)
- added JP1: TRM, Connector_PinHeader_2.54mm:PinHeader_1x02_P2.54mm_Vertical, F.Cu at (156.0, 29.8)
- added L1: 6.8u, Inductor_SMD:L_Coilcraft_XAL6020-XXX, F.Cu at (83.7, 69.3)
- added L2: 8.2u, LHRS_Passives:74439369082, F.Cu at (334.0, 197.8)
- added Q1: IRLML0030, Package_TO_SOT_SMD:SOT-23, F.Cu at (46.7, 81.3)
- added Q10: IRLML0030, Package_TO_SOT_SMD:SOT-23, F.Cu at (90.5, 31.7)
- added Q11: IRLML0030, Package_TO_SOT_SMD:SOT-23, F.Cu at (90.5, 36.1)
- added Q12: IRLML0030, Package_TO_SOT_SMD:SOT-23, F.Cu at (90.5, 40.6)
- added Q13: NVMFWS1D7N04XMT1G, OBBB Footprints:NVMFWS3D0P04M8LT1G, F.Cu at (132.1, 247.3)
- added Q14: NVMFWS1D7N04XMT1G, OBBB Footprints:NVMFWS3D0P04M8LT1G, F.Cu at (132.1, 256.0)
- added Q15: NVMFWS1D7N04XMT1G, OBBB Footprints:NVMFWS3D0P04M8LT1G, F.Cu at (178.1, 251.5)
- added Q16: NVMFWS1D7N04XMT1G, OBBB Footprints:NVMFWS3D0P04M8LT1G, F.Cu at (178.1, 260.2)
- added Q17: NVMFWS1D7N04XMT1G, OBBB Footprints:NVMFWS3D0P04M8LT1G, F.Cu at (219.1, 248.7)
- added Q18: NVMFWS1D7N04XMT1G, OBBB Footprints:NVMFWS3D0P04M8LT1G, F.Cu at (219.1, 257.4)
- added Q19: NVMFWS1D7N04XMT1G, OBBB Footprints:NVMFWS3D0P04M8LT1G, F.Cu at (259.6, 249.0)
- added Q2: IRLML0030, Package_TO_SOT_SMD:SOT-23, F.Cu at (46.7, 85.7)
- added Q20: NVMFWS1D7N04XMT1G, OBBB Footprints:NVMFWS3D0P04M8LT1G, F.Cu at (259.6, 257.8)
- added Q3: NVMFWS1D7N04XMT1G, OBBB Footprints:NVMFWS3D0P04M8LT1G, F.Cu at (57.1, 247.8)
- added Q4: NVMFWS1D7N04XMT1G, OBBB Footprints:NVMFWS3D0P04M8LT1G, F.Cu at (57.2, 256.6)
- added Q5: NVMFWS1D7N04XMT1G, OBBB Footprints:NVMFWS3D0P04M8LT1G, F.Cu at (112.0, 94.5)
- added Q6: NVMFWS1D7N04XMT1G, OBBB Footprints:NVMFWS3D0P04M8LT1G, F.Cu at (112.0, 103.2)
- added Q7: 2N7002, Package_TO_SOT_SMD:SOT-23, F.Cu at (90.5, 57.4)
- added Q8: NVMFWS1D7N04XMT1G, OBBB Footprints:NVMFWS3D0P04M8LT1G, F.Cu at (90.2, 247.2)
- added Q9: NVMFWS1D7N04XMT1G, OBBB Footprints:NVMFWS3D0P04M8LT1G, F.Cu at (90.2, 255.9)
- added R1: 10k, Resistor_SMD:R_0603_1608Metric_Pad0.98x0.95mm_HandSolder, F.Cu at (152.4, 83.6)
- added R10: 118k, Resistor_SMD:R_0603_1608Metric_Pad0.98x0.95mm_HandSolder, F.Cu at (50.8, 75.3)
- added R100: 4.7k, Resistor_SMD:R_0603_1608Metric_Pad0.98x0.95mm_HandSolder, F.Cu at (34.2, 117.3)
- added R101: 10, Resistor_SMD:R_0603_1608Metric_Pad0.98x0.95mm_HandSolder, F.Cu at (38.5, 99.8)
- added R102: 10k, Resistor_SMD:R_0603_1608Metric_Pad0.98x0.95mm_HandSolder, F.Cu at (38.5, 102.3)
- added R103: 10k, Resistor_SMD:R_0603_1608Metric_Pad0.98x0.95mm_HandSolder, F.Cu at (38.5, 104.8)
- added R104: 22, Resistor_SMD:R_0603_1608Metric_Pad0.98x0.95mm_HandSolder, F.Cu at (38.5, 107.3)
- added R105: 22, Resistor_SMD:R_0603_1608Metric_Pad0.98x0.95mm_HandSolder, F.Cu at (38.5, 109.8)
- added R106: 10k, Resistor_SMD:R_0603_1608Metric_Pad0.98x0.95mm_HandSolder, F.Cu at (38.5, 112.3)
- added R107: 10k, Resistor_SMD:R_0603_1608Metric_Pad0.98x0.95mm_HandSolder, F.Cu at (38.5, 114.8)
- added R108: 10k, Resistor_SMD:R_0603_1608Metric_Pad0.98x0.95mm_HandSolder, F.Cu at (38.5, 117.3)
- added R109: 220, Resistor_SMD:R_0603_1608Metric_Pad0.98x0.95mm_HandSolder, F.Cu at (42.9, 99.8)
- added R11: 10k, Resistor_SMD:R_0603_1608Metric_Pad0.98x0.95mm_HandSolder, F.Cu at (50.8, 77.8)
- added R110: 4.7k, Resistor_SMD:R_0603_1608Metric_Pad0.98x0.95mm_HandSolder, F.Cu at (42.9, 102.3)
- added R111: 10k, Resistor_SMD:R_0603_1608Metric_Pad0.98x0.95mm_HandSolder, F.Cu at (42.9, 104.8)
- added R112: 10k, Resistor_SMD:R_0603_1608Metric_Pad0.98x0.95mm_HandSolder, F.Cu at (42.9, 107.3)
- added R113: 10k, Resistor_SMD:R_0603_1608Metric_Pad0.98x0.95mm_HandSolder, F.Cu at (42.9, 109.8)
- added R114: 4.7k, Resistor_SMD:R_0603_1608Metric_Pad0.98x0.95mm_HandSolder, F.Cu at (42.9, 112.3)
- added R115: 470, Resistor_SMD:R_0603_1608Metric_Pad0.98x0.95mm_HandSolder, F.Cu at (42.9, 114.8)
- added R116: 1.3k, Resistor_SMD:R_0603_1608Metric_Pad0.98x0.95mm_HandSolder, F.Cu at (89.8, 107.8)
- added R117: 1.3k, Resistor_SMD:R_0603_1608Metric_Pad0.98x0.95mm_HandSolder, F.Cu at (89.8, 110.3)
- added R118: 100k, Resistor_SMD:R_0603_1608Metric_Pad0.98x0.95mm_HandSolder, F.Cu at (341.5, 201.3)
- added R119: 19.1k, Resistor_SMD:R_0603_1608Metric_Pad0.98x0.95mm_HandSolder, F.Cu at (341.5, 202.9)
- added R12: 10k, Resistor_SMD:R_0603_1608Metric_Pad0.98x0.95mm_HandSolder, F.Cu at (55.1, 67.8)
- added R120: 60, Resistor_SMD:R_0603_1608Metric_Pad0.98x0.95mm_HandSolder, F.Cu at (151.5, 29.7)
- added R121: 60, Resistor_SMD:R_0603_1608Metric_Pad0.98x0.95mm_HandSolder, F.Cu at (151.5, 32.2)
- added R122: 1.3k, Resistor_SMD:R_0603_1608Metric_Pad0.98x0.95mm_HandSolder, F.Cu at (140.1, 98.7)
- added R123: 1.3k, Resistor_SMD:R_0603_1608Metric_Pad0.98x0.95mm_HandSolder, F.Cu at (140.1, 101.2)
- added R124: 1.3k, Resistor_SMD:R_0603_1608Metric_Pad0.98x0.95mm_HandSolder, F.Cu at (140.1, 103.7)
- added R125: 1.3k, Resistor_SMD:R_0603_1608Metric_Pad0.98x0.95mm_HandSolder, F.Cu at (140.1, 106.2)
- added R126: 1.3k, Resistor_SMD:R_0603_1608Metric_Pad0.98x0.95mm_HandSolder, F.Cu at (140.1, 108.8)
- added R127: 1.3k, Resistor_SMD:R_0603_1608Metric_Pad0.98x0.95mm_HandSolder, F.Cu at (140.1, 111.3)
- added R128: 10k, Resistor_SMD:R_0603_1608Metric_Pad0.98x0.95mm_HandSolder, F.Cu at (38.5, 39.8)
- added R129: 22, Resistor_SMD:R_0603_1608Metric_Pad0.98x0.95mm_HandSolder, F.Cu at (42.9, 22.2)
- added R13: 100k, Resistor_SMD:R_0603_1608Metric_Pad0.98x0.95mm_HandSolder, F.Cu at (55.1, 70.3)
- added R130: 22, Resistor_SMD:R_0603_1608Metric_Pad0.98x0.95mm_HandSolder, F.Cu at (42.9, 24.7)
- added R131: 1k, Resistor_SMD:R_0603_1608Metric_Pad0.98x0.95mm_HandSolder, F.Cu at (42.9, 27.2)
- added R132: 1k, Resistor_SMD:R_0603_1608Metric_Pad0.98x0.95mm_HandSolder, F.Cu at (42.9, 29.7)
- added R133: 1k, Resistor_SMD:R_0603_1608Metric_Pad0.98x0.95mm_HandSolder, F.Cu at (42.9, 32.2)
- added R134: 10k, Resistor_SMD:R_0603_1608Metric_Pad0.98x0.95mm_HandSolder, F.Cu at (42.9, 34.7)
- added R135: 1k, Resistor_SMD:R_0603_1608Metric_Pad0.98x0.95mm_HandSolder, F.Cu at (42.9, 37.2)
- added R136: 10k, Resistor_SMD:R_0603_1608Metric_Pad0.98x0.95mm_HandSolder, F.Cu at (68.1, 78.4)
- added R137: 10k, Resistor_SMD:R_0603_1608Metric_Pad0.98x0.95mm_HandSolder, F.Cu at (68.1, 80.9)
- added R138: 10k, Resistor_SMD:R_0603_1608Metric_Pad0.98x0.95mm_HandSolder, F.Cu at (68.1, 83.4)
- added R139: 10k, Resistor_SMD:R_0603_1608Metric_Pad0.98x0.95mm_HandSolder, F.Cu at (68.1, 85.9)
- added R14: 118k, Resistor_SMD:R_0603_1608Metric_Pad0.98x0.95mm_HandSolder, F.Cu at (55.1, 72.8)
- added R140: 10k, Resistor_SMD:R_0603_1608Metric_Pad0.98x0.95mm_HandSolder, F.Cu at (68.1, 88.4)
- added R141: 33k, Resistor_SMD:R_0603_1608Metric_Pad0.98x0.95mm_HandSolder, F.Cu at (68.1, 90.9)
- added R142: 22k, Resistor_SMD:R_0603_1608Metric_Pad0.98x0.95mm_HandSolder, F.Cu at (68.1, 93.4)
- added R143: 0, Resistor_SMD:R_0603_1608Metric_Pad0.98x0.95mm_HandSolder, F.Cu at (68.1, 95.9)
- added R15: 10k, Resistor_SMD:R_0603_1608Metric_Pad0.98x0.95mm_HandSolder, F.Cu at (55.1, 75.3)
- added R16: 10k, Resistor_SMD:R_0603_1608Metric_Pad0.98x0.95mm_HandSolder, F.Cu at (69.9, 255.5)
- added R17: 10k, Resistor_SMD:R_0603_1608Metric_Pad0.98x0.95mm_HandSolder, F.Cu at (129.2, 102.2)
- added R18: 100k, Resistor_SMD:R_0603_1608Metric_Pad0.98x0.95mm_HandSolder, F.Cu at (81.5, 51.3)
- added R19: 100k, Resistor_SMD:R_0603_1608Metric_Pad0.98x0.95mm_HandSolder, F.Cu at (81.5, 53.8)
- added R2: 1k, Resistor_SMD:R_0603_1608Metric_Pad0.98x0.95mm_HandSolder, F.Cu at (46.4, 67.8)
- added R20: 49.9k, Resistor_SMD:R_0603_1608Metric_Pad0.98x0.95mm_HandSolder, F.Cu at (81.5, 56.4)
- added R21: 200k, Resistor_SMD:R_0603_1608Metric_Pad0.98x0.95mm_HandSolder, F.Cu at (81.5, 58.9)
- added R22: 26.1k, Resistor_SMD:R_0603_1608Metric_Pad0.98x0.95mm_HandSolder, F.Cu at (81.5, 61.4)
- added R23: 100k, Resistor_SMD:R_0603_1608Metric_Pad0.98x0.95mm_HandSolder, F.Cu at (81.5, 63.9)
- added R24: 100k, Resistor_SMD:R_0603_1608Metric_Pad0.98x0.95mm_HandSolder, F.Cu at (85.8, 51.3)
- added R25: 30k, Resistor_SMD:R_0603_1608Metric_Pad0.98x0.95mm_HandSolder, F.Cu at (85.8, 53.8)
- added R26: 1.3k, Resistor_SMD:R_0603_1608Metric_Pad0.98x0.95mm_HandSolder, F.Cu at (85.8, 56.4)
- added R27: 1.3k, Resistor_SMD:R_0603_1608Metric_Pad0.98x0.95mm_HandSolder, F.Cu at (85.8, 58.9)
- added R28: 25m, Resistor_SMD:R_2512_6332Metric_Pad1.40x3.35mm_HandSolder, F.Cu at (75.1, 67.6)
- added R29: 100k, Resistor_SMD:R_0603_1608Metric_Pad0.98x0.95mm_HandSolder, F.Cu at (85.8, 61.4)
- added R3: 100k, Resistor_SMD:R_0603_1608Metric_Pad0.98x0.95mm_HandSolder, F.Cu at (46.4, 70.3)
- added R30: 8.66k, Resistor_SMD:R_0603_1608Metric_Pad0.98x0.95mm_HandSolder, F.Cu at (85.8, 63.9)
- added R31: 10k, Resistor_SMD:R_0603_1608Metric_Pad0.98x0.95mm_HandSolder, F.Cu at (103.9, 254.9)
- added R32: 10k, Resistor_SMD:R_0603_1608Metric_Pad0.98x0.95mm_HandSolder, F.Cu at (136.0, 29.7)
- added R33: 1k, Resistor_SMD:R_0603_1608Metric_Pad0.98x0.95mm_HandSolder, F.Cu at (136.0, 32.2)
- added R34: 4.7k, Resistor_SMD:R_0603_1608Metric_Pad0.98x0.95mm_HandSolder, F.Cu at (136.0, 34.7)
- added R35: 200k, Resistor_SMD:R_0603_1608Metric_Pad0.98x0.95mm_HandSolder, F.Cu at (155.1, 48.3)
- added R36: 100k, Resistor_SMD:R_0603_1608Metric_Pad0.98x0.95mm_HandSolder, F.Cu at (155.1, 50.9)
- added R37: 470k, Resistor_SMD:R_0603_1608Metric_Pad0.98x0.95mm_HandSolder, F.Cu at (155.1, 53.4)
- added R38: 402k, Resistor_SMD:R_1206_3216Metric_Pad1.30x1.75mm_HandSolder, F.Cu at (123.9, 1.53)
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Routing:
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- added copper zone on F.Cu, net /Main Diode ORs/Ideal Diode1/DIODE_VOUT
- added copper zone on F.Cu, net /Main Diode ORs/Ideal Diode1/SRC
- added copper zone on F.Cu, net /Main Diode ORs/Ideal Diode1/VIN
- added copper zone on F.Cu, net /Main Diode ORs/Ideal Diode2/SRC
- added copper zone on F.Cu, net /Main Diode ORs/Ideal Diode2/VIN
- added copper zone on F.Cu, net /Main Diode ORs/Ideal Diode3/SRC
- added copper zone on F.Cu, net /Main Diode ORs/Ideal Diode3/VIN
- added copper zone on F.Cu, net /Ouput/12V_OUT
- added copper zone on F.Cu, net /Ouput/Ideal Diode/SRC
- added copper zone on F.Cu, net /Ouput/Ideal Diode/VIN
- added copper zone on F.Cu, net /Supp Input/CC Buck/CC_VIN
- added copper zone on F.Cu, net /Supp Input/Ideal Diode3/SRC
- added copper zone on F.Cu, net /Supp Input/Ideal Diode4/SRC
- added copper zone on F.Cu, net /Supp Input/Ideal Diode4/VIN
- added copper zone on F.Cu, net /Supp Input/SUPP_FUSED

Commit message: Js a lil
Parts:
- SW1: value SW_SPDT -> BOOT
- TP49: value BOOT -> BOOT0
- TP50: value RESET -> NSRT
- moved D45 354.8 mm to (389.7, -23.6), turned to 180 degrees
- moved D43 354.3 mm to (389.7, -18.2), turned to 180 degrees
- moved R135 351.8 mm to (389.7, -21.8), turned to 180 degrees
- moved R134 351.2 mm to (389.7, -20.1), turned to 180 degrees
- moved Reset 344.8 mm to (372.9, -21.7)
- moved R128 341.5 mm to (375.1, -18.2)
- moved C106 340.8 mm to (370.8, -18.2), turned to 180 degrees
- moved SW1 333.0 mm to (382.3, -19.3)
- moved C107 332.5 mm to (347.0, -75.5)
- moved J12 319.6 mm to (352.7, -7.55), turned to 180 degrees
- moved C112 309.7 mm to (327.5, -81.5), turned to 90 degrees
- moved R129 305.5 mm to (343.8, -30.2)
- moved R130 305.5 mm to (343.8, -27.7)
- moved J13 304.3 mm to (346.9, -11.6)
- moved U13 296.9 mm to (334.5, -68.5)
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- renumbered Reset1 to Reset
Routing:
- net Net-(D43-A2): track 0.00 -> 13.5 mm
- net /MCU/STM32G491VET/NRST: track 0.00 -> 12.2 mm
- net /MCU/STM32G491VET/BOOT0: track 0.00 -> 5.58 mm
- net +3V3: track 0.00 -> 4.52 mm
- net Net-(D45-K): track 0.00 -> 1.77 mm
Other:
- board text added: "3V3"
- board text added: "GND"
- board text added: "SWCLK"
- board text added: "SWDIO"

Commit message: continue working soon
Parts:
- removed F5: 5A, LHRS_Power:Fuse-3557-2
- removed F6: Fuse, LHRS_Power:Fuse-3557-2
- removed F8: TBD, LHRS_Power:Fuse-3557-2
- removed Q1, Q11, Q12, Q2: IRLML0030, Package_TO_SOT_SMD:SOT-23
- removed R2, R4, R62, R64: 1k, Resistor_SMD:R_0603_1608Metric_Pad0.98x0.95mm_HandSolder
- removed R3, R5, R6, R63, R65, R7, R73, R74: 100k, Resistor_SMD:R_0603_1608Metric_Pad0.98x0.95mm_HandSolder
- removed R69, R70, R71, R72: 10k, Resistor_SMD:R_0603_1608Metric_Pad0.98x0.95mm_HandSolder
- removed Reset: Reset, LHRS_Special:TL3365AF180QG
- added C114: 1000u, Capacitor_SMD:CP_Elec_10x12.5, F.Cu at (-151.9, -1.72)
- added D46: VSSAF522-M3/H, LHRS_Passives:SODFL5026X125N, F.Cu at (-214.8, -4.37)
- added J11: CAN_NANO_01x03, LHRS_Connectors:Molex_Nano-Fit_105309-xx03_1x03_P2.50mm_Vertical, F.Cu at (11.6, 263.9)
- added J16: Conn_01x02, Connector_PinHeader_1.00mm:PinHeader_1x02_P1.00mm_Vertical, F.Cu at (-48.3, 343.4)
- added R144: 47k, Resistor_SMD:R_0603_1608Metric_Pad0.98x0.95mm_HandSolder, F.Cu at (-46.3, 342.9)
- added Reset1: Reset, LHRS_Special:TL3365AF180QG, F.Cu at (-195.6, 263.6)
- added U7: CN150B110-12, OBBB Footprints:lvc_dcdc, F.Cu at (-242.8, 72.8)
- C12, C32, C33, C34, C35, C36, C45, C47, C48, C52, D17, R1, R10, R11, R116, R117, R136, R137, R14, R15, R16, R17, R20, R23, R24, R26, R27, R43, R51, R52, R53, R66, R67, R75, R76, R77, R78, R79, R8, R80, R88, R89, R9, R90, R91, R92, R93, R94: moved to B.Cu
- R61: value 470k -> 47k; moved to B.Cu
- R68: value 220k -> 22k; moved to B.Cu
- SW1: value BOOT -> SW_SPDT
- TP49: value BOOT0 -> BOOT
- TP50: value NSRT -> RESET
- moved TP49 692.4 mm to (-253.6, 232.6)
- moved TP50 692.4 mm to (-274.9, 233.9)
- moved C100 632.6 mm to (-266.6, 188.5)
- moved C101 632.6 mm to (-266.6, 191.0)
- moved C102 632.6 mm to (-241.1, 218.7)
- moved C103 632.6 mm to (-266.6, 193.5)
- moved C104 632.6 mm to (-266.6, 196.1)
- moved C105 632.6 mm to (-266.6, 198.6)
- moved C106 632.6 mm to (-206.4, 240.7)
- moved C107 632.6 mm to (-230.2, 183.4)
- moved C108 632.6 mm to (-266.6, 206.1)
- moved C109 632.6 mm to (-262.3, 188.5)
- moved C110 632.6 mm to (-262.3, 191.0)
- moved C111 632.6 mm to (-262.3, 193.5)
- moved C112 632.6 mm to (-249.7, 177.4)
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Connections:
- net /MCU/HSS_SCLK renamed /HSS_SCLK
- net /MCU/HV_PC_FAULT renamed /MCU/STM32G491VET/PD3
- net /MCU/HV_SC_FAULT renamed /MCU/STM32G491VET/PD4
- net LV_ENABLE renamed /Supp Input/LV_ENABLE
- C28 pad 1: /Supp Input/SUPP_V -> /SUPP_V
- C29 pad 1: /Supp Input/SUPP_I -> /SUPP_I
- C41 pad 1: /HV Input/HV Input/HV_IN_V -> /HV_IN_V
- C44 pad 1: /HV Input/HV Input/HV_IN_I -> /HV_IN_I
- C46 pad 1: Net-(U7-IN+) -> /HV Input/HV -> 12V/HV_IN
- C47 pad 1: Net-(U7-IN+) -> /HV Input/HV -> 12V/HV_IN
- C54 pad 1: /HV Input/HV -> 12V/HV_V_OUT -> /HV_OUT_V
- C55 pad 1: /HV Input/HV -> 12V/HV_I_OUT -> /HV_OUT_I
- C61 pad 1: /Main Diode ORs/Ideal Diode1/DIODE_VOUT -> /Main Diode ORs/12V_FUSED
- C65 pad 1: /Main Diode ORs/Ideal Diode1/DIODE_VOUT -> /Main Diode ORs/12V_FUSED
- C69 pad 1: /Main Diode ORs/Ideal Diode1/DIODE_VOUT -> /Main Diode ORs/12V_FUSED
- C79 pad 1: /Ouput/LVC_V -> /LV_V
- C80 pad 1: /Ouput/LVC_I -> /LV_I
- C83 pad 2: /Ouput/HSS/OUTPUT1 -> /Ouput/BPS_FUSED
- C86 pad 2: /Ouput/HSS/HSS_SNS -> /HSS_SNS
- D30 pad 1: /Ouput/HSS/OUTPUT1 -> /Ouput/BPS_FUSED
- D31 pad 2: /Ouput/HSS/OUTPUT1 -> /Ouput/BPS_FUSED
- D8 pad 1: /Supp Input/CC Buck/CHG_CC -> /CHG_CC
- F10 pad 2: /Ouput/HSS/OUTPUT1 -> /Ouput/BPS_FUSED
- IC1 pad 1: /Supp Input/Ideal Diode3/DIODE_EN -> DIODE_EN
- IC2 pad 1: /Supp Input/Ideal Diode1/DIODE_EN -> DIODE_EN
- IC4 pad 1: /Main Diode ORs/LVD_ENABLE -> DIODE_EN
- IC5 pad 1: /Main Diode ORs/Ideal Diode2/DIODE_EN -> DIODE_EN
- IC6 pad 1: /Main Diode ORs/Ideal Diode3/DIODE_EN -> DIODE_EN
- IC8 pad 5: /Ouput/HSS/LIMP_HOME -> /LIMP_HOME
- J6 pad 1: unconnected-(J6-Pin_1-Pad1) -> /HV Input/HV -> 12V/HV_IN-
- J6 pad 2: /HV Input/HV -> 12V/HV_IN -> /HV Input/HV -> 12V/HV_IN+
- J7 pad 1: unconnected-(J7-Pin_1-Pad1) -> /HV Input/HV -> 12V/HV_OUT-
- J7 pad 2: unconnected-(J7-Pin_2-Pad2) -> /HV Input/HV -> 12V/HV_OUT+
- Q10 pad 3: /Main Diode ORs/LVD_ENABLE -> DIODE_EN
- Q14 pad 5: /Main Diode ORs/Ideal Diode1/DIODE_VOUT -> /Main Diode ORs/12V_FUSED
- Q14 pad 6: /Main Diode ORs/Ideal Diode1/DIODE_VOUT -> /Main Diode ORs/12V_FUSED
- Q14 pad 7: /Main Diode ORs/Ideal Diode1/DIODE_VOUT -> /Main Diode ORs/12V_FUSED
- Q14 pad 8: /Main Diode ORs/Ideal Diode1/DIODE_VOUT -> /Main Diode ORs/12V_FUSED
- Q14 pad 9: /Main Diode ORs/Ideal Diode1/DIODE_VOUT -> /Main Diode ORs/12V_FUSED
- Q16 pad 5: /Main Diode ORs/Ideal Diode1/DIODE_VOUT -> /Main Diode ORs/12V_FUSED
- Q16 pad 6: /Main Diode ORs/Ideal Diode1/DIODE_VOUT -> /Main Diode ORs/12V_FUSED
- Q16 pad 7: /Main Diode ORs/Ideal Diode1/DIODE_VOUT -> /Main Diode ORs/12V_FUSED
- Q16 pad 8: /Main Diode ORs/Ideal Diode1/DIODE_VOUT -> /Main Diode ORs/12V_FUSED
- Q16 pad 9: /Main Diode ORs/Ideal Diode1/DIODE_VOUT -> /Main Diode ORs/12V_FUSED
- Q18 pad 5: /Main Diode ORs/Ideal Diode1/DIODE_VOUT -> /Main Diode ORs/12V_FUSED
- Q18 pad 6: /Main Diode ORs/Ideal Diode1/DIODE_VOUT -> /Main Diode ORs/12V_FUSED
- Q18 pad 7: /Main Diode ORs/Ideal Diode1/DIODE_VOUT -> /Main Diode ORs/12V_FUSED
- Q18 pad 8: /Main Diode ORs/Ideal Diode1/DIODE_VOUT -> /Main Diode ORs/12V_FUSED
- Q18 pad 9: /Main Diode ORs/Ideal Diode1/DIODE_VOUT -> /Main Diode ORs/12V_FUSED
- R107 pad 2: /Ouput/HSS/LIMP_HOME -> /LIMP_HOME
- R108 pad 1: /Ouput/HSS/DI_MODE -> /DI_MODE
- R109 pad 1: /Ouput/HSS/MISO -> /MISO
- R111 pad 1: /Ouput/HSS/MISO -> /MISO
- R113 pad 2: /Ouput/HSS/DI_MODE -> /DI_MODE
- R114 pad 2: /Ouput/HSS/HSS_SNS -> /HSS_SNS
- R139 pad 2: /Fans/FAN_A_PWM -> /Fans/FAN_B_PWM
- R23 pad 2: /Supp Input/CC Buck/CHG_CC -> /CHG_CC
- R24 pad 2: /Supp Input/CC Buck/CHG_PG -> /CHG_PG
- R27 pad 1: /Supp Input/CC Buck/CHG_PG -> /CHG_PG
- R32 pad 2: /Supp Input/SUPP_V -> /SUPP_V
- R33 pad 1: /Supp Input/SUPP_V -> /SUPP_V
- R34 pad 2: /Supp Input/SUPP_I -> /SUPP_I
- R37 pad 1: /Main Diode ORs/LVD_ENABLE -> DIODE_EN
- R45 pad 2: /HV Input/HV Input/HV_IN_V -> /HV_IN_V
- R50 pad 2: /HV Input/HV Input/HV_IN_I -> /HV_IN_I
- R58 pad 2: /HV Input/HV -> 12V/HV_V_OUT -> /HV_OUT_V
- R59 pad 1: /HV Input/HV -> 12V/HV_V_OUT -> /HV_OUT_V
- R60 pad 2: /HV Input/HV -> 12V/HV_I_OUT -> /HV_OUT_I
- R61 pad 2: /Main Diode ORs/LVD_ENABLE -> DIODE_EN
- R68 pad 1: /Main Diode ORs/LVD_ENABLE -> DIODE_EN
- R81 pad 1: /Main Diode ORs/Ideal Diode1/DIODE_VOUT -> /Main Diode ORs/12V_FUSED
- R82 pad 1: /Main Diode ORs/12V_FUSED -> /Main Diode ORs/Ideal Diode1/VIN
- R96 pad 2: /Ouput/LVC_V -> /LV_V
- R97 pad 1: /Ouput/LVC_V -> /LV_V
- R98 pad 2: /Ouput/LVC_I -> /LV_I
- TP10 pad 1: /Supp Input/SUPP_V -> /SUPP_V
- TP23 pad 1: /HV Input/HV -> 12V/HV_V_OUT -> /HV_OUT_V
- TP26 pad 1: /Main Diode ORs/LVD_ENABLE -> DIODE_EN
- TP27 pad 1: /Main Diode ORs/Ideal Diode2/DIODE_EN -> DIODE_EN
- TP28 pad 1: /Main Diode ORs/Ideal Diode3/DIODE_EN -> DIODE_EN
- TP29 pad 1: /Main Diode ORs/Ideal Diode1/DIODE_VOUT -> /Main Diode ORs/12V_FUSED
- TP40 pad 1: /Ouput/LVC_V -> /LV_V
- U1 pad 3: /Supp Input/CC Buck/CHG_PG -> /CHG_PG
- U1 pad 4: /Supp Input/CC Buck/CHG_CC -> /CHG_CC
- U13 pad 15: /MCU/HV_VICOR_TEMP -> /HV_DCDC_TEMP
- U13 pad 16: /MCU/SUPP_I -> /SUPP_I
- U13 pad 17: /MCU/SUPP_V -> /SUPP_V
- U13 pad 18: /MCU/HSS_SNS -> /HSS_SNS
- U13 pad 2: /MCU/CHG_PG -> /CHG_PG
- U13 pad 25: /MCU/HV_IN_I -> /HV_IN_I
- U13 pad 26: /MCU/HV_IN_V -> /HV_IN_V
- U13 pad 27: /MCU/HV_OUT_I -> /HV_OUT_I
- U13 pad 28: /MCU/HV_OUT_V -> /HV_OUT_V
- U13 pad 3: /MCU/CHG_CC -> /CHG_CC
- U13 pad 32: /MCU/LV_ISNS -> /LV_I
- U13 pad 33: /MCU/LV_VSNS -> /LV_V
- U13 pad 65: /MCU/DI_MODE -> /DI_MODE
- U13 pad 66: /MCU/LIMP_HOME -> /LIMP_HOME
- U13 pad 78: /MCU/I2C_SCL -> /Fans/I2C_SDA
- U13 pad 91: /MCU/MISO -> /MISO
- U13 pad 96: /MCU/I2C_SCL -> /Fans/I2C_SCL
- U14 pad 1: /Fans/FAN_SDA -> /Fans/I2C_SDA
- U14 pad 2: /Fans/FAN_SCL -> /Fans/I2C_SCL
Routing:
- net Net-(D43-A2): track 13.5 -> 0.00 mm
- net /MCU/STM32G491VET/NRST: track 12.2 -> 0.00 mm
- net /MCU/STM32G491VET/BOOT0: track 5.58 -> 0.00 mm
- net +3V3: track 4.52 -> 0.00 mm
- net /12V -> 3.3V/12V -> 5V Buck Converter/CB: track 0.00 -> 2.46 mm
- net Net-(D45-K): track 1.77 -> 0.00 mm
- added copper zone on F.Cu, net /12V -> 3.3V/12V -> 5V Buck Converter/FB
- added copper zone on F.Cu, net /12V -> 3.3V/12V -> 5V Buck Converter/SW
- added copper zone on F.Cu, net /12V -> 3.3V/12V -> 5V Buck Converter/V_out_5V
- added copper zone on F.Cu, net /12V -> 3.3V/12V_IN
- added copper zone on F.Cu, net /Main Diode ORs/12V_FUSED
- added copper zone on F.Cu, net /Supp Input/Ideal Diode1/SRC
- added copper zone on F.Cu, net Net-(D35-K)
- removed copper zone on F.Cu, net /Main Diode ORs/Ideal Diode1/DIODE_VOUT
Other:
- board text removed: "For Instructional Use Only."
- board text removed: "SOLIDWORKS Educational Product."

Commit message: save
Parts:
- removed C114, C72: 1000u, Capacitor_SMD:CP_Elec_10x12.5
- removed TP17, TP18: LV_GND, TestPoint:TestPoint_THTPad_D3.0mm_Drill1.5mm
- removed TP22: Earf, TestPoint:TestPoint_THTPad_D3.0mm_Drill1.5mm
- removed TP27: PS_DIODE_EN, TestPoint:TestPoint_Loop_D2.50mm_Drill1.0mm_LowProfile
- removed TP28: HV_DIODE_EN, TestPoint:TestPoint_Loop_D2.50mm_Drill1.0mm_LowProfile
- removed TP33: 12V_IN, TestPoint:TestPoint_THTPad_D3.0mm_Drill1.5mm
- removed TP34: HSS_IN, TestPoint:TestPoint_THTPad_D3.0mm_Drill1.5mm
- removed TP36: 12V_OUT, TestPoint:TestPoint_THTPad_D3.0mm_Drill1.5mm
- C12, C32, C33, C34, C35, C36, R10, R11, R43, R61, R66, R67, R68, R77, R78, R8, R9: moved to F.Cu
- C30, C56, C81, D14, D37, Q7, R100, R12, R123, R124, R125, R126, R127, R13, R18, R19, R21, R22, R31, R32, R33, R34, R56, R58, R59, R60, R81, R82, R96, R97, R98: moved to B.Cu
- D15: value HV24V_LED -> DIODE_VOUT_LED
- moved R126 534.7 mm to (-161.0, -48.5)
- moved R127 531.5 mm to (-157.7, -41.6)
- moved R123 531.5 mm to (-157.7, -52.7)
- moved D41 530.3 mm to (-161.0, -50.0)
- moved R125 527.1 mm to (-153.3, -46.2), turned to 180 degrees
- moved D42 527.1 mm to (-157.7, -43.2)
- moved D38 527.0 mm to (-157.7, -54.2)
- moved R122 527.0 mm to (-153.3, -56.9)
- moved D37 522.7 mm to (-153.3, -55.3)
- moved D40 522.7 mm to (-153.3, -47.7)
- moved R124 522.1 mm to (-148.4, -52.1)
- moved D39 517.7 mm to (-148.4, -53.7)
- moved J16 299.0 mm to (-164.7, 68.0)
- moved R144 299.0 mm to (-162.7, 67.5)
- moved R82 269.5 mm to (-117.7, 64.9)
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Routing:
- net Net-(U13-PF1-OSC_OUT): track 0.00 -> 8.75 mm
- net Net-(U13-PF0-OSC_IN): track 0.00 -> 8.72 mm
- net Net-(IC4-VCP): track 5.74 -> 0.00 mm
- net /Main Diode ORs/Ideal Diode1/VIN: track 0.00 -> 5.74 mm
- net +3V3: track 0.00 -> 4.89 mm, vias 0 -> 3
- net /HV Input/HV -> 12V/Voltage + Current Sense/VOUT: track 0.00 -> 2.42 mm, vias 0 -> 1
- net /Ouput/Voltage + Current Sense/VOUT: track 0.00 -> 2.42 mm, vias 0 -> 1
- net /Supp Input/Voltage + Current Sense/VOUT: track 0.00 -> 2.42 mm, vias 0 -> 1
- net /HV_OUT_V: track 0.00 -> 1.56 mm
- net /LV_V: track 0.00 -> 1.56 mm
- net /SUPP_V: track 0.00 -> 1.56 mm
- net LV_GND: track 0.00 -> 1.32 mm
- net /Supp Input/SUPP_FUSED: track 0.00 -> 1.20 mm, vias 0 -> 1
- net /Main Diode ORs/12V_FUSED: track 0.00 -> 1.20 mm, vias 0 -> 1
- net /HV Input/HV -> 12V/OUT+: track 0.00 -> 1.20 mm, vias 0 -> 1
Other:
- board outline added: 145.3 x 92.4 mm
