File: hardware/HV_protection.kicad_sch (KiCad schematic)
At the start: 37 parts, among them J9 HV_IN, U3 TMCS1107A3BQDR, U4 AMC3330, U5 TLV6001DCK

Commit message: addressed
Parts:
- R34, R39: LSCS P/N C23162 -> (none)
Changed lines of the file:
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@@
-			)
-		)
-		(property "LSCS P/N" "C23162"
-			(at 241.3 57.15 90)
-			(hide yes)
-			(show_name no)
-			(do_not_autoplace no)
-			(effects
-				(font
-					(size 1.27 1.27)
-				)
 			)
 		)
@@
 			(at 195.58 57.15 90)
 			(hide yes)
-			(show_name no)
-			(do_not_autoplace no)
-			(effects
-				(font
-					(size 1.27 1.27)
-				)
-			)
-		)
-		(property "LSCS P/N" "C23162"
-			(at 195.58 57.15 90)
-			(hide yes)

Commit message: update kicad sharepoint
Parts:
- added TP54: LV_GND, TestPoint:TestPoint_THTPad_D3.0mm_Drill1.5mm, symbol Connector:TestPoint
- C15: LCSC P/N C1636 -> C14663
- C19: LCSC P/N C1622 -> C62774
- J9: footprint LHRS_Connectors:105313-2102 -> LHRS_Connectors:AMASS_XT30UPB-M_1x02_P5.0mm_Vertical
Connections:
- net LV_GND: now also TP54.1
Other:
- moved on the sheet: TP10, TP11, TP12, TP13

Commit message: sorry im omw
Parts:
- TP10, TP11: footprint TestPoint:TestPoint_THTPad_D3.0mm_Drill1.5mm -> TestPoint:TestPoint_Loop_D2.50mm_Drill1.0mm_LowProfile
Changed lines of the file:
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@@
 			)
 		)
-		(property "Footprint" "TestPoint:TestPoint_THTPad_D3.0mm_Drill1.5mm"
+		(property "Footprint" "TestPoint:TestPoint_Loop_D2.50mm_Drill1.0mm_LowProfile"
 			(at 217.17 27.94 0)
 			(hide yes)
@@
 			)
 		)
-		(property "Footprint" "TestPoint:TestPoint_THTPad_D3.0mm_Drill1.5mm"
+		(property "Footprint" "TestPoint:TestPoint_Loop_D2.50mm_Drill1.0mm_LowProfile"
 			(at 229.87 27.94 0)
 			(hide yes)

Commit message: craigenyah
Parts:
- renumbered C8 to C32, C9 to C33, C10 to C34, C11 to C35, C12 to C36, C13 to C37, C14 to C38, C15 to C39, C16 to C40, C17 to C41, C19 to C42, C18 to C43, C20 to C44, D11 to D12, F8 to F4, J9 to J5, R27 to R38, R28 to R39, R29 to R40, R30 to R41, R31 to R42, R32 to R43, R33 to R44, R34 to R45, R35 to R46, R36 to R47, R38 to R48, R37 to R49, R39 to R50, TP9 to TP13, TP10 to TP14, TP11 to TP15, TP12 to TP16, TP13 to TP17, TP54 to TP18, U3 to U4, U4 to U5, U5 to U6

Commit message: save
Parts:
- removed TP17, TP18: LV_GND, TestPoint:TestPoint_THTPad_D3.0mm_Drill1.5mm, symbol Connector:TestPoint
Changed lines of the file:
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@@
-		)
-	)
-	(hierarchical_label "LV_GND"
-		(shape passive)
-		(at 250.19 27.94 270)
-		(effects
-			(font
-				(size 1.27 1.27)
-			)
-			(justify right)
 		)
 	)
@@
 			)
 			(justify left)
-		)
-	)
-	(hierarchical_label "LV_GND"
-		(shape passive)
-		(at 262.89 27.94 270)
-		(effects
-			(font
-				(size 1.27 1.27)
-			)
-			(justify right)
 		)
 	)
@@
 	)
 	(symbol
-		(lib_id "Connector:TestPoint")
-		(at 250.19 27.94 0)
-		(unit 1)
-		(body_style 1)
-		(exclude_from_sim no)
-		(in_bom yes)
-		(on_board yes)
-		(in_pos_files yes)
-		(dnp no)
-		(fields_autoplaced yes)
-		(property "Reference" "TP17"
-			(at 252.73 23.3679 0)
-			(show_name no)
-			(do_not_autoplace no)
-			(effects
-				(font
-					(size 1.27 1.27)
-				)
-				(justify left)
-			)
-		)
-		(property "Value" "LV_GND"
-			(at 252.73 25.9079 0)
-			(show_name no)
-			(do_not_autoplace no)
-			(effects
-				(font
-					(size 1.27 1.27)
-				)
-				(justify left)
-			)
-		)
-		(property "Footprint" "TestPoint:TestPoint_THTPad_D3.0mm_Drill1.5mm"
-			(at 255.27 27.94 0)
-			(hide yes)
-			(show_name no)
-			(do_not_autoplace no)
-			(effects
-				(font
-					(size 1.27 1.27)
-				)
-			)
-		)
-		(property "Datasheet" ""
-			(at 255.27 27.94 0)
-			(hide yes)
-			(show_name no)
-			(do_not_autoplace no)
-			(effects
-				(font
-					(size 1.27 1.27)
-				)
-			)
-		)
-		(property "Description" "test point"
-			(at 250.19 27.94 0)
-			(hide yes)
-			(show_name no)
-			(do_not_autoplace no)
-			(effects
-				(font
-					(size 1.27 1.27)
-				)
-			)
-		)
-		(property "LCSC" ""
-			(at 250.19 27.94 0)
-			(hide yes)
-			(show_name no)
-			(do_not_autoplace no)
-			(effects
-				(font
-					(size 1.27 1.27)
-				)
-			)
-		)
-		(pin "1"
-		)
-		(instances
-			(project "PS-LVCarrier"
-				(path "/9bab2d9d-20f3-40ef-8545-e1299efec47e/4f26e4eb-a337-4f9d-865d-e2c0801c36ac/22cc1fb0-4176-4c01-b88e-6af93ab0f3a2"
-					(reference "TP17")
-					(unit 1)
-				)
-			)
-		)
-	)
-	(symbol
 		(lib_id "Device:R")
 		(at 87.63 134.62 0)
@@
 					(unit 1)
 				)
-			)
-		)
-	)
-	(symbol
-		(lib_id "Connector:TestPoint")
-		(at 262.89 27.94 0)
-		(unit 1)
-		(body_style 1)
-		(exclude_from_sim no)
-		(in_bom yes)
-		(on_board yes)
-		(in_pos_files yes)
-		(dnp no)
-		(fields_autoplaced yes)
-		(property "Reference" "TP18"
-			(at 265.43 23.3679 0)
-			(show_name no)
-			(do_not_autoplace no)
-			(effects
-				(font
-					(size 1.27 1.27)
-				)
-				(justify left)
-			)
-		)
-		(property "Value" "LV_GND"
-			(at 265.43 25.9079 0)
-			(show_name no)
-			(do_not_autoplace no)
-			(effects
-				(font
-					(size 1.27 1.27)
-				)
-				(justify left)
-			)
-		)
-		(property "Footprint" "TestPoint:TestPoint_THTPad_D3.0mm_Drill1.5mm"
-			(at 267.97 27.94 0)
-			(hide yes)
-			(show_name no)
-			(do_not_autoplace no)
-			(effects
-				(font
-					(size 1.27 1.27)
-				)
-			)
-		)
-		(property "Datasheet" ""
-			(at 267.97 27.94 0)
-			(hide yes)
-			(show_name no)
-			(do_not_autoplace no)
-			(effects
-				(font
-					(size 1.27 1.27)
-				)
-			)
-		)
-		(property "Description" "test point"
-			(at 262.89 27.94 0)
-			(hide yes)
-			(show_name no)
-			(do_not_autoplace no)
-			(effects
-				(font
-					(size 1.27 1.27)
-				)
-			)
-		)
-		(property "LCSC" ""
-			(at 262.89 27.94 0)
-			(hide yes)
-			(show_name no)
-			(do_not_autoplace no)
-			(effects
-				(font
-					(size 1.27 1.27)
-				)
-			)
-		)
-		(pin "1"
-		)
-		(instances
-			(project "PS-LVCarrier"
-				(path "/9bab2d9d-20f3-40ef-8545-e1299efec47e/4f26e4eb-a337-4f9d-865d-e2c0801c36ac/22cc1fb0-4176-4c01-b88e-6af93ab0f3a2"
-					(reference "TP18")
-					(unit 1)
-				)

Commit message: switch, stll working
Parts:
- TP13, TP16: footprint TestPoint:TestPoint_THTPad_D3.0mm_Drill1.5mm -> TestPoint:TestPoint_Loop_D2.50mm_Drill1.0mm_LowProfile
Changed lines of the file:
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@@
 			)
 		)
-		(property "Footprint" "TestPoint:TestPoint_THTPad_D3.0mm_Drill1.5mm"
+		(property "Footprint" "TestPoint:TestPoint_Loop_D2.50mm_Drill1.0mm_LowProfile"
 			(at 195.58 27.94 0)
 			(hide yes)
@@
 			)
 		)
-		(property "Footprint" "TestPoint:TestPoint_THTPad_D3.0mm_Drill1.5mm"
+		(property "Footprint" "TestPoint:TestPoint_Loop_D2.50mm_Drill1.0mm_LowProfile"
 			(at 242.57 27.94 0)
 			(hide yes)

Commit message: switch to laptop
Parts:
- F4: footprint LHRS_Power:Fuse-3557-2 -> LHRS_Power:HV-Fuse
Changed lines of the file:
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@@
 			)
 		)
-		(property "Footprint" "LHRS_Power:Fuse-3557-2"
+		(property "Footprint" "LHRS_Power:HV-Fuse"
 			(at 72.39 50.038 90)
 			(hide yes)

Commit message: switch to pc...
Connections:
- net DCDC_IN renamed LDO_OUT
Changed lines of the file:
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@@
 		(color 0 0 0 0)
 	)
-	(junction
-		(at 114.3 167.64)
-		(diameter 0)
-		(color 0 0 0 0)
-	)
 	(bus_entry
 		(at 252.73 60.96)
@@
 	(wire
 		(pts
-			(xy 111.76 167.64) (xy 114.3 167.64)
-		)
-		(stroke
-			(width 0)
-			(type default)
-		)
-	)
-	(wire
-		(pts
 			(xy 129.54 130.81) (xy 144.78 130.81)
 		)
@@
 		)
 	)
+	(wire
+		(pts
+			(xy 132.08 105.41) (xy 132.08 111.76)
+		)
+		(stroke
+			(width 0)
+			(type default)
+		)
+	)
 	(bus
 		(pts
@@
 	(wire
 		(pts
-			(xy 114.3 167.64) (xy 116.84 167.64)
-		)
-		(stroke
-			(width 0)
-			(type default)
-		)
-	)
-	(wire
-		(pts
 			(xy 224.79 127) (xy 238.76 127)
 		)
@@
 		)
 	)
-	(label "DCDC_IN"
-		(at 132.08 111.76 0)
-		(effects
-			(font
-				(size 1.27 1.27)
-			)
-			(justify left bottom)
-		)
-	)
 	(label "HV_IN_V"
 		(at 207.01 60.96 180)
@@
 	)
 	(label "LDO_OUT"
-		(at 111.76 167.64 180)
+		(at 114.3 167.64 180)
 		(effects
 			(font
@@
 		(effects
 			(font
-				(size 1.27 1.27)
-			)
-			(justify left bottom)
-		)
-	)
-	(label "DCDC_IN"
-		(at 116.84 167.64 0)
-		(effects
-			(font
