File: hardware/idealdiode.kicad_sch (KiCad schematic)
At the start: 9 parts, among them IC9 AP74502QTA8-7, Q21 NVMFWS1D7N04XMT1G, Q22 NVMFWS1D7N04XMT1G

Commit message: addressed
Parts:
- C115: renamed from C93; LSCS P/N C15849 -> (none)
- C117: renamed from C95; LSCS P/N C15849 -> (none)
- D34: renamed from D30; LSCS P/N C78419 -> (none)
- IC12: renamed from IC9; LSCS P/N C48989247 -> (none)
- Q27: renamed from Q21; LSCS P/N C133142 -> (none)
- Q29: renamed from Q22; LSCS P/N C133142 -> (none)
- renumbered C94 to C116, TP37 to TP43, TP38 to TP44

Commit message: try smth on laptop
Parts:
- added C51: 47u, Capacitor_SMD:C_0603_1608Metric_Pad1.08x0.95mm_HandSolder, symbol Device:C
- IC12: value AP74502QTA8-7 -> AP74502HQTA8-7
Connections:
- net DIODE_VIN: now also C51.1
- net LV_GND: now also C51.2
Other:
- moved on the sheet: C115, C116, C117, D34, IC12, Q27, Q29

Commit message: update kicad sharepoint
Parts:
- removed TP44: DIODE_VOUT, symbol Connector:TestPoint
- added D19: ORB_IN, LED_SMD:LED_0603_1608Metric_Pad1.05x0.95mm_HandSolder, symbol Device:LED
- added R54: 10k, Resistor_SMD:R_0603_1608Metric_Pad0.98x0.95mm_HandSolder, symbol Device:R
- C115, C117: LCSC P/N (none) -> C22387800
Connections:
- net DIODE_VIN: now also R54.1
- net LV_GND: now also D19.1 (K)
- new net: D19.2 (A), R54.2

Commit message: sorry im omw
Parts:
- C115, C117: value 1 uF -> 1u; LCSC P/N C22387800 -> C15849
- TP43: footprint (none) -> TestPoint:TestPoint_THTPad_D3.0mm_Drill1.5mm
Changed lines of the file:
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@@
 			)
 		)
-		(property "Value" "1 uF"
+		(property "Value" "1u"
 			(at 64.77 59.6899 0)
 			(show_name no)
@@
 			)
 		)
-		(property "LCSC P/N" "C22387800"
+		(property "LCSC P/N" "C15849"
 			(at 60.96 58.42 0)
 			(hide yes)
@@
 			)
 		)
-		(property "Value" "1 uF"
+		(property "Value" "1u"
 			(at 151.13 58.4199 0)
 			(show_name no)
@@
 			)
 		)
-		(property "LCSC P/N" "C22387800"
+		(property "LCSC P/N" "C15849"
 			(at 147.32 57.15 0)
 			(hide yes)
@@
 			)
 		)
-		(property "Footprint" ""
+		(property "Footprint" "TestPoint:TestPoint_THTPad_D3.0mm_Drill1.5mm"
 			(at 40.64 115.57 0)
 			(hide yes)

Commit message: craigenyah
Parts:
- renumbered C51 to C1, C115 to C2, C116 to C3, C117 to C4, D19 to D4, D34 to D5, IC12 to IC1, Q27 to Q3, Q29 to Q4, R54 to R16, TP43 to TP3

Commit message: switch, stll working
Parts:
- TP3: footprint TestPoint:TestPoint_THTPad_D3.0mm_Drill1.5mm -> TestPoint:TestPoint_Loop_D2.50mm_Drill1.0mm_LowProfile
Changed lines of the file:
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@@
 			)
 		)
-		(property "Footprint" "TestPoint:TestPoint_THTPad_D3.0mm_Drill1.5mm"
+		(property "Footprint" "TestPoint:TestPoint_Loop_D2.50mm_Drill1.0mm_LowProfile"
 			(at 40.64 115.57 0)
 			(hide yes)

Commit message: switch to pc...
Changed lines of the file:
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@@
-		)
-	)
-	(label "VIN"
-		(at 138.43 80.01 180)
-		(effects
-			(font
-				(size 1.27 1.27)
-			)
-			(justify right bottom)
-		)
-	)
-	(label "VIN"
-		(at 72.39 53.34 0)
-		(effects
-			(font
-				(size 1.27 1.27)
-			)
-			(justify left bottom)
 		)
 	)
@@
 		)
 	)
+	(hierarchical_label "DIODE_VIN"
+		(shape input)
+		(at 138.43 80.01 0)
+		(effects
+			(font
+				(size 1.27 1.27)
+			)
+			(justify left)
+		)
+	)
