File: hardware/diodeors.kicad_sch (KiCad schematic)
At the start: 29 parts, among them Q33 IRLML0030, Q34 IRLML0030, Q35 IRLML0030

Commit message: update kicad sharepoint
Parts:
- added D30: HV24V_LED, LED_SMD:LED_0603_1608Metric_Pad1.05x0.95mm_HandSolder, symbol Device:LED
- added R83: 10k, Resistor_SMD:R_0603_1608Metric_Pad0.98x0.95mm_HandSolder, symbol Device:R
- added TP30, TP31, TP33: DIODE_EN, symbol Connector:TestPoint
- added TP38: LV_ENABLE, symbol Connector:TestPoint
- added TP42: DIODE_VOUT, symbol Connector:TestPoint
- C111: footprint (none) -> Capacitor_SMD:C_0603_1608Metric_Pad1.08x0.95mm_HandSolder; LCSC P/N (none) -> C14663
Connections:
- net Ideal Diode1/DIODE_VOUT: now also R83.1, TP42.1
- net Ideal Diode2/DIODE_EN: now also TP30.1
- net Ideal Diode3/DIODE_EN: now also TP31.1
- net LVD_ENABLE: now also TP33.1
- net LV_ENABLE: now also TP38.1
- net LV_GND: now also D30.1 (K)
- new net: D30.2 (A), R83.2
Other:
- moved on the sheet: F4

Commit message: sorry im omw
Parts:
- F4: footprint (none) -> LHRS_Power:Fuse-3557-2
- R113: LCSC P/N C21190 -> (none)
- TP30: value DIODE_EN -> PS_DIODE_EN; footprint (none) -> TestPoint:TestPoint_Loop_D2.50mm_Drill1.0mm_LowProfile
- TP31: value DIODE_EN -> HV_DIODE_EN; footprint (none) -> TestPoint:TestPoint_Loop_D2.50mm_Drill1.0mm_LowProfile
- TP33: value DIODE_EN -> SUPP_DIODE_EN; footprint (none) -> TestPoint:TestPoint_Loop_D2.50mm_Drill1.0mm_LowProfile
- TP38: value LV_ENABLE -> LV_EN_TP; footprint (none) -> TestPoint:TestPoint_Loop_D2.50mm_Drill1.0mm_LowProfile
- TP42: footprint (none) -> TestPoint:TestPoint_THTPad_D3.0mm_Drill1.5mm
Changed lines of the file:
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@@
 			)
 		)
-		(property "Footprint" ""
+		(property "Footprint" "LHRS_Power:Fuse-3557-2"
 			(at 198.12 56.388 90)
 			(hide yes)
@@
 			)
 		)
-		(property "Value" "DIODE_EN"
+		(property "Value" "SUPP_DIODE_EN"
 			(at 92.71 55.1179 0)
 			(show_name no)
@@
 			)
 		)
-		(property "Footprint" ""
+		(property "Footprint" "TestPoint:TestPoint_Loop_D2.50mm_Drill1.0mm_LowProfile"
 			(at 90.17 57.15 0)
 			(hide yes)
@@
 			)
 		)
-		(property "Footprint" ""
+		(property "Footprint" "TestPoint:TestPoint_THTPad_D3.0mm_Drill1.5mm"
 			(at 185.42 54.61 0)
 			(hide yes)
@@
 			)
 		)
-		(property "Value" "LV_ENABLE"
+		(property "Value" "LV_EN_TP"
 			(at 58.166 47.752 0)
 			(show_name no)
@@
 			)
 		)
-		(property "Footprint" ""
+		(property "Footprint" "TestPoint:TestPoint_Loop_D2.50mm_Drill1.0mm_LowProfile"
 			(at 52.07 53.34 0)
 			(hide yes)
@@
 			)
 		)
-		(property "LCSC P/N" "C21190"
+		(property "LCSC P/N" ""
 			(at 54.61 38.1 0)
 			(hide yes)
@@
 			)
 		)
-		(property "Value" "DIODE_EN"
+		(property "Value" "PS_DIODE_EN"
 			(at 92.71 100.8379 0)
 			(show_name no)
@@
 			)
 		)
-		(property "Footprint" ""
+		(property "Footprint" "TestPoint:TestPoint_Loop_D2.50mm_Drill1.0mm_LowProfile"
 			(at 90.17 102.87 0)
 			(hide yes)
@@
 			)
 		)
-		(property "Value" "DIODE_EN"
+		(property "Value" "HV_DIODE_EN"
 			(at 92.71 146.5579 0)
 			(show_name no)
@@
 			)
 		)
-		(property "Footprint" ""
+		(property "Footprint" "TestPoint:TestPoint_Loop_D2.50mm_Drill1.0mm_LowProfile"
 			(at 90.17 148.59 0)
 			(hide yes)

Commit message: craigenyah
Parts:
- renumbered C111 to C57, D30 to D15, D33 to D16, F4 to F6, Q33 to Q10, Q34 to Q11, Q35 to Q12, R113 to R61, R108 to R62, R152 to R63, R116 to R64, R153 to R65, R112 to R66, R151 to R67, R124 to R68, R109 to R69, R110 to R70, R117 to R71, R118 to R72, R111 to R73, R119 to R74, R6 to R75, R7 to R76, R4 to R77, R5 to R78, R8 to R79, R9 to R80, R83 to R81, R120 to R82, R121 to R83, R123 to R84, TP38 to TP25, TP33 to TP26, TP30 to TP27, TP31 to TP28, TP42 to TP29

Commit message: continue working soon
Parts:
- removed C57: 100n, Capacitor_SMD:C_0603_1608Metric_Pad1.08x0.95mm_HandSolder, symbol Device:C_Small
- removed D16: DISABLE_LED, LED_SMD:LED_0603_1608Metric_Pad1.05x0.95mm_HandSolder, symbol Device:LED
- removed F6: Fuse, LHRS_Power:Fuse-3557-2, symbol Device:Fuse
- removed Q10, Q11, Q12: IRLML0030, Package_TO_SOT_SMD:SOT-23, symbol Transistor_FET:IRLML0030
- removed R61: 470k, Resistor_SMD:R_0603_1608Metric_Pad0.98x0.95mm_HandSolder, symbol Device:R
- removed R62, R64, R66: 1k, Resistor_SMD:R_0603_1608Metric_Pad0.98x0.95mm_HandSolder, symbol Device:R
- removed R63, R65, R67, R73, R74: 100k, Resistor_SMD:R_0603_1608Metric_Pad0.98x0.95mm_HandSolder, symbol Device:R
- removed R68: 220k, Resistor_SMD:R_0603_1608Metric_Pad0.98x0.95mm_HandSolder, symbol Device:R
- removed R69, R70, R71, R72, R84: 10k, Resistor_SMD:R_0603_1608Metric_Pad0.98x0.95mm_HandSolder, symbol Device:R
- removed R82: 4.3k, Resistor_SMD:R_0603_1608Metric_Pad0.98x0.95mm_HandSolder, symbol Device:R
- removed R83: 33k, Resistor_SMD:R_0603_1608Metric_Pad0.98x0.95mm_HandSolder, symbol Device:R
- removed TP25: LV_EN_TP, TestPoint:TestPoint_Loop_D2.50mm_Drill1.0mm_LowProfile, symbol Connector:TestPoint
- added J16: Conn_01x02, Connector_PinHeader_1.00mm:PinHeader_1x02_P1.00mm_Vertical, symbol Connector_Generic:Conn_01x02
- added R144: 47k, Resistor_SMD:R_0603_1608Metric_Pad0.98x0.95mm_HandSolder, symbol Device:R
Connections:
- net Ideal Diode1/DIODE_VOUT is gone; now on net 12V_FUSED: R81.1, TP29.1
- net Ideal Diode3/DIODE_EN is gone; now on net DIODE_EN: TP28.1
- net LVD_ENABLE is gone; now on net DIODE_EN: TP26.1
- net PS_12V_FUSED: now also J16.2 (Pin_2)
- net Ideal Diode2/DIODE_EN renamed DIODE_EN
- net DIODE_EN: now also R144.2
- new net: J16.1 (Pin_1), R144.1
Other:
- note removed: "12.6V × 10/43 = 2.93V"
- note removed: "LEVEL SHIFTER (for mcu signal) 12->3.3V"

Commit message: save
Parts:
- removed TP27: PS_DIODE_EN, TestPoint:TestPoint_Loop_D2.50mm_Drill1.0mm_LowProfile, symbol Connector:TestPoint
- removed TP28: HV_DIODE_EN, TestPoint:TestPoint_Loop_D2.50mm_Drill1.0mm_LowProfile, symbol Connector:TestPoint
- D15: value HV24V_LED -> DIODE_VOUT_LED
Changed lines of the file:
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@@
-	)
-	(junction
-		(at 95.25 148.59)
-		(diameter 0)
-		(color 0 0 0 0)
 	)
 	(junction
@@
 		(color 0 0 0 0)
 	)
-	(junction
-		(at 95.25 102.87)
-		(diameter 0)
-		(color 0 0 0 0)
-	)
 	(wire
 		(pts
@@
 	(wire
 		(pts
-			(xy 95.25 148.59) (xy 107.95 148.59)
-		)
-		(stroke
-			(width 0)
-			(type default)
-		)
-	)
-	(wire
-		(pts
 			(xy 172.72 54.61) (xy 180.34 54.61)
 		)
@@
 	(wire
 		(pts
-			(xy 71.12 102.87) (xy 95.25 102.87)
-		)
-		(stroke
-			(width 0)
-			(type default)
-		)
-	)
-	(wire
-		(pts
 			(xy 95.25 71.12) (xy 95.25 69.85)
 		)
@@
 	(wire
 		(pts
-			(xy 71.12 148.59) (xy 95.25 148.59)
+			(xy 71.12 148.59) (xy 107.95 148.59)
 		)
 		(stroke
@@
 	(wire
 		(pts
-			(xy 95.25 102.87) (xy 107.95 102.87)
+			(xy 71.12 102.87) (xy 107.95 102.87)
 		)
 		(stroke
@@
 			)
 		)
-		(property "Value" "HV24V_LED"
+		(property "Value" "DIODE_VOUT_LED"
 			(at 184.15 70.1674 90)
 			(show_name no)
@@
 				(path "/9bab2d9d-20f3-40ef-8545-e1299efec47e/1bb70e84-a5b9-4a48-ae28-663d6ef6e6b1"
 					(reference "D15")
-					(unit 1)
-				)
-			)
-		)
-	)
-	(symbol
-		(lib_id "Connector:TestPoint")
-		(at 95.25 102.87 0)
-		(mirror y)
-		(unit 1)
-		(body_style 1)
-		(exclude_from_sim no)
-		(in_bom yes)
-		(on_board yes)
-		(in_pos_files yes)
-		(dnp no)
-		(property "Reference" "TP27"
-			(at 92.71 98.2979 0)
-			(show_name no)
-			(do_not_autoplace no)
-			(effects
-				(font
-					(size 1.27 1.27)
-				)
-				(justify left)
-			)
-		)
-		(property "Value" "PS_DIODE_EN"
-			(at 92.71 100.8379 0)
-			(show_name no)
-			(do_not_autoplace no)
-			(effects
-				(font
-					(size 1.27 1.27)
-				)
-				(justify left)
-			)
-		)
-		(property "Footprint" "TestPoint:TestPoint_Loop_D2.50mm_Drill1.0mm_LowProfile"
-			(at 90.17 102.87 0)
-			(hide yes)
-			(show_name no)
-			(do_not_autoplace no)
-			(effects
-				(font
-					(size 1.27 1.27)
-				)
-			)
-		)
-		(property "Datasheet" ""
-			(at 90.17 102.87 0)
-			(hide yes)
-			(show_name no)
-			(do_not_autoplace no)
-			(effects
-				(font
-					(size 1.27 1.27)
-				)
-			)
-		)
-		(property "Description" "test point"
-			(at 95.25 102.87 0)
-			(hide yes)
-			(show_name no)
-			(do_not_autoplace no)
-			(effects
-				(font
-					(size 1.27 1.27)
-				)
-			)
-		)
-		(property "LCSC" ""
-			(at 95.25 102.87 0)
-			(hide yes)
-			(show_name no)
-			(do_not_autoplace no)
-			(effects
-				(font
-					(size 1.27 1.27)
-				)
-			)
-		)
-		(pin "1"
-		)
-		(instances
-			(project "PS-LVCarrier"
-				(path "/9bab2d9d-20f3-40ef-8545-e1299efec47e/1bb70e84-a5b9-4a48-ae28-663d6ef6e6b1"
-					(reference "TP27")
 					(unit 1)
 				)
@@
 					(unit 1)
 				)
-			)
-		)
-	)
-	(symbol
-		(lib_id "Connector:TestPoint")
-		(at 95.25 148.59 0)
-		(mirror y)
-		(unit 1)
-		(body_style 1)
-		(exclude_from_sim no)
-		(in_bom yes)
-		(on_board yes)
-		(in_pos_files yes)
-		(dnp no)
-		(property "Reference" "TP28"
-			(at 92.71 144.0179 0)
-			(show_name no)
-			(do_not_autoplace no)
-			(effects
-				(font
-					(size 1.27 1.27)
-				)
-				(justify left)
-			)
-		)
-		(property "Value" "HV_DIODE_EN"
-			(at 92.71 146.5579 0)
-			(show_name no)
-			(do_not_autoplace no)
-			(effects
-				(font
-					(size 1.27 1.27)
-				)
-				(justify left)
-			)
-		)
-		(property "Footprint" "TestPoint:TestPoint_Loop_D2.50mm_Drill1.0mm_LowProfile"
-			(at 90.17 148.59 0)
-			(hide yes)
-			(show_name no)
-			(do_not_autoplace no)
-			(effects
-				(font
-					(size 1.27 1.27)
-				)
-			)
-		)
-		(property "Datasheet" ""
-			(at 90.17 148.59 0)
-			(hide yes)
-			(show_name no)
-			(do_not_autoplace no)
-			(effects
-				(font
-					(size 1.27 1.27)
-				)
-			)
-		)
-		(property "Description" "test point"
-			(at 95.25 148.59 0)
-			(hide yes)
-			(show_name no)
-			(do_not_autoplace no)
-			(effects
-				(font
-					(size 1.27 1.27)
-				)
-			)
-		)
-		(property "LCSC" ""
-			(at 95.25 148.59 0)
-			(hide yes)
-			(show_name no)
-			(do_not_autoplace no)
-			(effects
-				(font
-					(size 1.27 1.27)
-				)
-			)
-		)
-		(pin "1"
-		)
-		(instances
-			(project "PS-LVCarrier"
-				(path "/9bab2d9d-20f3-40ef-8545-e1299efec47e/1bb70e84-a5b9-4a48-ae28-663d6ef6e6b1"
-					(reference "TP28")
-					(unit 1)
-				)

Commit message: switch, stll working
Parts:
- TP29: footprint TestPoint:TestPoint_THTPad_D3.0mm_Drill1.5mm -> TestPoint:TestPoint_Loop_D2.50mm_Drill1.0mm_LowProfile
Changed lines of the file:
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@@
 			)
 		)
-		(property "Footprint" "TestPoint:TestPoint_THTPad_D3.0mm_Drill1.5mm"
+		(property "Footprint" "TestPoint:TestPoint_Loop_D2.50mm_Drill1.0mm_LowProfile"
 			(at 185.42 54.61 0)
 			(hide yes)

Commit message: switch to laptop
Parts:
- J16: value Conn_01x02 -> in the off chance no supp pwr
Other:
- moved on the sheet: J16, R144
Changed lines of the file:
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@@
 	(wire
 		(pts
-			(xy 158.75 38.1) (xy 160.02 38.1)
+			(xy 171.45 38.1) (xy 172.72 38.1)
 		)
 		(stroke
@@
 	(global_label "DIODE_EN"
 		(shape input)
-		(at 160.02 38.1 0)
+		(at 172.72 38.1 0)
 		(fields_autoplaced yes)
 		(effects
@@
 		)
 		(property "Intersheetrefs" "${INTERSHEET_REFS}"
-			(at 172.0766 38.1 0)
+			(at 184.7766 38.1 0)
 			(hide yes)
 			(show_name no)
@@
 	)
 	(hierarchical_label "LV_GND"
-		(shape input)
+		(shape passive)
 		(at 180.34 71.12 270)
 		(effects
@@
 	)
 	(hierarchical_label "LV_GND"
-		(shape input)
+		(shape passive)
 		(at 147.32 162.56 270)
 		(effects
@@
 	)
 	(hierarchical_label "LV_GND"
-		(shape input)
+		(shape passive)
 		(at 147.32 71.12 270)
 		(effects
@@
 	(hierarchical_label "PS_12V_FUSED"
 		(shape input)
-		(at 151.13 35.56 0)
+		(at 163.83 35.56 0)
 		(effects
 			(font
@@
 	)
 	(hierarchical_label "LV_GND"
-		(shape input)
+		(shape passive)
 		(at 147.32 116.84 270)
 		(effects
@@
 	(symbol
 		(lib_id "Connector_Generic:Conn_01x02")
-		(at 146.05 38.1 180)
+		(at 158.75 38.1 180)
 		(unit 1)
 		(body_style 1)
@@
 		(fields_autoplaced yes)
 		(property "Reference" "J16"
-			(at 146.05 29.21 0)
-			(show_name no)
-			(do_not_autoplace no)
-			(effects
-				(font
-					(size 1.27 1.27)
-				)
-			)
-		)
-		(property "Value" "Conn_01x02"
-			(at 146.05 31.75 0)
+			(at 158.75 29.21 0)
+			(show_name no)
+			(do_not_autoplace no)
+			(effects
+				(font
+					(size 1.27 1.27)
+				)
+			)
+		)
+		(property "Value" "in the off chance no supp pwr"
+			(at 158.75 31.75 0)
 			(show_name no)
 			(do_not_autoplace no)
@@
 		)
 		(property "Footprint" "Connector_PinHeader_1.00mm:PinHeader_1x02_P1.00mm_Vertical"
-			(at 146.05 38.1 0)
+			(at 158.75 38.1 0)
 			(hide yes)
 			(show_name no)
@@
 		)
 		(property "Datasheet" ""
-			(at 146.05 38.1 0)
+			(at 158.75 38.1 0)
 			(hide yes)
 			(show_name no)
@@
 		)
 		(property "Description" "Generic connector, single row, 01x02, script generated (kicad-library-utils/schlib/autogen/connector/)"
-			(at 146.05 38.1 0)
+			(at 158.75 38.1 0)
 			(hide yes)
 			(show_name no)
@@
 	(symbol
 		(lib_id "Device:R")
-		(at 154.94 38.1 90)
+		(at 167.64 38.1 90)
 		(unit 1)
 		(body_style 1)
@@
 		(dnp no)
 		(property "Reference" "R144"
-			(at 152.654 40.894 90)
+			(at 165.354 40.894 90)
 			(show_name no)
 			(do_not_autoplace no)
@@
 		)
 		(property "Value" "47k"
-			(at 152.654 43.2054 90)
+			(at 165.354 43.2054 90)
 			(show_name no)
 			(do_not_autoplace no)
@@
 		)
 		(property "Footprint" "Resistor_SMD:R_0603_1608Metric_Pad0.98x0.95mm_HandSolder"
-			(at 154.94 39.878 90)
+			(at 167.64 39.878 90)
 			(hide yes)
 			(show_name no)
@@
 		)
 		(property "Datasheet" "https://www.mouser.com/ProductDetail/Vishay/CRCW06031K00FKEI?qs=%252B6g0mu59x7LmDUigK4duvw%3D%3D&srsltid=AfmBOoq-qbpfAjzhtzCNjmKpq35FQ1BHTaIyFUz28_1v8HZaKbIrwYgN"
-			(at 154.94 38.1 0)
+			(at 167.64 38.1 0)
 			(hide yes)
 			(show_name no)
@@
 		)
 		(property "Description" "Resistor"
-			(at 154.94 38.1 0)
+			(at 167.64 38.1 0)
 			(hide yes)
 			(show_name no)
@@
 		)
 		(property "P/N" "CRCW06031K00FKEI "
-			(at 154.94 38.1 0)
+			(at 167.64 38.1 0)
 			(hide yes)
 			(show_name no)
@@
 		)
 		(property "Assemble" "Y"
-			(at 154.94 38.1 0)
+			(at 167.64 38.1 0)
 			(hide yes)
 			(show_name no)
@@
 		)
 		(property "LCSC P/N" ""
-			(at 154.94 38.1 0)
+			(at 167.64 38.1 0)
 			(hide yes)
 			(show_name no)
@@
 		)
 		(property "LCSC" ""
-			(at 154.94 38.1 0)
-			(hide yes)
-			(show_name no)
+			(at 167.64 38.1 0)
+			(hide yes)
+			(show_name no)

Commit message: oops
Parts:
- R144: LCSC P/N (none) -> C25819; P/N CRCW06031K00FKEI -> CRCW060347K0FKECC
Changed lines of the file:
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@@
 			)
 		)
-		(property "P/N" "CRCW06031K00FKEI "
+		(property "P/N" "CRCW060347K0FKECC"
 			(at 167.64 38.1 0)
 			(hide yes)
@@
 			)
 		)
-		(property "LCSC P/N" ""
+		(property "LCSC P/N" "C25819"
 			(at 167.64 38.1 0)
 			(hide yes)
