File: hardware/outputs.kicad_sch (KiCad schematic)
At the start: 28 parts, among them J4 BPS_12V, J5 PDU_12V

Commit message: craigenyah
Parts:
- renumbered C43 to C70, C58 to C71, C59 to C72, C60 to C73, C61 to C74, D39 to D23, D42 to D24, D40 to D25, D41 to D26, D1 to D27, F5 to F7, F6 to F8, F7 to F9, J5 to J10, J4 to J9, R85 to R88, R88 to R89, R86 to R90, R10 to R91, R11 to R92, R87 to R93, R12 to R94, TP46 to TP33, TP48 to TP34, TP37 to TP35, TP40 to TP36, TP50 to TP37, TP1 to TP38
Changed lines of the file:
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@@
 		(in_pos_files yes)
 		(dnp no)
-		(property "Reference" "TP37"
+		(property "Reference" "TP35"
 			(at 165.0083 59.182 0)
 			(show_name no)
@@
 			(project "PS-LVCarrier"
 				(path "/9bab2d9d-20f3-40ef-8545-e1299efec47e/10a2a81d-fff8-4091-b6ef-9685e4bd9514"
-					(reference "TP37")
+					(reference "TP35")
 					(unit 1)
 				)
@@
 		(dnp no)
 		(fields_autoplaced yes)
-		(property "Reference" "R12"
+		(property "Reference" "R94"
 			(at 228.6 73.6599 0)
 			(show_name no)
@@
 			(project "PS-LVCarrier"
 				(path "/9bab2d9d-20f3-40ef-8545-e1299efec47e/10a2a81d-fff8-4091-b6ef-9685e4bd9514"
-					(reference "R12")
+					(reference "R94")
 					(unit 1)
 				)
@@
 		(dnp no)
 		(fields_autoplaced yes)
-		(property "Reference" "D40"
+		(property "Reference" "D25"
 			(at 140.97 129.8574 90)
 			(show_name no)
@@
 			(project "PS-LVCarrier"
 				(path "/9bab2d9d-20f3-40ef-8545-e1299efec47e/10a2a81d-fff8-4091-b6ef-9685e4bd9514"
-					(reference "D40")
+					(reference "D25")
 					(unit 1)
 				)
@@
 		(dnp no)
 		(fields_autoplaced yes)
-		(property "Reference" "TP1"
+		(property "Reference" "TP38"
 			(at 228.6 65.2779 0)
 			(show_name no)
@@
 			(project "PS-LVCarrier"
 				(path "/9bab2d9d-20f3-40ef-8545-e1299efec47e/10a2a81d-fff8-4091-b6ef-9685e4bd9514"
-					(reference "TP1")
+					(reference "TP38")
 					(unit 1)
 				)
@@
 		(in_pos_files yes)
 		(dnp no)
-		(property "Reference" "C58"
+		(property "Reference" "C71"
 			(at 74.93 120.0149 0)
 			(show_name no)
@@
 			(project "PS-LVCarrier"
 				(path "/9bab2d9d-20f3-40ef-8545-e1299efec47e/10a2a81d-fff8-4091-b6ef-9685e4bd9514"
-					(reference "C58")
+					(reference "C71")
 					(unit 1)
 				)
@@
 		(dnp no)
 		(fields_autoplaced yes)
-		(property "Reference" "R85"
+		(property "Reference" "R88"
 			(at 49.53 73.6599 0)
 			(show_name no)
@@
 			(project "PS-LVCarrier"
 				(path "/9bab2d9d-20f3-40ef-8545-e1299efec47e/10a2a81d-fff8-4091-b6ef-9685e4bd9514"
-					(reference "R85")
+					(reference "R88")
 					(unit 1)
 				)
@@
 		(in_pos_files yes)
 		(dnp no)
-		(property "Reference" "R10"
+		(property "Reference" "R91"
 			(at 161.29 77.4699 0)
 			(show_name no)
@@
 			(project "PS-LVCarrier"
 				(path "/9bab2d9d-20f3-40ef-8545-e1299efec47e/10a2a81d-fff8-4091-b6ef-9685e4bd9514"
-					(reference "R10")
+					(reference "R91")
 					(unit 1)
 				)
@@
 		(dnp no)
 		(fields_autoplaced yes)
-		(property "Reference" "R88"
+		(property "Reference" "R89"
 			(at 137.16 78.7399 0)
 			(show_name no)
@@
 			(project "PS-LVCarrier"
 				(path "/9bab2d9d-20f3-40ef-8545-e1299efec47e/10a2a81d-fff8-4091-b6ef-9685e4bd9514"
-					(reference "R88")
+					(reference "R89")
 					(unit 1)
 				)
@@
 		(dnp no)
 		(fields_autoplaced yes)
-		(property "Reference" "R87"
+		(property "Reference" "R93"
 			(at 226.06 120.6499 0)
 			(show_name no)
@@
 			(project "PS-LVCarrier"
 				(path "/9bab2d9d-20f3-40ef-8545-e1299efec47e/10a2a81d-fff8-4091-b6ef-9685e4bd9514"
-					(reference "R87")
+					(reference "R93")
 					(unit 1)
 				)
@@
 		(dnp no)
 		(fields_autoplaced yes)
-		(property "Reference" "F7"
+		(property "Reference" "F9"
 			(at 219.71 63.5 90)
 			(show_name no)
@@
 			(project "PS-LVCarrier"
 				(path "/9bab2d9d-20f3-40ef-8545-e1299efec47e/10a2a81d-fff8-4091-b6ef-9685e4bd9514"
-					(reference "F7")
+					(reference "F9")
 					(unit 1)
 				)
@@
 		(dnp no)
 		(fields_autoplaced yes)
-		(property "Reference" "TP50"
+		(property "Reference" "TP37"
 			(at 226.06 112.2679 0)
 			(show_name no)
@@
 			(project "PS-LVCarrier"
 				(path "/9bab2d9d-20f3-40ef-8545-e1299efec47e/10a2a81d-fff8-4091-b6ef-9685e4bd9514"
-					(reference "TP50")
+					(reference "TP37")
 					(unit 1)
 				)
@@
 		(dnp no)
 		(fields_autoplaced yes)
-		(property "Reference" "TP46"
+		(property "Reference" "TP33"
 			(at 49.53 65.2779 0)
 			(show_name no)
@@
 			(project "PS-LVCarrier"
 				(path "/9bab2d9d-20f3-40ef-8545-e1299efec47e/10a2a81d-fff8-4091-b6ef-9685e4bd9514"
-					(reference "TP46")
+					(reference "TP33")
 					(unit 1)
 				)
@@
 		(in_pos_files yes)
 		(dnp no)
-		(property "Reference" "J4"
+		(property "Reference" "J9"
 			(at 254.508 116.84 0)
 			(show_name no)
@@
 			(project "PS-LVCarrier"
 				(path "/9bab2d9d-20f3-40ef-8545-e1299efec47e/10a2a81d-fff8-4091-b6ef-9685e4bd9514"
-					(reference "J4")
+					(reference "J9")
 					(unit 1)
 				)
@@
 		(dnp no)
 		(fields_autoplaced yes)
-		(property "Reference" "D41"
+		(property "Reference" "D26"
 			(at 227.33 129.8574 90)
 			(show_name no)
@@
 			(project "PS-LVCarrier"
 				(path "/9bab2d9d-20f3-40ef-8545-e1299efec47e/10a2a81d-fff8-4091-b6ef-9685e4bd9514"
-					(reference "D41")
+					(reference "D26")
 					(unit 1)
 				)
@@
 		(in_pos_files yes)
 		(dnp no)
-		(property "Reference" "C60"
+		(property "Reference" "C73"
 			(at 99.06 120.6499 0)
 			(show_name no)
@@
 			(project "PS-LVCarrier"
 				(path "/9bab2d9d-20f3-40ef-8545-e1299efec47e/10a2a81d-fff8-4091-b6ef-9685e4bd9514"
-					(reference "C60")
+					(reference "C73")
 					(unit 1)
 				)
@@
 		(dnp no)
 		(fields_autoplaced yes)
-		(property "Reference" "D1"
+		(property "Reference" "D27"
 			(at 229.87 82.8674 90)
 			(show_name no)
@@
 			(project "PS-LVCarrier"
 				(path "/9bab2d9d-20f3-40ef-8545-e1299efec47e/10a2a81d-fff8-4091-b6ef-9685e4bd9514"
-					(reference "D1")
+					(reference "D27")
 					(unit 1)
 				)
@@
 		(dnp no)
 		(fields_autoplaced yes)
-		(property "Reference" "D42"
+		(property "Reference" "D24"
 			(at 138.43 87.9474 90)
 			(show_name no)
@@
 			(project "PS-LVCarrier"
 				(path "/9bab2d9d-20f3-40ef-8545-e1299efec47e/10a2a81d-fff8-4091-b6ef-9685e4bd9514"
-					(reference "D42")
+					(reference "D24")
 					(unit 1)
 				)
@@
 		(in_pos_files yes)
 		(dnp no)
-		(property "Reference" "F5"
+		(property "Reference" "F7"
 			(at 127 72.898 90)
 			(show_name no)
@@
 			(project "PS-LVCarrier"
 				(path "/9bab2d9d-20f3-40ef-8545-e1299efec47e/10a2a81d-fff8-4091-b6ef-9685e4bd9514"
-					(reference "F5")
+					(reference "F7")
 					(unit 1)
 				)
@@
 		(in_pos_files yes)
 		(dnp no)
-		(property "Reference" "C59"
+		(property "Reference" "C72"
 			(at 87.63 120.0149 0)
 			(show_name no)
@@
 			(project "PS-LVCarrier"
 				(path "/9bab2d9d-20f3-40ef-8545-e1299efec47e/10a2a81d-fff8-4091-b6ef-9685e4bd9514"
-					(reference "C59")
+					(reference "C72")
 					(unit 1)
 				)
@@
 		(dnp no)
 		(fields_autoplaced yes)
-		(property "Reference" "D39"
+		(property "Reference" "D23"
 			(at 50.8 82.8674 90)
 			(show_name no)
@@
 			(project "PS-LVCarrier"
 				(path "/9bab2d9d-20f3-40ef-8545-e1299efec47e/10a2a81d-fff8-4091-b6ef-9685e4bd9514"
-					(reference "D39")
+					(reference "D23")
 					(unit 1)
 				)
@@
 		(in_pos_files yes)
 		(dnp no)
-		(property "Reference" "C43"
+		(property "Reference" "C70"
 			(at 62.23 120.0149 0)
 			(show_name no)
@@
 			(project "PS-LVCarrier"
 				(path "/9bab2d9d-20f3-40ef-8545-e1299efec47e/10a2a81d-fff8-4091-b6ef-9685e4bd9514"
-					(reference "C43")
+					(reference "C70")
 					(unit 1)
 				)
@@
 		(dnp no)
 		(fields_autoplaced yes)
-		(property "Reference" "TP48"
+		(property "Reference" "TP34"
 			(at 139.7 112.2679 0)
 			(show_name no)
@@
 			(project "PS-LVCarrier"
 				(path "/9bab2d9d-20f3-40ef-8545-e1299efec47e/10a2a81d-fff8-4091-b6ef-9685e4bd9514"
-					(reference "TP48")
+					(reference "TP34")
 					(unit 1)
 				)
@@
 		(in_pos_files yes)
 		(dnp no)
-		(property "Reference" "C61"
+		(property "Reference" "C74"
 			(at 110.49 120.6499 0)
 			(show_name no)
@@
 			(project "PS-LVCarrier"
 				(path "/9bab2d9d-20f3-40ef-8545-e1299efec47e/10a2a81d-fff8-4091-b6ef-9685e4bd9514"
-					(reference "C61")
+					(reference "C74")
 					(unit 1)
 				)
@@
 		(in_pos_files yes)
 		(dnp no)
-		(property "Reference" "R11"
+		(property "Reference" "R92"
 			(at 162.052 87.7316 0)
 			(show_name no)
@@
 			(project "PS-LVCarrier"
 				(path "/9bab2d9d-20f3-40ef-8545-e1299efec47e/10a2a81d-fff8-4091-b6ef-9685e4bd9514"
-					(reference "R11")
+					(reference "R92")
 					(unit 1)
 				)
@@
 		(in_pos_files yes)
 		(dnp no)
-		(property "Reference" "TP40"
+		(property "Reference" "TP36"
 			(at 214.376 61.722 0)
 			(show_name no)
@@
 			(project "PS-LVCarrier"
 				(path "/9bab2d9d-20f3-40ef-8545-e1299efec47e/10a2a81d-fff8-4091-b6ef-9685e4bd9514"
-					(reference "TP40")
+					(reference "TP36")
 					(unit 1)
 				)
@@
 		(in_pos_files yes)
 		(dnp no)
-		(property "Reference" "F6"
+		(property "Reference" "F8"
 			(at 215.646 111.506 90)
 			(show_name no)
@@
 			(project "PS-LVCarrier"
 				(path "/9bab2d9d-20f3-40ef-8545-e1299efec47e/10a2a81d-fff8-4091-b6ef-9685e4bd9514"
-					(reference "F6")
+					(reference "F8")
 					(unit 1)
 				)
@@
 		(in_pos_files yes)
 		(dnp no)
-		(property "Reference" "J5"
+		(property "Reference" "J10"
 			(at 257.048 69.85 0)
 			(show_name no)
@@
 			(project "PS-LVCarrier"
 				(path "/9bab2d9d-20f3-40ef-8545-e1299efec47e/10a2a81d-fff8-4091-b6ef-9685e4bd9514"
-					(reference "J5")
+					(reference "J10")
 					(unit 1)
 				)
@@
 		(dnp no)
 		(fields_autoplaced yes)
-		(property "Reference" "R86"
+		(property "Reference" "R90"
 			(at 139.7 120.6499 0)
 			(show_name no)
@@
 			(project "PS-LVCarrier"
 				(path "/9bab2d9d-20f3-40ef-8545-e1299efec47e/10a2a81d-fff8-4091-b6ef-9685e4bd9514"
-					(reference "R86")
+					(reference "R90")
 					(unit 1)
 				)

Commit message: continue working soon
Parts:
- removed F8: TBD, LHRS_Power:Fuse-3557-2, symbol Device:Fuse
- added C114: 1000u, Capacitor_SMD:CP_Elec_10x12.5, symbol Device:C_Polarized_US
Connections:
- net 12V_FUSED: now also C114.1
- net LV_GND: now also C114.2

Commit message: save
Parts:
- removed C114, C72: 1000u, Capacitor_SMD:CP_Elec_10x12.5, symbol Device:C_Polarized_US
- removed TP33: 12V_IN, TestPoint:TestPoint_THTPad_D3.0mm_Drill1.5mm, symbol Connector:TestPoint
- removed TP34: HSS_IN, TestPoint:TestPoint_THTPad_D3.0mm_Drill1.5mm, symbol Connector:TestPoint
- removed TP36: 12V_OUT, TestPoint:TestPoint_THTPad_D3.0mm_Drill1.5mm, symbol Connector:TestPoint

Commit message: switch, stll working
Parts:
- TP37, TP38: footprint TestPoint:TestPoint_THTPad_D3.0mm_Drill1.5mm -> TestPoint:TestPoint_Loop_D2.50mm_Drill1.0mm_LowProfile
Changed lines of the file:
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@@
 			)
 		)
-		(property "Footprint" "TestPoint:TestPoint_THTPad_D3.0mm_Drill1.5mm"
+		(property "Footprint" "TestPoint:TestPoint_Loop_D2.50mm_Drill1.0mm_LowProfile"
 			(at 231.14 69.85 0)
 			(hide yes)
@@
 			)
 		)
-		(property "Footprint" "TestPoint:TestPoint_THTPad_D3.0mm_Drill1.5mm"
+		(property "Footprint" "TestPoint:TestPoint_Loop_D2.50mm_Drill1.0mm_LowProfile"
 			(at 228.6 116.84 0)
 			(hide yes)

Commit message: switch to laptop
Parts:
- J9: footprint LHRS_Connectors:AMASS_XT30UPB-M_1x02_P5.0mm_Vertical -> LHRS_Connectors:Molex_Nano-Fit_105309-xx02_1x02_P2.50mm_Vertical
Changed lines of the file:
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@@
 			)
 		)
-		(property "Footprint" "LHRS_Connectors:AMASS_XT30UPB-M_1x02_P5.0mm_Vertical"
+		(property "Footprint" "LHRS_Connectors:Molex_Nano-Fit_105309-xx02_1x02_P2.50mm_Vertical"
 			(at 250.19 116.84 0)
 			(hide yes)

Commit message: switch to pc...
Other:
- sheet Voltage + Current Sense ports: added VS; removed none
Changed lines of the file:
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@@
 	)
 	(junction
-		(at 45.72 132.08)
+		(at 54.61 132.08)
 		(diameter 0)
 		(color 0 0 0 0)
 	)
 	(junction
-		(at 93.98 132.08)
+		(at 80.01 132.08)
 		(diameter 0)
 		(color 0 0 0 0)
@@
 	)
 	(junction
-		(at 93.98 121.92)
+		(at 80.01 121.92)
 		(diameter 0)
 		(color 0 0 0 0)
@@
 	)
 	(junction
-		(at 58.42 132.08)
+		(at 67.31 121.92)
 		(diameter 0)
 		(color 0 0 0 0)
 	)
 	(junction
-		(at 223.52 116.84)
+		(at 67.31 132.08)
 		(diameter 0)
 		(color 0 0 0 0)
 	)
 	(junction
-		(at 45.72 121.92)
+		(at 223.52 116.84)
 		(diameter 0)
 		(color 0 0 0 0)
 	)
 	(junction
-		(at 46.99 69.85)
+		(at 54.61 121.92)
 		(diameter 0)
 		(color 0 0 0 0)
 	)
 	(junction
-		(at 58.42 121.92)
+		(at 46.99 69.85)
 		(diameter 0)
 		(color 0 0 0 0)
@@
 	(wire
 		(pts
-			(xy 58.42 121.92) (xy 45.72 121.92)
+			(xy 67.31 121.92) (xy 54.61 121.92)
 		)
 		(stroke
@@
 	(wire
 		(pts
-			(xy 105.41 123.19) (xy 105.41 121.92)
+			(xy 91.44 123.19) (xy 91.44 121.92)
 		)
 		(stroke
@@
 	(wire
 		(pts
-			(xy 58.42 121.92) (xy 58.42 123.19)
+			(xy 67.31 121.92) (xy 67.31 123.19)
 		)
 		(stroke
@@
 	(wire
 		(pts
-			(xy 93.98 121.92) (xy 93.98 123.19)
+			(xy 80.01 121.92) (xy 80.01 123.19)
 		)
 		(stroke
@@
 	(wire
 		(pts
-			(xy 45.72 121.92) (xy 45.72 119.38)
+			(xy 54.61 121.92) (xy 54.61 119.38)
 		)
 		(stroke
@@
 	(wire
 		(pts
-			(xy 45.72 132.08) (xy 45.72 130.81)
+			(xy 54.61 132.08) (xy 54.61 130.81)
 		)
 		(stroke
@@
 	(wire
 		(pts
-			(xy 45.72 133.35) (xy 45.72 132.08)
+			(xy 54.61 133.35) (xy 54.61 132.08)
 		)
 		(stroke
@@
 	(wire
 		(pts
-			(xy 58.42 121.92) (xy 93.98 121.92)
+			(xy 67.31 121.92) (xy 80.01 121.92)
 		)
 		(stroke
@@
 	(wire
 		(pts
-			(xy 58.42 130.81) (xy 58.42 132.08)
+			(xy 67.31 130.81) (xy 67.31 132.08)
 		)
 		(stroke
@@
 	(wire
 		(pts
-			(xy 105.41 132.08) (xy 105.41 130.81)
+			(xy 91.44 132.08) (xy 91.44 130.81)
 		)
 		(stroke
@@
 	(wire
 		(pts
-			(xy 58.42 132.08) (xy 93.98 132.08)
+			(xy 67.31 132.08) (xy 80.01 132.08)
 		)
 		(stroke
@@
 	(wire
 		(pts
-			(xy 105.41 121.92) (xy 93.98 121.92)
+			(xy 91.44 121.92) (xy 80.01 121.92)
 		)
 		(stroke
@@
 	(wire
 		(pts
-			(xy 93.98 132.08) (xy 105.41 132.08)
+			(xy 80.01 132.08) (xy 91.44 132.08)
 		)
 		(stroke
@@
 	(wire
 		(pts
-			(xy 45.72 132.08) (xy 58.42 132.08)
+			(xy 54.61 132.08) (xy 67.31 132.08)
 		)
 		(stroke
@@
 	(wire
 		(pts
-			(xy 45.72 123.19) (xy 45.72 121.92)
+			(xy 54.61 123.19) (xy 54.61 121.92)
 		)
 		(stroke
@@
 	(wire
 		(pts
+			(xy 95.25 67.31) (xy 99.06 67.31)
+		)
+		(stroke
+			(width 0)
+			(type default)
+		)
+	)
+	(wire
+		(pts
 			(xy 163.83 83.82) (xy 168.91 83.82)
 		)
@@
 	(wire
 		(pts
-			(xy 93.98 130.81) (xy 93.98 132.08)
+			(xy 80.01 130.81) (xy 80.01 132.08)
 		)
 		(stroke
@@
 		)
 	)
+	(hierarchical_label "VS"
+		(shape input)
+		(at 99.06 67.31 0)
+		(effects
+			(font
+				(size 1.27 1.27)
+			)
+			(justify left)
+		)
+	)
 	(hierarchical_label "HSS_FLT_WAKE"
 		(shape input)
@@
 	(hierarchical_label "12V_FUSED"
 		(shape input)
-		(at 45.72 119.38 180)
+		(at 54.61 119.38 180)
 		(effects
 			(font
@@
 	(hierarchical_label "LV_GND"
 		(shape passive)
-		(at 45.72 133.35 270)
+		(at 54.61 133.35 270)
 		(effects
 			(font
@@
 	(symbol
 		(lib_id "Device:C_Polarized_US")
-		(at 58.42 127 0)
+		(at 67.31 127 0)
 		(mirror y)
 		(unit 1)
@@
 		(dnp no)
 		(property "Reference" "C71"
-			(at 54.61 125.0949 0)
+			(at 63.5 125.0949 0)
 			(show_name no)
 			(do_not_autoplace no)
@@
 		)
 		(property "Value" "1000u"
-			(at 54.61 127.6349 0)
+			(at 63.5 127.6349 0)
 			(show_name no)
 			(do_not_autoplace no)
@@
 		)
 		(property "Footprint" "Capacitor_SMD:CP_Elec_10x12.5"
-			(at 58.42 127 0)
+			(at 67.31 127 0)
 			(hide yes)
 			(show_name no)
@@
 		)
 		(property "Datasheet" ""
-			(at 58.42 127 0)
+			(at 67.31 127 0)
 			(hide yes)
 			(show_name no)
@@
 		)
 		(property "Description" "Polarized capacitor, US symbol"
-			(at 58.42 127 0)
+			(at 67.31 127 0)
 			(hide yes)
 			(show_name no)
@@
 		)
 		(property "LCSC" ""
-			(at 58.42 127 0)
+			(at 67.31 127 0)
 			(hide yes)
 			(show_name no)
@@
 		)
 		(property "LCSC P/N" "C22387800"
-			(at 58.42 127 0)
+			(at 67.31 127 0)
 			(hide yes)
 			(show_name no)
@@
 	(symbol
 		(lib_id "Device:C")
-		(at 93.98 127 0)
+		(at 80.01 127 0)
 		(mirror y)
 		(unit 1)
@@
 		(dnp no)
 		(property "Reference" "C73"
-			(at 90.17 125.7299 0)
+			(at 76.2 125.7299 0)
 			(show_name no)
 			(do_not_autoplace no)
@@
 		)
 		(property "Value" "22u"
-			(at 90.17 128.2699 0)
+			(at 76.2 128.2699 0)
 			(show_name no)
 			(do_not_autoplace no)
@@
 		)
 		(property "Footprint" "Capacitor_SMD:C_0603_1608Metric_Pad1.08x0.95mm_HandSolder"
-			(at 93.0148 130.81 0)
+			(at 79.0448 130.81 0)
 			(hide yes)
 			(show_name no)
@@
 		)
 		(property "Datasheet" ""
-			(at 93.98 127 0)
+			(at 80.01 127 0)
 			(hide yes)
 			(show_name no)
@@
 		)
 		(property "Description" "Unpolarized capacitor"
-			(at 93.98 127 0)
+			(at 80.01 127 0)
 			(hide yes)
 			(show_name no)
@@
 		)
 		(property "P/N" "MLASU168SB5105KTNA01"
-			(at 93.98 127 0)
+			(at 80.01 127 0)
 			(hide yes)
 			(show_name no)
@@
 		)
 		(property "Assemble" "Y"
-			(at 93.98 127 0)
+			(at 80.01 127 0)
 			(hide yes)
 			(show_name no)
@@
 		)
 		(property "LCSC" ""
-			(at 93.98 127 0)
+			(at 80.01 127 0)
 			(hide yes)
 			(show_name no)
@@
 		)
 		(property "LCSC P/N" "C21122"
-			(at 93.98 127 0)
+			(at 80.01 127 0)
 			(hide yes)
 			(show_name no)
@@
 	(symbol
 		(lib_id "Device:C_Polarized_US")
-		(at 45.72 127 0)
+		(at 54.61 127 0)
 		(mirror y)
 		(unit 1)
@@
 		(dnp no)
 		(property "Reference" "C70"
-			(at 41.91 125.0949 0)
+			(at 50.8 125.0949 0)
 			(show_name no)
 			(do_not_autoplace no)
@@
 		)
 		(property "Value" "1000u"
-			(at 41.91 127.6349 0)
+			(at 50.8 127.6349 0)
 			(show_name no)
 			(do_not_autoplace no)
@@
 		)
 		(property "Footprint" "Capacitor_SMD:CP_Elec_10x12.5"
-			(at 45.72 127 0)
+			(at 54.61 127 0)
 			(hide yes)
 			(show_name no)
@@
 		)
 		(property "Datasheet" ""
-			(at 45.72 127 0)
+			(at 54.61 127 0)
 			(hide yes)
 			(show_name no)
@@
 		)
 		(property "Description" "Polarized capacitor, US symbol"
-			(at 45.72 127 0)
+			(at 54.61 127 0)
 			(hide yes)
 			(show_name no)
@@
 		)
 		(property "LCSC" ""
-			(at 45.72 127 0)
+			(at 54.61 127 0)
 			(hide yes)
 			(show_name no)
@@
 		)
 		(property "LCSC P/N" "C22387800"
-			(at 45.72 127 0)
+			(at 54.61 127 0)
 			(hide yes)
 			(show_name no)
@@
 	(symbol
 		(lib_id "Device:C")
-		(at 105.41 127 0)
+		(at 91.44 127 0)
 		(mirror y)
 		(unit 1)
@@
 		(dnp no)
 		(property "Reference" "C74"
-			(at 101.6 125.7299 0)
+			(at 87.63 125.7299 0)
 			(show_name no)
 			(do_not_autoplace no)
@@
 		)
 		(property "Value" "22u"
-			(at 101.6 128.2699 0)
+			(at 87.63 128.2699 0)
 			(show_name no)
 			(do_not_autoplace no)
@@
 		)
 		(property "Footprint" "Capacitor_SMD:C_0603_1608Metric_Pad1.08x0.95mm_HandSolder"
-			(at 104.4448 130.81 0)
+			(at 90.4748 130.81 0)
 			(hide yes)
 			(show_name no)
@@
 		)
 		(property "Datasheet" ""
-			(at 105.41 127 0)
+			(at 91.44 127 0)
 			(hide yes)
 			(show_name no)
@@
 		)
 		(property "Description" "Unpolarized capacitor"
-			(at 105.41 127 0)
+			(at 91.44 127 0)
 			(hide yes)
 			(show_name no)
@@
 		)
 		(property "P/N" "MLASU168SB5105KTNA01"
-			(at 105.41 127 0)
+			(at 91.44 127 0)
 			(hide yes)
 			(show_name no)
@@
 		)
 		(property "Assemble" "Y"
-			(at 105.41 127 0)
+			(at 91.44 127 0)
 			(hide yes)
 			(show_name no)
@@
 		)
 		(property "LCSC" ""
-			(at 105.41 127 0)
+			(at 91.44 127 0)
 			(hide yes)
 			(show_name no)
@@
 		)
 		(property "LCSC P/N" "C21122"
-			(at 105.41 127 0)
+			(at 91.44 127 0)
 			(hide yes)
 			(show_name no)
@@
 			(effects
 				(font
+					(size 1.27 1.27)
+				)
+				(justify right)
+			)
+		)
+		(pin "VS" input
+			(at 95.25 67.31 0)
+			(effects
+				(font

Commit message: oops
Parts:
- R94: P/N (none) -> CRCW060322K0FKEAHP
Changed lines of the file:
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@@
+			)
+		)
+		(property "P/N" "CRCW060322K0FKEAHP"
+			(at 226.06 74.93 0)
+			(hide yes)
+			(show_name no)
+			(do_not_autoplace no)
+			(effects
+				(font
+					(size 1.27 1.27)
+				)
 			)
 		)

Commit message: ahhahahahhahahhahahhahahhahhaa im so back
Connections:
- net LV_GND: now also J10.1 (Pin_1); no longer J10.2 (Pin_2)
- net PDU_FUSED: now also J10.2 (Pin_2); no longer J10.1 (Pin_1)
Changed lines of the file:
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@@
 	(wire
 		(pts
-			(xy 236.22 72.39) (xy 247.65 72.39)
+			(xy 236.22 67.31) (xy 247.65 67.31)
 		)
 		(stroke
@@
 	(hierarchical_label "LV_GND"
 		(shape passive)
-		(at 236.22 72.39 270)
+		(at 236.22 67.31 270)
 		(effects
 			(font
@@
 	(symbol
 		(lib_id "Connector_Generic:Conn_01x02")
-		(at 252.73 69.85 0)
+		(at 252.73 67.31 0)
 		(unit 1)
 		(body_style 1)
@@
 		(dnp no)
 		(property "Reference" "J10"
-			(at 257.048 69.85 0)
+			(at 257.048 67.31 0)
 			(show_name no)
 			(do_not_autoplace no)
@@
 		)
 		(property "Value" "PDU_12V"
-			(at 259.588 72.39 0)
+			(at 259.588 69.85 0)
 			(show_name no)
 			(do_not_autoplace no)
@@
 		)
 		(property "Footprint" "LHRS_Connectors:AMASS_XT30UPB-M_1x02_P5.0mm_Vertical"
-			(at 252.73 69.85 0)
+			(at 252.73 67.31 0)
 			(hide yes)
 			(show_name no)
@@
 		)
 		(property "Datasheet" ""
-			(at 252.73 69.85 0)
+			(at 252.73 67.31 0)
 			(hide yes)
 			(show_name no)
@@
 		)
 		(property "Description" "Generic connector, single row, 01x02, script generated (kicad-library-utils/schlib/autogen/connector/)"
-			(at 252.73 69.85 0)
+			(at 252.73 67.31 0)
 			(hide yes)
 			(show_name no)
@@
 		)
 		(property "LCSC" ""
-			(at 252.73 69.85 0)
-			(hide yes)
-			(show_name no)
+			(at 252.73 67.31 0)
+			(hide yes)
+			(show_name no)
