File: hardware/LVD.kicad_sch (KiCad schematic)
At the start: 0 parts

Commit message: review ts
Parts:
- added C87: C_Small, symbol Device:C_Small
- added R100: 470k, symbol Device:R
- added R98: 200k, symbol Device:R
- added R99: 100k, symbol Device:R
- added U16: TPS3840DL30DBVR, DBV0005A_N, symbol OBBB Symbols:TPS3840DL30DBVR
Connections:
- new net: R100.2, U16.1 (RESET_N)
- new net: R98.2, R99.1, U16.2 (VDD)
- new net: C87.1, U16.5 (CT)
- new net LVD_EN: R100.1
- new net LVD_IN: R98.1
- new net LVD_RESET: U16.4 (MR_N)
- new net LV_GND: C87.2, R99.2, U16.3 (GND)
Other:
- note added: "3.0 × (200k + 100k) / 100k = 3.0 × 3.0 = 9.00V"
- note added: "RESET active low"
- note added: "Reset time delay"
- note added: "TPS3840DL33DBVR: not available on JLC, 30 variant pretty much the same"
- note added: "V_rail_max = 10 × (200k + 100k) / 100k = 30V"
- note added: "manual reset, pull low to assert reset at RESET pin"
- note added: "trips when supp goes under 9V"

Commit message: addressed
Other:
- note added: "Vit- = 3V"
- note added: "default delay: 50us (open)"
- note added: "ok to float"
- moved on the sheet: C87, R100, R98, R99, U16

Commit message: update kicad sharepoint
Parts:
- added TP36: LVD_RESET, symbol Connector:TestPoint
- C87: value C_Small -> 10nf
Connections:
- net LVD_RESET: now also TP36.1
Other:
- note added: "10nf: 6.2ms"
- moved on the sheet: C87, R100, R98, R99, U16

Commit message: sorry im omw
Parts:
- C87: value 10nf -> 10n; footprint (none) -> Capacitor_SMD:C_0603_1608Metric_Pad1.08x0.95mm_HandSolder
- R100, R99: footprint (none) -> Resistor_SMD:R_0603_1608Metric_Pad0.98x0.95mm_HandSolder
- R98: footprint (none) -> Resistor_SMD:R_0603_1608Metric_Pad0.98x0.95mm_HandSolder; LCSC P/N (none) -> C25811
- TP36: footprint (none) -> TestPoint:TestPoint_Loop_D2.50mm_Drill1.0mm_LowProfile
- U16: footprint DBV0005A_N -> OBBB Footprints:TPS3840DL33DBVR
Changed lines of the file:
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@@
 			)
 		)
-		(property "Footprint" "DBV0005A_N"
+		(property "Footprint" "OBBB Footprints:TPS3840DL33DBVR"
 			(at 209.55 76.2 0)
 			(hide yes)
@@
 			)
 		)
-		(property "Footprint" ""
+		(property "Footprint" "Resistor_SMD:R_0603_1608Metric_Pad0.98x0.95mm_HandSolder"
 			(at 186.182 60.96 90)
 			(hide yes)
@@
 			)
 		)
-		(property "Footprint" ""
+		(property "Footprint" "Resistor_SMD:R_0603_1608Metric_Pad0.98x0.95mm_HandSolder"
 			(at 174.752 69.85 90)
 			(hide yes)
@@
 		)
 		(property "LCSC" ""
+			(at 176.53 69.85 0)
+			(hide yes)
+			(show_name no)
+			(do_not_autoplace no)
+			(effects
+				(font
+					(size 1.27 1.27)
+				)
+			)
+		)
+		(property "LCSC P/N" "C25811"
 			(at 176.53 69.85 0)
 			(hide yes)
@@
 			)
 		)
-		(property "Footprint" ""
+		(property "Footprint" "TestPoint:TestPoint_Loop_D2.50mm_Drill1.0mm_LowProfile"
 			(at 233.68 71.12 0)
 			(hide yes)
@@
 			)
 		)
-		(property "Value" "10nf"
+		(property "Value" "10n"
 			(at 232.41 87.6362 0)
 			(show_name no)
@@
 			)
 		)
-		(property "Footprint" ""
+		(property "Footprint" "Capacitor_SMD:C_0603_1608Metric_Pad1.08x0.95mm_HandSolder"
 			(at 229.87 86.36 0)
 			(hide yes)
@@
 			)
 		)
-		(property "Footprint" ""
+		(property "Footprint" "Resistor_SMD:R_0603_1608Metric_Pad0.98x0.95mm_HandSolder"
 			(at 174.752 82.55 90)
 			(hide yes)

Commit message: craigenyah
Parts:
- renumbered C87 to C31, R98 to R35, R99 to R36, R100 to R37, TP36 to TP12, U16 to U3
Changed lines of the file:
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@@
 		(dnp no)
 		(fields_autoplaced yes)
-		(property "Reference" "U16"
+		(property "Reference" "U3"
 			(at 209.55 60.96 0)
 			(show_name no)
@@
 			(project "PS-LVCarrier"
 				(path "/9bab2d9d-20f3-40ef-8545-e1299efec47e/b521073a-8409-41eb-9cdc-cffa14c92055/85de105f-0d3a-47c9-b24a-66aeb10ffd65"
-					(reference "U16")
+					(reference "U3")
 					(unit 1)
 				)
@@
 		(in_pos_files yes)
 		(dnp no)
-		(property "Reference" "R100"
+		(property "Reference" "R37"
 			(at 185.42 59.6899 0)
 			(show_name no)
@@
 			(project "PS-LVCarrier"
 				(path "/9bab2d9d-20f3-40ef-8545-e1299efec47e/b521073a-8409-41eb-9cdc-cffa14c92055/85de105f-0d3a-47c9-b24a-66aeb10ffd65"
-					(reference "R100")
+					(reference "R37")
 					(unit 1)
 				)
@@
 		(in_pos_files yes)
 		(dnp no)
-		(property "Reference" "R98"
+		(property "Reference" "R35"
 			(at 173.99 68.5799 0)
 			(show_name no)
@@
 			(project "PS-LVCarrier"
 				(path "/9bab2d9d-20f3-40ef-8545-e1299efec47e/b521073a-8409-41eb-9cdc-cffa14c92055/85de105f-0d3a-47c9-b24a-66aeb10ffd65"
-					(reference "R98")
+					(reference "R35")
 					(unit 1)
 				)
@@
 		(in_pos_files yes)
 		(dnp no)
-		(property "Reference" "TP36"
+		(property "Reference" "TP12"
 			(at 227.584 62.992 0)
 			(show_name no)
@@
 			(project "PS-LVCarrier"
 				(path "/9bab2d9d-20f3-40ef-8545-e1299efec47e/b521073a-8409-41eb-9cdc-cffa14c92055/85de105f-0d3a-47c9-b24a-66aeb10ffd65"
-					(reference "TP36")
+					(reference "TP12")
 					(unit 1)
 				)
@@
 		(dnp yes)
 		(fields_autoplaced yes)
-		(property "Reference" "C87"
+		(property "Reference" "C31"
 			(at 232.41 85.0962 0)
 			(show_name no)
@@
 			(project "PS-LVCarrier"
 				(path "/9bab2d9d-20f3-40ef-8545-e1299efec47e/b521073a-8409-41eb-9cdc-cffa14c92055/85de105f-0d3a-47c9-b24a-66aeb10ffd65"
-					(reference "C87")
+					(reference "C31")
 					(unit 1)
 				)
@@
 		(in_pos_files yes)
 		(dnp no)
-		(property "Reference" "R99"
+		(property "Reference" "R36"
 			(at 173.99 81.2799 0)
 			(show_name no)
@@
 			(project "PS-LVCarrier"
 				(path "/9bab2d9d-20f3-40ef-8545-e1299efec47e/b521073a-8409-41eb-9cdc-cffa14c92055/85de105f-0d3a-47c9-b24a-66aeb10ffd65"
-					(reference "R99")
+					(reference "R36")
 					(unit 1)
 				)

Commit message: oops
Parts:
- C31: LCSC P/N (none) -> C57112; P/N (none) -> MSASH168SB5103KTNA01
- U3: LCSC P/N (none) -> C2862542; P/N (none) -> TPS3840DL30DBVR
Changed lines of the file:
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@@
+			)
+		)
+		(property "LCSC P/N" "C2862542"
+			(at 209.55 76.2 0)
+			(hide yes)
+			(show_name no)
+			(do_not_autoplace no)
+			(effects
+				(font
+					(size 1.27 1.27)
+				)
+			)
+		)
+		(property "P/N" "TPS3840DL30DBVR"
+			(at 209.55 76.2 0)
+			(hide yes)
+			(show_name no)
+			(do_not_autoplace no)
+			(effects
+				(font
+					(size 1.27 1.27)
+				)
 			)
 		)
@@
 			(at 229.87 86.36 0)
 			(hide yes)
+			(show_name no)
+			(do_not_autoplace no)
+			(effects
+				(font
+					(size 1.27 1.27)
+				)
+			)
+		)
+		(property "LCSC P/N" "C57112"
+			(at 229.87 86.36 0)
+			(hide yes)
+			(show_name no)
+			(do_not_autoplace no)
+			(effects
+				(font
+					(size 1.27 1.27)
+				)
+			)
+		)
+		(property "P/N" "MSASH168SB5103KTNA01"
+			(at 229.87 86.36 0)
+			(hide yes)

Commit message: added most p/n, still in progress but saving
Parts:
- R35: P/N (none) -> 0603WAF2003T5E
- R36: Assemble (none) -> -- mixed values --; LCSC P/N (none) -> C25803; P/N (none) -> CRCW0603100KFKEE
- R37: LCSC P/N (none) -> C23178; P/N (none) -> 0603WAF4703T5E
Changed lines of the file:
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@@
+			)
+		)
+		(property "LCSC P/N" "C23178"
+			(at 187.96 60.96 0)
+			(hide yes)
+			(show_name no)
+			(do_not_autoplace no)
+			(effects
+				(font
+					(size 1.27 1.27)
+				)
+			)
+		)
+		(property "P/N" "0603WAF4703T5E"
+			(at 187.96 60.96 0)
+			(hide yes)
+			(show_name no)
+			(do_not_autoplace no)
+			(effects
+				(font
+					(size 1.27 1.27)
+				)
 			)
 		)
@@
 		)
 		(property "LCSC P/N" "C25811"
+			(at 176.53 69.85 0)
+			(hide yes)
+			(show_name no)
+			(do_not_autoplace no)
+			(effects
+				(font
+					(size 1.27 1.27)
+				)
+			)
+		)
+		(property "P/N" "0603WAF2003T5E"
 			(at 176.53 69.85 0)
 			(hide yes)
@@
 			)
 		)
-		(property "Description" "Resistor"
+		(property "Description" "-- mixed values --"
 			(at 176.53 82.55 0)
 			(hide yes)
@@
 			(at 176.53 82.55 0)
 			(hide yes)
+			(show_name no)
+			(do_not_autoplace no)
+			(effects
+				(font
+					(size 1.27 1.27)
+				)
+			)
+		)
+		(property "Assemble" "-- mixed values --"
+			(at 176.53 82.55 0)
+			(hide yes)
+			(show_name no)
+			(do_not_autoplace no)
+			(effects
+				(font
+					(size 1.27 1.27)
+				)
+			)
+		)
+		(property "LCSC P/N" "C25803"
+			(at 176.53 82.55 0)
+			(hide yes)
+			(show_name no)
+			(do_not_autoplace no)
+			(effects
+				(font
+					(size 1.27 1.27)
+				)
+			)
+		)
+		(property "P/N" "CRCW0603100KFKEE"
+			(at 176.53 82.55 0)
+			(hide yes)
