File: hardware/sensing.kicad_sch (KiCad schematic)
At the start: 7 parts, among them U1 TMCS1107A2UQDR

Commit message: update kicad sharepoint
Parts:
- added TP16: I_ADC, symbol Connector:TestPoint
- added TP27: V_ADC, symbol Connector:TestPoint
- C3: LCSC P/N C1636 -> C14663
Connections:
- net VOUT: now also TP16.1
- net V_ADC: now also TP27.1
Other:
- note added: "Use a 10× probe or a DMM"
- moved on the sheet: C1

Commit message: sorry im omw
Parts:
- TP16, TP27: footprint (none) -> TestPoint:TestPoint_Loop_D2.50mm_Drill1.0mm_LowProfile
Changed lines of the file:
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@@
 			)
 		)
-		(property "Footprint" ""
+		(property "Footprint" "TestPoint:TestPoint_Loop_D2.50mm_Drill1.0mm_LowProfile"
 			(at 134.62 55.88 0)
 			(hide yes)
@@
 			)
 		)
-		(property "Footprint" ""
+		(property "Footprint" "TestPoint:TestPoint_Loop_D2.50mm_Drill1.0mm_LowProfile"
 			(at 58.42 64.77 0)
 			(hide yes)

Commit message: craigenyah
Parts:
- renumbered C1 to C28, C2 to C29, C3 to C30, R1 to R32, R2 to R33, R3 to R34, TP27 to TP10, TP16 to TP11, U1 to U2
Changed lines of the file:
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@@
 		(dnp no)
 		(fields_autoplaced yes)
-		(property "Reference" "U1"
+		(property "Reference" "U2"
 			(at 102.87 40.64 0)
 			(show_name no)
@@
 			(project "PS-LVCarrier"
 				(path "/9bab2d9d-20f3-40ef-8545-e1299efec47e/10a2a81d-fff8-4091-b6ef-9685e4bd9514/a12cc91e-7ffe-4aca-bb00-a063147b4e50"
+					(reference "U10")
+					(unit 1)
+				)
+				(path "/9bab2d9d-20f3-40ef-8545-e1299efec47e/b521073a-8409-41eb-9cdc-cffa14c92055/37ef47ed-2aee-4ae2-b946-13f1b7a76e72"
+					(reference "U2")
+					(unit 1)
+				)
+				(path "/9bab2d9d-20f3-40ef-8545-e1299efec47e/4f26e4eb-a337-4f9d-865d-e2c0801c36ac/a57b6f22-cd56-4351-a5e4-2e9e02d85251/72c78d2c-2a65-43a0-ad78-90d0e31c028b"
 					(reference "U9")
-					(unit 1)
-				)
-				(path "/9bab2d9d-20f3-40ef-8545-e1299efec47e/b521073a-8409-41eb-9cdc-cffa14c92055/37ef47ed-2aee-4ae2-b946-13f1b7a76e72"
-					(reference "U1")
-					(unit 1)
-				)
-				(path "/9bab2d9d-20f3-40ef-8545-e1299efec47e/4f26e4eb-a337-4f9d-865d-e2c0801c36ac/a57b6f22-cd56-4351-a5e4-2e9e02d85251/72c78d2c-2a65-43a0-ad78-90d0e31c028b"
-					(reference "U13")
 					(unit 1)
 				)
@@
 		(dnp no)
 		(fields_autoplaced yes)
-		(property "Reference" "TP16"
+		(property "Reference" "TP11"
 			(at 132.08 51.3079 0)
 			(show_name no)
@@
 			(project "PS-LVCarrier"
 				(path "/9bab2d9d-20f3-40ef-8545-e1299efec47e/10a2a81d-fff8-4091-b6ef-9685e4bd9514/a12cc91e-7ffe-4aca-bb00-a063147b4e50"
-					(reference "TP25")
+					(reference "TP41")
 					(unit 1)
 				)
 				(path "/9bab2d9d-20f3-40ef-8545-e1299efec47e/b521073a-8409-41eb-9cdc-cffa14c92055/37ef47ed-2aee-4ae2-b946-13f1b7a76e72"
-					(reference "TP16")
+					(reference "TP11")
 					(unit 1)
 				)
@@
 		(in_pos_files yes)
 		(dnp no)
-		(property "Reference" "R3"
+		(property "Reference" "R34"
 			(at 134.366 59.436 0)
 			(show_name no)
@@
 			(project "PS-LVCarrier"
 				(path "/9bab2d9d-20f3-40ef-8545-e1299efec47e/10a2a81d-fff8-4091-b6ef-9685e4bd9514/a12cc91e-7ffe-4aca-bb00-a063147b4e50"
-					(reference "R50")
+					(reference "R98")
 					(unit 1)
 				)
 				(path "/9bab2d9d-20f3-40ef-8545-e1299efec47e/b521073a-8409-41eb-9cdc-cffa14c92055/37ef47ed-2aee-4ae2-b946-13f1b7a76e72"
-					(reference "R3")
+					(reference "R34")
 					(unit 1)
 				)
 				(path "/9bab2d9d-20f3-40ef-8545-e1299efec47e/4f26e4eb-a337-4f9d-865d-e2c0801c36ac/a57b6f22-cd56-4351-a5e4-2e9e02d85251/72c78d2c-2a65-43a0-ad78-90d0e31c028b"
-					(reference "R69")
+					(reference "R60")
 					(unit 1)
 				)
@@
 		(in_pos_files yes)
 		(dnp no)
-		(property "Reference" "C1"
+		(property "Reference" "C28"
 			(at 55.88 69.8562 0)
 			(show_name no)
@@
 			(project "PS-LVCarrier"
 				(path "/9bab2d9d-20f3-40ef-8545-e1299efec47e/10a2a81d-fff8-4091-b6ef-9685e4bd9514/a12cc91e-7ffe-4aca-bb00-a063147b4e50"
+					(reference "C79")
+					(unit 1)
+				)
+				(path "/9bab2d9d-20f3-40ef-8545-e1299efec47e/b521073a-8409-41eb-9cdc-cffa14c92055/37ef47ed-2aee-4ae2-b946-13f1b7a76e72"
 					(reference "C28")
 					(unit 1)
 				)
-				(path "/9bab2d9d-20f3-40ef-8545-e1299efec47e/b521073a-8409-41eb-9cdc-cffa14c92055/37ef47ed-2aee-4ae2-b946-13f1b7a76e72"
-					(reference "C1")
-					(unit 1)
-				)
 				(path "/9bab2d9d-20f3-40ef-8545-e1299efec47e/4f26e4eb-a337-4f9d-865d-e2c0801c36ac/a57b6f22-cd56-4351-a5e4-2e9e02d85251/72c78d2c-2a65-43a0-ad78-90d0e31c028b"
-					(reference "C31")
+					(reference "C54")
 					(unit 1)
 				)
@@
 		(in_pos_files yes)
 		(dnp no)
-		(property "Reference" "R2"
+		(property "Reference" "R33"
 			(at 69.85 69.8499 0)
 			(show_name no)
@@
 			(project "PS-LVCarrier"
 				(path "/9bab2d9d-20f3-40ef-8545-e1299efec47e/10a2a81d-fff8-4091-b6ef-9685e4bd9514/a12cc91e-7ffe-4aca-bb00-a063147b4e50"
-					(reference "R48")
+					(reference "R97")
 					(unit 1)
 				)
 				(path "/9bab2d9d-20f3-40ef-8545-e1299efec47e/b521073a-8409-41eb-9cdc-cffa14c92055/37ef47ed-2aee-4ae2-b946-13f1b7a76e72"
-					(reference "R2")
+					(reference "R33")
 					(unit 1)
 				)
 				(path "/9bab2d9d-20f3-40ef-8545-e1299efec47e/4f26e4eb-a337-4f9d-865d-e2c0801c36ac/a57b6f22-cd56-4351-a5e4-2e9e02d85251/72c78d2c-2a65-43a0-ad78-90d0e31c028b"
-					(reference "R68")
+					(reference "R59")
 					(unit 1)
 				)
@@
 		(in_pos_files yes)
 		(dnp no)
-		(property "Reference" "#PWR010"
+		(property "Reference" "#PWR014"
 			(at 124.46 54.61 0)
 			(hide yes)
@@
 			(project "PS-LVCarrier"
 				(path "/9bab2d9d-20f3-40ef-8545-e1299efec47e/10a2a81d-fff8-4091-b6ef-9685e4bd9514/a12cc91e-7ffe-4aca-bb00-a063147b4e50"
-					(reference "#PWR050")
+					(reference "#PWR033")
 					(unit 1)
 				)
 				(path "/9bab2d9d-20f3-40ef-8545-e1299efec47e/b521073a-8409-41eb-9cdc-cffa14c92055/37ef47ed-2aee-4ae2-b946-13f1b7a76e72"
-					(reference "#PWR010")
+					(reference "#PWR014")
 					(unit 1)
 				)
 				(path "/9bab2d9d-20f3-40ef-8545-e1299efec47e/4f26e4eb-a337-4f9d-865d-e2c0801c36ac/a57b6f22-cd56-4351-a5e4-2e9e02d85251/72c78d2c-2a65-43a0-ad78-90d0e31c028b"
-					(reference "#PWR062")
+					(reference "#PWR031")
 					(unit 1)
 				)
@@
 		(in_pos_files yes)
 		(dnp no)
-		(property "Reference" "R1"
+		(property "Reference" "R32"
 			(at 69.85 57.1499 0)
 			(show_name no)
@@
 			(project "PS-LVCarrier"
 				(path "/9bab2d9d-20f3-40ef-8545-e1299efec47e/10a2a81d-fff8-4091-b6ef-9685e4bd9514/a12cc91e-7ffe-4aca-bb00-a063147b4e50"
-					(reference "R47")
+					(reference "R96")
 					(unit 1)
 				)
 				(path "/9bab2d9d-20f3-40ef-8545-e1299efec47e/b521073a-8409-41eb-9cdc-cffa14c92055/37ef47ed-2aee-4ae2-b946-13f1b7a76e72"
-					(reference "R1")
+					(reference "R32")
 					(unit 1)
 				)
 				(path "/9bab2d9d-20f3-40ef-8545-e1299efec47e/4f26e4eb-a337-4f9d-865d-e2c0801c36ac/a57b6f22-cd56-4351-a5e4-2e9e02d85251/72c78d2c-2a65-43a0-ad78-90d0e31c028b"
-					(reference "R67")
+					(reference "R58")
 					(unit 1)
 				)
@@
 		(in_pos_files yes)
 		(dnp no)
-		(property "Reference" "C2"
+		(property "Reference" "C29"
 			(at 132.08 71.1262 0)
 			(show_name no)
@@
 			(project "PS-LVCarrier"
 				(path "/9bab2d9d-20f3-40ef-8545-e1299efec47e/10a2a81d-fff8-4091-b6ef-9685e4bd9514/a12cc91e-7ffe-4aca-bb00-a063147b4e50"
+					(reference "C80")
+					(unit 1)
+				)
+				(path "/9bab2d9d-20f3-40ef-8545-e1299efec47e/b521073a-8409-41eb-9cdc-cffa14c92055/37ef47ed-2aee-4ae2-b946-13f1b7a76e72"
 					(reference "C29")
 					(unit 1)
 				)
-				(path "/9bab2d9d-20f3-40ef-8545-e1299efec47e/b521073a-8409-41eb-9cdc-cffa14c92055/37ef47ed-2aee-4ae2-b946-13f1b7a76e72"
-					(reference "C2")
-					(unit 1)
-				)
 				(path "/9bab2d9d-20f3-40ef-8545-e1299efec47e/4f26e4eb-a337-4f9d-865d-e2c0801c36ac/a57b6f22-cd56-4351-a5e4-2e9e02d85251/72c78d2c-2a65-43a0-ad78-90d0e31c028b"
-					(reference "C33")
+					(reference "C55")
 					(unit 1)
 				)
@@
 		(in_pos_files yes)
 		(dnp no)
-		(property "Reference" "C3"
+		(property "Reference" "C30"
 			(at 151.638 59.944 0)
 			(show_name no)
@@
 			(project "PS-LVCarrier"
 				(path "/9bab2d9d-20f3-40ef-8545-e1299efec47e/10a2a81d-fff8-4091-b6ef-9685e4bd9514/a12cc91e-7ffe-4aca-bb00-a063147b4e50"
+					(reference "C81")
+					(unit 1)
+				)
+				(path "/9bab2d9d-20f3-40ef-8545-e1299efec47e/b521073a-8409-41eb-9cdc-cffa14c92055/37ef47ed-2aee-4ae2-b946-13f1b7a76e72"
 					(reference "C30")
 					(unit 1)
 				)
-				(path "/9bab2d9d-20f3-40ef-8545-e1299efec47e/b521073a-8409-41eb-9cdc-cffa14c92055/37ef47ed-2aee-4ae2-b946-13f1b7a76e72"
-					(reference "C3")
-					(unit 1)
-				)
 				(path "/9bab2d9d-20f3-40ef-8545-e1299efec47e/4f26e4eb-a337-4f9d-865d-e2c0801c36ac/a57b6f22-cd56-4351-a5e4-2e9e02d85251/72c78d2c-2a65-43a0-ad78-90d0e31c028b"
-					(reference "C35")
+					(reference "C56")
 					(unit 1)
 				)
@@
 		(in_pos_files yes)
 		(dnp no)
-		(property "Reference" "#PWR011"
+		(property "Reference" "#PWR015"
 			(at 148.59 60.96 0)
 			(hide yes)
@@
 			(project "PS-LVCarrier"
 				(path "/9bab2d9d-20f3-40ef-8545-e1299efec47e/10a2a81d-fff8-4091-b6ef-9685e4bd9514/a12cc91e-7ffe-4aca-bb00-a063147b4e50"
-					(reference "#PWR051")
+					(reference "#PWR034")
 					(unit 1)
 				)
 				(path "/9bab2d9d-20f3-40ef-8545-e1299efec47e/b521073a-8409-41eb-9cdc-cffa14c92055/37ef47ed-2aee-4ae2-b946-13f1b7a76e72"
-					(reference "#PWR011")
+					(reference "#PWR015")
 					(unit 1)
 				)
 				(path "/9bab2d9d-20f3-40ef-8545-e1299efec47e/4f26e4eb-a337-4f9d-865d-e2c0801c36ac/a57b6f22-cd56-4351-a5e4-2e9e02d85251/72c78d2c-2a65-43a0-ad78-90d0e31c028b"
-					(reference "#PWR063")
+					(reference "#PWR032")
 					(unit 1)
 				)
@@
 		(in_pos_files yes)
 		(dnp no)
-		(property "Reference" "TP27"
+		(property "Reference" "TP10"
 			(at 60.96 60.1979 0)
 			(show_name no)
@@
 			(project "PS-LVCarrier"
 				(path "/9bab2d9d-20f3-40ef-8545-e1299efec47e/10a2a81d-fff8-4091-b6ef-9685e4bd9514/a12cc91e-7ffe-4aca-bb00-a063147b4e50"
-					(reference "TP29")
+					(reference "TP40")
 					(unit 1)
 				)
 				(path "/9bab2d9d-20f3-40ef-8545-e1299efec47e/b521073a-8409-41eb-9cdc-cffa14c92055/37ef47ed-2aee-4ae2-b946-13f1b7a76e72"
-					(reference "TP27")
+					(reference "TP10")
 					(unit 1)
 				)
 				(path "/9bab2d9d-20f3-40ef-8545-e1299efec47e/4f26e4eb-a337-4f9d-865d-e2c0801c36ac/a57b6f22-cd56-4351-a5e4-2e9e02d85251/72c78d2c-2a65-43a0-ad78-90d0e31c028b"
-					(reference "TP28")
-					(unit 1)
-				)
+					(reference "TP23")
+					(unit 1)
+				)

Commit message: switch, stll working
Parts:
- removed TP10: V_ADC, TestPoint:TestPoint_Loop_D2.50mm_Drill1.0mm_LowProfile, symbol Connector:TestPoint
- removed TP11: I_ADC, TestPoint:TestPoint_Loop_D2.50mm_Drill1.0mm_LowProfile, symbol Connector:TestPoint
Changed lines of the file:
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@@
-	)
-	(junction
-		(at 129.54 55.88)
-		(diameter 0)
-		(color 0 0 0 0)
 	)
 	(junction
@@
 	)
 	(junction
-		(at 63.5 64.77)
-		(diameter 0)
-		(color 0 0 0 0)
-	)
-	(junction
 		(at 67.31 64.77)
 		(diameter 0)
@@
 	(wire
 		(pts
-			(xy 63.5 64.77) (xy 67.31 64.77)
+			(xy 59.69 64.77) (xy 67.31 64.77)
 		)
 		(stroke
@@
 		(pts
 			(xy 148.59 57.15) (xy 148.59 58.42)
-		)
-		(stroke
-			(width 0)
-			(type default)
-		)
-	)
-	(wire
-		(pts
-			(xy 59.69 64.77) (xy 63.5 64.77)
 		)
 		(stroke
@@
 	)
 	(symbol
-		(lib_id "Connector:TestPoint")
-		(at 129.54 55.88 0)
-		(unit 1)
-		(body_style 1)
-		(exclude_from_sim no)
-		(in_bom yes)
-		(on_board yes)
-		(in_pos_files yes)
-		(dnp no)
-		(fields_autoplaced yes)
-		(property "Reference" "TP11"
-			(at 132.08 51.3079 0)
-			(show_name no)
-			(do_not_autoplace no)
-			(effects
-				(font
-					(size 1.27 1.27)
-				)
-				(justify left)
-			)
-		)
-		(property "Value" "I_ADC"
-			(at 132.08 53.8479 0)
-			(show_name no)
-			(do_not_autoplace no)
-			(effects
-				(font
-					(size 1.27 1.27)
-				)
-				(justify left)
-			)
-		)
-		(property "Footprint" "TestPoint:TestPoint_Loop_D2.50mm_Drill1.0mm_LowProfile"
-			(at 134.62 55.88 0)
-			(hide yes)
-			(show_name no)
-			(do_not_autoplace no)
-			(effects
-				(font
-					(size 1.27 1.27)
-				)
-			)
-		)
-		(property "Datasheet" ""
-			(at 134.62 55.88 0)
-			(hide yes)
-			(show_name no)
-			(do_not_autoplace no)
-			(effects
-				(font
-					(size 1.27 1.27)
-				)
-			)
-		)
-		(property "Description" "test point"
-			(at 129.54 55.88 0)
-			(hide yes)
-			(show_name no)
-			(do_not_autoplace no)
-			(effects
-				(font
-					(size 1.27 1.27)
-				)
-			)
-		)
-		(property "LCSC" ""
-			(at 129.54 55.88 0)
-			(hide yes)
-			(show_name no)
-			(do_not_autoplace no)
-			(effects
-				(font
-					(size 1.27 1.27)
-				)
-			)
-		)
-		(pin "1"
-		)
-		(instances
-			(project "PS-LVCarrier"
-				(path "/9bab2d9d-20f3-40ef-8545-e1299efec47e/10a2a81d-fff8-4091-b6ef-9685e4bd9514/a12cc91e-7ffe-4aca-bb00-a063147b4e50"
-					(reference "TP41")
-					(unit 1)
-				)
-				(path "/9bab2d9d-20f3-40ef-8545-e1299efec47e/b521073a-8409-41eb-9cdc-cffa14c92055/37ef47ed-2aee-4ae2-b946-13f1b7a76e72"
-					(reference "TP11")
-					(unit 1)
-				)
-				(path "/9bab2d9d-20f3-40ef-8545-e1299efec47e/4f26e4eb-a337-4f9d-865d-e2c0801c36ac/a57b6f22-cd56-4351-a5e4-2e9e02d85251/72c78d2c-2a65-43a0-ad78-90d0e31c028b"
-					(reference "TP24")
-					(unit 1)
-				)
-			)
-		)
-	)
-	(symbol
 		(lib_id "Device:R")
 		(at 129.54 60.96 0)
@@
 					(unit 1)
 				)
-			)
-		)
-	)
-	(symbol
-		(lib_id "Connector:TestPoint")
-		(at 63.5 64.77 0)
-		(mirror y)
-		(unit 1)
-		(body_style 1)
-		(exclude_from_sim no)
-		(in_bom yes)
-		(on_board yes)
-		(in_pos_files yes)
-		(dnp no)
-		(property "Reference" "TP10"
-			(at 60.96 60.1979 0)
-			(show_name no)
-			(do_not_autoplace no)
-			(effects
-				(font
-					(size 1.27 1.27)
-				)
-				(justify left)
-			)
-		)
-		(property "Value" "V_ADC"
-			(at 60.96 62.7379 0)
-			(show_name no)
-			(do_not_autoplace no)
-			(effects
-				(font
-					(size 1.27 1.27)
-				)
-				(justify left)
-			)
-		)
-		(property "Footprint" "TestPoint:TestPoint_Loop_D2.50mm_Drill1.0mm_LowProfile"
-			(at 58.42 64.77 0)
-			(hide yes)
-			(show_name no)
-			(do_not_autoplace no)
-			(effects
-				(font
-					(size 1.27 1.27)
-				)
-			)
-		)
-		(property "Datasheet" ""
-			(at 58.42 64.77 0)
-			(hide yes)
-			(show_name no)
-			(do_not_autoplace no)
-			(effects
-				(font
-					(size 1.27 1.27)
-				)
-			)
-		)
-		(property "Description" "test point"
-			(at 63.5 64.77 0)
-			(hide yes)
-			(show_name no)
-			(do_not_autoplace no)
-			(effects
-				(font
-					(size 1.27 1.27)
-				)
-			)
-		)
-		(property "LCSC" ""
-			(at 63.5 64.77 0)
-			(hide yes)
-			(show_name no)
-			(do_not_autoplace no)
-			(effects
-				(font
-					(size 1.27 1.27)
-				)
-			)
-		)
-		(pin "1"
-		)
-		(instances
-			(project "PS-LVCarrier"
-				(path "/9bab2d9d-20f3-40ef-8545-e1299efec47e/10a2a81d-fff8-4091-b6ef-9685e4bd9514/a12cc91e-7ffe-4aca-bb00-a063147b4e50"
-					(reference "TP40")
-					(unit 1)
-				)
-				(path "/9bab2d9d-20f3-40ef-8545-e1299efec47e/b521073a-8409-41eb-9cdc-cffa14c92055/37ef47ed-2aee-4ae2-b946-13f1b7a76e72"
-					(reference "TP10")
-					(unit 1)
-				)
-				(path "/9bab2d9d-20f3-40ef-8545-e1299efec47e/4f26e4eb-a337-4f9d-865d-e2c0801c36ac/a57b6f22-cd56-4351-a5e4-2e9e02d85251/72c78d2c-2a65-43a0-ad78-90d0e31c028b"
-					(reference "TP23")
-					(unit 1)
-				)

Commit message: switch to pc...
Connections:
- net +3V3 renamed VS
- net VOUT: no longer names the net of R34.1, U2.7 (VOUT)
Changed lines of the file:
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@@
 	(wire
 		(pts
-			(xy 148.59 57.15) (xy 148.59 58.42)
+			(xy 148.59 55.88) (xy 148.59 58.42)
 		)
 		(stroke
@@
 			(width 0)
 			(type default)
-		)
-	)
-	(label "VS"
-		(at 119.38 50.8 0)
-		(effects
-			(font
-				(size 1.27 1.27)
-			)
-			(justify left bottom)
-		)
-	)
-	(label "VOUT"
-		(at 125.73 55.88 180)
-		(effects
-			(font
-				(size 1.27 1.27)
-			)
-			(justify right bottom)
-		)
-	)
-	(label "VS"
-		(at 148.59 58.42 0)
-		(effects
-			(font
-				(size 1.27 1.27)
-			)
-			(justify left bottom)
 		)
 	)
@@
 		)
 	)
+	(hierarchical_label "VS"
+		(shape input)
+		(at 148.59 55.88 0)
+		(effects
+			(font
+				(size 1.27 1.27)
+			)
+			(justify left)
+		)
+	)
 	(hierarchical_label "LV_GND"
 		(shape passive)
@@
 			)
 			(justify right)
+		)
+	)
+	(hierarchical_label "VS"
+		(shape input)
+		(at 124.46 50.8 0)
+		(effects
+			(font
+				(size 1.27 1.27)
+			)
+			(justify left)
 		)
 	)
@@
 	)
 	(symbol
-		(lib_id "power:+3V3")
-		(at 124.46 50.8 0)
-		(unit 1)
-		(body_style 1)
-		(exclude_from_sim no)
-		(in_bom yes)
-		(on_board yes)
-		(in_pos_files yes)
-		(dnp no)
-		(property "Reference" "#PWR014"
-			(at 124.46 54.61 0)
-			(hide yes)
-			(show_name no)
-			(do_not_autoplace no)
-			(effects
-				(font
-					(size 1.27 1.27)
-				)
-			)
-		)
-		(property "Value" "+3V3"
-			(at 123.952 46.228 0)
-			(show_name no)
-			(do_not_autoplace no)
-			(effects
-				(font
-					(size 1.27 1.27)
-				)
-			)
-		)
-		(property "Footprint" ""
-			(at 124.46 50.8 0)
-			(hide yes)
-			(show_name no)
-			(do_not_autoplace no)
-			(effects
-				(font
-					(size 1.27 1.27)
-				)
-			)
-		)
-		(property "Datasheet" ""
-			(at 124.46 50.8 0)
-			(hide yes)
-			(show_name no)
-			(do_not_autoplace no)
-			(effects
-				(font
-					(size 1.27 1.27)
-				)
-			)
-		)
-		(property "Description" "Power symbol creates a global label with name \"+3V3\""
-			(at 124.46 50.8 0)
-			(hide yes)
-			(show_name no)
-			(do_not_autoplace no)
-			(effects
-				(font
-					(size 1.27 1.27)
-				)
-			)
-		)
-		(pin "1"
-		)
-		(instances
-			(project "PS-LVCarrier"
-				(path "/9bab2d9d-20f3-40ef-8545-e1299efec47e/10a2a81d-fff8-4091-b6ef-9685e4bd9514/a12cc91e-7ffe-4aca-bb00-a063147b4e50"
-					(reference "#PWR033")
-					(unit 1)
-				)
-				(path "/9bab2d9d-20f3-40ef-8545-e1299efec47e/b521073a-8409-41eb-9cdc-cffa14c92055/37ef47ed-2aee-4ae2-b946-13f1b7a76e72"
-					(reference "#PWR014")
-					(unit 1)
-				)
-				(path "/9bab2d9d-20f3-40ef-8545-e1299efec47e/4f26e4eb-a337-4f9d-865d-e2c0801c36ac/a57b6f22-cd56-4351-a5e4-2e9e02d85251/72c78d2c-2a65-43a0-ad78-90d0e31c028b"
-					(reference "#PWR031")
-					(unit 1)
-				)
-			)
-		)
-	)
-	(symbol
 		(lib_id "Device:R")
 		(at 67.31 58.42 0)
@@
 					(unit 1)
 				)
-			)
-		)
-	)
-	(symbol
-		(lib_id "power:+3V3")
-		(at 148.59 57.15 0)
-		(unit 1)
-		(body_style 1)
-		(exclude_from_sim no)
-		(in_bom yes)
-		(on_board yes)
-		(in_pos_files yes)
-		(dnp no)
-		(property "Reference" "#PWR015"
-			(at 148.59 60.96 0)
-			(hide yes)
-			(show_name no)
-			(do_not_autoplace no)
-			(effects
-				(font
-					(size 1.27 1.27)
-				)
-			)
-		)
-		(property "Value" "+3V3"
-			(at 148.082 52.578 0)
-			(show_name no)
-			(do_not_autoplace no)
-			(effects
-				(font
-					(size 1.27 1.27)
-				)
-			)
-		)
-		(property "Footprint" ""
-			(at 148.59 57.15 0)
-			(hide yes)
-			(show_name no)
-			(do_not_autoplace no)
-			(effects
-				(font
-					(size 1.27 1.27)
-				)
-			)
-		)
-		(property "Datasheet" ""
-			(at 148.59 57.15 0)
-			(hide yes)
-			(show_name no)
-			(do_not_autoplace no)
-			(effects
-				(font
-					(size 1.27 1.27)
-				)
-			)
-		)
-		(property "Description" "Power symbol creates a global label with name \"+3V3\""
-			(at 148.59 57.15 0)
-			(hide yes)
-			(show_name no)
-			(do_not_autoplace no)
-			(effects
-				(font
-					(size 1.27 1.27)
-				)
-			)
-		)
-		(pin "1"
-		)
-		(instances
-			(project "PS-LVCarrier"
-				(path "/9bab2d9d-20f3-40ef-8545-e1299efec47e/10a2a81d-fff8-4091-b6ef-9685e4bd9514/a12cc91e-7ffe-4aca-bb00-a063147b4e50"
-					(reference "#PWR034")
-					(unit 1)
-				)
-				(path "/9bab2d9d-20f3-40ef-8545-e1299efec47e/b521073a-8409-41eb-9cdc-cffa14c92055/37ef47ed-2aee-4ae2-b946-13f1b7a76e72"
-					(reference "#PWR015")
-					(unit 1)
-				)
-				(path "/9bab2d9d-20f3-40ef-8545-e1299efec47e/4f26e4eb-a337-4f9d-865d-e2c0801c36ac/a57b6f22-cd56-4351-a5e4-2e9e02d85251/72c78d2c-2a65-43a0-ad78-90d0e31c028b"
-					(reference "#PWR032")
-					(unit 1)
-				)

Commit message: oops
Parts:
- C28, C30: P/N (none) -> MLASH168SB7104KTNA01
- C29: P/N (none) -> MSASU105SB5473KFNA01
- U2: LCSC P/N (none) -> C3684136; P/N (none) -> TMCS1107A2UQDR
Changed lines of the file:
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@@
+			)
+		)
+		(property "LCSC P/N" "C3684136"
+			(at 85.09 50.8 0)
+			(hide yes)
+			(show_name no)
+			(do_not_autoplace no)
+			(effects
+				(font
+					(size 1.27 1.27)
+				)
+			)
+		)
+		(property "P/N" "TMCS1107A2UQDR"
+			(at 85.09 50.8 0)
+			(hide yes)
+			(show_name no)
+			(do_not_autoplace no)
+			(effects
+				(font
+					(size 1.27 1.27)
+				)
 			)
 		)
@@
 		)
 		(property "LCSC" ""
+			(at 59.69 71.12 0)
+			(hide yes)
+			(show_name no)
+			(do_not_autoplace no)
+			(effects
+				(font
+					(size 1.27 1.27)
+				)
+			)
+		)
+		(property "P/N" "MLASH168SB7104KTNA01"
 			(at 59.69 71.12 0)
 			(hide yes)
@@
 			)
 		)
+		(property "P/N" "MSASU105SB5473KFNA01"
+			(at 129.54 72.39 0)
+			(hide yes)
+			(show_name no)
+			(do_not_autoplace no)
+			(effects
+				(font
+					(size 1.27 1.27)
+				)
+			)
+		)
 		(pin "2"
 		)
@@
 			(at 148.59 60.96 0)
 			(hide yes)
+			(show_name no)
+			(do_not_autoplace no)
+			(effects
+				(font
+					(size 1.27 1.27)
+				)
+			)
+		)
+		(property "P/N" "MLASH168SB7104KTNA01"
+			(at 148.59 60.96 0)
+			(hide yes)

Commit message: added most p/n, still in progress but saving
Parts:
- R32: Assemble (none) -> -- mixed values --; Mouser Part Number (none) -> -- mixed values --; P/N CRCW060310K0FKEI -> -- mixed values --
- R33: Assemble (none) -> -- mixed values --
- R34: Assemble Y -> -- mixed values --; LCSC P/N (none) -> C23162
Changed lines of the file:
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@@
 			)
 		)
-		(property "Datasheet" "https://www.mouser.com/ProductDetail/Vishay/CRCW06034K70FKEA?qs=4E3O%252BEEZcdLDG%2FSk4GmlWQ%3D%3D&srsltid=AfmBOoqcFOp_RyXq2yrOgJIYefuosjeBTcR7TE2c5E8zthdTaDTezlM7"
+		(property "Datasheet" "-- mixed values --"
 			(at 129.54 60.96 0)
 			(hide yes)
@@
 			)
 		)
-		(property "Assemble" "Y"
+		(property "Assemble" "-- mixed values --"
 			(at 129.54 60.96 90)
 			(hide yes)
@@
 		)
 		(property "LCSC" ""
+			(at 129.54 60.96 0)
+			(hide yes)
+			(show_name no)
+			(do_not_autoplace no)
+			(effects
+				(font
+					(size 1.27 1.27)
+				)
+			)
+		)
+		(property "LCSC P/N" "C23162"
 			(at 129.54 60.96 0)
 			(hide yes)
@@
 			)
 		)
-		(property "Datasheet" ""
+		(property "Datasheet" "-- mixed values --"
 			(at 67.31 71.12 0)
 			(hide yes)
@@
 		)
 		(property "LCSC" ""
+			(at 67.31 71.12 0)
+			(hide yes)
+			(show_name no)
+			(do_not_autoplace no)
+			(effects
+				(font
+					(size 1.27 1.27)
+				)
+			)
+		)
+		(property "Assemble" "-- mixed values --"
 			(at 67.31 71.12 0)
 			(hide yes)
@@
 			)
 		)
-		(property "Datasheet" ""
+		(property "Datasheet" "-- mixed values --"
 			(at 67.31 58.42 0)
 			(hide yes)
@@
 			)
 		)
-		(property "Description" "Resistor"
+		(property "Description" "-- mixed values --"
 			(at 67.31 58.42 0)
 			(hide yes)
@@
 			)
 		)
-		(property "P/N" "CRCW060310K0FKEI "
+		(property "P/N" "-- mixed values --"
 			(at 67.31 58.42 90)
 			(hide yes)
@@
 			(at 67.31 58.42 0)
 			(hide yes)
+			(show_name no)
+			(do_not_autoplace no)
+			(effects
+				(font
+					(size 1.27 1.27)
+				)
+			)
+		)
+		(property "Assemble" "-- mixed values --"
+			(at 67.31 58.42 0)
+			(hide yes)
+			(show_name no)
+			(do_not_autoplace no)
+			(effects
+				(font
+					(size 1.27 1.27)
+				)
+			)
+		)
+		(property "Mouser Part Number" "-- mixed values --"
+			(at 67.31 58.42 0)
+			(hide yes)
