File: hardware/HSS.kicad_sch (KiCad schematic)
At the start: 29 parts, among them IC8 TPS2HCS08AQPWPRQ1

Commit message: switch to laptop
Connections:
- net FLT_WAKE: no longer IC8.12 (~{FLT_}/_~{WAKE_SIG}), R112.1
- net SPI_CS: no longer IC8.15 (NCS), R104.2
- new net HSS_FLT_WAKE: IC8.12 (~{FLT_}/_~{WAKE_SIG}), R112.1
- new net HSS_SPI_CS: IC8.15 (NCS), R104.2
Changed lines of the file:
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@@
 	(wire
 		(pts
-			(xy 142.24 140.97) (xy 132.08 140.97)
+			(xy 146.05 140.97) (xy 132.08 140.97)
 		)
 		(stroke
@@
 	(wire
 		(pts
-			(xy 63.5 95.25) (xy 55.88 95.25)
+			(xy 67.31 95.25) (xy 55.88 95.25)
 		)
 		(stroke
@@
 		)
 	)
-	(label "FLT_WAKE"
-		(at 142.24 140.97 180)
+	(label "HSS_FLT_WAKE"
+		(at 146.05 140.97 180)
 		(effects
 			(font
@@
 		)
 	)
-	(label "SPI_CS"
+	(label "HSS_SPI_CS"
 		(at 97.79 99.06 0)
 		(effects
@@
 		)
 	)
-	(label "SPI_CS"
-		(at 63.5 95.25 180)
+	(label "HSS_SPI_CS"
+		(at 67.31 95.25 180)
 		(effects
 			(font
@@
 		)
 	)
-	(label "FLT_WAKE"
+	(label "HSS_FLT_WAKE"
 		(at 97.79 88.9 0)
 		(effects

Commit message: save me
Connections:
- net HSS_MOSI: no longer R105.1, R106.2
- new net HSS_SCLK: R105.1, R106.2
Changed lines of the file:
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@@
 		)
 	)
-	(label "HSS_MOSI"
+	(label "HSS_SCLK"
 		(at 88.9 168.91 180)
 		(effects

Commit message: switch to pc...
Connections:
- net HSS_SCLK is gone; now on net HSS_MOSI: R105.1, R106.2
Changed lines of the file:
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@@
 	)
 	(junction
+		(at 114.3 39.37)
+		(diameter 0)
+		(color 0 0 0 0)
+	)
+	(junction
 		(at 44.45 95.25)
 		(diameter 0)
@@
 	)
 	(junction
-		(at 114.3 39.37)
-		(diameter 0)
-		(color 0 0 0 0)
-	)
-	(junction
 		(at 102.87 39.37)
 		(diameter 0)
@@
 	(wire
 		(pts
-			(xy 114.3 39.37) (xy 121.92 39.37)
+			(xy 114.3 39.37) (xy 118.11 39.37)
 		)
 		(stroke
@@
 		)
 	)
-	(label "HSS_SCLK"
+	(label "HSS_MOSI"
 		(at 88.9 168.91 180)
 		(effects
@@
 		)
 	)
-	(label "VBB"
-		(at 118.11 78.74 180)
-		(effects
-			(font
-				(size 1.27 1.27)
-			)
-			(justify right bottom)
-		)
-	)
 	(label "HSS_SNS"
 		(at 161.29 128.27 0)
@@
 		)
 	)
-	(label "VBB"
-		(at 121.92 39.37 180)
-		(effects
-			(font
-				(size 1.27 1.27)
-			)
-			(justify right bottom)
-		)
-	)
 	(label "VDD"
 		(at 58.42 44.45 180)
@@
 		)
 	)
+	(hierarchical_label "12V_HSS"
+		(shape input)
+		(at 118.11 39.37 0)
+		(effects
+			(font
+				(size 1.27 1.27)
+			)
+			(justify left)
+		)
+	)

Commit message: remapped pins
Connections:
- net HSS_MOSI: no longer R105.1, R106.2
- new net HSS_SCLK: R105.1, R106.2
Changed lines of the file:
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@@
 		)
 	)
-	(label "HSS_MOSI"
+	(label "HSS_SCLK"
 		(at 88.9 168.91 180)
 		(effects

Commit message: oops
Parts:
- C83: P/N (none) -> MLASH168SB7104KTNA01
- C85: LCSC P/N C696901 -> C15849; P/N (none) -> MLASU168SB5105KTNA01
- C86: P/N (none) -> MSASU105SB5473KFNA01
- R101: P/N (none) -> CRCW060310R0FKEE
- R104: LCSC P/N (none) -> C2930077; P/N (none) -> FRC0603F22R0TS
- R105, R99: LCSC P/N C23162 -> C2930077; P/N (none) -> FRC0603F22R0TS
- R109: LCSC P/N (none) -> C22356650; P/N (none) -> RCA03220RJLF
- R115: LCSC P/N (none) -> C23179; P/N (none) -> CRCW1206470RFKEA
Changed lines of the file:
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@@
 			)
 		)
+		(property "P/N" "CRCW060310R0FKEE"
+			(at 44.45 44.45 90)
+			(hide yes)
+			(show_name no)
+			(do_not_autoplace no)
+			(effects
+				(font
+					(size 1.27 1.27)
+				)
+			)
+		)
 		(pin "2"
 		)
@@
 			)
 		)
-		(property "LCSC P/N" "C23162"
+		(property "LCSC P/N" "C2930077"
 			(at 41.91 168.91 90)
 			(hide yes)
@@
 			)
 		)
+		(property "P/N" "FRC0603F22R0TS"
+			(at 41.91 168.91 90)
+			(hide yes)
+			(show_name no)
+			(do_not_autoplace no)
+			(effects
+				(font
+					(size 1.27 1.27)
+				)
+			)
+		)
 		(pin "2"
 		)
@@
 			)
 		)
+		(property "P/N" "MLASH168SB7104KTNA01"
+			(at 78.74 137.16 0)
+			(hide yes)
+			(show_name no)
+			(do_not_autoplace no)
+			(effects
+				(font
+					(size 1.27 1.27)
+				)
+			)
+		)
 		(pin "2"
 		)
@@
 			)
 		)
-		(property "LCSC P/N" ""
+		(property "LCSC P/N" "C23179"
 			(at 181.61 121.92 0)
 			(hide yes)
@@
 			)
 		)
+		(property "P/N" "CRCW1206470RFKEA "
+			(at 181.61 121.92 0)
+			(hide yes)
+			(show_name no)
+			(do_not_autoplace no)
+			(effects
+				(font
+					(size 1.27 1.27)
+				)
+			)
+		)
 		(pin "2"
 		)
@@
 			)
 		)
+		(property "P/N" "MSASU105SB5473KFNA01"
+			(at 171.45 133.35 0)
+			(hide yes)
+			(show_name no)
+			(do_not_autoplace no)
+			(effects
+				(font
+					(size 1.27 1.27)
+				)
+			)
+		)
 		(pin "2"
 		)
@@
 			)
 		)
+		(property "LCSC P/N" "C2930077"
+			(at 52.07 95.25 90)
+			(hide yes)
+			(show_name no)
+			(do_not_autoplace no)
+			(effects
+				(font
+					(size 1.27 1.27)
+				)
+			)
+		)
+		(property "P/N" "FRC0603F22R0TS"
+			(at 52.07 95.25 90)
+			(hide yes)
+			(show_name no)
+			(do_not_autoplace no)
+			(effects
+				(font
+					(size 1.27 1.27)
+				)
+			)
+		)
 		(pin "2"
 		)
@@
 			)
 		)
-		(property "LCSC P/N" "C696901"
+		(property "LCSC P/N" "C15849"
 			(at 102.87 44.45 0)
 			(hide yes)
@@
 			)
 		)
+		(property "P/N" "MLASU168SB5105KTNA01"
+			(at 102.87 44.45 0)
+			(hide yes)
+			(show_name no)
+			(do_not_autoplace no)
+			(effects
+				(font
+					(size 1.27 1.27)
+				)
+			)
+		)
 		(pin "2"
 		)
@@
 			)
 		)
-		(property "LCSC P/N" "C23162"
+		(property "LCSC P/N" "C2930077"
 			(at 74.93 168.91 90)
 			(hide yes)
@@
 			)
 		)
+		(property "P/N" "FRC0603F22R0TS"
+			(at 74.93 168.91 90)
+			(hide yes)
+			(show_name no)
+			(do_not_autoplace no)
+			(effects
+				(font
+					(size 1.27 1.27)
+				)
+			)
+		)
 		(pin "2"
 		)
@@
 			(at 111.76 93.98 90)
 			(hide yes)
+			(show_name no)
+			(do_not_autoplace no)
+			(effects
+				(font
+					(size 1.27 1.27)
+				)
+			)
+		)
+		(property "LCSC P/N" "C22356650"
+			(at 111.76 93.98 90)
+			(hide yes)
+			(show_name no)
+			(do_not_autoplace no)
+			(effects
+				(font
+					(size 1.27 1.27)
+				)
+			)
+		)
+		(property "P/N" "RCA03220RJLF"
+			(at 111.76 93.98 90)
+			(hide yes)

Commit message: added most p/n, still in progress but saving
Parts:
- C82: P/N (none) -> CL10B474KA8NNNC
- C84: LCSC P/N C100040 -> C1588; P/N (none) -> MLASU063SB7102KFNA01
- C87: LCSC P/N C77047 -> (none)
- D30: LCSC P/N C84263 -> -- mixed values --; P/N (none) -> -- mixed values --
- F10: footprint LHRS_Power:Fuse-3557-2 -> -- mixed values --; Digikey P/N 36-3557-2-ND -> -- mixed values --; LCSC P/N C3205238 -> -- mixed values --; Mouser P/N 534-3557-2 -> -- mixed values --; P/N 3557-2 -> -- mixed values --
- R100, R110: Assemble (none) -> -- mixed values --; P/N (none) -> CRCW06034K70FKEA
- R102, R103, R106, R107, R108, R111, R112, R113: Assemble (none) -> -- mixed values --; Mouser Part Number (none) -> -- mixed values --; P/N (none) -> -- mixed values --
- R114: Assemble (none) -> -- mixed values --; LCSC P/N C21190 -> C23162; P/N (none) -> CRCW06034K70FKEA

Commit message: more pns i go now
Parts:
- D30: LCSC P/N -- mixed values -- -> (none); P/N -- mixed values -- -> (none)
- F10: footprint -- mixed values -- -> LHRS_Power:Fuse-3557-2; LCSC P/N -- mixed values -- -> C352820; P/N -- mixed values -- -> 3557-2
- TP42: now left out of the parts list
Changed lines of the file:
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@@
 		(body_style 1)
 		(exclude_from_sim no)
-		(in_bom yes)
+		(in_bom no)
 		(on_board yes)
 		(in_pos_files yes)
@@
 			)
 		)
-		(property "Footprint" "-- mixed values --"
+		(property "Footprint" "LHRS_Power:Fuse-3557-2"
 			(at 46.99 132.588 90)
 			(hide yes)
@@
 			)
 		)
-		(property "P/N" "-- mixed values --"
+		(property "P/N" "3557-2"
 			(at 46.99 130.81 0)
 			(hide yes)
@@
 			)
 		)
-		(property "LCSC P/N" "-- mixed values --"
+		(property "LCSC P/N" "C352820"
 			(at 46.99 130.81 0)
 			(hide yes)
@@
 			)
 		)
-		(property "LCSC P/N" "-- mixed values --"
+		(property "LCSC P/N" ""
 			(at 52.07 140.97 0)
 			(hide yes)
@@
 			)
 		)
-		(property "P/N" "-- mixed values --"
+		(property "P/N" ""
 			(at 52.07 140.97 0)
 			(hide yes)

Commit message: done
Parts:
- C87: LCSC P/N (none) -> C53084536; P/N (none) -> CC0603X5R25V225KN
Changed lines of the file:
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@@
 			)
 		)
-		(property "LCSC P/N" ""
+		(property "LCSC P/N" "C53084536"
 			(at 193.04 121.92 0)
 			(hide yes)
@@
 			(at 193.04 121.92 0)
 			(hide yes)
+			(show_name no)
+			(do_not_autoplace no)
+			(effects
+				(font
+					(size 1.27 1.27)
+				)
+			)
+		)
+		(property "P/N" "CC0603X5R25V225KN"
+			(at 193.04 121.92 0)
+			(hide yes)
