File: hardware/USB.kicad_sch (KiCad schematic)
At the start: 6 parts, among them J17 USB_C_Receptacle_USB2.0_16P

Commit message: remapped pins
Changed lines of the file:
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@@
+		)
+	)
+	(label "CC2"
+		(at 72.39 55.88 180)
+		(effects
+			(font
+				(size 1.27 1.27)
+			)
+			(justify right bottom)
+		)
+	)
+	(label "CC2"
+		(at 129.54 33.02 0)
+		(effects
+			(font
+				(size 1.27 1.27)
+			)
+			(justify left bottom)
 		)
 	)
@@
 		)
 	)
-	(hierarchical_label "USB_5V"
-		(shape output)
-		(at 87.63 43.18 90)
+	(label "CC1"
+		(at 121.92 33.02 0)
 		(effects
 			(font
 				(size 1.27 1.27)
 			)
-			(justify left)
+			(justify left bottom)
 		)
 	)
-	(hierarchical_label "CC1"
-		(shape bidirectional)
-		(at 72.39 53.34 0)
+	(label "CC1"
+		(at 72.39 53.34 180)
+		(effects
+			(font
+				(size 1.27 1.27)
+			)
+			(justify right bottom)
+		)
+	)
+	(hierarchical_label "USB_5V"
+		(shape output)
+		(at 87.63 43.18 90)
 		(effects
 			(font
@@
 			)
 			(justify right)
-		)
-	)
-	(hierarchical_label "CC2"
-		(shape bidirectional)
-		(at 72.39 55.88 0)
-		(effects
-			(font
-				(size 1.27 1.27)
-			)
-			(justify left)
 		)
 	)
@@
 		(effects
 			(font
-				(size 1.27 1.27)
-			)
-			(justify right)
-		)
-	)
-	(hierarchical_label "CC1"
-		(shape bidirectional)
-		(at 121.92 33.02 180)
-		(effects
-			(font
-				(size 1.27 1.27)
-			)
-			(justify right)
-		)
-	)
-	(hierarchical_label "CC2"
-		(shape bidirectional)
-		(at 129.54 33.02 180)
-		(effects
-			(font

Commit message: added most p/n, still in progress but saving
Parts:
- C72: Mouser P/N (none) -> -- mixed values --; Mouser Part Number (none) -> -- mixed values --
- R2, R3: P/N (none) -> CRCW06035K10FKEC
Changed lines of the file:
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@@
 			)
 		)
-		(property "Description" "Unpolarized capacitor"
+		(property "Description" "-- mixed values --"
 			(at 87.63 54.61 0)
 			(hide yes)
@@
 		)
 		(property "LCSC P/N" "C440198"
+			(at 87.63 54.61 0)
+			(hide yes)
+			(show_name no)
+			(do_not_autoplace no)
+			(effects
+				(font
+					(size 1.27 1.27)
+				)
+			)
+		)
+		(property "Mouser P/N" "-- mixed values --"
+			(at 87.63 54.61 0)
+			(hide yes)
+			(show_name no)
+			(do_not_autoplace no)
+			(effects
+				(font
+					(size 1.27 1.27)
+				)
+			)
+		)
+		(property "Mouser Part Number" "-- mixed values --"
 			(at 87.63 54.61 0)
 			(hide yes)
@@
 		)
 		(property "LCSC P/N" "C23186"
+			(at 123.19 39.37 90)
+			(hide yes)
+			(show_name no)
+			(do_not_autoplace no)
+			(effects
+				(font
+					(size 1.27 1.27)
+				)
+			)
+		)
+		(property "P/N" "CRCW06035K10FKEC "
 			(at 123.19 39.37 90)
 			(hide yes)
@@
 			(at 130.81 39.37 90)
 			(hide yes)
+			(show_name no)
+			(do_not_autoplace no)
+			(effects
+				(font
+					(size 1.27 1.27)
+				)
+			)
+		)
+		(property "P/N" "CRCW06035K10FKEC "
+			(at 130.81 39.37 90)
+			(hide yes)

Commit message: more pns i go now
Parts:
- J17: now left out of the parts list
Changed lines of the file:
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@@
 		(body_style 1)
 		(exclude_from_sim no)
-		(in_bom yes)
+		(in_bom no)
 		(on_board yes)
 		(in_pos_files yes)

Commit message: save changes
Parts:
- C72: Mouser P/N -- mixed values -- -> (none)
Changed lines of the file:
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@@
-			)
-		)
-		(property "Mouser P/N" "-- mixed values --"
-			(at 87.63 54.61 0)
-			(hide yes)
-			(show_name no)
-			(do_not_autoplace no)
-			(effects
-				(font
-					(size 1.27 1.27)
-				)
 			)
 		)
