File: hardware/supplementalbattery.kicad_sch (KiCad schematic)
At the start: 25 parts, among them J2 LV_ENABLE, J3 SUPP, Q10 IRLML0030

Commit message: switch to pc...
Connections:
- net CC Buck/CC_VOUT: now also D3.1 (K); no longer D3.2 (A)
- net LV_GND: now also D3.2 (A); no longer D3.1 (K)
Other:
- sheet Voltage + Current Sense ports: added VS; removed none
- moved on the sheet: D3
Changed lines of the file:
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@@
 	)
 	(junction
-		(at 68.58 120.65)
-		(diameter 0)
-		(color 0 0 0 0)
-	)
-	(junction
 		(at 59.69 120.65)
 		(diameter 0)
@@
 	(wire
 		(pts
-			(xy 161.29 128.27) (xy 163.83 128.27)
+			(xy 161.29 129.54) (xy 163.83 129.54)
 		)
 		(stroke
@@
 	(wire
 		(pts
-			(xy 68.58 120.65) (xy 73.66 120.65)
-		)
-		(stroke
-			(width 0)
-			(type default)
-		)
-	)
-	(wire
-		(pts
 			(xy 54.61 158.75) (xy 68.58 158.75)
 		)
@@
 	(wire
 		(pts
+			(xy 161.29 127) (xy 165.1 127)
+		)
+		(stroke
+			(width 0)
+			(type default)
+		)
+	)
+	(wire
+		(pts
 			(xy 186.69 88.9) (xy 189.23 88.9)
 		)
@@
 		)
 	)
-	(global_label "LVD_ENABLE"
+	(global_label "DIODE_EN"
 		(shape input)
 		(at 123.19 168.91 180)
@@
 		)
 		(property "Intersheetrefs" "${INTERSHEET_REFS}"
-			(at 108.8353 168.91 0)
+			(at 111.1334 168.91 0)
 			(hide yes)
 			(show_name no)
@@
 		)
 	)
-	(global_label "LVD_ENABLE"
-		(shape input)
-		(at 73.66 120.65 0)
-		(fields_autoplaced yes)
-		(effects
-			(font
-				(size 1.27 1.27)
-			)
-			(justify left)
-		)
-		(property "Intersheetrefs" "${INTERSHEET_REFS}"
-			(at 88.0147 120.65 0)
-			(hide yes)
-			(show_name no)
-			(do_not_autoplace no)
-			(effects
-				(font
-					(size 1.27 1.27)
-				)
-				(justify left)
-			)
-		)
-	)
 	(hierarchical_label "LV_GND"
 		(shape bidirectional)
@@
 		)
 	)
+	(hierarchical_label "VS"
+		(shape input)
+		(at 165.1 127 0)
+		(effects
+			(font
+				(size 1.27 1.27)
+			)
+			(justify left)
+		)
+	)
 	(hierarchical_label "SUPP_12V_FUSED"
 		(shape output)
-		(at 163.83 128.27 0)
+		(at 163.83 129.54 0)
 		(effects
 			(font
@@
 	(symbol
 		(lib_id "Device:D_Zener")
-		(at 194.31 87.63 90)
+		(at 194.31 87.63 270)
 		(unit 1)
 		(body_style 1)
@@
 					(size 1.27 1.27)
 				)
-				(justify right)
+				(justify left)
 			)
 		)
@@
 					(size 1.27 1.27)
 				)
-				(justify right)
+				(justify left)
 			)
 		)
@@
 		)
 		(pin "SENSE_OUT" output
-			(at 161.29 128.27 0)
+			(at 161.29 129.54 0)
 			(effects
 				(font
@@
 			(effects
 				(font
+					(size 1.27 1.27)
+				)
+				(justify right)
+			)
+		)
+		(pin "VS" input
+			(at 161.29 127 0)
+			(effects
+				(font

Commit message: switch to pc
Connections:
- net LV_ENABLE-: now reaches J2.2 (Pin_2)
- no-connect marks 1 -> 0
Changed lines of the file:
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@@
 		(color 0 0 0 0)
-	)
-	(no_connect
-		(at 44.45 180.34)
 	)
 	(bus_entry
@@
 		(pts
 			(xy 54.61 144.78) (xy 54.61 147.32)
+		)
+		(stroke
+			(width 0)
+			(type default)
+		)
+	)
+	(wire
+		(pts
+			(xy 57.15 180.34) (xy 44.45 180.34)
 		)
 		(stroke
@@
 		(effects
 			(font
+				(size 1.27 1.27)
+			)
+			(justify right bottom)
+		)
+	)
+	(label "LV_ENABLE-"
+		(at 57.15 180.34 180)
+		(effects
+			(font

Commit message: oops
Parts:
- C57: P/N (none) -> MLASH168SB7104KTNA01
- R61: LCSC P/N (none) -> C25819; P/N CRCW06031K00FKEI -> CRCW060347K0FKECC
- R68: LCSC P/N C21190 -> C31850; P/N CRCW06031K00FKEI -> CRCW060322K0FKEAHP
- R82: LCSC P/N C23162 -> C2907165; P/N CRCW06034K30FKTA -> CRCW06034K30FKEA
- R83: LCSC P/N C25804 -> C22356655; P/N CRCW060310K0FKEI -> RCA0333KJLF
Changed lines of the file:
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@@
 			)
 		)
-		(property "P/N" "CRCW060310K0FKEI "
+		(property "P/N" "RCA0333KJLF"
 			(at 231.14 123.19 0)
 			(hide yes)
@@
 			)
 		)
-		(property "LCSC P/N" "C25804"
+		(property "LCSC P/N" "C22356655"
 			(at 231.14 123.19 0)
 			(hide yes)
@@
 			)
 		)
-		(property "P/N" "CRCW06031K00FKEI "
+		(property "P/N" "CRCW060322K0FKEAHP"
 			(at 59.69 125.73 0)
 			(hide yes)
@@
 			)
 		)
-		(property "LCSC P/N" "C21190"
+		(property "LCSC P/N" "C31850"
 			(at 59.69 125.73 0)
 			(hide yes)
@@
 			)
 		)
+		(property "P/N" "MLASH168SB7104KTNA01"
+			(at 241.3 135.89 0)
+			(hide yes)
+			(show_name no)
+			(do_not_autoplace no)
+			(effects
+				(font
+					(size 1.27 1.27)
+				)
+			)
+		)
 		(pin "2"
 		)
@@
 			)
 		)
-		(property "P/N" "CRCW06034K30FKTA "
+		(property "P/N" "CRCW06034K30FKEA"
 			(at 214.63 133.35 0)
 			(hide yes)
@@
 			)
 		)
-		(property "LCSC P/N" "C23162"
+		(property "LCSC P/N" "C2907165"
 			(at 214.63 133.35 0)
 			(hide yes)
@@
 			)
 		)
-		(property "P/N" "CRCW06031K00FKEI "
+		(property "P/N" "CRCW060347K0FKECC"
 			(at 52.07 120.65 0)
 			(hide yes)
@@
 			)
 		)
-		(property "LCSC P/N" ""
+		(property "LCSC P/N" "C25819"
 			(at 52.07 120.65 0)
 			(hide yes)

Commit message: ahhahahahhahahhahahhahahhahhaa im so back
Connections:
- net LV_ENABLE: now also J2.2 (Pin_2); no longer J2.1 (Pin_1)
- net LV_ENABLE-: now also J2.1 (Pin_1); no longer J2.2 (Pin_2)
- net LV_GND: now also J3.1 (Pin_1); no longer J3.2 (Pin_2)
- net at F2.1: now also J3.2 (Pin_2); no longer J3.1 (Pin_1)
Other:
- moved on the sheet: J3
Changed lines of the file:
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@@
 	(wire
 		(pts
-			(xy 100.33 130.81) (xy 102.87 130.81)
+			(xy 100.33 125.73) (xy 102.87 125.73)
 		)
 		(stroke
@@
 	(wire
 		(pts
-			(xy 57.15 180.34) (xy 44.45 180.34)
+			(xy 57.15 177.8) (xy 44.45 177.8)
 		)
 		(stroke
@@
 	(wire
 		(pts
-			(xy 44.45 177.8) (xy 57.15 177.8)
+			(xy 44.45 180.34) (xy 57.15 180.34)
 		)
 		(stroke
@@
 	)
 	(label "LV_ENABLE-"
-		(at 57.15 180.34 180)
+		(at 57.15 177.8 180)
 		(effects
 			(font
@@
 	)
 	(label "LV_ENABLE"
-		(at 57.15 177.8 180)
+		(at 57.15 180.34 180)
 		(effects
 			(font
@@
 	(hierarchical_label "LV_GND"
 		(shape bidirectional)
-		(at 102.87 130.81 270)
+		(at 102.87 125.73 270)
 		(effects
 			(font
@@
 	(symbol
 		(lib_id "Connector_Generic:Conn_01x02")
-		(at 95.25 128.27 0)
+		(at 95.25 125.73 0)
 		(mirror y)
 		(unit 1)
@@
 		(fields_autoplaced yes)
 		(property "Reference" "J3"
-			(at 95.25 121.92 0)
+			(at 95.25 119.38 0)
 			(show_name no)
 			(do_not_autoplace no)
@@
 		)
 		(property "Value" "SUPP"
-			(at 95.25 124.46 0)
+			(at 95.25 121.92 0)
 			(show_name no)
 			(do_not_autoplace no)
@@
 		)
 		(property "Footprint" "LHRS_Connectors:AMASS_XT30UPB-M_1x02_P5.0mm_Vertical"
-			(at 95.25 128.27 0)
+			(at 95.25 125.73 0)
 			(hide yes)
 			(show_name no)
@@
 		)
 		(property "Datasheet" ""
-			(at 95.25 128.27 0)
+			(at 95.25 125.73 0)
 			(hide yes)
 			(show_name no)
@@
 		)
 		(property "Description" "Generic connector, single row, 01x02, script generated (kicad-library-utils/schlib/autogen/connector/)"
-			(at 95.25 128.27 0)
+			(at 95.25 125.73 0)
 			(hide yes)
 			(show_name no)
@@
 		)
 		(property "LCSC" ""
-			(at 95.25 128.27 0)
+			(at 95.25 125.73 0)
 			(hide yes)
 			(show_name no)

Commit message: added most p/n, still in progress but saving
Parts:
- D2: value ORA_OUT -> ORA_OUT_LED; footprint LED_SMD:LED_0603_1608Metric_Pad1.05x0.95mm_HandSolder -> -- mixed values --
- F2: LCSC P/N (none) -> -- mixed values --
- R11, R15, R84, R9: Assemble Y -> -- mixed values --; Mouser Part Number (none) -> -- mixed values --; P/N CRCW060310K0FKEI -> -- mixed values --
- R12: Assemble (none) -> -- mixed values --; Mouser Part Number (none) -> -- mixed values --; P/N (none) -> -- mixed values --
- R13: Assemble (none) -> -- mixed values --; LCSC P/N C177867 -> C25803; P/N (none) -> CRCW0603100KFKEE
- R66, R67, R68, R83: Assemble Y -> -- mixed values --
- TP2: value ORA_OUT -> ORA_OUT_TP; footprint TestPoint:TestPoint_Loop_D2.50mm_Drill1.0mm_LowProfile -> -- mixed values --
Changed lines of the file:
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@@
 			)
 		)
-		(property "Assemble" "Y"
+		(property "Assemble" "-- mixed values --"
 			(at 231.14 123.19 0)
 			(hide yes)
@@
 			)
 		)
-		(property "Datasheet" "https://www.mouser.com/ProductDetail/Vishay/CRCW06031K00FKEI?qs=%252B6g0mu59x7LmDUigK4duvw%3D%3D&srsltid=AfmBOoq-qbpfAjzhtzCNjmKpq35FQ1BHTaIyFUz28_1v8HZaKbIrwYgN"
+		(property "Datasheet" "-- mixed values --"
 			(at 59.69 125.73 0)
 			(hide yes)
@@
 			)
 		)
-		(property "Assemble" "Y"
+		(property "Assemble" "-- mixed values --"
 			(at 59.69 125.73 0)
 			(hide yes)
@@
 			)
 		)
-		(property "Description" "Resistor"
+		(property "Description" "-- mixed values --"
 			(at 54.61 153.67 0)
 			(hide yes)
@@
 			)
 		)
-		(property "Assemble" "Y"
+		(property "Assemble" "-- mixed values --"
 			(at 54.61 153.67 0)
 			(hide yes)
@@
 			)
 		)
-		(property "Description" "Resistor"
+		(property "Description" "-- mixed values --"
 			(at 151.13 87.63 0)
 			(hide yes)
@@
 			)
 		)
-		(property "LCSC P/N" "C177867"
+		(property "LCSC P/N" "C25803"
 			(at 151.13 87.63 0)
 			(hide yes)
@@
 		)
 		(property "LCSC" ""
+			(at 151.13 87.63 0)
+			(hide yes)
+			(show_name no)
+			(do_not_autoplace no)
+			(effects
+				(font
+					(size 1.27 1.27)
+				)
+			)
+		)
+		(property "Assemble" "-- mixed values --"
+			(at 151.13 87.63 0)
+			(hide yes)
+			(show_name no)
+			(do_not_autoplace no)
+			(effects
+				(font
+					(size 1.27 1.27)
+				)
+			)
+		)
+		(property "P/N" "CRCW0603100KFKEE"
 			(at 151.13 87.63 0)
 			(hide yes)
@@
 			)
 		)
-		(property "Datasheet" "https://www.mouser.com/ProductDetail/Vishay/CRCW060310K0FKEI?qs=3qWEzBg5KnKofE%252B8acPBRA%3D%3D&srsltid=AfmBOoqKim6ih2rJJ1EIhwDCT-JirqUJIep-ZlqxnK3BQM3p3g1ka950"
+		(property "Datasheet" "-- mixed values --"
 			(at 63.5 93.98 0)
 			(hide yes)
@@
 			)
 		)
-		(property "Description" "Resistor"
+		(property "Description" "-- mixed values --"
 			(at 63.5 93.98 0)
 			(hide yes)
@@
 			)
 		)
-		(property "P/N" "CRCW060310K0FKEI "
+		(property "P/N" "-- mixed values --"
 			(at 63.5 93.98 0)
 			(hide yes)
@@
 			)
 		)
-		(property "Assemble" "Y"
+		(property "Assemble" "-- mixed values --"
 			(at 63.5 93.98 0)
 			(hide yes)
@@
 		)
 		(property "LCSC" ""
+			(at 63.5 93.98 0)
+			(hide yes)
+			(show_name no)
+			(do_not_autoplace no)
+			(effects
+				(font
+					(size 1.27 1.27)
+				)
+			)
+		)
+		(property "Mouser Part Number" "-- mixed values --"
 			(at 63.5 93.98 0)
 			(hide yes)
@@
 			)
 		)
-		(property "Datasheet" "https://www.mouser.com/ProductDetail/Vishay/CRCW06031K00FKEI?qs=%252B6g0mu59x7LmDUigK4duvw%3D%3D&srsltid=AfmBOoq-qbpfAjzhtzCNjmKpq35FQ1BHTaIyFUz28_1v8HZaKbIrwYgN"
+		(property "Datasheet" "-- mixed values --"
 			(at 54.61 140.97 0)
 			(hide yes)
@@
 			)
 		)
-		(property "Assemble" "Y"
+		(property "Assemble" "-- mixed values --"
 			(at 54.61 140.97 0)
 			(hide yes)
@@
 			)
 		)
-		(property "Datasheet" ""
+		(property "Datasheet" "-- mixed values --"
 			(at 124.46 78.74 0)
 			(hide yes)
@@
 			)
 		)
-		(property "Description" "Resistor"
+		(property "Description" "-- mixed values --"
 			(at 124.46 78.74 0)
 			(hide yes)
@@
 		)
 		(property "LCSC" ""
+			(at 124.46 78.74 0)
+			(hide yes)
+			(show_name no)
+			(do_not_autoplace no)
+			(effects
+				(font
+					(size 1.27 1.27)
+				)
+			)
+		)
+		(property "Assemble" "-- mixed values --"
+			(at 124.46 78.74 0)
+			(hide yes)
+			(show_name no)
+			(do_not_autoplace no)
+			(effects
+				(font
+					(size 1.27 1.27)
+				)
+			)
+		)
+		(property "Mouser Part Number" "-- mixed values --"
+			(at 124.46 78.74 0)
+			(hide yes)
+			(show_name no)
+			(do_not_autoplace no)
+			(effects
+				(font
+					(size 1.27 1.27)
+				)
+			)
+		)
+		(property "P/N" "-- mixed values --"
 			(at 124.46 78.74 0)
 			(hide yes)
@@
 			)
 		)
-		(property "Datasheet" "https://www.mouser.com/ProductDetail/Vishay/CRCW060310K0FKEI?qs=3qWEzBg5KnKofE%252B8acPBRA%3D%3D&srsltid=AfmBOoqKim6ih2rJJ1EIhwDCT-JirqUJIep-ZlqxnK3BQM3p3g1ka950"
+		(property "Datasheet" "-- mixed values --"
 			(at 207.01 93.98 0)
 			(hide yes)
@@
 			)
 		)
-		(property "Description" "Resistor"
+		(property "Description" "-- mixed values --"
 			(at 207.01 93.98 0)
 			(hide yes)
@@
 			)
 		)
-		(property "P/N" "CRCW060310K0FKEI "
+		(property "P/N" "-- mixed values --"
 			(at 207.01 93.98 0)
 			(hide yes)
@@
 			)
 		)
-		(property "Assemble" "Y"
+		(property "Assemble" "-- mixed values --"
 			(at 207.01 93.98 0)
 			(hide yes)
@@
 		)
 		(property "LCSC" ""
+			(at 207.01 93.98 0)
+			(hide yes)
+			(show_name no)
+			(do_not_autoplace no)
+			(effects
+				(font
+					(size 1.27 1.27)
+				)
+			)
+		)
+		(property "Mouser Part Number" "-- mixed values --"
 			(at 207.01 93.98 0)
 			(hide yes)
@@
 			)
 		)
-		(property "Datasheet" "https://www.mouser.com/ProductDetail/Vishay/CRCW060310K0FKEI?qs=3qWEzBg5KnKofE%252B8acPBRA%3D%3D&srsltid=AfmBOoqKim6ih2rJJ1EIhwDCT-JirqUJIep-ZlqxnK3BQM3p3g1ka950"
+		(property "Datasheet" "-- mixed values --"
 			(at 231.14 135.89 0)
 			(hide yes)
@@
 			)
 		)
-		(property "Description" "Resistor"
+		(property "Description" "-- mixed values --"
 			(at 231.14 135.89 0)
 			(hide yes)
@@
 			)
 		)
-		(property "P/N" "CRCW060310K0FKEI "
+		(property "P/N" "-- mixed values --"
 			(at 231.14 135.89 0)
 			(hide yes)
@@
 			)
 		)
-		(property "Assemble" "Y"
+		(property "Assemble" "-- mixed values --"
 			(at 231.14 135.89 0)
 			(hide yes)
@@
 		)
 		(property "LCSC" ""
+			(at 231.14 135.89 0)
+			(hide yes)
+			(show_name no)
+			(do_not_autoplace no)
+			(effects
+				(font
+					(size 1.27 1.27)
+				)
+			)
+		)
+		(property "Mouser Part Number" "-- mixed values --"
 			(at 231.14 135.89 0)
 			(hide yes)
@@
 			)
 		)
-		(property "Value" "ORA_OUT"
+		(property "Value" "ORA_OUT_TP"
 			(at 127 71.6279 0)
 			(show_name no)
@@
 			)
 		)
-		(property "Footprint" "TestPoint:TestPoint_Loop_D2.50mm_Drill1.0mm_LowProfile"
+		(property "Footprint" "-- mixed values --"
 			(at 129.54 73.66 0)
 			(hide yes)
@@
 			)
 		)
-		(property "Description" "test point"
+		(property "Description" "-- mixed values --"
 			(at 124.46 73.66 0)
 			(hide yes)
@@
 		)
 		(property "LCSC" ""
+			(at 124.46 73.66 0)
+			(hide yes)
+			(show_name no)
+			(do_not_autoplace no)
+			(effects
+				(font
+					(size 1.27 1.27)
+				)
+			)
+		)
+		(property "Sim.Pins" "-- mixed values --"
 			(at 124.46 73.66 0)
 			(hide yes)
@@
 			)
 		)
+		(property "LCSC P/N" "-- mixed values --"
+			(at 109.22 128.27 90)
+			(hide yes)
+			(show_name no)
+			(do_not_autoplace no)
+			(effects
+				(font
+					(size 1.27 1.27)
+				)
+			)
+		)
 		(pin "2"
 		)
@@
 			)
 		)
-		(property "Datasheet" "https://www.mouser.com/ProductDetail/Vishay/CRCW060310K0FKEI?qs=3qWEzBg5KnKofE%252B8acPBRA%3D%3D&srsltid=AfmBOoqKim6ih2rJJ1EIhwDCT-JirqUJIep-ZlqxnK3BQM3p3g1ka950"
+		(property "Datasheet" "-- mixed values --"
 			(at 63.5 55.88 0)
 			(hide yes)
@@
 			)
 		)
-		(property "Description" "Resistor"
+		(property "Description" "-- mixed values --"
 			(at 63.5 55.88 0)
 			(hide yes)
@@
 			)
 		)
-		(property "P/N" "CRCW060310K0FKEI "
+		(property "P/N" "-- mixed values --"
 			(at 63.5 55.88 0)
 			(hide yes)
@@
 			)
 		)
-		(property "Assemble" "Y"
+		(property "Assemble" "-- mixed values --"
 			(at 63.5 55.88 0)
 			(hide yes)
@@
 		)
 		(property "LCSC" ""
+			(at 63.5 55.88 0)
+			(hide yes)
+			(show_name no)
+			(do_not_autoplace no)
+			(effects
+				(font
+					(size 1.27 1.27)
+				)
+			)
+		)
+		(property "Mouser Part Number" "-- mixed values --"
 			(at 63.5 55.88 0)
 			(hide yes)
@@
 			)
 		)
-		(property "Value" "ORA_OUT"
+		(property "Value" "ORA_OUT_LED"
 			(at 128.27 89.2174 90)
 			(show_name no)
@@
 			)
 		)
-		(property "Footprint" "LED_SMD:LED_0603_1608Metric_Pad1.05x0.95mm_HandSolder"
+		(property "Footprint" "-- mixed values --"
 			(at 124.46 86.36 0)
 			(hide yes)
@@
 			)
 		)
-		(property "Description" "Light emitting diode"
+		(property "Description" "-- mixed values --"
 			(at 124.46 86.36 0)
 			(hide yes)
@@
 			)
 		)
-		(property "Sim.Pins" "1=K 2=A"
+		(property "Sim.Pins" "-- mixed values --"
 			(at 124.46 86.36 0)
 			(hide yes)

Commit message: more pns i go now
Parts:
- D2: footprint -- mixed values -- -> LED_SMD:LED_0603_1608Metric_Pad1.05x0.95mm_HandSolder
- F2: LCSC P/N -- mixed values -- -> C352820; P/N (none) -> 3557-2
- J2, J3, TP25: now left out of the parts list
- TP2: footprint -- mixed values -- -> TestPoint:TestPoint_Loop_D2.50mm_Drill1.0mm_LowProfile; now left out of the parts list
Changed lines of the file:
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@@
 		(body_style 1)
 		(exclude_from_sim no)
-		(in_bom yes)
+		(in_bom no)
 		(on_board yes)
 		(in_pos_files yes)
@@
 		(body_style 1)
 		(exclude_from_sim no)
-		(in_bom yes)
+		(in_bom no)
 		(on_board yes)
 		(in_pos_files yes)
@@
 		(body_style 1)
 		(exclude_from_sim no)
-		(in_bom yes)
+		(in_bom no)
 		(on_board yes)
 		(in_pos_files yes)
@@
 			)
 		)
-		(property "Footprint" "-- mixed values --"
+		(property "Footprint" "TestPoint:TestPoint_Loop_D2.50mm_Drill1.0mm_LowProfile"
 			(at 129.54 73.66 0)
 			(hide yes)
@@
 			)
 		)
-		(property "LCSC P/N" "-- mixed values --"
+		(property "LCSC P/N" "C352820"
+			(at 109.22 128.27 90)
+			(hide yes)
+			(show_name no)
+			(do_not_autoplace no)
+			(effects
+				(font
+					(size 1.27 1.27)
+				)
+			)
+		)
+		(property "P/N" "3557-2"
 			(at 109.22 128.27 90)
 			(hide yes)
@@
 			)
 		)
-		(property "Footprint" "-- mixed values --"
+		(property "Footprint" "LED_SMD:LED_0603_1608Metric_Pad1.05x0.95mm_HandSolder"
 			(at 124.46 86.36 0)
 			(hide yes)
@@
 		(body_style 1)
 		(exclude_from_sim no)
-		(in_bom yes)
+		(in_bom no)
 		(on_board yes)
 		(in_pos_files yes)

Commit message: finishing up pns
Parts:
- D2: LCSC P/N (none) -> C125103; P/N (none) -> LTST-C193TBKT-5A
- D3: now not fitted; now left out of the parts list
Changed lines of the file:
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@@
 		(body_style 1)
 		(exclude_from_sim no)
-		(in_bom yes)
+		(in_bom no)
 		(on_board yes)
 		(in_pos_files yes)
-		(dnp no)
+		(dnp yes)
 		(fields_autoplaced yes)
 		(property "Reference" "D3"
@@
 			(at 124.46 86.36 90)
 			(hide yes)
+			(show_name no)
+			(do_not_autoplace no)
+			(effects
+				(font
+					(size 1.27 1.27)
+				)
+			)
+		)
+		(property "LCSC P/N" "C125103"
+			(at 124.46 86.36 90)
+			(hide yes)
+			(show_name no)
+			(do_not_autoplace no)
+			(effects
+				(font
+					(size 1.27 1.27)
+				)
+			)
+		)
+		(property "P/N" "LTST-C193TBKT-5A"
+			(at 124.46 86.36 90)
+			(hide yes)
